File: KiCad/TC_Interface_Board/TC_Interface_Board.kicad_sch (KiCad schematic)
At the start: 21 parts, among them J1_24V Conn_01x04, J1_CN1_24V Conn_01x03, J2_CN2_9V_Main02 Conn_01x02, J3_CN3_9V_Main01 Conn_01x02, Q1 DTC143X (C143 NPN), Q2 DTC143X (C143 NPN), U1 LM2596S-ADJ (SHARP IR3M03A)

Commit message: UPDATE
Parts:
- added J4_BUS_MONITER: Conn_01x05, symbol Connector_Generic:Conn_01x05
- added L1_Inductor: L_Ferrite, symbol Device:L_Ferrite
- renumbered J1_24V to J1_24V_ROW
Connections:
- net at D4.1 (K): now also U1.4 (FB), L1_Inductor.1
- net at D4.2 (A): now also R6.1
- net at J1_24V_ROW.1 (Pin_1): now also C2.1, C3.2, U1.3 (GND)
- net at J1_24V_ROW.4 (Pin_4): now also C2.2, U1.1 (VIN)
- net at R6.2: now also U1.2 (OUT)
- net at C3.1: now also L1_Inductor.2
Other:
- note added: "BUS to OC interface"
- note added: "DC DC Invert DV24V -> DC9V"
- moved on the sheet: C1, C2, C3, D1, D2, D3, D4, D5, J1_24V_ROW, Q1, Q2, R1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

Commit message: UPDATE
Parts:
- R2: value 120Ω -> 10KΩ
- R4: value R -> 11KΩ
- R5: value R -> 0.55Ω
- R6: value 1kΩ -> 110Ω
Changed lines of the file:
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@@
 			)
 		)
-		(property "Value" "R"
+		(property "Value" "0.55Ω"
 			(at 52.0699 93.98 0)
 			(effects
@@
 			)
 		)
-		(property "Value" "120Ω"
+		(property "Value" "10KΩ"
 			(at 35.56 152.3999 0)
 			(effects
@@
 			)
 		)
-		(property "Value" "1kΩ"
+		(property "Value" "110Ω"
 			(at 130.81 36.83 90)
 			(effects
@@
 			)
 		)
-		(property "Value" "R"
+		(property "Value" "11KΩ"
 			(at 55.88 137.1599 0)
 			(effects

Commit message: UPDATE
Connections:
- net at D5.1 (K): now also J1_24V_ROW.4 (Pin_4)
- net at D5.2 (A): now also C2.2, U1.1 (VIN)
Other:
- moved on the sheet: D5
Changed lines of the file:
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@@
+	(wire
+		(pts
+			(xy 30.48 33.02) (xy 36.83 33.02)
+		)
+		(stroke
+			(width 0)
+			(type default)
+		)
+	)
 	(wire
 		(pts
@@
 	(wire
 		(pts
-			(xy 30.48 33.02) (xy 52.07 33.02)
-		)
-		(stroke
-			(width 0)
-			(type default)
-		)
-	)
-	(wire
-		(pts
 			(xy 52.07 43.18) (xy 52.07 40.64)
+		)
+		(stroke
+			(width 0)
+			(type default)
+		)
+	)
+	(wire
+		(pts
+			(xy 44.45 33.02) (xy 52.07 33.02)
 		)
 		(stroke
@@
 	(symbol
 		(lib_id "Device:D")
-		(at 146.05 153.67 0)
+		(at 40.64 33.02 0)
 		(unit 1)
 		(exclude_from_sim no)
@@
 		(fields_autoplaced yes)
 		(property "Reference" "D5"
-			(at 146.05 147.32 0)
+			(at 40.64 26.67 0)
 			(effects
 				(font
@@
 		)
 		(property "Value" "24V?"
-			(at 146.05 149.86 0)
+			(at 40.64 29.21 0)
 			(effects
 				(font
@@
 		)
 		(property "Footprint" "Diode_THT:D_DO-41_SOD81_P7.62mm_Horizontal"
-			(at 146.05 153.67 0)
+			(at 40.64 33.02 0)
 			(effects
 				(font
@@
 		)
 		(property "Datasheet" "~"
-			(at 146.05 153.67 0)
+			(at 40.64 33.02 0)
 			(effects
 				(font
@@
 		)
 		(property "Description" "Diode"
-			(at 146.05 153.67 0)
+			(at 40.64 33.02 0)
 			(effects
 				(font
@@
 		)
 		(property "Sim.Device" "D"
-			(at 146.05 153.67 0)
+			(at 40.64 33.02 0)
 			(effects
 				(font
@@
 		)
 		(property "Sim.Pins" "1=K 2=A"
-			(at 146.05 153.67 0)
-			(effects
-				(font
+			(at 40.64 33.02 0)
+			(effects
+				(font

Commit message: UPDATE
Parts:
- removed Q1, Q2: DTC143X (C143 NPN), Package_TO_SOT_THT:TO-92_Inline, symbol Transistor_BJT:DTC143X
- added Q1, Q2: DTC143E, Package_TO_SOT_THT:TO-92_Inline, symbol Transistor_BJT:DTC143E
Changed lines of the file:
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@@
-	)
-	(symbol
-		(lib_id "Transistor_BJT:DTC143X")
-		(at 73.66 95.25 0)
-		(unit 1)
-		(exclude_from_sim no)
-		(in_bom yes)
-		(on_board yes)
-		(dnp no)
-		(property "Reference" "Q1"
-			(at 78.74 93.9799 0)
-			(effects
-				(font
-					(size 1.27 1.27)
-				)
-				(justify left)
-			)
-		)
-		(property "Value" "DTC143X (C143 NPN)"
-			(at 78.74 96.5199 0)
-			(effects
-				(font
-					(size 1.27 1.27)
-				)
-				(justify left)
-			)
-		)
-		(property "Footprint" "Package_TO_SOT_THT:TO-92_Inline"
-			(at 67.31 86.614 0)
-			(effects
-				(font
-					(size 1.27 1.27)
-				)
-				(justify left)
-			)
-		)
-		(property "Datasheet" ""
-			(at 73.66 95.25 0)
-			(effects
-				(font
-					(size 1.27 1.27)
-				)
-				(justify left)
-				(hide yes)
-			)
-		)
-		(property "Description" "Digital NPN Transistor, 4k7/10k, SOT-23"
-			(at 73.66 95.25 0)
-			(effects
-				(font
-					(size 1.27 1.27)
-				)
-				(hide yes)
-			)
-		)
-		(pin "2"
-		)
-		(pin "1"
-		)
-		(pin "3"
-		)
-		(instances
-			(project ""
-				(path "/bd09a545-618a-47d2-a0b1-f0d03750b68a"
-					(reference "Q1")
-					(unit 1)
-				)
-			)
-		)
 	)
 	(symbol
@@
 	)
 	(symbol
+		(lib_id "Transistor_BJT:DTC143E")
+		(at 81.28 172.72 0)
+		(unit 1)
+		(exclude_from_sim no)
+		(in_bom yes)
+		(on_board yes)
+		(dnp no)
+		(fields_autoplaced yes)
+		(property "Reference" "Q2"
+			(at 86.36 171.4499 0)
+			(effects
+				(font
+					(size 1.27 1.27)
+				)
+				(justify left)
+			)
+		)
+		(property "Value" "DTC143E"
+			(at 86.36 173.9899 0)
+			(effects
+				(font
+					(size 1.27 1.27)
+				)
+				(justify left)
+			)
+		)
+		(property "Footprint" "Package_TO_SOT_THT:TO-92_Inline"
+			(at 81.28 172.72 0)
+			(effects
+				(font
+					(size 1.27 1.27)
+				)
+				(justify left)
+				(hide yes)
+			)
+		)
+		(property "Datasheet" ""
+			(at 81.28 172.72 0)
+			(effects
+				(font
+					(size 1.27 1.27)
+				)
+				(justify left)
+				(hide yes)
+			)
+		)
+		(property "Description" "Digital NPN Transistor, 4k7/4k7, SOT-23"
+			(at 81.28 172.72 0)
+			(effects
+				(font
+					(size 1.27 1.27)
+				)
+				(hide yes)
+			)
+		)
+		(pin "1"
+		)
+		(pin "2"
+		)
+		(pin "3"
+		)
+		(instances
+			(project ""
+				(path "/bd09a545-618a-47d2-a0b1-f0d03750b68a"
+					(reference "Q2")
+					(unit 1)
+				)
+			)
+		)
+	)
+	(symbol
 		(lib_id "Device:D")
 		(at 40.64 33.02 0)
@@
 	)
 	(symbol
-		(lib_id "Transistor_BJT:DTC143X")
-		(at 83.82 179.07 0)
-		(unit 1)
-		(exclude_from_sim no)
-		(in_bom yes)
-		(on_board yes)
-		(dnp no)
-		(property "Reference" "Q2"
-			(at 88.9 177.7999 0)
-			(effects
-				(font
-					(size 1.27 1.27)
-				)
-				(justify left)
-			)
-		)
-		(property "Value" "DTC143X (C143 NPN)"
-			(at 88.9 180.3399 0)
-			(effects
-				(font
-					(size 1.27 1.27)
-				)
-				(justify left)
-			)
-		)
-		(property "Footprint" "Package_TO_SOT_THT:TO-92_Inline"
-			(at 77.47 170.434 0)
-			(effects
-				(font
-					(size 1.27 1.27)
-				)
-				(justify left)
-				(hide yes)
-			)
-		)
-		(property "Datasheet" ""
-			(at 83.82 179.07 0)
-			(effects
-				(font
-					(size 1.27 1.27)
-				)
-				(justify left)
-				(hide yes)
-			)
-		)
-		(property "Description" "Digital NPN Transistor, 4k7/10k, SOT-23"
-			(at 83.82 179.07 0)
-			(effects
-				(font
-					(size 1.27 1.27)
-				)
-				(hide yes)
-			)
-		)
-		(pin "2"
-		)
-		(pin "1"
-		)
-		(pin "3"
-		)
-		(instances
-			(project "TC_Interface_Board"
-				(path "/bd09a545-618a-47d2-a0b1-f0d03750b68a"
-					(reference "Q2")
-					(unit 1)
-				)
-			)
-		)
-	)
-	(symbol
 		(lib_id "Device:D")
 		(at 123.19 167.64 0)
@@
 					(unit 1)
 				)
+			)
+		)
+	)
+	(symbol
+		(lib_id "Transistor_BJT:DTC143E")
+		(at 80.01 160.02 0)
+		(unit 1)
+		(exclude_from_sim no)
+		(in_bom yes)
+		(on_board yes)
+		(dnp no)
+		(property "Reference" "Q1"
+			(at 85.09 158.7499 0)
+			(effects
+				(font
+					(size 1.27 1.27)
+				)
+				(justify left)
+			)
+		)
+		(property "Value" "DTC143E"
+			(at 85.09 161.2899 0)
+			(effects
+				(font
+					(size 1.27 1.27)
+				)
+				(justify left)
+			)
+		)
+		(property "Footprint" "Package_TO_SOT_THT:TO-92_Inline"
+			(at 68.072 153.162 0)
+			(effects
+				(font
+					(size 1.27 1.27)
+				)
+				(justify left)
+			)
+		)
+		(property "Datasheet" ""
+			(at 80.01 160.02 0)
+			(effects
+				(font
+					(size 1.27 1.27)
+				)
+				(justify left)
+				(hide yes)
+			)
+		)
+		(property "Description" "Digital NPN Transistor, 4k7/4k7, SOT-23"
+			(at 80.01 160.02 0)
+			(effects
+				(font
+					(size 1.27 1.27)
+				)
+				(hide yes)
+			)
+		)
+		(pin "3"
+		)
+		(pin "2"
+		)
+		(pin "1"
+		)
+		(instances
+			(project ""
+				(path "/bd09a545-618a-47d2-a0b1-f0d03750b68a"
+					(reference "Q1")
+					(unit 1)
+				)

Commit message: UPDATE
Parts:
- renumbered C2 to C1, C1 to C2, D5 to D1, D1 to D2, D2 to D3, D3 to D4, D4 to D5, J1_24V_ROW to J1_24V_ROW1, J1_CN1_24V to J1_CN1_24V1, J2_CN2_9V_Main02 to J2_CN2_9V_Main1, J3_CN3_9V_Main01 to J3_CN3_9V_Main1, J4_BUS_MONITER to J4_BUS_MONITER1, L1_Inductor to L1_Inductor1, R5 to R4, R4 to R5
Changed lines of the file:
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@@
 		(on_board yes)
 		(dnp no)
-		(property "Reference" "R5"
+		(property "Reference" "R4"
 			(at 49.5299 93.98 0)
 			(effects
@@
 			(project ""
 				(path "/bd09a545-618a-47d2-a0b1-f0d03750b68a"
-					(reference "R5")
+					(reference "R4")
 					(unit 1)
 				)
@@
 		(dnp no)
 		(fields_autoplaced yes)
-		(property "Reference" "D4"
+		(property "Reference" "D5"
 			(at 149.86 35.5599 90)
 			(effects
@@
 			(project ""
 				(path "/bd09a545-618a-47d2-a0b1-f0d03750b68a"
-					(reference "D4")
+					(reference "D5")
 					(unit 1)
 				)
@@
 		(dnp no)
 		(fields_autoplaced yes)
-		(property "Reference" "J3_CN3_9V_Main01"
+		(property "Reference" "J3_CN3_9V_Main1"
 			(at 233.68 82.5499 0)
 			(effects
@@
 			(project ""
 				(path "/bd09a545-618a-47d2-a0b1-f0d03750b68a"
-					(reference "J3_CN3_9V_Main01")
+					(reference "J3_CN3_9V_Main1")
 					(unit 1)
 				)
@@
 		(dnp no)
 		(fields_autoplaced yes)
-		(property "Reference" "D5"
+		(property "Reference" "D1"
 			(at 40.64 26.67 0)
 			(effects
@@
 			(project ""
 				(path "/bd09a545-618a-47d2-a0b1-f0d03750b68a"
-					(reference "D5")
+					(reference "D1")
 					(unit 1)
 				)
@@
 		(dnp no)
 		(fields_autoplaced yes)
-		(property "Reference" "J1_24V_ROW"
+		(property "Reference" "J1_24V_ROW1"
 			(at 25.4 26.67 0)
 			(effects
@@
 			(project ""
 				(path "/bd09a545-618a-47d2-a0b1-f0d03750b68a"
-					(reference "J1_24V_ROW")
+					(reference "J1_24V_ROW1")
 					(unit 1)
 				)
@@
 		(on_board yes)
 		(dnp no)
-		(property "Reference" "C2"
+		(property "Reference" "C1"
 			(at 55.88 34.2899 0)
 			(effects
@@
 			(project ""
 				(path "/bd09a545-618a-47d2-a0b1-f0d03750b68a"
-					(reference "C2")
+					(reference "C1")
 					(unit 1)
 				)
@@
 		(on_board yes)
 		(dnp no)
-		(property "Reference" "D1"
+		(property "Reference" "D2"
 			(at 123.19 135.89 0)
 			(effects
@@
 			(project ""
 				(path "/bd09a545-618a-47d2-a0b1-f0d03750b68a"
-					(reference "D1")
+					(reference "D2")
 					(unit 1)
 				)
@@
 		(on_board yes)
 		(dnp no)
-		(property "Reference" "J1_CN1_24V"
+		(property "Reference" "J1_CN1_24V1"
 			(at 233.68 106.6799 0)
 			(effects
@@
 			(project ""
 				(path "/bd09a545-618a-47d2-a0b1-f0d03750b68a"
-					(reference "J1_CN1_24V")
+					(reference "J1_CN1_24V1")
 					(unit 1)
 				)
@@
 		(dnp no)
 		(fields_autoplaced yes)
-		(property "Reference" "J2_CN2_9V_Main02"
+		(property "Reference" "J2_CN2_9V_Main1"
 			(at 233.68 92.7099 0)
 			(effects
@@
 			(project "TC_Interface_Board"
 				(path "/bd09a545-618a-47d2-a0b1-f0d03750b68a"
-					(reference "J2_CN2_9V_Main02")
+					(reference "J2_CN2_9V_Main1")
 					(unit 1)
 				)
@@
 		(dnp no)
 		(fields_autoplaced yes)
-		(property "Reference" "C1"
+		(property "Reference" "C2"
 			(at 90.17 138.4299 0)
 			(effects
@@
 			(project ""
 				(path "/bd09a545-618a-47d2-a0b1-f0d03750b68a"
-					(reference "C1")
+					(reference "C2")
 					(unit 1)
 				)
@@
 		(dnp no)
 		(fields_autoplaced yes)
-		(property "Reference" "J4_BUS_MONITER"
+		(property "Reference" "J4_BUS_MONITER1"
 			(at 26.67 80.01 0)
 			(effects
@@
 			(project ""
 				(path "/bd09a545-618a-47d2-a0b1-f0d03750b68a"
-					(reference "J4_BUS_MONITER")
+					(reference "J4_BUS_MONITER1")
 					(unit 1)
 				)
@@
 		(dnp no)
 		(fields_autoplaced yes)
-		(property "Reference" "L1_Inductor"
+		(property "Reference" "L1_Inductor1"
 			(at 167.64 35.5599 0)
 			(effects
@@
 			(project ""
 				(path "/bd09a545-618a-47d2-a0b1-f0d03750b68a"
-					(reference "L1_Inductor")
+					(reference "L1_Inductor1")
 					(unit 1)
 				)
@@
 		(on_board yes)
 		(dnp no)
-		(property "Reference" "R4"
+		(property "Reference" "R5"
 			(at 55.88 134.6199 0)
 			(effects
@@
 			(project ""
 				(path "/bd09a545-618a-47d2-a0b1-f0d03750b68a"
-					(reference "R4")
+					(reference "R5")
 					(unit 1)
 				)
@@
 		(dnp no)
 		(fields_autoplaced yes)
-		(property "Reference" "D3"
+		(property "Reference" "D4"
 			(at 123.19 161.29 0)
 			(effects
@@
 			(project ""
 				(path "/bd09a545-618a-47d2-a0b1-f0d03750b68a"
-					(reference "D3")
+					(reference "D4")
 					(unit 1)
 				)
@@
 		(dnp no)
 		(fields_autoplaced yes)
-		(property "Reference" "D2"
+		(property "Reference" "D3"
 			(at 123.19 147.32 0)
 			(effects
@@
 			(project ""
 				(path "/bd09a545-618a-47d2-a0b1-f0d03750b68a"
-					(reference "D2")
-					(unit 1)
-				)
+					(reference "D3")
+					(unit 1)
+				)

Commit message: UPDATE
Connections:
- net at D5.2 (A): no longer R6.1
- net at D1.1 (K): no longer J1_24V_ROW1.4 (Pin_4)
- net at R6.2: no longer U1.2 (OUT)
- net at L1_Inductor1.2: no longer C3.1
- now unconnected: C1.1, C1.2, C3.2, D1.2 (A), D5.1 (K), J1_24V_ROW1.1 (Pin_1), L1_Inductor1.1, U1.1 (VIN), U1.3 (GND), U1.4 (FB)
Changed lines of the file:
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@@
-		)
-	)
-	(junction
-		(at 52.07 40.64)
-		(diameter 0)
-		(color 0 0 0 0)
-	)
-	(junction
-		(at 147.32 33.02)
-		(diameter 0)
-		(color 0 0 0 0)
-	)
-	(junction
-		(at 52.07 33.02)
-		(diameter 0)
-		(color 0 0 0 0)
-	)
-	(junction
-		(at 104.14 43.18)
-		(diameter 0)
-		(color 0 0 0 0)
-	)
-	(wire
-		(pts
-			(xy 30.48 33.02) (xy 36.83 33.02)
-		)
-		(stroke
-			(width 0)
-			(type default)
-		)
-	)
-	(wire
-		(pts
-			(xy 104.14 53.34) (xy 104.14 43.18)
-		)
-		(stroke
-			(width 0)
-			(type default)
-		)
-	)
-	(wire
-		(pts
-			(xy 30.48 40.64) (xy 52.07 40.64)
-		)
-		(stroke
-			(width 0)
-			(type default)
-		)
-	)
-	(wire
-		(pts
-			(xy 165.1 53.34) (xy 104.14 53.34)
-		)
-		(stroke
-			(width 0)
-			(type default)
-		)
-	)
-	(wire
-		(pts
-			(xy 104.14 43.18) (xy 52.07 43.18)
-		)
-		(stroke
-			(width 0)
-			(type default)
-		)
-	)
-	(wire
-		(pts
-			(xy 165.1 40.64) (xy 165.1 45.72)
-		)
-		(stroke
-			(width 0)
-			(type default)
-		)
-	)
-	(wire
-		(pts
-			(xy 134.62 40.64) (xy 147.32 40.64)
-		)
-		(stroke
-			(width 0)
-			(type default)
-		)
-	)
-	(wire
-		(pts
-			(xy 116.84 33.02) (xy 147.32 33.02)
-		)
-		(stroke
-			(width 0)
-			(type default)
-		)
-	)
-	(wire
-		(pts
-			(xy 147.32 33.02) (xy 165.1 33.02)
-		)
-		(stroke
-			(width 0)
-			(type default)
-		)
-	)
-	(wire
-		(pts
-			(xy 127 38.1) (xy 127 40.64)
-		)
-		(stroke
-			(width 0)
-			(type default)
-		)
-	)
-	(wire
-		(pts
-			(xy 52.07 33.02) (xy 91.44 33.02)
-		)
-		(stroke
-			(width 0)
-			(type default)
 		)
 	)
@@
 		)
 		(stroke
-			(width 0)
-			(type default)
-		)
-	)
-	(wire
-		(pts
-			(xy 116.84 38.1) (xy 127 38.1)
-		)
-		(stroke
-			(width 0)
-			(type default)
-		)
-	)
-	(wire
-		(pts
-			(xy 52.07 43.18) (xy 52.07 40.64)
-		)
-		(stroke
-			(width 0)
-			(type default)
-		)
-	)
-	(wire
-		(pts
-			(xy 44.45 33.02) (xy 52.07 33.02)
-		)
-		(stroke

Commit message: UPDATE
Parts:
- C1: footprint Diode_THT:D_5W_P5.08mm_Vertical_AnodeUp -> Capacitor_THT:CP_Radial_D5.0mm_P2.50mm
- C2: footprint Diode_THT:D_DO-15_P12.70mm_Horizontal -> Capacitor_THT:CP_Radial_D5.0mm_P2.50mm
- C3: footprint Diode_THT:D_DO-15_P5.08mm_Vertical_AnodeUp -> Capacitor_THT:CP_Radial_D5.0mm_P2.50mm
- J4_BUS_MONITER1: footprint (none) -> Connector_JST:JST_VH_B5P-VH-B_1x05_P3.96mm_Vertical
- L1_Inductor1: footprint (none) -> Capacitor_THT:CP_Radial_D13.0mm_P7.50mm
- R2: footprint (none) -> Resistor_THT:R_Axial_DIN0207_L6.3mm_D2.5mm_P7.62mm_Horizontal
Changed lines of the file:
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@@
 			)
 		)
-		(property "Footprint" "Diode_THT:D_5W_P5.08mm_Vertical_AnodeUp"
+		(property "Footprint" "Capacitor_THT:CP_Radial_D5.0mm_P2.50mm"
 			(at 35.052 44.704 0)
 			(effects
@@
 			)
 		)
-		(property "Footprint" ""
+		(property "Footprint" "Resistor_THT:R_Axial_DIN0207_L6.3mm_D2.5mm_P7.62mm_Horizontal"
 			(at 31.242 151.13 90)
 			(effects
@@
 					(size 1.27 1.27)
 				)
+				(hide yes)
 			)
 		)
@@
 			)
 		)
-		(property "Footprint" "Diode_THT:D_DO-15_P12.70mm_Horizontal"
+		(property "Footprint" "Capacitor_THT:CP_Radial_D5.0mm_P2.50mm"
 			(at 87.3252 143.51 0)
 			(effects
@@
 		(on_board yes)
 		(dnp no)
-		(fields_autoplaced yes)
 		(property "Reference" "J4_BUS_MONITER1"
 			(at 26.67 80.01 0)
@@
 			)
 		)
-		(property "Footprint" ""
-			(at 26.67 91.44 0)
-			(effects
-				(font
-					(size 1.27 1.27)
-				)
-				(hide yes)
+		(property "Footprint" "Connector_JST:JST_VH_B5P-VH-B_1x05_P3.96mm_Vertical"
+			(at 44.958 103.124 0)
+			(effects
+				(font
+					(size 1.27 1.27)
+				)
 			)
 		)
@@
 			)
 		)
-		(property "Footprint" ""
+		(property "Footprint" "Capacitor_THT:CP_Radial_D13.0mm_P7.50mm"
 			(at 165.1 36.83 0)
 			(effects
@@
 			)
 		)
-		(property "Footprint" "Diode_THT:D_DO-15_P5.08mm_Vertical_AnodeUp"
+		(property "Footprint" "Capacitor_THT:CP_Radial_D5.0mm_P2.50mm"
 			(at 155.702 56.134 0)
 			(effects

Commit message: UPDATE
Parts:
- added U1: IR3M03A, Package_DIP:DIP-8_W7.62mm, symbol Sharp_Legacy_IC:IR3M03A
- R5: footprint Resistor_THT:R_Axial_DIN0207_L6.3mm_D2.5mm_P7.62mm_Horizontal -> Resistor_THT:R_Axial_DIN0207_L6.3mm_D2.5mm_P10.16mm_Horizontal
- renumbered U1 to U2
Changed lines of the file:
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@@
+	)
+	(symbol
+		(lib_id "Sharp_Legacy_IC:IR3M03A")
+		(at 205.74 40.64 0)
+		(unit 1)
+		(exclude_from_sim no)
+		(in_bom yes)
+		(on_board yes)
+		(dnp no)
+		(fields_autoplaced yes)
+		(property "Reference" "U1"
+			(at 205.105 27.94 0)
+			(effects
+				(font
+					(size 1.27 1.27)
+				)
+			)
+		)
+		(property "Value" "IR3M03A"
+			(at 205.105 30.48 0)
+			(effects
+				(font
+					(size 1.27 1.27)
+				)
+			)
+		)
+		(property "Footprint" "Package_DIP:DIP-8_W7.62mm"
+			(at 206.248 48.768 0)
+			(effects
+				(font
+					(size 1.27 1.27)
+				)
+				(hide yes)
+			)
+		)
+		(property "Datasheet" ""
+			(at 205.74 40.64 0)
+			(effects
+				(font
+					(size 1.27 1.27)
+				)
+				(hide yes)
+			)
+		)
+		(property "Description" ""
+			(at 205.74 40.64 0)
+			(effects
+				(font
+					(size 1.27 1.27)
+				)
+				(hide yes)
+			)
+		)
+		(pin "5"
+		)
+		(pin "7"
+		)
+		(pin "1"
+		)
+		(pin "3"
+		)
+		(pin "2"
+		)
+		(pin "4"
+		)
+		(pin "6"
+		)
+		(pin "8"
+		)
+		(instances
+			(project ""
+				(path "/bd09a545-618a-47d2-a0b1-f0d03750b68a"
+					(reference "U1")
+					(unit 1)
+				)
+			)
+		)
 	)
 	(symbol
@@
 			)
 		)
-		(property "Footprint" "Resistor_THT:R_Axial_DIN0207_L6.3mm_D2.5mm_P7.62mm_Horizontal"
+		(property "Footprint" "Resistor_THT:R_Axial_DIN0207_L6.3mm_D2.5mm_P10.16mm_Horizontal"
 			(at 16.51 128.27 0)
 			(effects
@@
 		(on_board yes)
 		(dnp no)
-		(property "Reference" "U1"
+		(property "Reference" "U2"
 			(at 104.14 25.4 0)
 			(effects
@@
 			(project ""
 				(path "/bd09a545-618a-47d2-a0b1-f0d03750b68a"
-					(reference "U1")
-					(unit 1)
-				)
+					(reference "U2")
+					(unit 1)
+				)
