File: KiCad/TC_Interface_Board/TC_Interface_Board.kicad_sch (KiCad schematic)
At the start: 30 parts, among them J1 Conn_01x05, J1_24V1 JST_VH_01x04, J1_CN1 JST_VH_01x03, J2 Conn_01x05, J2_CN1 JST_VH_01x02, J3 Conn_01x05, J3_CN1 JST_VH_01x02, J4 Conn_01x05, J5 Conn_01x05, J6 Conn_01x05, J7 Conn_01x05, J8 Conn_01x05, Q1 DTC143E, Q2 DTC143E, U1 MC34063AP

Commit message: UPDATE
Parts:
- R6: footprint Resistor_THT:R_Axial_DIN0207_L6.3mm_D2.5mm_P15.24mm_Horizontal -> Resistor_THT:R_Axial_DIN0204_L3.6mm_D1.6mm_P7.62mm_Horizontal
- renumbered Q2 to Q1, Q1 to Q2
Connections:
- net +24V: now also R2.1
- net CMD_IN: now also D1.1 (K); no longer D2.1 (K), R6.1
- net GND: now also D2.2 (A), R1.2, R6.2; no longer D1.2 (A), R2.2, R5.1
- net MC34063_SW_NODE: now also R5.1; no longer R1.2
- net TC_CMD_BUS: now also D2.1 (K), Q1.2 (C); no longer D1.1 (K), Q2.3 (B)
- net at D5.1 (K): no longer R6.2
- net at R4.1, U1.5 (Vfb): now also R6.1; no longer R5.2
- net at C1.1, D3.1 (K), U1.6 (Vin): now also R5.2; no longer R1.1
- net at Q1.3 (B), Q2.2 (C), R3.1: now also R2.2
- removed net Q2C_NODE: D2.2 (A), Q1.2 (C), R2.1
- new net: D1.2 (A), Q2.3 (B), R1.1
Other:
- moved on the sheet: D1, D2, R1, R2, R5, R6

Commit message: UPDATE
Parts:
- R5: footprint Resistor_THT:R_Axial_DIN0207_L6.3mm_D2.5mm_P7.62mm_Horizontal -> Resistor_THT:R_Axial_DIN0309_L9.0mm_D3.2mm_P12.70mm_Horizontal
Connections:
- net MC34063_TC: now also D5.1 (K), R5.2
- net at C1.1, D3.1 (K), U1.6 (Vin): no longer R5.2
- net Q2_BASE: now reaches D1.2 (A), Q2.3 (B), R1.1
Other:
- moved on the sheet: D5
Changed lines of the file:
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@@
 	)
 	(junction
-		(at 81.28 57.15)
-		(diameter 0)
-		(color 0 0 0 0)
-	)
-	(junction
 		(at 121.92 36.83)
 		(diameter 0)
@@
 	)
 	(junction
+		(at 100.33 80.01)
+		(diameter 0)
+		(color 0 0 0 0)
+	)
+	(junction
 		(at 64.77 93.98)
 		(diameter 0)
@@
 	)
 	(junction
+		(at 100.33 59.69)
+		(diameter 0)
+		(color 0 0 0 0)
+	)
+	(junction
 		(at 151.13 116.84)
 		(diameter 0)
@@
 	(wire
 		(pts
-			(xy 208.28 110.49) (xy 153.67 110.49)
+			(xy 153.67 110.49) (xy 209.55 110.49)
 		)
 		(stroke
@@
 	(wire
 		(pts
+			(xy 100.33 59.69) (xy 100.33 80.01)
+		)
+		(stroke
+			(width 0)
+			(type default)
+		)
+	)
+	(wire
+		(pts
 			(xy 87.63 31.75) (xy 102.87 31.75)
 		)
@@
 	(wire
 		(pts
+			(xy 110.49 54.61) (xy 100.33 54.61)
+		)
+		(stroke
+			(width 0)
+			(type default)
+		)
+	)
+	(wire
+		(pts
 			(xy 41.91 50.8) (xy 67.31 50.8)
 		)
@@
 	(wire
 		(pts
-			(xy 124.46 80.01) (xy 90.17 80.01)
+			(xy 124.46 80.01) (xy 100.33 80.01)
 		)
 		(stroke
@@
 	(wire
 		(pts
-			(xy 133.35 142.24) (xy 151.13 142.24)
+			(xy 100.33 80.01) (xy 90.17 80.01)
 		)
 		(stroke
@@
 	(wire
 		(pts
-			(xy 151.13 41.91) (xy 158.75 41.91)
+			(xy 133.35 142.24) (xy 151.13 142.24)
 		)
 		(stroke
@@
 	(wire
 		(pts
-			(xy 57.15 116.84) (xy 57.15 57.15)
+			(xy 151.13 41.91) (xy 158.75 41.91)
 		)
 		(stroke
@@
 	(wire
 		(pts
-			(xy 52.07 80.01) (xy 52.07 133.35)
+			(xy 57.15 116.84) (xy 57.15 57.15)
 		)
 		(stroke
@@
 	(wire
 		(pts
-			(xy 99.06 139.7) (xy 115.57 139.7)
+			(xy 52.07 80.01) (xy 52.07 133.35)
 		)
 		(stroke
@@
 	(wire
 		(pts
-			(xy 130.81 41.91) (xy 151.13 41.91)
+			(xy 99.06 139.7) (xy 115.57 139.7)
 		)
 		(stroke
@@
 	(wire
 		(pts
-			(xy 81.28 64.77) (xy 81.28 57.15)
+			(xy 130.81 41.91) (xy 151.13 41.91)
 		)
 		(stroke
@@
 	(wire
 		(pts
-			(xy 110.49 64.77) (xy 81.28 64.77)
-		)
-		(stroke
-			(width 0)
-			(type default)
-		)
-	)
-	(wire
-		(pts
 			(xy 115.57 109.22) (xy 133.35 109.22)
 		)
@@
 	(wire
 		(pts
-			(xy 153.67 111.76) (xy 153.67 137.16)
+			(xy 118.11 54.61) (xy 209.55 54.61)
 		)
 		(stroke
@@
 	(wire
 		(pts
-			(xy 153.67 109.22) (xy 138.43 109.22)
+			(xy 153.67 111.76) (xy 153.67 137.16)
 		)
 		(stroke
@@
 	(wire
 		(pts
-			(xy 55.88 124.46) (xy 66.04 124.46)
+			(xy 153.67 109.22) (xy 138.43 109.22)
 		)
 		(stroke
@@
 	(wire
 		(pts
-			(xy 179.07 40.64) (xy 189.23 40.64)
+			(xy 55.88 124.46) (xy 66.04 124.46)
 		)
 		(stroke
@@
 	(wire
 		(pts
-			(xy 83.82 137.16) (xy 99.06 137.16)
+			(xy 209.55 110.49) (xy 209.55 54.61)
 		)
 		(stroke
@@
 	(wire
 		(pts
-			(xy 130.81 31.75) (xy 158.75 31.75)
+			(xy 83.82 137.16) (xy 99.06 137.16)
 		)
 		(stroke
@@
 	(wire
 		(pts
-			(xy 44.45 29.21) (xy 44.45 93.98)
+			(xy 130.81 31.75) (xy 158.75 31.75)
 		)
 		(stroke
@@
 	(wire
 		(pts
-			(xy 187.96 96.52) (xy 215.9 96.52)
+			(xy 44.45 29.21) (xy 44.45 93.98)
 		)
 		(stroke
@@
 	(wire
 		(pts
-			(xy 77.47 57.15) (xy 81.28 57.15)
+			(xy 187.96 96.52) (xy 215.9 96.52)
 		)
 		(stroke
@@
 	(wire
 		(pts
-			(xy 208.28 40.64) (xy 196.85 40.64)
+			(xy 77.47 57.15) (xy 81.28 57.15)
 		)
 		(stroke
@@
 	(wire
 		(pts
-			(xy 208.28 40.64) (xy 208.28 110.49)
-		)
-		(stroke
-			(width 0)
-			(type default)
-		)
-	)
-	(wire
-		(pts
 			(xy 115.57 134.62) (xy 133.35 134.62)
 		)
@@
 	(wire
 		(pts
-			(xy 67.31 31.75) (xy 67.31 34.29)
+			(xy 110.49 59.69) (xy 100.33 59.69)
 		)
 		(stroke
@@
 	(wire
 		(pts
-			(xy 110.49 59.69) (xy 110.49 64.77)
+			(xy 67.31 31.75) (xy 67.31 34.29)
 		)
 		(stroke
@@
 	(wire
 		(pts
+			(xy 100.33 54.61) (xy 100.33 59.69)
+		)
+		(stroke
+			(width 0)
+			(type default)
+		)
+	)
+	(wire
+		(pts
 			(xy 151.13 142.24) (xy 151.13 116.84)
 		)
@@
 		)
 	)
-	(label "OC_DRIVE_NODE"
-		(at 153.67 53.34 0)
+	(label "MC34063_TC"
+		(at 107.95 80.01 0)
 		(effects
 			(font
@@
 		)
 	)
-	(label "MC34063_TC"
-		(at 107.95 80.01 0)
+	(label "TC_CMD_BUS"
+		(at 151.13 46.99 0)
 		(effects
 			(font
@@
 		)
 	)
-	(label "TC_CMD_BUS"
-		(at 151.13 46.99 0)
+	(label "CMD_IN"
+		(at 46.99 38.1 0)
 		(effects
 			(font
@@
 		)
 	)
-	(label "CMD_IN"
-		(at 46.99 38.1 0)
+	(label "Q2_BASE"
+		(at 83.82 36.83 0)
 		(effects
 			(font
@@
 			)
 		)
-		(property "Footprint" "Resistor_THT:R_Axial_DIN0207_L6.3mm_D2.5mm_P7.62mm_Horizontal"
+		(property "Footprint" "Resistor_THT:R_Axial_DIN0309_L9.0mm_D3.2mm_P12.70mm_Horizontal"
 			(at 114.3 57.912 90)
 			(effects
@@
 	(symbol
 		(lib_id "Device:D")
-		(at 193.04 40.64 0)
+		(at 114.3 54.61 0)
 		(unit 1)
 		(exclude_from_sim no)
@@
 		(fields_autoplaced yes)
 		(property "Reference" "D5"
-			(at 193.04 34.29 0)
+			(at 114.3 48.26 0)
 			(effects
 				(font
@@
 		)
 		(property "Value" "1N4148"
-			(at 193.04 36.83 0)
+			(at 114.3 50.8 0)
 			(effects
 				(font
@@
 		)
 		(property "Footprint" "Diode_THT:D_DO-35_SOD27_P10.16mm_Horizontal"
-			(at 193.04 40.64 0)
+			(at 114.3 54.61 0)
 			(effects
 				(font
@@
 		)
 		(property "Datasheet" "~"
-			(at 193.04 40.64 0)
+			(at 114.3 54.61 0)
 			(effects
 				(font
@@
 		)
 		(property "Description" "Diode"
-			(at 193.04 40.64 0)
+			(at 114.3 54.61 0)
 			(effects
 				(font
@@
 		)
 		(property "Sim.Device" "D"
-			(at 193.04 40.64 0)
+			(at 114.3 54.61 0)
 			(effects
 				(font
@@
 		)
 		(property "Sim.Pins" "1=K 2=A"
-			(at 193.04 40.64 0)
+			(at 114.3 54.61 0)
 			(effects
 				(font

Commit message: UPDATE
Connections:
- net CMD_IN: now also R3.1
- net MC34063_TC: now also C1.1; no longer C2.1, D5.1 (K), R5.2
- net at D3.1 (K), U1.6 (Vin): no longer C1.1
- net at Q1.3 (B), Q2.2 (C), R2.2: no longer R3.1
- new net: C2.1, D5.1 (K), R5.2
Other:
- moved on the sheet: C1, C2

Commit message: UPDATE
Parts:
- R3: footprint Resistor_THT:R_Axial_DIN0207_L6.3mm_D2.5mm_P7.62mm_Horizontal -> Resistor_THT:R_Axial_DIN0207_L6.3mm_D2.5mm_P10.16mm_Horizontal
Connections:
- net +24V: now also D3.1 (K); no longer D3.2 (A), R3.2
- net at U1.6 (Vin): now also C2.1, D5.1 (K), R5.2; no longer D3.1 (K)
- new net: D3.2 (A), R3.2
Other:
- moved on the sheet: D3, R3
Changed lines of the file:
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@@
 	)
 	(junction
-		(at 153.67 109.22)
-		(diameter 0)
-		(color 0 0 0 0)
-	)
-	(junction
 		(at 81.28 63.5)
 		(diameter 0)
@@
 	)
 	(junction
-		(at 69.85 133.35)
+		(at 87.63 31.75)
 		(diameter 0)
 		(color 0 0 0 0)
 	)
 	(junction
-		(at 87.63 31.75)
+		(at 133.35 116.84)
 		(diameter 0)
 		(color 0 0 0 0)
 	)
 	(junction
-		(at 133.35 116.84)
+		(at 100.33 62.23)
 		(diameter 0)
 		(color 0 0 0 0)
@@
 	(wire
 		(pts
+			(xy 109.22 69.85) (xy 109.22 62.23)
+		)
+		(stroke
+			(width 0)
+			(type default)
+		)
+	)
+	(wire
+		(pts
 			(xy 57.15 57.15) (xy 64.77 57.15)
 		)
@@
 	(wire
 		(pts
+			(xy 86.36 57.15) (xy 77.47 57.15)
+		)
+		(stroke
+			(width 0)
+			(type default)
+		)
+	)
+	(wire
+		(pts
 			(xy 87.63 31.75) (xy 102.87 31.75)
 		)
@@
 	(wire
 		(pts
-			(xy 148.59 52.07) (xy 153.67 52.07)
-		)
-		(stroke
-			(width 0)
-			(type default)
-		)
-	)
-	(wire
-		(pts
-			(xy 77.47 69.85) (xy 77.47 57.15)
-		)
-		(stroke
-			(width 0)
-			(type default)
-		)
-	)
-	(wire
-		(pts
-			(xy 69.85 133.35) (xy 52.07 133.35)
+			(xy 124.46 69.85) (xy 109.22 69.85)
 		)
 		(stroke
@@
 	(wire
 		(pts
-			(xy 147.32 69.85) (xy 147.32 72.39)
+			(xy 109.22 62.23) (xy 100.33 62.23)
 		)
 		(stroke
@@
 	(wire
 		(pts
-			(xy 115.57 137.16) (xy 133.35 137.16)
+			(xy 147.32 69.85) (xy 147.32 72.39)
 		)
 		(stroke
@@
 	(wire
 		(pts
-			(xy 99.06 137.16) (xy 115.57 137.16)
+			(xy 115.57 137.16) (xy 133.35 137.16)
 		)
 		(stroke
@@
 	(wire
 		(pts
-			(xy 85.09 111.76) (xy 99.06 111.76)
+			(xy 99.06 137.16) (xy 115.57 137.16)
 		)
 		(stroke
@@
 	(wire
 		(pts
-			(xy 133.35 142.24) (xy 151.13 142.24)
+			(xy 85.09 111.76) (xy 99.06 111.76)
 		)
 		(stroke
@@
 	(wire
 		(pts
-			(xy 151.13 41.91) (xy 158.75 41.91)
+			(xy 133.35 142.24) (xy 151.13 142.24)
 		)
 		(stroke
@@
 	(wire
 		(pts
-			(xy 57.15 116.84) (xy 57.15 57.15)
+			(xy 151.13 41.91) (xy 158.75 41.91)
 		)
 		(stroke
@@
 	(wire
 		(pts
-			(xy 52.07 80.01) (xy 52.07 133.35)
+			(xy 57.15 116.84) (xy 57.15 57.15)
 		)
 		(stroke
@@
 	(wire
 		(pts
-			(xy 52.07 80.01) (xy 82.55 80.01)
-		)
-		(stroke
-			(width 0)
-			(type default)
-		)
-	)
-	(wire
-		(pts
 			(xy 99.06 134.62) (xy 115.57 134.62)
 		)
@@
 	(wire
 		(pts
-			(xy 124.46 69.85) (xy 77.47 69.85)
-		)
-		(stroke
-			(width 0)
-			(type default)
-		)
-	)
-	(wire
-		(pts
 			(xy 106.68 80.01) (xy 106.68 66.04)
 		)
@@
 	(wire
 		(pts
-			(xy 153.67 52.07) (xy 153.67 109.22)
-		)
-		(stroke
-			(width 0)
-			(type default)
-		)
-	)
-	(wire
-		(pts
 			(xy 115.57 111.76) (xy 133.35 111.76)
 		)
@@
 	(wire
 		(pts
-			(xy 55.88 124.46) (xy 66.04 124.46)
+			(xy 86.36 52.07) (xy 86.36 57.15)
 		)
 		(stroke
@@
 	(wire
 		(pts
-			(xy 69.85 139.7) (xy 83.82 139.7)
+			(xy 55.88 124.46) (xy 66.04 124.46)
 		)
 		(stroke
@@
 	(wire
 		(pts
-			(xy 66.04 116.84) (xy 73.66 116.84)
+			(xy 69.85 139.7) (xy 83.82 139.7)
 		)
 		(stroke
@@
 	(wire
 		(pts
-			(xy 153.67 137.16) (xy 182.88 137.16)
+			(xy 66.04 116.84) (xy 73.66 116.84)
 		)
 		(stroke
@@
 	(wire
 		(pts
-			(xy 215.9 96.52) (xy 215.9 31.75)
+			(xy 153.67 137.16) (xy 182.88 137.16)
 		)
 		(stroke
@@
 	(wire
 		(pts
-			(xy 66.04 124.46) (xy 69.85 124.46)
+			(xy 215.9 96.52) (xy 215.9 31.75)
 		)
 		(stroke
@@
 	(wire
 		(pts
-			(xy 69.85 139.7) (xy 69.85 133.35)
+			(xy 66.04 124.46) (xy 69.85 124.46)
 		)
 		(stroke
@@
 	(wire
 		(pts
-			(xy 69.85 124.46) (xy 69.85 133.35)
+			(xy 69.85 124.46) (xy 69.85 139.7)
 		)
 		(stroke
@@
 	(wire
 		(pts
-			(xy 140.97 52.07) (xy 72.39 52.07)
-		)
-		(stroke
-			(width 0)
-			(type default)
-		)
-	)
-	(wire
-		(pts
 			(xy 99.06 142.24) (xy 115.57 142.24)
 		)
@@
 	(wire
 		(pts
+			(xy 72.39 52.07) (xy 78.74 52.07)
+		)
+		(stroke
+			(width 0)
+			(type default)
+		)
+	)
+	(wire
+		(pts
 			(xy 133.35 119.38) (xy 142.24 119.38)
 		)
@@
 	(symbol
 		(lib_id "Device:D")
-		(at 68.58 57.15 180)
+		(at 68.58 57.15 0)
 		(unit 1)
 		(exclude_from_sim no)
@@
 		(dnp no)
 		(property "Reference" "D3"
-			(at 71.628 58.928 0)
+			(at 65.532 55.372 0)
 			(effects
 				(font
@@
 		)
 		(property "Value" "1N4007"
-			(at 71.628 61.468 0)
+			(at 65.532 52.832 0)
 			(effects
 				(font
@@
 		(dnp no)
 		(property "Reference" "C2"
-			(at 96.012 56.134 90)
+			(at 96.52 59.182 90)
 			(effects
 				(font
@@
 		)
 		(property "Value" "1000uF 35V"
-			(at 100.076 53.848 90)
+			(at 100.584 56.896 90)
 			(effects
 				(font
@@
 	(symbol
 		(lib_id "Device:R")
-		(at 144.78 52.07 90)
+		(at 82.55 52.07 90)
 		(unit 1)
 		(exclude_from_sim no)
@@
 		(dnp no)
 		(property "Reference" "R3"
-			(at 137.922 48.006 90)
+			(at 89.662 51.562 90)
 			(effects
 				(font
@@
 		)
 		(property "Value" "10k"
-			(at 137.922 50.546 90)
+			(at 89.662 54.102 90)
 			(effects
 				(font
 					(size 1.27 1.27)
 				)
-				(hide yes)
 			)
 		)
-		(property "Footprint" "Resistor_THT:R_Axial_DIN0207_L6.3mm_D2.5mm_P7.62mm_Horizontal"
-			(at 144.78 53.848 90)
+		(property "Footprint" "Resistor_THT:R_Axial_DIN0207_L6.3mm_D2.5mm_P10.16mm_Horizontal"
+			(at 82.55 53.848 90)
 			(effects
 				(font
@@
 		)
 		(property "Datasheet" "~"
-			(at 144.78 52.07 0)
+			(at 82.55 52.07 0)
 			(effects
 				(font
@@
 		)
 		(property "Description" "Resistor"
-			(at 144.78 52.07 0)
+			(at 82.55 52.07 0)
 			(effects
 				(font
@@
 		)
 		(property "Value" "PWR_FLAG"
-			(at 82.55 53.848 0)
+			(at 82.804 59.182 0)
 			(effects
 				(font

Commit message: UPDATE
Connections:
- net TC_CMD_BUS is gone; now on net MC34063_SW_NODE: D2.1 (K), J1.2 (Pin_2), J2.2 (Pin_2), J3.2 (Pin_2), J4.2 (Pin_2), J5.2 (Pin_2), J6.2 (Pin_2), J7.2 (Pin_2), J8.2 (Pin_2), Q1.2 (C)
- net MC34063_SW_NODE: no longer R5.1, U1.1 (SwC), U1.7 (Ipk), U1.8 (DC)
- new net: R5.1, U1.1 (SwC), U1.7 (Ipk), U1.8 (DC)
Changed lines of the file:
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@@
 	)
 	(junction
-		(at 77.47 57.15)
-		(diameter 0)
-		(color 0 0 0 0)
-	)
-	(junction
 		(at 147.32 87.63)
 		(diameter 0)
@@
 	)
 	(junction
+		(at 101.6 62.23)
+		(diameter 0)
+		(color 0 0 0 0)
+	)
+	(junction
 		(at 115.57 134.62)
 		(diameter 0)
@@
 	)
 	(junction
-		(at 100.33 59.69)
-		(diameter 0)
-		(color 0 0 0 0)
-	)
-	(junction
 		(at 102.87 31.75)
 		(diameter 0)
@@
 	(wire
 		(pts
-			(xy 72.39 57.15) (xy 77.47 57.15)
+			(xy 153.67 110.49) (xy 209.55 110.49)
 		)
 		(stroke
@@
 	(wire
 		(pts
-			(xy 153.67 110.49) (xy 209.55 110.49)
+			(xy 101.6 59.69) (xy 101.6 62.23)
 		)
 		(stroke
@@
 	(wire
 		(pts
-			(xy 72.39 44.45) (xy 72.39 52.07)
+			(xy 101.6 62.23) (xy 100.33 62.23)
 		)
 		(stroke
@@
 	(wire
 		(pts
-			(xy 67.31 34.29) (xy 67.31 40.64)
+			(xy 72.39 44.45) (xy 72.39 52.07)
 		)
 		(stroke
@@
 	(wire
 		(pts
-			(xy 158.75 31.75) (xy 158.75 33.02)
+			(xy 67.31 34.29) (xy 67.31 40.64)
 		)
 		(stroke
@@
 	(wire
 		(pts
-			(xy 86.36 57.15) (xy 77.47 57.15)
+			(xy 158.75 31.75) (xy 158.75 33.02)
 		)
 		(stroke
@@
 	(wire
 		(pts
+			(xy 118.11 59.69) (xy 147.32 59.69)
+		)
+		(stroke
+			(width 0)
+			(type default)
+		)
+	)
+	(wire
+		(pts
+			(xy 86.36 57.15) (xy 72.39 57.15)
+		)
+		(stroke
+			(width 0)
+			(type default)
+		)
+	)
+	(wire
+		(pts
 			(xy 102.87 41.91) (xy 102.87 49.53)
 		)
@@
 	(wire
 		(pts
-			(xy 109.22 62.23) (xy 100.33 62.23)
+			(xy 109.22 62.23) (xy 101.6 62.23)
 		)
 		(stroke
@@
 	(wire
 		(pts
-			(xy 100.33 59.69) (xy 100.33 62.23)
+			(xy 110.49 59.69) (xy 101.6 59.69)
 		)
 		(stroke
@@
 	(wire
 		(pts
-			(xy 100.33 54.61) (xy 100.33 59.69)
+			(xy 100.33 54.61) (xy 100.33 62.23)
 		)
 		(stroke
@@
 	(wire
 		(pts
-			(xy 86.36 52.07) (xy 86.36 57.15)
-		)
-		(stroke
-			(width 0)
-			(type default)
-		)
-	)
-	(wire
-		(pts
 			(xy 55.88 124.46) (xy 66.04 124.46)
 		)
@@
 	(wire
 		(pts
+			(xy 86.36 52.07) (xy 86.36 57.15)
+		)
+		(stroke
+			(width 0)
+			(type default)
+		)
+	)
+	(wire
+		(pts
 			(xy 81.28 66.04) (xy 81.28 63.5)
 		)
@@
 	(wire
 		(pts
-			(xy 147.32 59.69) (xy 118.11 59.69)
-		)
-		(stroke
-			(width 0)
-			(type default)
-		)
-	)
-	(wire
-		(pts
 			(xy 83.82 134.62) (xy 99.06 134.62)
 		)
@@
 	(wire
 		(pts
-			(xy 110.49 59.69) (xy 100.33 59.69)
-		)
-		(stroke
-			(width 0)
-			(type default)
-		)
-	)
-	(wire
-		(pts
 			(xy 67.31 31.75) (xy 67.31 34.29)
 		)
@@
 	)
 	(label "MC34063_SW_NODE"
-		(at 147.32 74.93 90)
+		(at 151.13 74.93 90)
 		(effects
 			(font
@@
 					(unit 1)
 				)
-			)
-		)
-	)
-	(symbol
-		(lib_id "power:PWR_FLAG")
-		(at 77.47 57.15 0)
-		(unit 1)
-		(exclude_from_sim no)
-		(in_bom yes)
-		(on_board yes)
-		(dnp no)
-		(property "Reference" "#FLG03"
-			(at 77.47 55.245 0)
-			(effects
-				(font
-					(size 1.27 1.27)
-				)
-				(hide yes)
-			)
-		)
-		(property "Value" "PWR_FLAG"
-			(at 82.804 59.182 0)
-			(effects
-				(font
-					(size 1.27 1.27)
-				)
-			)
-		)
-		(property "Footprint" ""
-			(at 77.47 57.15 0)
-			(effects
-				(font
-					(size 1.27 1.27)
-				)
-				(hide yes)
-			)
-		)
-		(property "Datasheet" "~"
-			(at 77.47 57.15 0)
-			(effects
-				(font
-					(size 1.27 1.27)
-				)
-				(hide yes)
-			)
-		)
-		(property "Description" "Special symbol for telling ERC where power comes from"
-			(at 77.47 57.15 0)
-			(effects
-				(font
-					(size 1.27 1.27)
-				)
-				(hide yes)
-			)
-		)
-		(pin "1"
-		)
-		(instances
-			(project ""
-				(path "/bd09a545-618a-47d2-a0b1-f0d03750b68a"
-					(reference "#FLG03")
-					(unit 1)
-				)

Commit message: UPDATE
Connections:
- net MC34063_SW_NODE renamed TC_CMD_BUS
Changed lines of the file:
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@@
 		)
 	)
-	(label "MC34063_SW_NODE"
+	(label "TC_CMD_BUS"
 		(at 151.13 74.93 90)
 		(effects

Commit message: UPDATE
Parts:
- L1_Inductor1: value L_Ferrite -> 330uH
- R1: value 0.22 -> 220
- R2: value 220 -> 10k
- R3: value 10k -> 1k2
- R5: value 1k -> 0R22
Changed lines of the file:
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@@
 		(dnp no)
 		(property "Reference" "R6"
-			(at 164.592 99.314 90)
+			(at 167.386 99.06 90)
 			(effects
 				(font
@@
 		)
 		(property "Value" "1.2k"
-			(at 164.592 101.854 90)
+			(at 167.386 101.6 90)
 			(effects
 				(font
@@
 		(dnp no)
 		(property "Reference" "R4"
-			(at 162.814 86.868 90)
+			(at 168.91 92.456 90)
 			(effects
 				(font
@@
 		)
 		(property "Value" "6.2k"
-			(at 162.56 88.9 90)
+			(at 168.656 94.488 90)
 			(effects
 				(font
@@
 		(dnp no)
 		(property "Reference" "D3"
-			(at 65.532 55.372 0)
+			(at 68.326 55.372 0)
 			(effects
 				(font
@@
 		)
 		(property "Value" "1N4007"
-			(at 65.532 52.832 0)
+			(at 68.326 52.832 0)
 			(effects
 				(font
@@
 			)
 		)
-		(property "Value" "10k"
+		(property "Value" "1k2"
 			(at 89.662 54.102 90)
 			(effects
@@
 			)
 		)
-		(property "Value" "220"
+		(property "Value" "10k"
 			(at 67.31 71.1199 0)
 			(effects
@@
 			)
 		)
-		(property "Value" "1k"
+		(property "Value" "0R22"
 			(at 114.554 64.77 90)
 			(effects
@@
 			)
 		)
-		(property "Value" "L_Ferrite"
+		(property "Value" "330uH"
 			(at 161.29 69.8499 0)
 			(effects
@@
 			)
 		)
-		(property "Value" "0.22"
+		(property "Value" "220"
 			(at 81.28 45.974 90)
 			(effects

Commit message: UPdate
Parts:
- R4: value 6.2k -> 6k2
- R6: value 1.2k -> 1k
