File: KiCad/TC_Interface_Board/TC_Interface_Board.kicad_pcb (KiCad board)
At the start: 2 copper layers, 30 parts, among them J10 Conn_01x05, J11 Conn_01x05, J1_24V_ROW1 Conn_01x04, J1_CN1_24V1 Conn_01x03, J2_CN2_9V_Main1 Conn_01x02, J3_CN3_9V_Main1 Conn_01x02, J4 Conn_01x05, J5 Conn_01x05, J6 Conn_01x05, J7 Conn_01x05, J8 Conn_01x05, J9 Conn_01x05, Q1 DTC143E, Q2 DTC143E, U1 MC34063AP

Commit message: UPDATE
Parts:
- D4: value 630mV -> 630mV 1N5819
- D5: value 24V? -> 24V 1N4006
Connections:
- J4 pad 4: Net-(J4-Pin_4) -> Net-(J10-Pin_4)
- J5 pad 4: Net-(J4-Pin_4) -> Net-(J10-Pin_4)
- J6 pad 4: Net-(J4-Pin_4) -> Net-(J10-Pin_4)
- J7 pad 4: Net-(J4-Pin_4) -> Net-(J10-Pin_4)
Routing:
- net Net-(J4-Pin_4): track 58.6 -> 0.00 mm
- net Net-(J10-Pin_4): track 125.0 -> 183.5 mm
Changed lines of the file:
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@@
 	(net 21 "Net-(U1-Vfb)")
 	(net 22 "Net-(J10-Pin_4)")
-	(net 23 "Net-(J4-Pin_4)")
-	(net 24 "unconnected-(J5-Pin_1-Pad1)")
-	(net 25 "unconnected-(J6-Pin_1-Pad1)")
-	(net 26 "unconnected-(J7-Pin_1-Pad1)")
+	(net 23 "unconnected-(J5-Pin_1-Pad1)")
+	(net 24 "unconnected-(J6-Pin_1-Pad1)")
+	(net 25 "unconnected-(J7-Pin_1-Pad1)")
 	(footprint "Capacitor_THT:CP_Radial_D5.0mm_P2.50mm"
 		(layer "F.Cu")
@@
 			(remove_unused_layers no)
 			(roundrect_rratio 0.092593)
-			(net 24 "unconnected-(J5-Pin_1-Pad1)")
+			(net 23 "unconnected-(J5-Pin_1-Pad1)")
 			(pinfunction "Pin_1")
 			(pintype "passive")
@@
 			(layers "*.Cu" "*.Mask")
 			(remove_unused_layers no)
-			(net 23 "Net-(J4-Pin_4)")
+			(net 22 "Net-(J10-Pin_4)")
 			(pinfunction "Pin_4")
 			(pintype "passive")
@@
 			)
 		)
-		(property "Value" "630mV"
+		(property "Value" "630mV 1N5819"
 			(at 3.81 2.47 0)
 			(layer "F.Fab")
@@
 			(remove_unused_layers no)
 			(roundrect_rratio 0.092593)
-			(net 25 "unconnected-(J6-Pin_1-Pad1)")
+			(net 24 "unconnected-(J6-Pin_1-Pad1)")
 			(pinfunction "Pin_1")
 			(pintype "passive")
@@
 			(layers "*.Cu" "*.Mask")
 			(remove_unused_layers no)
-			(net 23 "Net-(J4-Pin_4)")
+			(net 22 "Net-(J10-Pin_4)")
 			(pinfunction "Pin_4")
 			(pintype "passive")
@@
 			(layers "*.Cu" "*.Mask")
 			(remove_unused_layers no)
-			(net 23 "Net-(J4-Pin_4)")
+			(net 22 "Net-(J10-Pin_4)")
 			(pinfunction "Pin_4")
 			(pintype "passive")
@@
 			)
 		)
-		(property "Value" "24V?"
+		(property "Value" "24V  1N4006"
 			(at 3.81 2.47 0)
 			(layer "F.Fab")
@@
 			(remove_unused_layers no)
 			(roundrect_rratio 0.092593)
-			(net 26 "unconnected-(J7-Pin_1-Pad1)")
+			(net 25 "unconnected-(J7-Pin_1-Pad1)")
 			(pinfunction "Pin_1")
 			(pintype "passive")
@@
 			(layers "*.Cu" "*.Mask")
 			(remove_unused_layers no)
-			(net 23 "Net-(J4-Pin_4)")
+			(net 22 "Net-(J10-Pin_4)")
 			(pinfunction "Pin_4")
 			(pintype "passive")
@@
 	)
 	(segment
+		(start 135.81 89.18)
+		(end 135.86 89.23)
+		(width 0.2)
+		(layer "F.Cu")
+		(net 22)
+	)
+	(segment
 		(start 157.485216 41.07)
 		(end 160.32 41.07)
@@
 	)
 	(segment
+		(start 135.81 69.57)
+		(end 135.81 89.18)
+		(width 0.2)
+		(layer "F.Cu")
+		(net 22)
+	)
+	(segment
 		(start 165.18 36.21)
 		(end 165.32 36.35)
@@
 	)
 	(segment
+		(start 135.86 89.23)
+		(end 135.86 108.19)
+		(width 0.2)
+		(layer "F.Cu")
+		(net 22)
+	)
+	(segment
 		(start 157.02 67.07)
 		(end 157.14 67.19)
@@
 	)
 	(segment
-		(start 165.32 36.35)
-		(end 169.37 36.35)
+		(start 135.86 108.19)
+		(end 135.4 108.65)
 		(width 0.2)
 		(layer "F.Cu")
@@
 	)
 	(segment
-		(start 171.54 52.62)
-		(end 171.19 52.97)
+		(start 165.32 36.35)
+		(end 169.37 36.35)
 		(width 0.2)
 		(layer "F.Cu")
@@
 	)
 	(segment
-		(start 157.22 108.64)
-		(end 156.97 108.89)
+		(start 135.4 108.65)
+		(end 135.4 127.67)
 		(width 0.2)
 		(layer "F.Cu")
@@
 	)
 	(segment
-		(start 160.32 41.07)
-		(end 165.18 36.21)
+		(start 171.54 52.62)
+		(end 171.19 52.97)
 		(width 0.2)
 		(layer "F.Cu")
@@
 	)
 	(segment
-		(start 135.81 89.18)
-		(end 135.86 89.23)
-		(width 0.2)
-		(layer "F.Cu")
-		(net 23)
-	)
-	(segment
-		(start 135.81 69.57)
-		(end 135.81 89.18)
-		(width 0.2)
-		(layer "F.Cu")
-		(net 23)
-	)
-	(segment
-		(start 135.86 89.23)
-		(end 135.86 108.19)
-		(width 0.2)
-		(layer "F.Cu")
-		(net 23)
-	)
-	(segment
-		(start 135.86 108.19)
-		(end 135.4 108.65)
+		(start 135.4 127.67)
+		(end 135.59 127.86)
 		(width 0.2)
 		(layer "F.Cu")
-		(net 23)
+		(net 22)
 	)
 	(segment
-		(start 135.4 108.65)
-		(end 135.4 127.67)
+		(start 157.22 108.64)
+		(end 156.97 108.89)
 		(width 0.2)
 		(layer "F.Cu")
-		(net 23)
+		(net 22)
 	)
 	(segment
-		(start 135.4 127.67)
-		(end 135.59 127.86)
+		(start 160.32 41.07)
+		(end 165.18 36.21)
 		(width 0.2)
 		(layer "F.Cu")
-		(net 23)
+		(net 22)
 	)
 	(embedded_fonts no)

Commit message: UPDATE
Routing:
- net Net-(J10-Pin_4): track 183.5 -> 205.0 mm, vias 0 -> 2
- net Net-(D1-K): track 152.8 -> 174.2 mm, vias 0 -> 2
Changed lines of the file:
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@@
+		(net 1)
+	)
+	(via
+		(at 127.94 79.56)
+		(size 2.7)
+		(drill 1.3)
+		(layers "F.Cu" "B.Cu")
+		(net 1)
+	)
+	(via
+		(at 149.12 80.14)
+		(size 2.7)
+		(drill 1.3)
+		(layers "F.Cu" "B.Cu")
 		(net 1)
 	)
@@
 	)
 	(segment
+		(start 149.12 80.14)
+		(end 128.52 80.14)
+		(width 0.2)
+		(layer "B.Cu")
+		(net 1)
+	)
+	(segment
 		(start 149.02 125.1)
 		(end 149.32 125.4)
@@
 	)
 	(segment
+		(start 128.52 80.14)
+		(end 127.94 79.56)
+		(width 0.2)
+		(layer "B.Cu")
+		(net 1)
+	)
+	(segment
 		(start 166.52 124.81)
 		(end 149.31 124.81)
@@
 	(segment
 		(start 157.22 89.23)
-		(end 157.22 108.64)
+		(end 157.22 99.11)
 		(width 0.2)
 		(layer "F.Cu")
@@
 	)
 	(segment
+		(start 157.22 99.17)
+		(end 157.22 108.64)
+		(width 0.2)
+		(layer "F.Cu")
+		(net 22)
+	)
+	(segment
 		(start 171.19 52.97)
 		(end 171.16 52.94)
@@
 		(net 22)
 	)
+	(via
+		(at 135.9 98.74)
+		(size 2.7)
+		(drill 1.3)
+		(layers "F.Cu" "B.Cu")
+		(net 22)
+	)
+	(via
+		(at 157.22 99.17)
+		(size 2.7)
+		(drill 1.3)
+		(layers "F.Cu" "B.Cu")
+		(net 22)
+	)
+	(segment
+		(start 157.22 99.17)
+		(end 136.33 99.17)
+		(width 0.2)
+		(layer "B.Cu")
+		(net 22)
+	)
+	(segment
+		(start 136.33 99.17)
+		(end 135.9 98.74)
+		(width 0.2)
+		(layer "B.Cu")
+		(net 22)
+	)

Commit message: UPDATE
Routing:
- net Net-(D1-K): track 174.2 -> 167.6 mm, vias 2 -> 4
Changed lines of the file:
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@@
+	)
+	(via
+		(at 166 121.15)
+		(size 2.7)
+		(drill 1.3)
+		(layers "F.Cu" "B.Cu")
+		(net 1)
+	)
+	(via
+		(at 148.9 120.7)
+		(size 2.7)
+		(drill 1.3)
+		(layers "F.Cu" "B.Cu")
+		(net 1)
 	)
 	(via
@@
 	)
 	(segment
-		(start 148.99 124.91)
-		(end 149.32 125.24)
+		(start 149.35 121.15)
+		(end 148.9 120.7)
 		(width 0.2)
 		(layer "B.Cu")
@@
 	)
 	(segment
-		(start 149.31 124.81)
-		(end 149.02 125.1)
-		(width 0.2)
-		(layer "B.Cu")
-		(net 1)
-	)
-	(segment
-		(start 149.32 125.4)
-		(end 149.32 127.94)
-		(width 0.2)
-		(layer "B.Cu")
-		(net 1)
-	)
-	(segment
-		(start 149.09 124.81)
-		(end 148.99 124.91)
+		(start 166 121.15)
+		(end 149.35 121.15)
 		(width 0.2)
 		(layer "B.Cu")
@@
 	)
 	(segment
-		(start 149.02 125.1)
-		(end 149.32 125.4)
-		(width 0.2)
-		(layer "B.Cu")
-		(net 1)
-	)
-	(segment
 		(start 128.52 80.14)
 		(end 127.94 79.56)
 		(width 0.2)
 		(layer "B.Cu")
-		(net 1)
-	)
-	(segment
-		(start 166.52 124.81)
-		(end 149.31 124.81)
-		(width 0.2)
-		(layer "B.Cu")
-		(net 1)
-	)
-	(segment
-		(start 149.32 125.24)
-		(end 149.32 127.94)
-		(width 0.2)
-		(layer "B.Cu")

Commit message: UPDATE
Parts:
- C1, C2, C3, D1, D2, D3, D4, D5, J10, J11, J1_24V_ROW1, J1_CN1_24V1, J2_CN2_9V_Main1, J3_CN3_9V_Main1, J4, J5, J6, J7, J8, J9, L1_Inductor1, Q1, Q2, R1, R2, R3, R4, R5, R6, U1: moved to B.Cu
- moved R6 62.0 mm to (112.0, 60.1), turned to 0 degrees
- moved Q1 55.9 mm to (115.1, 118.8), turned to 0 degrees
- moved D3 55.7 mm to (115.2, 80.3)
- moved R2 53.6 mm to (116.2, 93.3)
- moved C3 52.5 mm to (116.8, 52.9)
- moved Q2 50.9 mm to (117.6, 110.6), turned to 0 degrees
- moved C2 48.0 mm to (119.0, 42.2)
- moved D1 47.0 mm to (119.5, 124.8)
- moved R3 46.8 mm to (119.6, 87.9)
- moved D2 45.3 mm to (120.4, 90.6)
- moved R1 45.2 mm to (120.4, 101.9), turned to 180 degrees
- moved J5 39.0 mm to (162.5, 108.7), turned to 180 degrees
- moved R5 39.0 mm to (123.5, 48.7)
- moved R4 38.9 mm to (123.6, 65.2), turned to 180 degrees
- moved J4 38.6 mm to (162.3, 127.9), turned to 180 degrees
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
Commit message: UPDATE
Routing:
- net Net-(D3-A): track 234.7 -> 231.2 mm
Changed lines of the file:
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@@
 			(at 3.81 -2.47 90)
 			(layer "B.Fab")
+			(hide yes)
 			(effects
 				(font
@@
 	)
 	(segment
-		(start 146.506428 132.42)
-		(end 146.236428 132.69)
-		(width 0.2)
-		(layer "B.Cu")
-		(net 19)
-	)
-	(segment
 		(start 124.876428 84.38)
 		(end 124.876428 70.37)
@@
 	)
 	(segment
-		(start 146.116428 132.57)
-		(end 124.576428 132.57)
-		(width 0.2)
-		(layer "B.Cu")
-		(net 19)
-	)
-	(segment
-		(start 158.343928 141)
-		(end 158.343928 133.4775)
-		(width 0.2)
-		(layer "B.Cu")
-		(net 19)
-	)
-	(segment
 		(start 124.786428 84.29)
 		(end 124.876428 84.38)
@@
 	)
 	(segment
-		(start 146.236428 132.69)
-		(end 146.116428 132.57)
+		(start 158.343928 133.96)
+		(end 146.506428 133.96)
 		(width 0.2)
 		(layer "B.Cu")
@@
 	)
 	(segment
-		(start 158.343928 133.4775)
-		(end 157.316428 132.45)
-		(width 0.2)
-		(layer "B.Cu")
-		(net 19)
-	)
-	(segment
-		(start 124.576428 132.57)
-		(end 124.576428 132.46)
-		(width 0.2)
-		(layer "B.Cu")
-		(net 19)
-	)
-	(segment
-		(start 124.576428 132.46)
-		(end 124.856428 132.18)
-		(width 0.2)
-		(layer "B.Cu")
-		(net 19)
-	)
-	(segment
 		(start 146.696428 108.65)
 		(end 146.696428 127.67)
@@
 	)
 	(segment
+		(start 124.856428 133.856428)
+		(end 124.856428 127.94)
+		(width 0.2)
+		(layer "B.Cu")
+		(net 19)
+	)
+	(segment
 		(start 146.236428 108.19)
 		(end 146.696428 108.65)
@@
 	)
 	(segment
-		(start 157.316428 132.45)
-		(end 146.706428 132.45)
-		(width 0.2)
-		(layer "B.Cu")
-		(net 19)
-	)
-	(segment
 		(start 156.916428 51.33)
 		(end 156.916428 45.72)
@@
 	)
 	(segment
-		(start 146.706428 132.45)
-		(end 146.506428 132.65)
+		(start 156.926428 51.34)
+		(end 156.916428 51.33)
 		(width 0.2)
 		(layer "B.Cu")
@@
 	)
 	(segment
-		(start 156.926428 51.34)
-		(end 156.916428 51.33)
+		(start 125.126428 108.89)
+		(end 125.126428 89.48)
 		(width 0.2)
 		(layer "B.Cu")
@@
 	)
 	(segment
-		(start 124.856428 132.18)
-		(end 124.856428 127.94)
+		(start 146.306428 61.96)
+		(end 156.926428 51.34)
 		(width 0.2)
 		(layer "B.Cu")
@@
 	)
 	(segment
-		(start 125.126428 108.89)
-		(end 125.126428 89.48)
+		(start 158.343928 141)
+		(end 158.343928 133.96)
 		(width 0.2)
 		(layer "B.Cu")
@@
 	)
 	(segment
-		(start 146.306428 61.96)
-		(end 156.926428 51.34)
+		(start 146.506428 127.86)
+		(end 146.506428 133.96)
 		(width 0.2)
 		(layer "B.Cu")
@@
 	)
 	(segment
-		(start 146.506428 132.65)
-		(end 146.506428 127.86)
+		(start 146.506428 133.96)
+		(end 124.96 133.96)
 		(width 0.2)
 		(layer "B.Cu")
@@
 	)
 	(segment
+		(start 124.96 133.96)
+		(end 124.856428 133.856428)
+		(width 0.2)
+		(layer "B.Cu")
+		(net 19)
+	)
+	(segment
 		(start 124.876428 70.37)
 		(end 125.076428 70.17)
@@
 		(width 0.2)
 		(layer "B.Cu")
-		(net 19)
-	)
-	(segment
-		(start 146.506428 127.86)
-		(end 146.506428 132.42)
-		(width 0.2)
-		(layer "B.Cu")

Commit message: UPDATE
Parts:
- moved R4 0.05 mm to (123.5, 65.2)
Connections:
- U1 pad 6: unconnected-(U1-Vin-Pad6) -> Net-(D5-K)
Routing:
- net Net-(D5-K): track 40.7 -> 73.3 mm
- net Net-(D1-A): track 123.1 -> 123.7 mm
- net Net-(D2-K): track 72.7 -> 72.1 mm

Commit message: UPDATE
Parts:
- C1, C2, C3, D1, D2, D3, D4, D5, J10, J11, J1_24V_ROW1, J1_CN1_24V1, J2_CN2_9V_Main1, J3_CN3_9V_Main1, J4, J5, J6, J7, J8, J9, L1_Inductor1, Q1, Q2, R1, R2, R3, R4, R5, R6, U1: moved to F.Cu
- moved R6 62.0 mm to (174.0, 60.1), turned to 180 degrees
- moved Q1 55.9 mm to (171.0, 118.8), turned to 180 degrees
- moved D3 55.7 mm to (170.9, 80.3)
- moved R2 53.6 mm to (169.8, 93.3)
- moved C3 52.5 mm to (169.3, 52.9)
- moved Q2 50.9 mm to (168.5, 110.6), turned to 180 degrees
- moved C2 48.0 mm to (167.0, 42.2)
- moved D1 47.0 mm to (166.5, 124.8)
- moved R3 46.8 mm to (166.4, 87.9)
- moved D2 45.3 mm to (165.7, 90.6)
- moved R1 45.2 mm to (165.6, 101.9), turned to 0 degrees
- moved J5 39.0 mm to (123.5, 108.7), turned to 0 degrees
- moved R5 39.0 mm to (162.5, 48.7)
- moved R4 39.0 mm to (162.5, 65.2), turned to 0 degrees
- moved J4 38.6 mm to (123.7, 127.9), turned to 0 degrees
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Connections:
- J1_24V_ROW1 pad 2: unconnected-(J1_24V_ROW1-Pin_2-Pad2) -> Net-(D4-A)
- J1_24V_ROW1 pad 3: unconnected-(J1_24V_ROW1-Pin_3-Pad3) -> Net-(D3-A)
Routing:
- net Net-(D4-A): track 335.6 -> 351.3 mm
- net Net-(D3-A): track 231.2 -> 240.7 mm
Other:
- board text added: "2026.1.29"
- board text removed: "2026.1.26"

Commit message: UPDATE
Routing:
- net Net-(D1-A): track 123.7 -> 121.5 mm
- net Net-(D2-K): track 72.1 -> 71.4 mm
Changed lines of the file:
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@@
-	)
-	(segment
-		(start 165.67 93.266428)
-		(end 165.67 90.62)
-		(width 1)
-		(layer "F.Cu")
-		(net 4)
 	)
 	(segment
@@
 	)
 	(segment
-		(start 162.78 96.136428)
-		(end 165.616428 93.3)
-		(width 1)
-		(layer "F.Cu")
-		(net 4)
-	)
-	(segment
-		(start 163.02 123.44)
-		(end 162.78 123.44)
-		(width 0.2)
+		(start 165.67 90.62)
+		(end 165.67 92.45)
+		(width 1)
 		(layer "F.Cu")
 		(net 4)
@@
 	)
 	(segment
-		(start 163.696428 124.116428)
-		(end 163.02 123.44)
-		(width 1)
-		(layer "F.Cu")
-		(net 4)
-	)
-	(segment
 		(start 147.4425 140.91)
 		(end 150.8025 137.55)
@@
 	)
 	(segment
+		(start 163.68 124.223572)
+		(end 163.7 124.243572)
+		(width 0.2)
+		(layer "F.Cu")
+		(net 4)
+	)
+	(segment
 		(start 160.7325 137.7125)
 		(end 160.69 137.67)
@@
 	)
 	(segment
+		(start 165.67 92.45)
+		(end 163.68 94.44)
+		(width 1)
+		(layer "F.Cu")
+		(net 4)
+	)
+	(segment
 		(start 163.696428 124.24)
 		(end 163.696428 124.116428)
@@
 	)
 	(segment
-		(start 162.78 123.44)
-		(end 162.78 96.136428)
-		(width 1)
-		(layer "F.Cu")
-		(net 4)
-	)
-	(segment
 		(start 160.7325 140.91)
 		(end 160.7325 137.7125)
@@
 	)
 	(segment
+		(start 163.68 94.44)
+		(end 163.68 124.223572)
+		(width 1)
+		(layer "F.Cu")
+		(net 4)
+	)
+	(segment
 		(start 160.69 137.67)
 		(end 160.81 137.55)
@@
 	)
 	(segment
-		(start 172.73 132.43)
-		(end 171.64 132.43)
-		(width 0.2)
-		(layer "F.Cu")
-		(net 8)
-	)
-	(segment
-		(start 172.73 132.43)
-		(end 166.52 132.43)
+		(start 166.84 132.56)
+		(end 166.71 132.43)
 		(width 1)
 		(layer "F.Cu")
@@
 	)
 	(segment
-		(start 158.6 148.02)
-		(end 163.16 148.02)
-		(width 1)
-		(layer "F.Cu")
-		(net 8)
-	)
-	(segment
 		(start 130.99 148.02)
 		(end 144.58 148.02)
@@
 	)
 	(segment
+		(start 173.11 132.56)
+		(end 166.84 132.56)
+		(width 1)
+		(layer "F.Cu")
+		(net 8)
+	)
+	(segment
 		(start 131.656428 144.52)
 		(end 131.6725 144.503928)
@@
 	)
 	(segment
+		(start 173.11 138.07)
+		(end 163.16 148.02)
+		(width 1)
+		(layer "F.Cu")
+		(net 8)
+	)
+	(segment
 		(start 172.99 118.84)
 		(end 171 118.84)
@@
 	)
 	(segment
-		(start 172.73 138.45)
-		(end 172.73 132.43)
-		(width 1)
-		(layer "F.Cu")
-		(net 8)
-	)
-	(segment
 		(start 144.58 148.02)
 		(end 158.6 148.02)
@@
 	)
 	(segment
-		(start 172.98 132.43)
-		(end 173.11 132.56)
-		(width 0.2)
-		(layer "F.Cu")
-		(net 8)
-	)
-	(segment
 		(start 130.99 145.203572)
 		(end 130.966428 145.18)
@@
 	)
 	(segment
-		(start 163.16 148.02)
-		(end 172.73 138.45)
-		(width 1)
-		(layer "F.Cu")
-		(net 8)
-	)
-	(segment
 		(start 131.6725 144.503928)
 		(end 131.6725 141)
@@
 	)
 	(segment
+		(start 166.71 132.43)
+		(end 166.52 132.43)
+		(width 1)
+		(layer "F.Cu")
+		(net 8)
+	)
+	(segment
 		(start 173.19 118.81)
 		(end 173.19 110.52)
@@
 	)
 	(segment
+		(start 163.16 148.02)
+		(end 158.6 148.02)
+		(width 1)
+		(layer "F.Cu")
+		(net 8)
+	)
+	(segment
 		(start 173.19 110.52)
 		(end 173.11 110.44)
@@
 	)
 	(segment
-		(start 171.64 132.43)
-		(end 172.98 132.43)
-		(width 0.2)
-		(layer "F.Cu")
-		(net 8)
-	)
-	(segment
 		(start 131.626428 144.52)
 		(end 131.656428 144.52)
@@
 		(layer "F.Cu")
 		(net 8)
+	)
+	(segment
+		(start 173.11 138.07)
+		(end 173.11 132.56)
+		(width 1)
+		(layer "F.Cu")
+		(net 8)
