File: KiCad/TC_Interface_Board/TC_Interface_Board.kicad_pcb (KiCad board)
At the start: 2 copper layers, 30 parts, among them J10 Conn_01x05, J11 Conn_01x05, J1_24V_ROW1 Conn_01x04, J1_CN1_24V1 Conn_01x03, J2_CN2_9V_Main1 Conn_01x02, J3_CN3_9V_Main1 Conn_01x02, J4 Conn_01x05, J5 Conn_01x05, J6 Conn_01x05, J7 Conn_01x05, J8 Conn_01x05, J9 Conn_01x05, Q1 DTC143E, Q2 DTC143E, U1 MC34063AP

Commit message: UPDATE
Parts:
- moved D2 0.97 mm to (166.3, 89.9)
- moved R1 0.32 mm to (165.9, 101.8)
Routing:
- net Net-(D1-A): track 121.5 -> 119.9 mm
- net Net-(D2-A): track 12.5 -> 13.3 mm
Changed lines of the file:
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@@
 	(footprint "Resistor_THT:R_Axial_DIN0207_L6.3mm_D2.5mm_P7.62mm_Horizontal"
 		(layer "F.Cu")
-		(at 165.64 101.92)
+		(at 165.94 101.81)
 		(descr "Resistor, Axial_DIN0207 series, Axial, Horizontal, pin pitch=7.62mm, 0.25W = 1/4W, length*diameter=6.3*2.5mm^2, http://cdn-reichelt.de/documents/datenblatt/B400/1_4W%23YAG.pdf")
 		(tags "Resistor Axial_DIN0207 series Axial Horizontal pin pitch 7.62mm 0.25W = 1/4W length 6.3mm diameter 2.5mm")
@@
 	(footprint "Diode_THT:D_DO-41_SOD81_P7.62mm_Horizontal"
 		(layer "F.Cu")
-		(at 165.67 90.62 -90)
+		(at 166.34 89.92 -90)
 		(descr "Diode, DO-41_SOD81 series, Axial, Horizontal, pin pitch=7.62mm, length*diameter=5.2*2.7mm^2, https://www.diodes.com/assets/Package-Files/DO-41-Plastic.pdf")
 		(tags "Diode DO-41_SOD81 series Axial Horizontal pin pitch 7.62mm  length 5.2mm diameter 2.7mm")
@@
 	(footprint "Connector_JST:JST_VH_B3P-VH-B_1x03_P3.96mm_Vertical"
 		(layer "F.Cu")
-		(at 123.7525 141)
+		(at 123.74 141.01)
 		(descr "JST VH PBT series connector, B3P-VH-B (http://www.jst-mfg.com/product/pdf/eng/eVH.pdf), generated with kicad-footprint-generator")
 		(tags "connector JST VH vertical")
@@
 		(start 165.96 110.62)
 		(end 165.96 102.24)
-		(width 1)
+		(width 0.8)
 		(layer "F.Cu")
 		(net 2)
 	)
 	(segment
-		(start 165.64 101.92)
-		(end 165.64 98.27)
-		(width 1)
+		(start 165.94 97.94)
+		(end 166.34 97.54)
+		(width 0.2)
 		(layer "F.Cu")
 		(net 2)
@@
 	)
 	(segment
+		(start 165.94 101.81)
+		(end 165.94 97.94)
+		(width 0.8)
+		(layer "F.Cu")
+		(net 2)
+	)
+	(segment
 		(start 162.43 58.71)
 		(end 162.43 60.646428)
@@
 	)
 	(segment
-		(start 130.966428 145.18)
-		(end 131.626428 144.52)
-		(width 1)
-		(layer "F.Cu")
-		(net 8)
-	)
-	(segment
 		(start 168.68 110.44)
 		(end 168.5 110.62)
@@
 	)
 	(segment
-		(start 130.99 148.02)
-		(end 144.58 148.02)
-		(width 1)
-		(layer "F.Cu")
-		(net 8)
-	)
-	(segment
 		(start 173.16 118.84)
 		(end 173.19 118.81)
@@
 	)
 	(segment
-		(start 131.656428 144.52)
-		(end 131.6725 144.503928)
-		(width 0.2)
-		(layer "F.Cu")
-		(net 8)
-	)
-	(segment
 		(start 158.71 145.33)
 		(end 158.71 147.91)
@@
 	)
 	(segment
+		(start 131.72 148.02)
+		(end 144.58 148.02)
+		(width 1)
+		(layer "F.Cu")
+		(net 8)
+	)
+	(segment
 		(start 144.58 148.02)
 		(end 158.6 148.02)
@@
 	)
 	(segment
-		(start 130.99 145.203572)
-		(end 130.966428 145.18)
-		(width 0.2)
+		(start 173.11 132.56)
+		(end 173.11 118.96)
+		(width 1)
 		(layer "F.Cu")
 		(net 8)
 	)
 	(segment
-		(start 173.11 132.56)
-		(end 173.11 118.96)
-		(width 1)
+		(start 131.72 148.02)
+		(end 131.66 147.96)
+		(width 0.2)
 		(layer "F.Cu")
 		(net 8)
@@
 	)
 	(segment
-		(start 131.6725 144.503928)
-		(end 131.6725 141)
-		(width 1)
-		(layer "F.Cu")
-		(net 8)
-	)
-	(segment
 		(start 173.26 110.29)
 		(end 173.26 101.92)
@@
 	)
 	(segment
-		(start 131.626428 144.52)
-		(end 131.656428 144.52)
-		(width 0.2)
-		(layer "F.Cu")
-		(net 8)
-	)
-	(segment
 		(start 143.4825 143.7925)
 		(end 144.69 145)
@@
 	)
 	(segment
-		(start 130.61 148.4)
-		(end 130.99 148.02)
-		(width 0.2)
+		(start 131.66 147.96)
+		(end 131.66 141.01)
+		(width 1)
 		(layer "F.Cu")
 		(net 8)
@@
 	)
 	(segment
-		(start 130.99 148.02)
-		(end 130.99 145.203572)
-		(width 1)
-		(layer "F.Cu")
-		(net 8)
-	)
-	(segment
 		(start 167.15 117.53)
 		(end 167.15 110.62)
@@
 		(start 167.23 102.62)
 		(end 169.81 100.04)
-		(width 1)
+		(width 0.8)
 		(layer "F.Cu")
 		(net 9)
@@
 		(start 167.23 110.62)
 		(end 167.23 102.62)
-		(width 1)
+		(width 0.8)
 		(layer "F.Cu")
 		(net 9)
@@
 		(start 169.81 85.64)
 		(end 169.81 84.51)
-		(width 0.2)
+		(width 1)
 		(layer "F.Cu")
 		(net 16)

Commit message: UPDATE
Routing:
- net Net-(D5-K): track 73.3 -> 66.8 mm

Commit message: UPDATE
Parts:
- moved R4 1.47 mm to (162.5, 63.7)
- moved R3 0.59 mm to (166.4, 87.3)
Routing:
- net Net-(D4-A): track 351.3 -> 347.8 mm
- net Net-(U1-Vfb): track 22.1 -> 23.6 mm
- net Net-(D1-K): track 167.8 -> 166.6 mm
- net Net-(D3-K): track 11.3 -> 12.1 mm

Commit message: UPDATE
Parts:
- moved J7 0.67 mm to (123.9, 70.2)
- renumbered J1_CN1_24V1 to J1_CN1, J2_CN2_9V_Main1 to J2_CN2, J3_CN3_9V_Main1 to J3_CN3
Other:
- board outline added: 68.9 x 121.6 mm
Changed lines of the file:
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@@
 		)
 		(fp_text user "K"
-			(at 0 -2.1 90)
+			(at 0.12 2.11 180)
 			(layer "F.SilkS")
 			(effects
@@
 		(descr "JST VH PBT series connector, B2P-VH-B (http://www.jst-mfg.com/product/pdf/eng/eVH.pdf), generated with kicad-footprint-generator")
 		(tags "connector JST VH vertical")
-		(property "Reference" "J3_CN3_9V_Main1"
+		(property "Reference" "J3_CN3"
 			(at 2.31 -5.51 0)
 			(layer "F.SilkS")
@@
 		(descr "JST VH PBT series connector, B2P-VH-B (http://www.jst-mfg.com/product/pdf/eng/eVH.pdf), generated with kicad-footprint-generator")
 		(tags "connector JST VH vertical")
-		(property "Reference" "J2_CN2_9V_Main1"
+		(property "Reference" "J2_CN2"
 			(at 2.0775 -5.93 0)
 			(layer "F.SilkS")
@@
 		)
 		(fp_text user "K"
-			(at 0 -2.1 90)
+			(at -0.01 2.323572 90)
 			(layer "F.SilkS")
 			(effects
@@
 		)
 		(fp_text user "K"
-			(at 0 -2.1 90)
+			(at 0 2.323572 90)
 			(layer "F.Fab")
 			(effects
@@
 		(tags "THT DIP DIL PDIP 2.54mm 7.62mm 300mil")
 		(property "Reference" "U1"
-			(at 3.81 -2.33 90)
+			(at 3.785 11.62 90)
 			(layer "F.SilkS")
 			(effects
@@
 		(descr "JST VH PBT series connector, B3P-VH-B (http://www.jst-mfg.com/product/pdf/eng/eVH.pdf), generated with kicad-footprint-generator")
 		(tags "connector JST VH vertical")
-		(property "Reference" "J1_CN1_24V1"
+		(property "Reference" "J1_CN1"
 			(at 4.07 -5.93 0)
 			(layer "F.SilkS")
@@
 	(footprint "Connector_JST:JST_VH_B5P-VH-B_1x05_P3.96mm_Vertical"
 		(layer "F.Cu")
-		(at 123.93 69.57)
+		(at 123.88 70.24)
 		(descr "JST VH PBT series connector, B5P-VH-B (http://www.jst-mfg.com/product/pdf/eng/eVH.pdf), generated with kicad-footprint-generator")
 		(tags "connector JST VH vertical")
@@
 		)
 	)
+	(gr_rect
+		(start 108.8 32.13)
+		(end 177.69 153.68)
+		(stroke
+			(width 0.05)
+			(type default)
+		)
+		(fill no)
+		(layer "Edge.Cuts")
+	)
 	(image
 		(at 143.028214 93.288861)
@@
 	)
 	(segment
-		(start 163.696428 124.24)
-		(end 163.696428 124.116428)
-		(width 0.2)
-		(layer "F.Cu")
-		(net 4)
-	)
-	(segment
 		(start 160.7325 140.91)
 		(end 160.7325 137.7125)
@@
 		(start 132.87 55.08)
 		(end 129.13 51.34)
-		(width 4)
+		(width 2)
 		(layer "F.Cu")
 		(net 16)
@@
 		(start 139.75 61.96)
 		(end 132.87 55.08)
-		(width 4)
+		(width 2)
 		(layer "F.Cu")
 		(net 16)

Commit message: UPDATE
Other:
- board text added: "2026.1.30"
- board text removed: "2026.1.29"
Changed lines of the file:
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@@
 		)
 	)
-	(gr_text "2026.1.29"
+	(gr_text "2026.1.30"
 		(at 212 194 0)
 		(layer "F.Cu")

Commit message: UPDATE
Parts:
- removed J1_CN1: Conn_01x03, Connector_JST:JST_VH_B3P-VH-B_1x03_P3.96mm_Vertical
- removed J2_CN2, J3_CN3: Conn_01x02, Connector_JST:JST_VH_B2P-VH-B_1x02_P3.96mm_Vertical
- added J1_CN1_24V1: Conn_01x03, Connector_JST:JST_VH_B3P-VH-B_1x03_P3.96mm_Vertical, F.Cu at (123.6, 140.7)
- added J2_CN2_9V_Main1: Conn_01x02, Connector_JST:JST_VH_B2P-VH-B_1x02_P3.96mm_Vertical, F.Cu at (143.5, 140.5)
- added J3_CN3_9V_Main1: Conn_01x02, Connector_JST:JST_VH_B2P-VH-B_1x02_P3.96mm_Vertical, F.Cu at (156.9, 140.3)
Connections:
- net Net-(D4-A) renamed GND

Commit message: UPDATE
Parts:
- R1: value 220Ω -> 220
- R2: value 10KΩ -> 10K
- R3: value 1.2kΩ -> 1.2K
- R4: value 0.55Ω -> 6.2K
- R5: value 11KΩ -> 0.22
- R6: value 110Ω -> 1K
Connections:
- net Net-(D3-A) renamed -24V
Changed lines of the file:
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@@
 	(net 14 "unconnected-(J10-Pin_1-Pad1)")
 	(net 15 "unconnected-(J11-Pin_1-Pad1)")
-	(net 16 "Net-(D3-A)")
+	(net 16 "-24V")
 	(net 17 "GND")
 	(net 18 "Net-(U1-Vfb)")
@@
 			)
 		)
-		(property "Value" "110Ω"
+		(property "Value" "1K"
 			(at 3.81 2.37 0)
 			(layer "F.Fab")
@@
 			)
 		)
-		(property "Value" "220Ω"
+		(property "Value" "220"
 			(at 3.81 2.37 0)
 			(layer "F.Fab")
@@
 			(net 12 "unconnected-(J8-Pin_1-Pad1)")
 			(pinfunction "Pin_1")
-			(pintype "passive")
+			(pintype "passive+no_connect")
 		)
 		(pad "2" thru_hole circle
@@
 			(layers "*.Cu" "*.Mask")
 			(remove_unused_layers no)
-			(net 16 "Net-(D3-A)")
+			(net 16 "-24V")
 			(pinfunction "Pin_5")
 			(pintype "passive")
@@
 			)
 		)
-		(property "Value" "10KΩ"
+		(property "Value" "10K"
 			(at 3.81 2.37 90)
 			(layer "F.Fab")
@@
 			(layers "*.Cu" "*.Mask")
 			(remove_unused_layers no)
-			(net 16 "Net-(D3-A)")
+			(net 16 "-24V")
 			(pintype "passive")
 		)
@@
 			(net 13 "unconnected-(J9-Pin_1-Pad1)")
 			(pinfunction "Pin_1")
-			(pintype "passive")
+			(pintype "passive+no_connect")
 		)
 		(pad "2" thru_hole circle
@@
 			(layers "*.Cu" "*.Mask")
 			(remove_unused_layers no)
-			(net 16 "Net-(D3-A)")
+			(net 16 "-24V")
 			(pinfunction "Pin_5")
 			(pintype "passive")
@@
 			)
 		)
-		(property "Value" "1.2kΩ"
+		(property "Value" "1.2K"
 			(at 10.83 -2.243572 90)
 			(layer "F.Fab")
@@
 			(net 20 "unconnected-(J5-Pin_1-Pad1)")
 			(pinfunction "Pin_1")
-			(pintype "passive")
+			(pintype "passive+no_connect")
 		)
 		(pad "2" thru_hole circle
@@
 			(layers "*.Cu" "*.Mask")
 			(remove_unused_layers no)
-			(net 16 "Net-(D3-A)")
+			(net 16 "-24V")
 			(pinfunction "Pin_5")
 			(pintype "passive")
@@
 			)
 		)
-		(property "Value" "11KΩ"
+		(property "Value" "0.22"
 			(at 5.08 2.37 90)
 			(layer "F.Fab")
@@
 			(layers "*.Cu" "*.Mask")
 			(remove_unused_layers no)
-			(net 16 "Net-(D3-A)")
+			(net 16 "-24V")
 			(pinfunction "A")
 			(pintype "passive")
@@
 			(net 21 "unconnected-(J6-Pin_1-Pad1)")
 			(pinfunction "Pin_1")
-			(pintype "passive")
+			(pintype "passive+no_connect")
 		)
 		(pad "2" thru_hole circle
@@
 			(layers "*.Cu" "*.Mask")
 			(remove_unused_layers no)
-			(net 16 "Net-(D3-A)")
+			(net 16 "-24V")
 			(pinfunction "Pin_5")
 			(pintype "passive")
@@
 			(layers "*.Cu" "*.Mask")
 			(remove_unused_layers no)
-			(net 16 "Net-(D3-A)")
+			(net 16 "-24V")
 			(pinfunction "Pin_2")
 			(pintype "passive")
@@
 			(layers "*.Cu" "*.Mask")
 			(remove_unused_layers no)
-			(net 16 "Net-(D3-A)")
+			(net 16 "-24V")
 			(pinfunction "Pin_3")
 			(pintype "passive")
@@
 			(layers "*.Cu" "*.Mask")
 			(remove_unused_layers no)
-			(net 16 "Net-(D3-A)")
+			(net 16 "-24V")
 			(pinfunction "Pin_4")
 			(pintype "passive")
@@
 			(layers "*.Cu" "*.Mask")
 			(remove_unused_layers no)
-			(net 16 "Net-(D3-A)")
+			(net 16 "-24V")
 			(pinfunction "Pin_5")
 			(pintype "passive")
@@
 			(net 15 "unconnected-(J11-Pin_1-Pad1)")
 			(pinfunction "Pin_1")
-			(pintype "passive")
+			(pintype "passive+no_connect")
 		)
 		(pad "2" thru_hole circle
@@
 			(layers "*.Cu" "*.Mask")
 			(remove_unused_layers no)
-			(net 16 "Net-(D3-A)")
+			(net 16 "-24V")
 			(pinfunction "Pin_5")
 			(pintype "passive")
@@
 			(layers "*.Cu" "*.Mask")
 			(remove_unused_layers no)
-			(net 16 "Net-(D3-A)")
+			(net 16 "-24V")
 			(pinfunction "A")
 			(pintype "passive")
@@
 			(net 14 "unconnected-(J10-Pin_1-Pad1)")
 			(pinfunction "Pin_1")
-			(pintype "passive")
+			(pintype "passive+no_connect")
 		)
 		(pad "2" thru_hole circle
@@
 			(layers "*.Cu" "*.Mask")
 			(remove_unused_layers no)
-			(net 16 "Net-(D3-A)")
+			(net 16 "-24V")
 			(pinfunction "Pin_5")
 			(pintype "passive")
@@
 			(net 22 "unconnected-(J7-Pin_1-Pad1)")
 			(pinfunction "Pin_1")
-			(pintype "passive")
+			(pintype "passive+no_connect")
 		)
 		(pad "2" thru_hole circle
@@
 			(layers "*.Cu" "*.Mask")
 			(remove_unused_layers no)
-			(net 16 "Net-(D3-A)")
+			(net 16 "-24V")
 			(pinfunction "Pin_5")
 			(pintype "passive")
@@
 			)
 		)
-		(property "Value" "0.55Ω"
+		(property "Value" "6.2K"
 			(at 3.81 2.37 0)
 			(layer "F.Fab")

Commit message: update
Other:
- board text added: "2026.2.1"
- board text removed: "2026.1.30"
Changed lines of the file:
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@@
 		)
 	)
-	(gr_text "2026.1.30"
+	(gr_text "2026.2.1"
 		(at 212 194 0)
 		(layer "F.Cu")
