File: KiCad/TC_Interface_Board/TC_Interface_Board.kicad_pcb (KiCad board)
At the start: 2 copper layers, 68.9 x 121.6 mm, 30 parts, among them J1 Conn_01x05, J1_24V1 JST_VH_01x04, J1_CN1 JST_VH_01x03, J2 Conn_01x05, J2_CN1 JST_VH_01x02, J3 Conn_01x05, J3_CN1 JST_VH_01x02, J4 Conn_01x05, J5 Conn_01x05, J6 Conn_01x05, J7 Conn_01x05, J8 Conn_01x05, Q1 DTC143E, Q2 DTC143E, U1 MC34063AP

Commit message: UPDATE
Parts:
- R6: footprint Resistor_THT:R_Axial_DIN0207_L6.3mm_D2.5mm_P15.24mm_Horizontal -> Resistor_THT:R_Axial_DIN0204_L3.6mm_D1.6mm_P7.62mm_Horizontal
- moved R6 7.73 mm to (166.3, 60.2), turned to 0 degrees
Connections:
- D1 pad 1: /TC_CMD_BUS -> /CMD_IN
- D1 pad 2: GND -> Net-(D1-A)
- D2 pad 1: /CMD_IN -> Net-(D2-K)
- D2 pad 2: /Q2C_NODE -> GND
- D5 pad 1: Net-(D5-K) -> unconnected-(D5-K-Pad1)
- Q1 pad 2: Net-(Q1-C) -> Net-(D2-K)
- Q1 pad 3: /TC_CMD_BUS -> Net-(Q1-B)
- Q2 pad 2: /Q2C_NODE -> Net-(Q1-B)
- Q2 pad 3: Net-(Q1-C) -> Net-(D1-A)
- R1 pad 1: Net-(D3-K) -> Net-(D1-A)
- R1 pad 2: /MC34063_SW_NODE -> GND
- R2 pad 1: /Q2C_NODE -> +24V
- R2 pad 2: GND -> Net-(Q1-B)
- R3 pad 1: Net-(Q1-C) -> Net-(Q1-B)
- R5 pad 1: GND -> /MC34063_SW_NODE
- R5 pad 2: Net-(U1-Vfb) -> Net-(D3-K)
- R6 pad 1: /CMD_IN -> Net-(U1-Vfb)
- R6 pad 2: Net-(D5-K) -> GND
Routing:
- net Net-(D5-K): track 66.5 -> 0.00 mm
- net (no net): track 55.4 -> 105.5 mm
- net /MC34063_SW_NODE: track 0.00 -> 16.4 mm
- net Net-(D1-A): track 0.00 -> 13.3 mm
- net GND: track 522.3 -> 511.9 mm
- net +24V: track 240.7 -> 243.4 mm

Commit message: UPDATE
Parts:
- R5: footprint Resistor_THT:R_Axial_DIN0207_L6.3mm_D2.5mm_P7.62mm_Horizontal -> Resistor_THT:R_Axial_DIN0309_L9.0mm_D3.2mm_P12.70mm_Horizontal
- moved D5 1.37 mm to (145.1, 37.3)
- moved R5 1.27 mm to (162.4, 47.4)
- moved R2 0.84 mm to (169.9, 93.8)
Connections:
- net Net-(D1-A) renamed /Q2_BASE
- D2 pad 1: Net-(D2-K) -> /TC_CMD_BUS
- D5 pad 1: unconnected-(D5-K-Pad1) -> /MC34063_TC
- Q1 pad 2: Net-(D2-K) -> /TC_CMD_BUS
- R5 pad 2: Net-(D3-K) -> /MC34063_TC
Changed lines of the file:
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@@
 	(net 17 "Net-(D3-K)")
 	(net 18 "unconnected-(J7-Pin_1-Pad1)")
-	(net 19 "Net-(D1-A)")
-	(net 20 "Net-(D2-K)")
-	(net 21 "Net-(Q1-B)")
-	(net 22 "unconnected-(D5-K-Pad1)")
+	(net 19 "/Q2_BASE")
+	(net 20 "Net-(Q1-B)")
 	(footprint "Connector_JST:JST_VH_B5P-VH-B_1x05_P3.96mm_Vertical"
 		(layer "F.Cu")
@@
 		(tags "CP Radial series Radial pin pitch 2.50mm diameter 5mm height 7mm Electrolytic Capacitor")
 		(property "Reference" "C3"
-			(at 1.14 5.43 90)
+			(at -2.02 2.19 90)
 			(layer "F.SilkS")
 			(effects
@@
 			(layers "*.Cu" "*.Mask")
 			(remove_unused_layers no)
-			(net 19 "Net-(D1-A)")
+			(net 19 "/Q2_BASE")
 			(pintype "passive")
 		)
@@
 	(footprint "Resistor_THT:R_Axial_DIN0207_L6.3mm_D2.5mm_P7.62mm_Horizontal"
 		(layer "F.Cu")
-		(at 169.8498 92.9894 90)
+		(at 169.92 93.83 90)
 		(descr "Resistor, Axial_DIN0207 series, Axial, Horizontal, pin pitch=7.62mm, 0.25W = 1/4W, length*diameter=6.3*2.5mm^2, http://cdn-reichelt.de/documents/datenblatt/B400/1_4W%23YAG.pdf")
 		(tags "Resistor Axial_DIN0207 series Axial Horizontal pin pitch 7.62mm 0.25W = 1/4W length 6.3mm diameter 2.5mm")
@@
 			(layers "*.Cu" "*.Mask")
 			(remove_unused_layers no)
-			(net 21 "Net-(Q1-B)")
+			(net 20 "Net-(Q1-B)")
 			(pintype "passive")
 		)
@@
 			(layers "*.Cu" "*.Mask")
 			(remove_unused_layers no)
-			(net 21 "Net-(Q1-B)")
+			(net 20 "Net-(Q1-B)")
 			(pintype "passive")
 		)
@@
 			(remove_unused_layers no)
 			(roundrect_rratio 0.15625)
-			(net 20 "Net-(D2-K)")
+			(net 10 "/TC_CMD_BUS")
 			(pinfunction "K")
 			(pintype "passive")
@@
 			(layers "*.Cu" "*.Mask")
 			(remove_unused_layers no)
-			(net 19 "Net-(D1-A)")
+			(net 19 "/Q2_BASE")
 			(pinfunction "A")
 			(pintype "passive")
@@
 			(layers "*.Cu" "*.Mask")
 			(remove_unused_layers no)
-			(net 21 "Net-(Q1-B)")
+			(net 20 "Net-(Q1-B)")
 			(pinfunction "C")
 			(pintype "passive")
@@
 			(layers "*.Cu" "*.Mask")
 			(remove_unused_layers no)
-			(net 19 "Net-(D1-A)")
+			(net 19 "/Q2_BASE")
 			(pinfunction "B")
 			(pintype "input")
@@
 		)
 	)
-	(footprint "Resistor_THT:R_Axial_DIN0207_L6.3mm_D2.5mm_P7.62mm_Horizontal"
+	(footprint "Resistor_THT:R_Axial_DIN0309_L9.0mm_D3.2mm_P12.70mm_Horizontal"
 		(layer "F.Cu")
-		(at 162.51 48.69 -90)
-		(descr "Resistor, Axial_DIN0207 series, Axial, Horizontal, pin pitch=7.62mm, 0.25W = 1/4W, length*diameter=6.3*2.5mm^2, http://cdn-reichelt.de/documents/datenblatt/B400/1_4W%23YAG.pdf")
-		(tags "Resistor Axial_DIN0207 series Axial Horizontal pin pitch 7.62mm 0.25W = 1/4W length 6.3mm diameter 2.5mm")
+		(at 162.36 47.43 -90)
+		(descr "Resistor, Axial_DIN0309 series, Axial, Horizontal, pin pitch=12.7mm, 0.5W = 1/2W, length*diameter=9*3.2mm^2, http://cdn-reichelt.de/documents/datenblatt/B400/1_4W%23YAG.pdf")
+		(tags "Resistor Axial_DIN0309 series Axial Horizontal pin pitch 12.7mm 0.5W = 1/2W length 9mm diameter 3.2mm")
 		(property "Reference" "R5"
-			(at 3.81 -2.37 270)
+			(at 6.35 -2.72 270)
 			(layer "F.SilkS")
 			(effects
@@
 		)
 		(property "Value" "1k"
-			(at 3.81 2.37 270)
+			(at 6.35 2.72 270)
 			(layer "F.Fab")
 			(effects
@@
 		(attr through_hole)
 		(fp_line
-			(start 0.54 1.37)
-			(end 7.08 1.37)
-			(stroke
-				(width 0.12)
-				(type solid)
-			)
-			(layer "F.SilkS")
-		)
-		(fp_line
-			(start 7.08 1.37)
-			(end 7.08 1.04)
-			(stroke
-				(width 0.12)
-				(type solid)
-			)
-			(layer "F.SilkS")
-		)
-		(fp_line
-			(start 0.54 1.04)
-			(end 0.54 1.37)
-			(stroke
-				(width 0.12)
-				(type solid)
-			)
-			(layer "F.SilkS")
-		)
-		(fp_line
-			(start 0.54 -1.04)
-			(end 0.54 -1.37)
+			(start 1.04 0)
+			(end 1.73 0)
 			(stroke
 				(width 0.12)
@@
 		)
 		(fp_line
-			(start 0.54 -1.37)
-			(end 7.08 -1.37)
+			(start 11.66 0)
+			(end 10.97 0)
 			(stroke
 				(width 0.12)
@@
 			(layer "F.SilkS")
 		)
-		(fp_line
-			(start 7.08 -1.37)
-			(end 7.08 -1.04)
+		(fp_rect
+			(start 1.73 -1.72)
+			(end 10.97 1.72)
 			(stroke
 				(width 0.12)
 				(type solid)
 			)
+			(fill no)
 			(layer "F.SilkS")
 		)
 		(fp_rect
-			(start -1.05 -1.5)
-			(end 8.67 1.5)
+			(start -1.05 -1.85)
+			(end 13.75 1.85)
 			(stroke
 				(width 0.05)
@@
 		(fp_line
 			(start 0 0)
-			(end 0.66 0)
+			(end 1.85 0)
 			(stroke
 				(width 0.1)
@@
 		)
 		(fp_line
-			(start 7.62 0)
-			(end 6.96 0)
+			(start 12.7 0)
+			(end 10.85 0)
 			(stroke
 				(width 0.1)
@@
 		)
 		(fp_rect
-			(start 0.66 -1.25)
-			(end 6.96 1.25)
+			(start 1.85 -1.6)
+			(end 10.85 1.6)
 			(stroke
 				(width 0.1)
@@
 		)
 		(fp_text user "${REFERENCE}"
-			(at 3.81 0 270)
+			(at 6.35 0 270)
 			(layer "F.Fab")
 			(effects
@@
 		)
 		(pad "2" thru_hole circle
-			(at 7.62 0 270)
+			(at 12.7 0 270)
 			(size 1.6 1.6)
 			(drill 0.8)
 			(layers "*.Cu" "*.Mask")
 			(remove_unused_layers no)
-			(net 17 "Net-(D3-K)")
+			(net 8 "/MC34063_TC")
 			(pintype "passive")
 		)
 		(embedded_fonts no)
-		(model "${KICAD9_3DMODEL_DIR}/Resistor_THT.3dshapes/R_Axial_DIN0207_L6.3mm_D2.5mm_P7.62mm_Horizontal.step"
+		(model "${KICAD9_3DMODEL_DIR}/Resistor_THT.3dshapes/R_Axial_DIN0309_L9.0mm_D3.2mm_P12.70mm_Horizontal.step"
 			(offset
 				(xyz 0 0 0)
@@
 		(tags "CP Radial series Radial pin pitch 2.50mm diameter 5mm height 7mm Electrolytic Capacitor")
 		(property "Reference" "C1"
-			(at 1.25 -3.75 0)
+			(at 1.54 3.93 0)
 			(layer "F.SilkS")
 			(effects
@@
 			(layers "*.Cu" "*.Mask")
 			(remove_unused_layers no)
-			(net 20 "Net-(D2-K)")
+			(net 10 "/TC_CMD_BUS")
 			(pinfunction "C")
 			(pintype "passive")
@@
 			(layers "*.Cu" "*.Mask")
 			(remove_unused_layers no)
-			(net 21 "Net-(Q1-B)")
+			(net 20 "Net-(Q1-B)")
 			(pinfunction "B")
 			(pintype "input")
@@
 	(footprint "Diode_THT:D_DO-35_SOD27_P10.16mm_Horizontal"
 		(layer "F.Cu")
-		(at 143.74 37.25 180)
+		(at 145.11 37.29 180)
 		(descr "Diode, DO-35_SOD27 series, Axial, Horizontal, pin pitch=10.16mm, length*diameter=4*2mm^2, http://www.diodes.com/_files/packages/DO-35.pdf")
 		(tags "Diode DO-35_SOD27 series Axial Horizontal pin pitch 10.16mm  length 4mm diameter 2mm")
@@
 			(remove_unused_layers no)
 			(roundrect_rratio 0.15625)
-			(net 22 "unconnected-(D5-K-Pad1)")
+			(net 8 "/MC34063_TC")
 			(pinfunction "K")
 			(pintype "passive")

Commit message: UPDATE
Parts:
- moved R2 9.03 mm to (169.8, 84.8), turned to -90 degrees
Connections:
- C1 pad 1: Net-(D3-K) -> /MC34063_TC
- C2 pad 1: /MC34063_TC -> Net-(D5-K)
- D5 pad 1: /MC34063_TC -> Net-(D5-K)
- R3 pad 1: Net-(Q1-B) -> /CMD_IN
- R5 pad 2: /MC34063_TC -> Net-(D5-K)
Routing:
- net (no net): track 105.5 -> 78.6 mm
- net Net-(Q1-B): track 0.00 -> 26.9 mm
Changed lines of the file:
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@@
 	(net 19 "/Q2_BASE")
 	(net 20 "Net-(Q1-B)")
+	(net 21 "Net-(D5-K)")
 	(footprint "Connector_JST:JST_VH_B5P-VH-B_1x05_P3.96mm_Vertical"
 		(layer "F.Cu")
@@
 	(footprint "Resistor_THT:R_Axial_DIN0207_L6.3mm_D2.5mm_P7.62mm_Horizontal"
 		(layer "F.Cu")
-		(at 169.92 93.83 90)
+		(at 169.82 84.8 -90)
 		(descr "Resistor, Axial_DIN0207 series, Axial, Horizontal, pin pitch=7.62mm, 0.25W = 1/4W, length*diameter=6.3*2.5mm^2, http://cdn-reichelt.de/documents/datenblatt/B400/1_4W%23YAG.pdf")
 		(tags "Resistor Axial_DIN0207 series Axial Horizontal pin pitch 7.62mm 0.25W = 1/4W length 6.3mm diameter 2.5mm")
 		(property "Reference" "R2"
-			(at 1.21 2.49 90)
+			(at 3.9 -2.37 90)
 			(layer "F.SilkS")
 			(effects
@@
 		(attr through_hole)
 		(fp_line
-			(start 7.08 -1.37)
-			(end 7.08 -1.04)
+			(start 0.54 1.37)
+			(end 7.08 1.37)
 			(stroke
 				(width 0.12)
@@
 		)
 		(fp_line
-			(start 0.54 -1.37)
-			(end 7.08 -1.37)
+			(start 7.08 1.37)
+			(end 7.08 1.04)
 			(stroke
 				(width 0.12)
@@
 		)
 		(fp_line
-			(start 0.54 -1.04)
-			(end 0.54 -1.37)
+			(start 0.54 1.04)
+			(end 0.54 1.37)
 			(stroke
 				(width 0.12)
@@
 		)
 		(fp_line
-			(start 0.54 1.04)
-			(end 0.54 1.37)
+			(start 0.54 -1.04)
+			(end 0.54 -1.37)
 			(stroke
 				(width 0.12)
@@
 		)
 		(fp_line
-			(start 7.08 1.37)
-			(end 7.08 1.04)
+			(start 0.54 -1.37)
+			(end 7.08 -1.37)
 			(stroke
 				(width 0.12)
@@
 		)
 		(fp_line
-			(start 0.54 1.37)
-			(end 7.08 1.37)
+			(start 7.08 -1.37)
+			(end 7.08 -1.04)
 			(stroke
 				(width 0.12)
@@
 		)
 		(fp_line
-			(start 7.62 0)
-			(end 6.96 0)
+			(start 0 0)
+			(end 0.66 0)
 			(stroke
 				(width 0.1)
@@
 		)
 		(fp_line
-			(start 0 0)
-			(end 0.66 0)
+			(start 7.62 0)
+			(end 6.96 0)
 			(stroke
 				(width 0.1)
@@
 		)
 		(pad "1" thru_hole circle
-			(at 0 0 90)
+			(at 0 0 270)
 			(size 1.6 1.6)
 			(drill 0.8)
@@
 		)
 		(pad "2" thru_hole circle
-			(at 7.62 0 90)
+			(at 7.62 0 270)
 			(size 1.6 1.6)
 			(drill 0.8)
@@
 			(layers "*.Cu" "*.Mask")
 			(remove_unused_layers no)
-			(net 20 "Net-(Q1-B)")
+			(net 12 "/CMD_IN")
 			(pintype "passive")
 		)
@@
 		(tags "Diode DO-41_SOD81 series Axial Horizontal pin pitch 7.62mm  length 5.2mm diameter 2.7mm")
 		(property "Reference" "D1"
-			(at 3.81 -2.47 270)
+			(at 6.95 -2.19 270)
 			(layer "F.SilkS")
 			(effects
@@
 		)
 		(fp_text user "K"
-			(at 0 -2.1 270)
+			(at 4.08 -2.34 270)
 			(layer "F.SilkS")
 			(effects
@@
 			(remove_unused_layers no)
 			(roundrect_rratio 0.15625)
-			(net 8 "/MC34063_TC")
+			(net 21 "Net-(D5-K)")
 			(pintype "passive")
 		)
@@
 			(layers "*.Cu" "*.Mask")
 			(remove_unused_layers no)
-			(net 8 "/MC34063_TC")
+			(net 21 "Net-(D5-K)")
 			(pintype "passive")
 		)
@@
 			(remove_unused_layers no)
 			(roundrect_rratio 0.15625)
-			(net 17 "Net-(D3-K)")
+			(net 8 "/MC34063_TC")
 			(pintype "passive")
 		)
@@
 			(remove_unused_layers no)
 			(roundrect_rratio 0.15625)
-			(net 8 "/MC34063_TC")
+			(net 21 "Net-(D5-K)")
 			(pinfunction "K")
 			(pintype "passive")
@@
 	)
 	(segment
-		(start 169.9006 99.8728)
-		(end 169.8498 99.822)
-		(width 0.2)
-		(layer "F.Cu")
-		(net 0)
-	)
-	(segment
 		(start 167.321 42.4039)
 		(end 167.0861 42.169)
@@
 	)
 	(segment
-		(start 167.2082 111.221)
-		(end 167.23 111.221)
-		(width 0.2)
-		(layer "F.Cu")
-		(net 0)
-	)
-	(segment
 		(start 156.46 51.44)
 		(end 156.46 45.463572)
@@
 	)
 	(segment
-		(start 167.2082 117.5882)
-		(end 167.2082 111.221)
-		(width 0.6)
-		(layer "F.Cu")
-		(net 0)
-	)
-	(segment
-		(start 167.23 102.5434)
-		(end 169.9006 99.8728)
-		(width 0.6)
-		(layer "F.Cu")
-		(net 0)
-	)
-	(segment
 		(start 150.12 37.25)
 		(end 152.54 39.67)
@@
 	)
 	(segment
-		(start 167.23 110.62)
-		(end 167.23 102.5434)
-		(width 0.6)
-		(layer "F.Cu")
-		(net 0)
-	)
-	(segment
 		(start 167.5 80.29)
 		(end 167.49 80.3)
@@
 	)
 	(segment
-		(start 168.46 118.84)
-		(end 167.2082 117.5882)
-		(width 0.6)
-		(layer "F.Cu")
-		(net 0)
-	)
-	(segment
 		(start 159.136428 63.9)
 		(end 160.386428 62.65)
@@
 	)
 	(segment
-		(start 169.8498 99.822)
-		(end 169.8498 92.9894)
-		(width 0.6)
-		(layer "F.Cu")
-		(net 0)
-	)
-	(segment
 		(start 163.87 57.08)
 		(end 159.49 52.7)
@@
 		(net 19)
 	)
+	(segment
+		(start 169.9006 99.8728)
+		(end 169.8498 99.822)
+		(width 0.2)
+		(layer "F.Cu")
+		(net 20)
+	)
+	(segment
+		(start 167.2082 111.221)
+		(end 167.23 111.221)
+		(width 0.2)
+		(layer "F.Cu")
+		(net 20)
+	)
+	(segment
+		(start 167.2082 117.5882)
+		(end 167.2082 111.221)
+		(width 0.6)
+		(layer "F.Cu")
+		(net 20)
+	)
+	(segment
+		(start 167.23 102.5434)
+		(end 169.9006 99.8728)
+		(width 0.6)
+		(layer "F.Cu")
+		(net 20)
+	)
+	(segment
+		(start 167.23 110.62)
+		(end 167.23 102.5434)
+		(width 0.6)
+		(layer "F.Cu")
+		(net 20)
+	)
+	(segment
+		(start 168.46 118.84)
+		(end 167.2082 117.5882)
+		(width 0.6)
+		(layer "F.Cu")
+		(net 20)
+	)
+	(segment
+		(start 169.8498 99.822)
+		(end 169.8498 92.9894)
+		(width 0.6)
+		(layer "F.Cu")
+		(net 20)
+	)
 	(embedded_fonts no)

Commit message: UPDATE
Parts:
- R3: footprint Resistor_THT:R_Axial_DIN0207_L6.3mm_D2.5mm_P7.62mm_Horizontal -> Resistor_THT:R_Axial_DIN0207_L6.3mm_D2.5mm_P10.16mm_Horizontal
- moved R5 12.8 mm to (162.4, 60.2), turned to 90 degrees
- moved D3 8.46 mm to (170.8, 71.8), turned to -90 degrees
- moved R3 0.15 mm to (166.4, 87.4)
Connections:
- D3 pad 1: Net-(D3-K) -> +24V
- D3 pad 2: +24V -> Net-(D3-A)
- R3 pad 2: +24V -> Net-(D3-A)
- U1 pad 6: Net-(D3-K) -> Net-(D5-K)
Routing:
- net (no net): track 78.6 -> 0.00 mm
- net Net-(D5-K): track 0.00 -> 64.8 mm
- net Net-(D3-A): track 0.00 -> 6.16 mm
- net /MC34063_SW_NODE: track 16.4 -> 14.4 mm
- net +24V: track 243.4 -> 242.6 mm

Commit message: UPdate
Parts:
- L1_Inductor1: value L_Ferrite -> 330uH
- R1: value 0.22 -> 220
- R2: value 220 -> 10k
- R3: value 10k -> 1k2
- R4: value 6.2k -> 6k2
- R5: value 1k -> 0R22
- R6: value 1.2k -> 1k
Connections:
- net /MC34063_SW_NODE renamed Net-(U1-DC)
Changed lines of the file:
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@@
 	(net 14 "unconnected-(J2-Pin_1-Pad1)")
 	(net 15 "unconnected-(J3-Pin_1-Pad1)")
-	(net 16 "/MC34063_SW_NODE")
+	(net 16 "Net-(U1-DC)")
 	(net 17 "Net-(D3-A)")
 	(net 18 "unconnected-(J7-Pin_1-Pad1)")
@@
 			)
 		)
-		(property "Value" "1.2k"
+		(property "Value" "1k"
 			(at 3.81 1.92 0)
 			(layer "F.Fab")
@@
 			)
 		)
-		(property "Value" "0.22"
+		(property "Value" "220"
 			(at 5.08 2.37 0)
 			(layer "F.Fab")
@@
 			)
 		)
-		(property "Value" "220"
+		(property "Value" "10k"
 			(at 3.81 2.37 90)
 			(layer "F.Fab")
@@
 			)
 		)
-		(property "Value" "10k"
+		(property "Value" "1k2"
 			(at 5.08 2.37 90)
 			(layer "F.Fab")
@@
 			)
 		)
-		(property "Value" "L_Ferrite"
+		(property "Value" "330uH"
 			(at 3.75 7.75 0)
 			(layer "F.Fab")
@@
 			)
 		)
-		(property "Value" "1k"
+		(property "Value" "0R22"
 			(at 6.35 2.72 90)
 			(layer "F.Fab")
@@
 			(layers "*.Cu" "*.Mask")
 			(remove_unused_layers no)
-			(net 16 "/MC34063_SW_NODE")
+			(net 16 "Net-(U1-DC)")
 			(pintype "passive")
 		)
@@
 			(remove_unused_layers no)
 			(roundrect_rratio 0.15625)
-			(net 16 "/MC34063_SW_NODE")
+			(net 16 "Net-(U1-DC)")
 			(pinfunction "SwC")
 			(pintype "open_collector")
@@
 			(layers "*.Cu" "*.Mask")
 			(remove_unused_layers no)
-			(net 16 "/MC34063_SW_NODE")
+			(net 16 "Net-(U1-DC)")
 			(pinfunction "Ipk")
 			(pintype "input")
@@
 			(layers "*.Cu" "*.Mask")
 			(remove_unused_layers no)
-			(net 16 "/MC34063_SW_NODE")
+			(net 16 "Net-(U1-DC)")
 			(pinfunction "DC")
 			(pintype "open_collector")
@@
 			)
 		)
-		(property "Value" "6.2k"
+		(property "Value" "6k2"
 			(at 3.81 2.37 0)
 			(layer "F.Fab")

Commit message: UPDATE
Parts:
- J1, J2, J3, J4, J5, J6, J7, J8: value Conn_01x05 -> JST_VH_01x05
- moved J3 15.9 mm to (139.7, 108.7), turned to 180 degrees
- moved J5 15.8 mm to (161.0, 127.5), turned to 180 degrees
- moved J2 15.7 mm to (139.6, 88.9), turned to 180 degrees
- moved J8 15.6 mm to (161.1, 70.0), turned to 180 degrees
- moved J4 15.5 mm to (139.2, 127.4), turned to 180 degrees
- moved J6 15.5 mm to (160.9, 108.6), turned to 180 degrees
- moved J1 15.4 mm to (139.6, 70.1), turned to 180 degrees
- moved J7 14.9 mm to (160.9, 88.8), turned to 180 degrees
Connections:
- net Net-(D3-A) renamed /CMD_IN_PROT
- net Net-(D4-K) renamed /SW_OUT
- net Net-(D5-K) renamed /+24V_FILT
- net Net-(Q1-B) renamed /Q1_BASE
- net Net-(U1-DC) renamed /I_SENSE
- net Net-(U1-Vfb) renamed /V_FB
- J1 pad 1: unconnected-(J1-Pin_1-Pad1) -> +24V
- J1 pad 2: /TC_CMD_BUS -> /+5V_OUT
- J1 pad 4: /+5V_OUT -> /TC_CMD_BUS
- J1 pad 5: +24V -> unconnected-(J1-Pin_5-Pad5)
- J2 pad 1: unconnected-(J2-Pin_1-Pad1) -> +24V
- J2 pad 2: /TC_CMD_BUS -> /+5V_OUT
- J2 pad 4: /+5V_OUT -> /TC_CMD_BUS
- J2 pad 5: +24V -> unconnected-(J2-Pin_5-Pad5)
- J3 pad 1: unconnected-(J3-Pin_1-Pad1) -> +24V
- J3 pad 2: /TC_CMD_BUS -> /+5V_OUT
- J3 pad 4: /+5V_OUT -> /TC_CMD_BUS
- J3 pad 5: +24V -> unconnected-(J3-Pin_5-Pad5)
- J4 pad 1: /TC_TX_REP -> +24V
- J4 pad 2: /TC_CMD_BUS -> /+5V_OUT
- J4 pad 4: /+5V_OUT -> /TC_CMD_BUS
- J4 pad 5: +24V -> /TC_TX_REP
- J5 pad 1: unconnected-(J5-Pin_1-Pad1) -> +24V
- J5 pad 2: /TC_CMD_BUS -> /+5V_OUT
- J5 pad 4: /+5V_OUT -> /TC_CMD_BUS
- J5 pad 5: +24V -> unconnected-(J5-Pin_5-Pad5)
- J6 pad 1: unconnected-(J6-Pin_1-Pad1) -> +24V
- J6 pad 2: /TC_CMD_BUS -> /+5V_OUT
- J6 pad 4: /+5V_OUT -> /TC_CMD_BUS
- J6 pad 5: +24V -> unconnected-(J6-Pin_5-Pad5)
- J7 pad 1: unconnected-(J7-Pin_1-Pad1) -> +24V
- J7 pad 2: /TC_CMD_BUS -> /+5V_OUT
- J7 pad 4: /+5V_OUT -> /TC_CMD_BUS
- J7 pad 5: +24V -> unconnected-(J7-Pin_5-Pad5)
- J8 pad 1: unconnected-(J8-Pin_1-Pad1) -> +24V
- J8 pad 2: /TC_CMD_BUS -> /+5V_OUT
- J8 pad 4: /+5V_OUT -> /TC_CMD_BUS
- J8 pad 5: +24V -> unconnected-(J8-Pin_5-Pad5)

Commit message: UPDATE
Routing:
- added copper zone on F.Cu, net +24V
- added copper zone on F.Cu, net GND
Changed lines of the file:
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@@
+	)
+	(segment
+		(start 135.96 37.09)
+		(end 136.12 37.25)
+		(width 2)
+		(layer "F.Cu")
+		(net 1)
 	)
 	(segment
@@
 	)
 	(segment
+		(start 129.14 39.97)
+		(end 131.95 37.16)
+		(width 2)
+		(layer "F.Cu")
+		(net 1)
+	)
+	(segment
 		(start 169.81 85.64)
 		(end 169.81 84.51)
@@
 	)
 	(segment
-		(start 129.14 45.72)
-		(end 129.14 39.97)
-		(width 2)
-		(layer "F.Cu")
-		(net 1)
-	)
-	(segment
 		(start 161.2 69.95)
 		(end 160.98 70.17)
@@
 	)
 	(segment
-		(start 131.86 37.25)
-		(end 136.12 37.25)
+		(start 129.14 51.33)
+		(end 129.14 39.97)
+		(width 2)
+		(layer "F.Cu")
+		(net 1)
+	)
+	(segment
+		(start 133.41 37.09)
+		(end 135.96 37.09)
 		(width 2)
 		(layer "F.Cu")
@@
 	)
 	(segment
+		(start 131.95 37.16)
+		(end 133.34 37.16)
+		(width 2)
+		(layer "F.Cu")
+		(net 1)
+	)
+	(segment
+		(start 133.34 37.16)
+		(end 133.41 37.09)
+		(width 2)
+		(layer "F.Cu")
+		(net 1)
+	)
+	(segment
 		(start 139.77 62.54)
 		(end 139.75 62.52)
@@
 	)
 	(segment
-		(start 129.14 51.33)
-		(end 129.14 45.72)
-		(width 2)
-		(layer "F.Cu")
-		(net 1)
-	)
-	(segment
 		(start 132.87 55.08)
 		(end 129.13 51.34)
@@
 	)
 	(segment
-		(start 129.14 39.97)
-		(end 131.86 37.25)
-		(width 2)
-		(layer "F.Cu")
-		(net 1)
-	)
-	(segment
 		(start 161.096428 133.96)
 		(end 161.2 133.856428)
@@
 		(start 174.01 63.43)
 		(end 174.01 60.771)
-		(width 0.6)
+		(width 0.8)
 		(layer "F.Cu")
 		(net 4)
@@
 		(start 173.56 101.81)
 		(end 173.56 64.06)
-		(width 0.6)
+		(width 0.8)
 		(layer "F.Cu")
 		(net 4)
@@
 		(start 173.56 64.06)
 		(end 174.1 63.52)
-		(width 0.6)
+		(width 0.8)
 		(layer "F.Cu")
 		(net 4)
@@
 		(net 21)
 	)
+	(zone
+		(net 4)
+		(net_name "GND")
+		(layer "F.Cu")
+		(hatch edge 0.5)
+		(priority 1)
+		(connect_pads
+			(clearance 0.5)
+		)
+		(min_thickness 0.25)
+		(filled_areas_thickness no)
+		(fill yes
+			(thermal_gap 0.5)
+			(thermal_bridge_width 0.5)
+		)
+		(polygon
+			(pts
+				(xy 142.69 34.51) (xy 142.62 52.65) (xy 141.43 53.35) (xy 142.06 56.49) (xy 137.06 52.84) (xy 135.5725 42.95)
+				(xy 137.1 41.07) (xy 137.94 39.12) (xy 138.15 34.37) (xy 142.83 34.51)
+			)
+		)
+	)
+	(zone
+		(net 1)
+		(net_name "+24V")
+		(layer "F.Cu")
+		(hatch edge 0.5)
+		(connect_pads
+			(clearance 0.5)
+		)
+		(min_thickness 0.25)
+		(filled_areas_thickness no)
+		(fill yes
+			(thermal_gap 0.5)
+			(thermal_bridge_width 0.5)
+		)
+		(polygon
+			(pts
+				(xy 134.52 38.28) (xy 134.38 45.07) (xy 134.31 54.96) (xy 129.71 50.77) (xy 129.78 40.16) (xy 132.43 37.93)
+				(xy 134.59 37.16)
+			)
+		)
+	)
 	(embedded_fonts no)

Commit message: UPDATE
Other:
- board text added: "2026.2.6"
- board text removed: "2026.2.1"
Changed lines of the file:
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@@
 		)
 	)
-	(gr_text "2026.2.1"
+	(gr_text "2026.2.6"
 		(at 212 194 0)
 		(layer "F.Cu")
