File: KiCad/TC_Interface_Board/_autosave-TC_Interface_Board.kicad_pcb (KiCad board)
At the start: 2 copper layers, 68.9 x 121.6 mm, 30 parts, among them J1 Conn_01x05, J1_24V1 JST_VH_01x04, J1_CN1 JST_VH_01x03, J2 Conn_01x05, J2_CN1 JST_VH_01x02, J3 Conn_01x05, J3_CN1 JST_VH_01x02, J4 Conn_01x05, J5 Conn_01x05, J6 Conn_01x05, J7 Conn_01x05, J8 Conn_01x05, Q1 DTC143E, Q2 DTC143E, U1 MC34063AP

Commit message: UPDATE
Connections:
- D1 pad 1: /TC_CMD_BUS -> /CMD_IN
- D1 pad 2: GND -> Net-(D1-A)
- D2 pad 1: /CMD_IN -> Net-(D2-K)
- Q1 pad 2: Net-(Q1-C) -> /Q2C_NODE
- Q1 pad 3: /TC_CMD_BUS -> Net-(Q1-B)
- Q2 pad 2: /Q2C_NODE -> /TC_CMD_BUS
- Q2 pad 3: Net-(Q1-C) -> Net-(D1-A)
- R1 pad 1: Net-(D3-K) -> Net-(D1-A)
- R1 pad 2: /MC34063_SW_NODE -> GND
- R3 pad 1: Net-(Q1-C) -> Net-(Q1-B)
- R6 pad 1: /CMD_IN -> Net-(D2-K)
Routing:
- net (no net): track 55.4 -> 28.5 mm
- net /Q2C_NODE: track 0.00 -> 26.9 mm
- net Net-(D1-A): track 0.00 -> 13.3 mm
- net GND: track 522.3 -> 511.9 mm
- net +24V: track 240.7 -> 243.4 mm
Changed lines of the file:
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@@
 	(net 18 "/MC34063_SW_NODE")
 	(net 19 "Net-(D3-K)")
-	(net 20 "Net-(Q1-C)")
-	(net 21 "unconnected-(J7-Pin_1-Pad1)")
+	(net 20 "unconnected-(J7-Pin_1-Pad1)")
+	(net 21 "Net-(D1-A)")
+	(net 22 "Net-(D2-K)")
+	(net 23 "Net-(Q1-B)")
 	(footprint "Connector_JST:JST_VH_B5P-VH-B_1x05_P3.96mm_Vertical"
 		(layer "F.Cu")
@@
 			(layers "*.Cu" "*.Mask")
 			(remove_unused_layers no)
-			(net 13 "/CMD_IN")
+			(net 22 "Net-(D2-K)")
 			(pintype "passive")
 		)
@@
 			(layers "*.Cu" "*.Mask")
 			(remove_unused_layers no)
-			(net 19 "Net-(D3-K)")
+			(net 21 "Net-(D1-A)")
 			(pintype "passive")
 		)
@@
 			(layers "*.Cu" "*.Mask")
 			(remove_unused_layers no)
-			(net 18 "/MC34063_SW_NODE")
+			(net 5 "GND")
 			(pintype "passive")
 		)
@@
 		(tags "Resistor Axial_DIN0207 series Axial Horizontal pin pitch 7.62mm 0.25W = 1/4W length 6.3mm diameter 2.5mm")
 		(property "Reference" "R3"
-			(at 3.81 -2.37 90)
+			(at 5.54 -2.32 90)
 			(layer "F.SilkS")
 			(effects
@@
 			(layers "*.Cu" "*.Mask")
 			(remove_unused_layers no)
-			(net 20 "Net-(Q1-C)")
+			(net 23 "Net-(Q1-B)")
 			(pintype "passive")
 		)
@@
 			(remove_unused_layers no)
 			(roundrect_rratio 0.15625)
-			(net 13 "/CMD_IN")
+			(net 22 "Net-(D2-K)")
 			(pinfunction "K")
 			(pintype "passive")
@@
 			(remove_unused_layers no)
 			(roundrect_rratio 0.113636)
-			(net 11 "/TC_CMD_BUS")
+			(net 13 "/CMD_IN")
 			(pinfunction "K")
 			(pintype "passive")
@@
 			(layers "*.Cu" "*.Mask")
 			(remove_unused_layers no)
-			(net 5 "GND")
+			(net 21 "Net-(D1-A)")
 			(pinfunction "A")
 			(pintype "passive")
@@
 			(layers "*.Cu" "*.Mask")
 			(remove_unused_layers no)
-			(net 14 "/Q2C_NODE")
+			(net 11 "/TC_CMD_BUS")
 			(pinfunction "C")
 			(pintype "passive")
@@
 			(layers "*.Cu" "*.Mask")
 			(remove_unused_layers no)
-			(net 20 "Net-(Q1-C)")
+			(net 21 "Net-(D1-A)")
 			(pinfunction "B")
 			(pintype "input")
@@
 			(layers "*.Cu" "*.Mask")
 			(remove_unused_layers no)
-			(net 20 "Net-(Q1-C)")
+			(net 14 "/Q2C_NODE")
 			(pinfunction "C")
 			(pintype "passive")
@@
 			(layers "*.Cu" "*.Mask")
 			(remove_unused_layers no)
-			(net 11 "/TC_CMD_BUS")
+			(net 23 "Net-(Q1-B)")
 			(pinfunction "B")
 			(pintype "input")
@@
 			(remove_unused_layers no)
 			(roundrect_rratio 0.092593)
-			(net 21 "unconnected-(J7-Pin_1-Pad1)")
+			(net 20 "unconnected-(J7-Pin_1-Pad1)")
 			(pinfunction "Pin_1")
 			(pintype "passive+no_connect")
@@
 	)
 	(segment
-		(start 169.9006 99.8728)
-		(end 169.8498 99.822)
-		(width 0.2)
-		(layer "F.Cu")
-		(net 0)
-	)
-	(segment
 		(start 162.43 58.71)
 		(end 162.43 60.646428)
@@
 	)
 	(segment
-		(start 167.2082 111.221)
-		(end 167.23 111.221)
-		(width 0.2)
-		(layer "F.Cu")
-		(net 0)
-	)
-	(segment
 		(start 158.28 60.67)
 		(end 158.27 60.66)
@@
 	)
 	(segment
-		(start 167.2082 117.5882)
-		(end 167.2082 111.221)
-		(width 0.6)
-		(layer "F.Cu")
-		(net 0)
-	)
-	(segment
-		(start 167.23 102.5434)
-		(end 169.9006 99.8728)
-		(width 0.6)
-		(layer "F.Cu")
-		(net 0)
-	)
-	(segment
-		(start 167.23 110.62)
-		(end 167.23 102.5434)
-		(width 0.6)
-		(layer "F.Cu")
-		(net 0)
-	)
-	(segment
 		(start 158.27 60.66)
 		(end 158.27 60.55)
@@
 	)
 	(segment
-		(start 168.46 118.84)
-		(end 167.2082 117.5882)
-		(width 0.6)
-		(layer "F.Cu")
-		(net 0)
-	)
-	(segment
 		(start 162.406428 60.67)
 		(end 158.28 60.67)
@@
 	)
 	(segment
-		(start 169.8498 99.822)
-		(end 169.8498 92.9894)
-		(width 0.6)
-		(layer "F.Cu")
-		(net 0)
-	)
-	(segment
 		(start 158.27 60.55)
 		(end 158.27 54.515)
@@
 	)
 	(segment
+		(start 170.86 69.95)
+		(end 170.86 70.41)
+		(width 0.2)
+		(layer "F.Cu")
+		(net 1)
+	)
+	(segment
 		(start 139.77 69.57)
 		(end 139.77 89.18)
@@
 	)
 	(segment
+		(start 170.86 69.95)
+		(end 170.876428 69.966428)
+		(width 0.2)
+		(layer "F.Cu")
+		(net 1)
+	)
+	(segment
 		(start 139.36 108.65)
 		(end 139.36 127.67)
@@
 	)
 	(segment
+		(start 170.876428 70.426428)
+		(end 170.876428 72.67)
+		(width 0.2)
+		(layer "F.Cu")
+		(net 1)
+	)
+	(segment
+		(start 170.86 70.41)
+		(end 170.876428 70.426428)
+		(width 0.2)
+		(layer "F.Cu")
+		(net 1)
+	)
+	(segment
 		(start 160.93 108.89)
 		(end 160.93 89.48)
@@
 	)
 	(segment
+		(start 176.1 101.81)
+		(end 173.37 101.81)
+		(width 0.2)
+		(layer "F.Cu")
+		(net 5)
+	)
+	(segment
 		(start 141.02 45.72)
 		(end 141.02 34.43)
@@
 	)
 	(segment
-		(start 165.96 102.24)
-		(end 165.64 101.92)
-		(width 0.2)
-		(layer "F.Cu")
-		(net 5)
-	)
-	(segment
-		(start 165.96 110.62)
-		(end 165.96 102.24)
-		(width 0.6)
-		(layer "F.Cu")
-		(net 5)
-	)
-	(segment
 		(start 173.16 118.84)
 		(end 173.19 118.81)
@@
 	)
 	(segment
-		(start 165.94 97.94)
-		(end 166.34 97.54)
-		(width 0.2)
-		(layer "F.Cu")
-		(net 5)
-	)
-	(segment
 		(start 143.256428 59.59)
 		(end 142.74 59.073572)
@@
 	)
 	(segment
+		(start 173.37 101.81)
+		(end 173.26 101.92)
+		(width 0.2)
+		(layer "F.Cu")
+		(net 5)
+	)
+	(segment
 		(start 156.7725 140.91)
 		(end 156.7725 143.3925)
@@
 	)
 	(segment
-		(start 165.64 98.27)
-		(end 165.67 98.24)
-		(width 0.2)
-		(layer "F.Cu")
-		(net 5)
-	)
-	(segment
 		(start 137.06 45.72)
 		(end 137.06 52.84)
@@
 	)
 	(segment
-		(start 165.94 101.81)
-		(end 165.94 97.94)
-		(width 0.8)
-		(layer "F.Cu")
-		(net 5)
-	)
-	(segment
 		(start 149.745 52.92)
 		(end 141.25 52.92)
@@
 		(net 13)
 	)
+	(segment
+		(start 169.9006 99.8728)
+		(end 169.8498 99.822)
+		(width 0.2)
+		(layer "F.Cu")
+		(net 14)
+	)
+	(segment
+		(start 167.2082 111.221)
+		(end 167.23 111.221)
+		(width 0.2)
+		(layer "F.Cu")
+		(net 14)
+	)
+	(segment
+		(start 167.2082 117.5882)
+		(end 167.2082 111.221)
+		(width 0.6)
+		(layer "F.Cu")
+		(net 14)
+	)
+	(segment
+		(start 167.23 102.5434)
+		(end 169.9006 99.8728)
+		(width 0.6)
+		(layer "F.Cu")
+		(net 14)
+	)
+	(segment
+		(start 167.23 110.62)
+		(end 167.23 102.5434)
+		(width 0.6)
+		(layer "F.Cu")
+		(net 14)
+	)
+	(segment
+		(start 168.46 118.84)
+		(end 167.2082 117.5882)
+		(width 0.6)
+		(layer "F.Cu")
+		(net 14)
+	)
+	(segment
+		(start 169.8498 99.822)
+		(end 169.8498 92.9894)
+		(width 0.6)
+		(layer "F.Cu")
+		(net 14)
+	)
+	(segment
+		(start 165.96 102.24)
+		(end 165.64 101.92)
+		(width 0.2)
+		(layer "F.Cu")
+		(net 21)
+	)
+	(segment
+		(start 165.96 110.62)
+		(end 165.96 102.24)
+		(width 0.6)
+		(layer "F.Cu")
+		(net 21)
+	)
+	(segment
+		(start 165.94 97.94)
+		(end 166.34 97.54)
+		(width 0.2)
+		(layer "F.Cu")
+		(net 21)
+	)
+	(segment
+		(start 165.64 98.27)
+		(end 165.67 98.24)
+		(width 0.2)
+		(layer "F.Cu")
+		(net 21)
+	)
+	(segment
+		(start 165.94 101.81)
+		(end 165.94 97.94)
+		(width 0.8)
+		(layer "F.Cu")
+		(net 21)
+	)
 	(embedded_fonts no)
