File: KiCad/TC_Interface_Board/_autosave-TC_Interface_Board.kicad_sch (KiCad schematic)
At the start: 30 parts, among them J1 Conn_01x05, J1_24V1 JST_VH_01x04, J1_CN1 JST_VH_01x03, J2 Conn_01x05, J2_CN1 JST_VH_01x02, J3 Conn_01x05, J3_CN1 JST_VH_01x02, J4 Conn_01x05, J5 Conn_01x05, J6 Conn_01x05, J7 Conn_01x05, J8 Conn_01x05, Q1 DTC143E, Q2 DTC143E, U1 MC34063AP

Commit message: UPDATE
Parts:
- renumbered Q2 to Q1, Q1 to Q2
Connections:
- net +24V: now also R2.1
- net CMD_IN: now also D1.1 (K); no longer D2.1 (K), R6.1
- net GND: now also D2.2 (A), R1.2; no longer D1.2 (A), R2.2
- net MC34063_SW_NODE: no longer R1.2
- net TC_CMD_BUS: no longer D1.1 (K), Q2.3 (B)
- net at C1.1, D3.1 (K), U1.6 (Vin): no longer R1.1
- net at Q1.3 (B), Q2.2 (C), R3.1: now also R2.2
- removed net Q2C_NODE: D2.2 (A), Q1.2 (C), R2.1
- new net: D2.1 (K), Q1.2 (C)
- new net: D1.2 (A), Q2.3 (B), R1.1
Other:
- moved on the sheet: D1, D2, R1, R2
