File: KiCad/ESP32S3_Snifar/ESP32S3_Snifar.kicad_pcb (KiCad board)
At the start: 2 copper layers, 95 x 70 mm, 14 parts, among them J1 Conn_01x04_Pin, U1 MOUDLE-SEEEDUINO-XIAO-ESP32S3

Commit message: UPDATE
Parts:
- added TP3: TestPoint, TestPoint:TestPoint_THTPad_D1.0mm_Drill0.5mm, F.Cu at (81.5, 38.0)
- added TP4: TestPoint, TestPoint:TestPoint_THTPad_D1.0mm_Drill0.5mm, F.Cu at (79.5, 58.4)
- moved TP1 1.93 mm to (60.9, 35.1)
- moved U1 0.88 mm to (98.7, 49.1)
- moved (R3)2.2k1 0.76 mm to (68.7, 38.1)
- moved D3 0.40 mm to (93.9, 62.4)
- moved (R2)100K1 0.40 mm to (53.3, 45.7)
- moved D1 0.34 mm to (94.0, 43.7)
- moved J1 0.32 mm to (37.2, 45.8)
- moved (R1)100K1 0.27 mm to (45.9, 38.1)
- moved D4 0.10 mm to (83.7, 71.4)
Routing:
- net Net-(D1-K): track 55.1 -> 60.2 mm
- net GND: track 193.5 -> 190.0 mm
- net Net-((R1)100K1-Pad2): track 30.2 -> 28.4 mm
- net Net-(D3-A): track 71.6 -> 72.5 mm
- net Net-(D1-A): track 68.8 -> 68.3 mm

Commit message: UPDATE
Parts:
- U1: footprint MOUDLE-SEEEDUINO-XIAO-ESP32S3:MOUDLE14P-SMD-2.54-21X17.8MM -> MOUDLE-SEEEDUINO-XIAO-ESP32S3:XIAO-ESP32S3-DIP
- moved U1 14.1 mm to (109.2, 58.5)

Commit message: UPDATE
Parts:
- J1: value Conn_01x04_Pin -> Conn_01x04_Socket; footprint Connector_PinHeader_2.54mm:PinHeader_1x04_P2.54mm_Vertical -> Connector_PinSocket_2.54mm:PinSocket_1x04_P2.54mm_Vertical
- moved J1 7.54 mm to (37.8, 53.3), turned to 180 degrees
Connections:
- (R1)100K1 pad 1: Net-(J1-Pin_1) -> Net-(J1-Pin_4)
- (R2)100K1 pad 2: GND -> Net-(D2-A)
- (R4)100K1 pad 1: Net-(J1-Pin_2) -> Net-(J1-Pin_3)
- (R5)100K1 pad 2: GND -> Net-(D2-A)
- D2 pad 2: GND -> Net-(D2-A)
- D4 pad 2: GND -> Net-(D2-A)
- J1 pad 1: Net-(J1-Pin_1) -> Net-(D2-A)
- J1 pad 2: Net-(J1-Pin_2) -> unconnected-(J1-Pin_2-Pad2)
- J1 pad 3: GND -> Net-(J1-Pin_3)
- J1 pad 4: unconnected-(J1-Pin_4-Pad4) -> Net-(J1-Pin_4)
- U1 pad 13: GND -> Net-(D2-A)
Routing:
- net GND: track 190.0 -> 0.00 mm
- net Net-(D2-A): track 0.00 -> 187.0 mm
- net Net-(J1-Pin_2): track 16.8 -> 0.00 mm
- net Net-(J1-Pin_3): track 0.00 -> 16.6 mm
- net Net-(J1-Pin_1): track 16.3 -> 0.00 mm
- net Net-(J1-Pin_4): track 0.00 -> 15.6 mm

Commit message: UPDATE
Parts:
- added Q2: DTC143E, Package_TO_SOT_THT:TO-92_Inline, F.Cu at (60.3, 76.2)
- added R7_220: 220Ω, Resistor_THT:R_Axial_DIN0204_L3.6mm_D1.6mm_P5.08mm_Vertical, F.Cu at (68.6, 73.7)
- added TP5: TestPoint, TestPoint:TestPoint_THTPad_D1.0mm_Drill0.5mm, F.Cu at (55.9, 54.9)
Connections:
- J1 pad 2: unconnected-(J1-Pin_2-Pad2) -> Net-(J1-Pin_2)
- U1 pad 10: unconnected-(U1-PA5_A9_D9_MISO-Pad10) -> Net-(U1-PA5_A9_D9_MISO)
- U1 pad 11: unconnected-(U1-PA6_A10_D10_MOSI-Pad11) -> Net-(U1-PA5_A9_D9_MISO)
- U1 pad 8: unconnected-(U1-PB09_D7_RX-Pad8) -> Net-(U1-PA5_A9_D9_MISO)
- U1 pad 9: unconnected-(U1-PA7_A8_D8_SCK-Pad9) -> Net-(U1-PA5_A9_D9_MISO)
Routing:
- net Net-(J1-Pin_2): track 0.00 -> 46.6 mm
- net Net-(U1-PA5_A9_D9_MISO): track 0.00 -> 43.0 mm
- net Net-(Q2-C): track 0.00 -> 8.29 mm
- net Net-(D2-A): track 187.0 -> 192.1 mm

Commit message: UPDATE
Parts:
- moved Q2 2.89 mm to (58.9, 73.7), turned to -90 degrees
Connections:
- Q2 pad 1: Net-(D2-A) -> Net-(Q2-B)
- Q2 pad 2: Net-(J1-Pin_2) -> Net-(D2-A)
- Q2 pad 3: Net-(Q2-C) -> Net-(J1-Pin_2)
- R7_220 pad 1: Net-(Q2-C) -> Net-(Q2-B)
- R7_220 pad 2: Net-(U1-PA5_A9_D9_MISO) -> Net-(U1-PA6_A10_D10_MOSI)
- U1 pad 10: Net-(U1-PA5_A9_D9_MISO) -> unconnected-(U1-PA5_A9_D9_MISO-Pad10)
- U1 pad 11: Net-(U1-PA5_A9_D9_MISO) -> Net-(U1-PA6_A10_D10_MOSI)
- U1 pad 8: Net-(U1-PA5_A9_D9_MISO) -> unconnected-(U1-PB09_D7_RX-Pad8)
- U1 pad 9: Net-(U1-PA5_A9_D9_MISO) -> unconnected-(U1-PA7_A8_D8_SCK-Pad9)
Routing:
- net Net-(U1-PA6_A10_D10_MOSI): track 0.00 -> 43.0 mm
- net Net-(U1-PA5_A9_D9_MISO): track 43.0 -> 0.00 mm
- net Net-(Q2-B): track 0.00 -> 9.89 mm
- net Net-(Q2-C): track 8.29 -> 0.00 mm
- net Net-(D2-A): track 192.1 -> 195.6 mm

Commit message: UPDATE
Parts:
- removed Q2: DTC143E, Package_TO_SOT_THT:TO-92_Inline
- added Q1: 2N7000, Package_TO_SOT_THT:TO-92_Inline, F.Cu at (62.4, 75.0)
Routing:
- net Net-(Q1-G): track 9.89 -> 6.22 mm
- net Net-(D2-A): track 195.6 -> 193.5 mm

Commit message: UPDATE
Parts:
- added (R5)100K2: 100kΩ, Resistor_THT:R_Axial_DIN0204_L3.6mm_D1.6mm_P5.08mm_Vertical, F.Cu at (68.6, 72.9)
- moved R7_220 3.95 mm to (68.6, 69.8)
- moved Q1 3.86 mm to (62.4, 71.1)
Connections:
- net Net-(D2-A) renamed GND
Routing:
- net GND: track 193.5 -> 200.7 mm
- net Net-(U1-PA6_A10_D10_MOSI): track 43.0 -> 46.9 mm
- net Net-(J1-Pin_2): track 46.1 -> 42.2 mm
- net Net-(Q1-G): track 6.22 -> 9.44 mm

Commit message: UPDATE
Parts:
- removed (R5)100K2: 100kΩ, Resistor_THT:R_Axial_DIN0204_L3.6mm_D1.6mm_P5.08mm_Vertical
- removed R7_220: 220Ω, Resistor_THT:R_Axial_DIN0204_L3.6mm_D1.6mm_P5.08mm_Vertical
- added (R9)100K1: 100kΩ, Resistor_THT:R_Axial_DIN0204_L3.6mm_D1.6mm_P5.08mm_Vertical, F.Cu at (68.6, 73.3)
- added R7_1: 220Ω, Resistor_THT:R_Axial_DIN0204_L3.6mm_D1.6mm_P5.08mm_Vertical, F.Cu at (68.5, 69.8)
- moved TP3 30.6 mm to (56.0, 55.0)
- moved TP5 23.8 mm to (79.4, 58.4)
- moved TP4 20.4 mm to (81.4, 38.0)
- moved TP2 7.06 mm to (60.5, 61.9)
Connections:
- TP3 pad 1: Net-(D1-A) -> Net-(J1-Pin_2)
- TP4 pad 1: Net-(D3-A) -> Net-(D1-A)
- TP5 pad 1: Net-(J1-Pin_2) -> Net-(D3-A)
Routing:
- net GND: track 200.7 -> 199.9 mm
