File: KiCad/ESP32S3_Snifar/ESP32S3_Snifar.kicad_pcb (KiCad board)
At the start: 2 copper layers, 95 x 70 mm, 33 parts, among them J1 Conn_01x04_Socket, J2 J2_Pi_01x06_Socket, Q1 2N7000, Q2 2N7000, U1 XIAO-ESP32S3

Commit message: UPDATE
Parts:
- TP1, TP2, TP3: footprint TestPoint:TestPoint_THTPad_2.0x2.0mm_Drill1.0mm -> TestPoint:TestPoint_Loop_D2.50mm_Drill1.0mm
- moved TP4 2.18 mm to (118.3, 63.9)
- moved TP3 2.01 mm to (122.1, 64.0)
Routing:
- net /Pi_Rx_MCU: track 93.5 -> 91.4 mm
- net /TC_MCU_RX: track 73.5 -> 71.4 mm

Commit message: UPDATE
Parts:
- moved TP1 0.64 mm to (83.8, 35.9)
Routing:
- net /SIG_DIV: track 131.7 -> 134.7 mm, vias 1 -> 0
Changed lines of the file:
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@@
 	(footprint "TestPoint:TestPoint_Loop_D2.50mm_Drill1.0mm"
 		(layer "F.Cu")
-		(at 83.9 36.51)
+		(at 83.78 35.88)
 		(descr "wire loop as test point, loop diameter 2.5mm, hole diameter 1.0mm")
 		(tags "test point wire loop bead")
@@
 	)
 	(segment
-		(start 83.905 35.755)
-		(end 83.9 35.75)
+		(start 124.34 78.06)
+		(end 124.399 78.001)
 		(width 0.2)
 		(layer "F.Cu")
@@
 	)
 	(segment
-		(start 119.18 35.755)
-		(end 120.6375 37.2125)
+		(start 83.91 35.75)
+		(end 83.78 35.88)
 		(width 0.2)
 		(layer "F.Cu")
@@
 	)
 	(segment
-		(start 83.91 35.76)
-		(end 83.905 35.755)
+		(start 83.905 35.755)
+		(end 83.9 35.75)
 		(width 0.2)
 		(layer "F.Cu")
@@
 	)
 	(segment
-		(start 83.92 35.77)
-		(end 83.91 35.76)
+		(start 124.399 78.001)
+		(end 124.399 35.79)
 		(width 0.2)
 		(layer "F.Cu")
@@
 	)
 	(segment
-		(start 83.905 35.755)
-		(end 119.18 35.755)
+		(start 83.91 35.76)
+		(end 83.905 35.755)
 		(width 0.2)
 		(layer "F.Cu")
@@
 	)
 	(segment
-		(start 53.74 40.48)
-		(end 53.7 40.52)
+		(start 83.9 35.77)
+		(end 58.45 35.77)
 		(width 0.2)
 		(layer "F.Cu")
@@
 	)
 	(segment
-		(start 53.74 40.48)
-		(end 57.71 36.51)
+		(start 83.91 35.76)
+		(end 83.9 35.77)
 		(width 0.2)
 		(layer "F.Cu")
@@
 	)
 	(segment
-		(start 53.7 40.52)
-		(end 53.66 40.56)
+		(start 83.92 35.77)
+		(end 83.91 35.76)
 		(width 0.2)
 		(layer "F.Cu")
@@
 	)
 	(segment
-		(start 83.91 35.76)
-		(end 83.9 35.77)
+		(start 83.87 35.79)
+		(end 83.78 35.88)
 		(width 0.2)
 		(layer "F.Cu")
@@
 	)
 	(segment
-		(start 83.9 35.77)
-		(end 83.9 36.51)
+		(start 124.399 35.79)
+		(end 83.87 35.79)
 		(width 0.2)
 		(layer "F.Cu")
@@
 	)
 	(segment
-		(start 57.71 36.51)
-		(end 83.9 36.51)
+		(start 122.14 78.06)
+		(end 124.34 78.06)
 		(width 0.2)
 		(layer "F.Cu")
 		(net 49)
 	)
-	(via
-		(at 120.6375 37.2125)
-		(size 0.6)
-		(drill 0.3)
-		(layers "F.Cu" "B.Cu")
-		(net 49)
-	)
 	(segment
-		(start 124.399 77.989)
-		(end 124.399 77.99)
-		(width 0.2)
-		(layer "B.Cu")
-		(net 49)
-	)
-	(segment
-		(start 53.66 40.56)
-		(end 53.66 44.1803)
+		(start 83.905 35.755)
+		(end 83.91 35.75)
 		(width 0.2)
-		(layer "B.Cu")
+		(layer "F.Cu")
 		(net 49)
 	)
 	(segment
-		(start 124.399 77.99)
-		(end 122.21 77.99)
+		(start 58.45 35.77)
+		(end 53.66 40.56)
 		(width 0.2)
-		(layer "B.Cu")
+		(layer "F.Cu")
 		(net 49)
 	)
 	(segment
-		(start 120.6375 37.2125)
-		(end 124.39 40.965)
+		(start 53.66 40.56)
+		(end 53.66 44.1803)
 		(width 0.2)
 		(layer "B.Cu")
@@
 	)
 	(segment
-		(start 124.39 77.98)
-		(end 124.399 77.989)
+		(start 122.21 77.99)
+		(end 122.14 78.06)
 		(width 0.2)
 		(layer "B.Cu")
@@
 		(width 0.2)
 		(layer "B.Cu")
-		(net 49)
-	)
-	(segment
-		(start 124.39 40.965)
-		(end 124.39 77.98)
-		(width 0.2)
-		(layer "B.Cu")
-		(net 49)
-	)
-	(segment
-		(start 122.21 77.99)
-		(end 122.14 78.06)
-		(width 0.2)
-		(layer "B.Cu")

Commit message: UPDATE Ver1.0
Parts:
- added M3: MountingHole_3.2mm_M3, MountingHole:MountingHole_3.2mm_M3, F.Cu at (34.1, 33.9)
- added M3: MountingHole_3.2mm_M3, MountingHole:MountingHole_3.2mm_M3, F.Cu at (34.0, 96.0)
- added M3: MountingHole_3.2mm_M3, MountingHole:MountingHole_3.2mm_M3, F.Cu at (121.0, 34.1)
- added M3: MountingHole_3.2mm_M3, MountingHole:MountingHole_3.2mm_M3, F.Cu at (121.1, 96.0)
Routing:
- net /SIG_DIV: track 134.7 -> 130.9 mm
- net Net-(JP3-B): vias 1 -> 0
Other:
- board text added: "TC106 Snidar ESP32S3 Ver 1.0 2026.03.04"

Commit message: UPDATE
Routing:
- net Net-(JP5-A): track 52.0 -> 51.2 mm
Changed lines of the file:
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@@
+	)
+	(segment
+		(start 109.39 37.18)
+		(end 109.41 37.2)
+		(width 0.2)
+		(layer "B.Cu")
+		(net 50)
 	)
 	(segment
@@
 	)
 	(segment
+		(start 107.2 37.38)
+		(end 107 37.18)
+		(width 0.2)
+		(layer "B.Cu")
+		(net 50)
+	)
+	(segment
+		(start 107.2 45.08)
+		(end 107.2 37.38)
+		(width 0.2)
+		(layer "B.Cu")
+		(net 50)
+	)
+	(segment
+		(start 105.49 45.09)
+		(end 107.19 45.09)
+		(width 0.2)
+		(layer "B.Cu")
+		(net 50)
+	)
+	(segment
 		(start 107.19 45.09)
 		(end 107.2 45.08)
@@
 	)
 	(segment
-		(start 109.39 37.18)
-		(end 109.41 37.2)
+		(start 105.49 62.96)
+		(end 105.49 45.09)
 		(width 0.2)
 		(layer "B.Cu")
@@
 	(segment
 		(start 104.14 64.31)
-		(end 105.2684 63.1816)
-		(width 0.2)
-		(layer "B.Cu")
-		(net 50)
-	)
-	(segment
-		(start 105.2684 63.1816)
-		(end 105.2684 45.09)
-		(width 0.2)
-		(layer "B.Cu")
-		(net 50)
-	)
-	(segment
-		(start 107.2 37.38)
-		(end 107 37.18)
-		(width 0.2)
-		(layer "B.Cu")
-		(net 50)
-	)
-	(segment
-		(start 105.2684 45.09)
-		(end 107.19 45.09)
-		(width 0.2)
-		(layer "B.Cu")
-		(net 50)
-	)
-	(segment
-		(start 107.2 45.08)
-		(end 107.2 37.38)
+		(end 105.49 62.96)
 		(width 0.2)
 		(layer "B.Cu")
@@
 	)
 	(segment
+		(start 102.91 62.82)
+		(end 102.92 62.81)
+		(width 0.2)
+		(layer "F.Cu")
+		(net 67)
+	)
+	(segment
 		(start 79.75 64.28)
 		(end 79.77 64.3)
@@
 	(segment
 		(start 79.75 62.81)
-		(end 79.7515 62.8115)
-		(width 0.2)
-		(layer "F.Cu")
-		(net 67)
-	)
-	(segment
-		(start 79.7515 62.8115)
-		(end 103.6225 62.8115)
-		(width 0.2)
-		(layer "F.Cu")
-		(net 67)
-	)
-	(segment
-		(start 79.75 64.28)
-		(end 79.75 62.81)
+		(end 79.76 62.82)
 		(width 0.2)
 		(layer "F.Cu")
@@
 		(net 67)
 	)
+	(segment
+		(start 79.76 62.82)
+		(end 102.91 62.82)
+		(width 0.2)
+		(layer "F.Cu")
+		(net 67)
+	)
+	(segment
+		(start 79.75 64.28)
+		(end 79.75 62.81)
+		(width 0.2)
+		(layer "F.Cu")
+		(net 67)
+	)
 	(via
-		(at 103.6225 62.8115)
+		(at 102.92 62.81)
 		(size 0.6)
 		(drill 0.3)
@@
 	)
 	(segment
-		(start 103.0581 39.0519)
+		(start 103.06 62.82)
+		(end 102.9 62.66)
+		(width 0.2)
+		(layer "B.Cu")
+		(net 67)
+	)
+	(segment
+		(start 102.9 62.66)
+		(end 102.9 39.21)
+		(width 0.2)
+		(layer "B.Cu")
+		(net 67)
+	)
+	(segment
+		(start 102.9 39.21)
 		(end 104.91 37.2)
-		(width 0.2)
-		(layer "B.Cu")
-		(net 67)
-	)
-	(segment
-		(start 103.6225 54.2108)
-		(end 103.0581 53.6464)
-		(width 0.2)
-		(layer "B.Cu")
-		(net 67)
-	)
-	(segment
-		(start 103.0581 53.6464)
-		(end 103.0581 39.0519)
-		(width 0.2)
-		(layer "B.Cu")
-		(net 67)
-	)
-	(segment
-		(start 103.6225 62.8115)
-		(end 103.6225 54.2108)
 		(width 0.2)
 		(layer "B.Cu")
@@
 	)
 	(segment
+		(start 94.67 66.91)
+		(end 91.99 66.91)
+		(width 0.2)
+		(layer "B.Cu")
+		(net 70)
+	)
+	(segment
+		(start 91.99 42.06)
+		(end 87.15 42.06)
+		(width 0.2)
+		(layer "B.Cu")
+		(net 70)
+	)
+	(segment
+		(start 106.66 66.9)
+		(end 102.89 66.9)
+		(width 0.2)
+		(layer "B.Cu")
+		(net 70)
+	)
+	(segment
+		(start 106.68 64.31)
+		(end 106.68 66.88)
+		(width 0.2)
+		(layer "B.Cu")
+		(net 70)
+	)
+	(segment
+		(start 106.68 66.88)
+		(end 106.66 66.9)
+		(width 0.2)
+		(layer "B.Cu")
+		(net 70)
+	)
+	(segment
 		(start 102.89 66.9)
-		(end 106.66 66.9)
-		(width 0.2)
-		(layer "B.Cu")
-		(net 70)
-	)
-	(segment
-		(start 102.87 57.78)
 		(end 102.87 66.88)
 		(width 0.2)
@@
 	)
 	(segment
-		(start 91.13 57.78)
-		(end 91.11 57.8)
-		(width 0.2)
-		(layer "B.Cu")
-		(net 70)
-	)
-	(segment
-		(start 91 42.04)
-		(end 90.98 42.06)
-		(width 0.2)
-		(layer "B.Cu")
-		(net 70)
-	)
-	(segment
 		(start 102.87 66.88)
-		(end 102.89 66.9)
-		(width 0.2)
-		(layer "B.Cu")
-		(net 70)
-	)
-	(segment
-		(start 91.11 57.8)
-		(end 91 57.69)
-		(width 0.2)
-		(layer "B.Cu")
-		(net 70)
-	)
-	(segment
-		(start 91 57.69)
-		(end 91 42.04)
-		(width 0.2)
-		(layer "B.Cu")
-		(net 70)
-	)
-	(segment
-		(start 90.98 42.06)
-		(end 87.15 42.06)
-		(width 0.2)
-		(layer "B.Cu")
-		(net 70)
-	)
-	(segment
-		(start 106.66 66.9)
-		(end 106.68 66.88)
-		(width 0.2)
-		(layer "B.Cu")
-		(net 70)
-	)
-	(segment
-		(start 106.68 66.88)
-		(end 106.68 64.31)
-		(width 0.2)
-		(layer "B.Cu")
-		(net 70)
-	)
-	(segment
-		(start 102.87 57.78)
-		(end 91.13 57.78)
-		(width 0.2)
-		(layer "B.Cu")
+		(end 102.87 66.91)
+		(width 0.2)
+		(layer "B.Cu")
+		(net 70)
+	)
+	(segment
+		(start 94.68 66.92)
+		(end 94.67 66.91)
+		(width 0.2)
+		(layer "B.Cu")
+		(net 70)
+	)
+	(segment
+		(start 102.87 66.91)
+		(end 94.42 66.91)
+		(width 0.2)
+		(layer "B.Cu")
+		(net 70)
+	)
+	(segment
+		(start 91.99 66.91)
+		(end 91.99 42.06)
+		(width 0.2)
+		(layer "B.Cu")

Commit message: UPDATE
Parts:
- removed M3 (x4): MountingHole_3.2mm_M3, MountingHole:MountingHole_3.2mm_M3
- added H1-M3: MountingHole, MountingHole:MountingHole_3.2mm_M3, F.Cu at (34.0, 34.0)
- added H2-M3: MountingHole, MountingHole:MountingHole_3.2mm_M3, F.Cu at (121.0, 34.1)
- added H3-M3: MountingHole, MountingHole:MountingHole_3.2mm_M3, F.Cu at (34.0, 95.9)
- added H4-M3: MountingHole, MountingHole:MountingHole_3.2mm_M3, F.Cu at (121.0, 96.0)
Routing:
- net /3.3V_Clamp: track 48.1 -> 49.9 mm

Commit message: UPDATE
Parts:
- moved J1 75.7 mm to (38.0, 61.7)
- moved J2 1.96 mm to (38.0, 53.0)
Routing:
- net /SIG_FOR_24V_or_15V: track 108.9 -> 32.1 mm, vias 1 -> 0
- net Net-(J1-Pin_3): track 68.1 -> 21.6 mm, vias 0 -> 1
- net Net-(JP4-A): track 45.5 -> 61.2 mm, vias 0 -> 1
- net /3.3V_Clamp: track 49.9 -> 36.0 mm
- net /Nano_CMD_BUS: track 76.7 -> 65.0 mm
- net /SIG_DIV: track 130.9 -> 139.9 mm, vias 0 -> 1
- net Net-(JP1-B): track 37.9 -> 29.9 mm
- net /Pi_Rx_MCU: track 91.4 -> 84.3 mm
- net Net-(JP3-B): track 82.2 -> 75.6 mm
- net /TC_MCU_RX: track 71.4 -> 66.0 mm
- net /Pi_Tx_MCU: track 71.6 -> 75.6 mm, vias 1 -> 0
- net /Pi_Rx: track 28.3 -> 24.3 mm, vias 0 -> 1
- net /MCU_RX: track 21.8 -> 18.6 mm
- net /TC_MOS_DRAIN: track 108.0 -> 104.9 mm
- net GND: track 184.0 -> 186.9 mm, vias 1 -> 0
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
Commit message: UPDATE
Routing:
- net /3.3V_Clamp: track 36.0 -> 53.0 mm
- net /Nano_CMD_BUS: track 65.0 -> 80.9 mm
- net /TC_MOS_DRAIN: track 104.9 -> 116.5 mm
- net /Pi_Tx_MCU: track 75.6 -> 86.8 mm
- net Net-(JP4-A): track 61.2 -> 50.7 mm
- net /MOS_GATE: track 42.5 -> 52.2 mm
- net Net-(JP1-B): track 29.9 -> 37.9 mm
- net /TC_MCU_RX: track 66.0 -> 73.4 mm
- net Net-(JP3-B): track 75.6 -> 82.3 mm
- net /Nano_MOS_DRAIN: track 49.8 -> 55.6 mm
- net /Pi_Rx_MCU: track 84.3 -> 90.0 mm
- net /SIG_DIV: track 139.9 -> 135.0 mm, vias 1 -> 0
- net /SIG_FOR_24V_or_15V: track 32.1 -> 36.9 mm
- net Net-(J1-Pin_3): track 21.6 -> 25.9 mm
- net GND: track 186.9 -> 190.4 mm
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
Commit message: UPDATE
Parts:
- JP1, JP2, JP5, JP6, JP7: footprint Connector_Wire:SolderWire-0.25sqmm_1x02_P4.5mm_D0.65mm_OD2mm -> Connector_PinHeader_2.54mm:PinHeader_1x02_P2.54mm_Vertical
- moved JP5 2.01 mm to (106.7, 38.2), turned to 90 degrees
- moved JP7 1.90 mm to (116.6, 43.0), turned to 90 degrees
- moved R8 1.31 mm to (46.2, 55.8)
- moved JP6 1.28 mm to (106.6, 43.1), turned to 90 degrees
- moved JP1 0.08 mm to (47.9, 75.8), turned to 90 degrees
- turned JP2 to 90 degrees
Routing:
- net /SIG_DIV: track 135.0 -> 137.8 mm
- net Net-(JP4-B): track 72.1 -> 74.9 mm
- net Net-(JP4-A): track 50.7 -> 53.5 mm
- net /SEND_BUS_OUT_FROM_ESP32S3: track 7.33 -> 9.29 mm
- net Net-(JP1-B): track 37.9 -> 39.7 mm
- net Net-(JP5-A): track 51.2 -> 52.9 mm
- net Net-(Q1-G): track 29.3 -> 30.7 mm
- net Net-(JP6-B): track 23.6 -> 24.6 mm
- net /MCU_RX: track 21.7 -> 21.1 mm
- net /MCU_TX_TRIG: track 32.4 -> 31.9 mm
Other:
- board text added: "2026.03.05"
- board text added: "TC OC sniffer XIAO ESP32S3"
- board text removed: "2026.03.04"
