File: KiCad/ESP32S3_Snifar/ESP32S3_Snifar.kicad_pcb (KiCad board)
At the start: 2 copper layers, 95 x 70 mm, 43 parts, among them J1 Conn_01x04_Socket, J2 J2_Pi_01x06_Socket, Q1 2N7000, Q2 2N7000, U1 XIAO-ESP32S3

Commit message: UPDATE
Routing:
- net Net-(JP1-B): track 30.6 -> 39.4 mm
- net /Pi_Rx_MCU: track 66.7 -> 71.3 mm
- net Net-(J1-Pin_3): track 21.6 -> 26.0 mm
- net /SIG_DIV: track 34.2 -> 38.4 mm
- net Net-(JP3-B): track 60.8 -> 63.7 mm
- net GND: track 235.2 -> 237.6 mm
- net /MOS_GATE: track 53.8 -> 55.8 mm
- net /Pi_Tx: track 35.3 -> 37.3 mm
- net /Pi_Tx_MCU: track 66.9 -> 68.8 mm
- net /SIG_FOR_24V_or_15V: track 75.5 -> 77.0 mm
- net /SEND_BUS_OUT_FROM_ESP32S3: track 8.15 -> 9.47 mm

Commit message: UPDATE
Routing:
- net /3.3V_Clamp: track 49.0 -> 51.7 mm
- net Net-(JP4-A): track 21.9 -> 24.2 mm
- net Net-(JP4-B): track 116.4 -> 118.5 mm
- net Net-(JP5-A): track 74.5 -> 76.5 mm
- net /Pi_Tx_MCU: track 68.8 -> 69.6 mm
Other:
- board text added: "FOR RaspberyPi UART PORT"

Commit message: UPDATE
Parts:
- moved R3 7.06 mm to (74.1, 40.5), turned to 180 degrees
Routing:
- net /SIG_DIV: track 38.4 -> 22.2 mm
- net Net-(R1-Pad1): track 23.9 -> 16.9 mm
Changed lines of the file:
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@@
 	(footprint "Resistor_THT:R_Axial_DIN0207_L6.3mm_D2.5mm_P7.62mm_Horizontal"
 		(layer "F.Cu")
-		(at 67.02 40.56)
+		(at 74.08 40.5 180)
 		(descr "Resistor, Axial_DIN0207 series, Axial, Horizontal, pin pitch=7.62mm, 0.25W = 1/4W, length*diameter=6.3*2.5mm^2, http://cdn-reichelt.de/documents/datenblatt/B400/1_4W%23YAG.pdf")
 		(tags "Resistor Axial_DIN0207 series Axial Horizontal pin pitch 7.62mm 0.25W = 1/4W length 6.3mm diameter 2.5mm")
 		(property "Reference" "R3"
-			(at 3.81 -2.37 0)
+			(at 3.48 2.24 0)
 			(layer "F.SilkS")
 			(effects
@@
 		)
 		(property "Value" "39k"
-			(at 3.81 2.37 0)
+			(at 3.64 -2.26 0)
 			(layer "F.Fab")
 			(effects
@@
 		(attr through_hole)
 		(fp_line
-			(start 0.54 -1.37)
-			(end 7.08 -1.37)
+			(start 7.08 1.37)
+			(end 7.08 1.04)
 			(stroke
 				(width 0.12)
@@
 		)
 		(fp_line
-			(start 0.54 -1.04)
-			(end 0.54 -1.37)
+			(start 7.08 -1.37)
+			(end 7.08 -1.04)
 			(stroke
 				(width 0.12)
@@
 		)
 		(fp_line
-			(start 0.54 1.04)
-			(end 0.54 1.37)
+			(start 0.54 1.37)
+			(end 7.08 1.37)
 			(stroke
 				(width 0.12)
@@
 		)
 		(fp_line
-			(start 0.54 1.37)
-			(end 7.08 1.37)
+			(start 0.54 1.04)
+			(end 0.54 1.37)
 			(stroke
 				(width 0.12)
@@
 		)
 		(fp_line
-			(start 7.08 -1.37)
-			(end 7.08 -1.04)
+			(start 0.54 -1.04)
+			(end 0.54 -1.37)
 			(stroke
 				(width 0.12)
@@
 		)
 		(fp_line
-			(start 7.08 1.37)
-			(end 7.08 1.04)
+			(start 0.54 -1.37)
+			(end 7.08 -1.37)
 			(stroke
 				(width 0.12)
@@
 		)
 		(fp_line
-			(start 0 0)
-			(end 0.66 0)
+			(start 7.62 0)
+			(end 6.96 0)
 			(stroke
 				(width 0.1)
@@
 		)
 		(fp_line
-			(start 7.62 0)
-			(end 6.96 0)
+			(start 0 0)
+			(end 0.66 0)
 			(stroke
 				(width 0.1)
@@
 		)
 		(pad "1" thru_hole circle
-			(at 0 0)
+			(at 0 0 180)
 			(size 1.6 1.6)
 			(drill 0.8)
@@
 		)
 		(pad "2" thru_hole circle
-			(at 7.62 0)
+			(at 7.62 0 180)
 			(size 1.6 1.6)
 			(drill 0.8)
@@
 		(tags "Diode DO-35_SOD27 series Axial Horizontal pin pitch 7.62mm  length 4mm diameter 2mm")
 		(property "Reference" "D1"
-			(at 3.62 -2.47 0)
+			(at 4.18 -2.4 0)
 			(layer "F.SilkS")
 			(effects
@@
 		)
 		(fp_text user "K"
-			(at -1.65 0.23 0)
+			(at -1.63 0.85 0)
 			(layer "F.SilkS")
 			(effects
@@
 	)
 	(segment
-		(start 62.33 46.69)
-		(end 60.25 46.69)
+		(start 89.99 50.77)
+		(end 89.99 49.21)
 		(width 0.2)
 		(layer "F.Cu")
@@
 	)
 	(segment
-		(start 89.99 50.77)
-		(end 89.99 49.94)
+		(start 62.33 46.69)
+		(end 60.25 46.69)
 		(width 0.2)
 		(layer "F.Cu")
@@
 	)
 	(segment
-		(start 62.38 46.74)
-		(end 62.33 46.69)
+		(start 62.38 49.21)
+		(end 62.38 46.74)
 		(width 0.2)
 		(layer "F.Cu")
@@
 	)
 	(segment
-		(start 109.2 49.09)
-		(end 109.2 50.77)
+		(start 89.99 49.21)
+		(end 62.38 49.21)
 		(width 0.2)
 		(layer "F.Cu")
@@
 	)
 	(segment
-		(start 109.2 50.77)
-		(end 89.99 50.77)
+		(start 109.22 49.07)
+		(end 109.2 49.09)
 		(width 0.2)
 		(layer "F.Cu")
@@
 	)
 	(segment
-		(start 109.22 49.07)
-		(end 109.2 49.09)
+		(start 109.2 49.09)
+		(end 109.2 50.77)
 		(width 0.2)
 		(layer "F.Cu")
@@
 	)
 	(segment
-		(start 89.99 49.94)
-		(end 62.38 49.94)
+		(start 62.38 46.74)
+		(end 62.33 46.69)
 		(width 0.2)
 		(layer "F.Cu")
@@
 	)
 	(segment
-		(start 62.38 49.94)
-		(end 62.38 46.74)
+		(start 109.2 50.77)
+		(end 89.99 50.77)
 		(width 0.2)
 		(layer "F.Cu")
@@
 	)
 	(segment
-		(start 79.53 42.06)
-		(end 79.54 42.05)
-		(width 0.2)
-		(layer "F.Cu")
-		(net 9)
-	)
-	(segment
 		(start 95.88 41.13)
 		(end 94.76 40.01)
@@
 	)
 	(segment
-		(start 84.12 40.01)
-		(end 94.76 40.01)
+		(start 79.53 42.06)
+		(end 79.54 42.05)
 		(width 0.2)
 		(layer "F.Cu")
@@
 	)
 	(segment
-		(start 79.54 42.05)
-		(end 82.08 42.05)
+		(start 116.6 41.15)
+		(end 116.58 41.13)
 		(width 0.2)
 		(layer "F.Cu")
@@
 	)
 	(segment
-		(start 82.08 42.05)
-		(end 84.12 40.01)
+		(start 116.58 41.13)
+		(end 95.88 41.13)
 		(width 0.2)
 		(layer "F.Cu")
@@
 	)
 	(segment
-		(start 116.6 41.15)
-		(end 116.58 41.13)
+		(start 85.93 40.01)
+		(end 94.76 40.01)
 		(width 0.2)
 		(layer "F.Cu")
@@
 	)
 	(segment
-		(start 116.58 41.13)
-		(end 95.88 41.13)
+		(start 79.54 42.05)
+		(end 83.89 42.05)
 		(width 0.2)
 		(layer "F.Cu")
@@
 	)
 	(segment
+		(start 83.89 42.05)
+		(end 85.93 40.01)
+		(width 0.2)
+		(layer "F.Cu")
+		(net 9)
+	)
+	(segment
 		(start 79.53 42.06)
 		(end 79.49 42.02)
@@
 	)
 	(segment
-		(start 74.64 40.56)
-		(end 74.64 42.61)
-		(width 0.2)
-		(layer "F.Cu")
-		(net 49)
-	)
-	(segment
 		(start 67.01 46.7)
 		(end 67.02 46.71)
@@
 	)
 	(segment
-		(start 74.6 42.65)
-		(end 60.3 42.65)
-		(width 0.2)
-		(layer "F.Cu")
-		(net 49)
-	)
-	(segment
-		(start 74.64 42.61)
-		(end 74.6 42.65)
-		(width 0.2)
-		(layer "F.Cu")
-		(net 49)
-	)
-	(segment
 		(start 60.2 40.49)
 		(end 53.77 40.49)
@@
 	)
 	(segment
-		(start 60.3 42.65)
-		(end 60.2 42.55)
+		(start 66.46 40.5)
+		(end 60.21 40.5)
 		(width 0.2)
-		(layer "F.Cu")
+		(layer "B.Cu")
 		(net 49)
 	)
 	(segment
-		(start 60.2 42.55)
-		(end 60.2 40.49)
+		(start 67.02 46.71)
+		(end 67.0998 46.7898)
 		(width 0.2)
-		(layer "F.Cu")
+		(layer "B.Cu")
 		(net 49)
 	)
 	(segment
-		(start 64 46.71)
-		(end 64 40.49)
+		(start 66.6675 46.71)
+		(end 64.01 46.71)
 		(width 0.2)
 		(layer "B.Cu")
@@
 	)
 	(segment
-		(start 67.02 46.71)
-		(end 67.0998 46.7898)
+		(start 64.01 46.71)
+		(end 64.01 40.5)
 		(width 0.2)
 		(layer "B.Cu")
@@
 	)
 	(segment
-		(start 66.6675 46.71)
-		(end 64 46.71)
-		(width 0.2)
-		(layer "B.Cu")
-		(net 49)
-	)
-	(segment
-		(start 64 40.49)
+		(start 60.21 40.5)
 		(end 60.2 40.49)
 		(width 0.2)
@@
 	)
 	(segment
-		(start 74.64 40.56)
-		(end 74.65 40.55)
-		(width 0.2)
-		(layer "B.Cu")
-		(net 49)
-	)
-	(segment
 		(start 104.14 64.31)
 		(end 104.14 65.145)
@@
 	)
 	(segment
-		(start 76.9583 43.7017)
-		(end 76.89 43.77)
-		(width 0.2)
-		(layer "F.Cu")
-		(net 64)
-	)
-	(segment
-		(start 92.4566 43.7017)
-		(end 76.9583 43.7017)
+		(start 76.89 46.62)
+		(end 76.8 46.71)
 		(width 0.2)
 		(layer "F.Cu")
@@
 	)
 	(segment
-		(start 92.49 43.6683)
-		(end 92.4566 43.7017)
+		(start 94.77 43.67)
+		(end 76.99 43.67)
 		(width 0.2)
 		(layer "F.Cu")
@@
 	)
 	(segment
-		(start 76.89 46.62)
-		(end 76.8 46.71)
+		(start 94.77 42.56)
+		(end 94.77 43.67)
 		(width 0.2)
 		(layer "F.Cu")
@@
 	(segment
 		(start 94.76 42.55)
-		(end 92.54 42.55)
+		(end 94.77 42.56)
 		(width 0.2)
 		(layer "F.Cu")
@@
 	)
 	(segment
-		(start 92.49 42.6)
-		(end 92.49 43.6683)
-		(width 0.2)
-		(layer "F.Cu")
-		(net 64)
-	)
-	(segment
-		(start 92.54 42.55)
-		(end 92.49 42.6)
+		(start 76.99 43.67)
+		(end 76.89 43.77)
 		(width 0.2)
 		(layer "F.Cu")
@@
 	)
 	(segment
-		(start 67.02 40.56)
-		(end 66.94 40.48)
-		(width 0.2)
-		(layer "F.Cu")
-		(net 71)
-	)
-	(segment
-		(start 71.97 44.44)
-		(end 71.97 51.79)
+		(start 77.42 40.5)
+		(end 77.42 51.93)
 		(width 0.2)
 		(layer "B.Cu")
@@
 	)
 	(segment
-		(start 71.97 51.79)
-		(end 72.11 51.93)
-		(width 0.2)
-		(layer "B.Cu")
-		(net 71)
-	)
-	(segment
-		(start 72.11 51.93)
+		(start 77.42 51.93)
 		(end 79.51 51.93)
 		(width 0.2)
@@
 	)
 	(segment
-		(start 67.02 44.44)
-		(end 71.97 44.44)
-		(width 0.2)
-		(layer "B.Cu")
-		(net 71)
-	)
-	(segment
-		(start 67.02 40.56)
-		(end 67.02 44.44)
+		(start 74.08 40.5)
+		(end 77.42 40.5)
 		(width 0.2)
 		(layer "B.Cu")

Commit message: UPDATE
Other:
- board text added: "TC106 Snidar ESP32S3 Ver 1.0 2026.03.10"
- board text removed: "TC106 Snidar ESP32S3 Ver 1.0 2026.03.04"
Changed lines of the file:
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@@
 		)
 	)
-	(gr_text "TC106 Snidar ESP32S3\nVer 1.0 2026.03.04"
+	(gr_text "TC106 Snidar ESP32S3\nVer 1.0 2026.03.10"
 		(at 39.5 91.68 90)
 		(layer "F.SilkS")

Commit message: UPDATE
Parts:
- moved TP6 0.06 mm to (60.2, 52.4)
Routing:
- net /Pi_Rx_MCU: track 71.3 -> 70.7 mm
Changed lines of the file:
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@@
 		)
 	)
-	(footprint "TestPoint:TestPoint_Loop_D2.50mm_Drill1.0mm"
-		(layer "F.Cu")
-		(at 60.25 52.35)
-		(descr "wire loop as test point, loop diameter 2.5mm, hole diameter 1.0mm")
-		(tags "test point wire loop bead")
-		(property "Reference" "TP6"
-			(at -0.22 4.6 0)
-			(layer "F.SilkS")
-			(hide yes)
-			(effects
-				(font
-					(size 1 1)
-					(thickness 0.15)
-				)
-			)
-		)
-		(property "Value" "TestPoint"
-			(at 0 -2.8 0)
-			(layer "F.Fab")
-			(effects
-				(font
-					(size 1 1)
-					(thickness 0.15)
-				)
-			)
-		)
-		(property "Datasheet" "~"
-			(at 0 0 0)
-			(unlocked yes)
-			(layer "F.Fab")
-			(hide yes)
-			(effects
-				(font
-					(size 1.27 1.27)
-					(thickness 0.15)
-				)
-			)
-		)
-		(property "Description" "test point"
-			(at 0 0 0)
-			(unlocked yes)
-			(layer "F.Fab")
-			(hide yes)
-			(effects
-				(font
-					(size 1.27 1.27)
-					(thickness 0.15)
-				)
-			)
-		)
-		(property ki_fp_filters "Pin* Test*")
-		(sheetname "/")
-		(sheetfile "ESP32S3_Snifar.kicad_sch")
-		(attr through_hole)
-		(fp_circle
-			(center 0 0)
-			(end 1.5 0)
-			(stroke
-				(width 0.12)
-				(type solid)
-			)
-			(fill no)
-			(layer "F.SilkS")
-		)
-		(fp_circle
-			(center 0 0)
-			(end 1.8 0)
-			(stroke
-				(width 0.05)
-				(type solid)
-			)
-			(fill no)
-			(layer "F.CrtYd")
-		)
-		(fp_line
-			(start -1.3 -0.2)
-			(end -1.3 0.2)
-			(stroke
-				(width 0.12)
-				(type solid)
-			)
-			(layer "F.Fab")
-		)
-		(fp_line
-			(start -1.3 0.2)
-			(end 1.3 0.2)
-			(stroke
-				(width 0.12)
-				(type solid)
-			)
-			(layer "F.Fab")
-		)
-		(fp_line
-			(start 1.3 -0.2)
-			(end -1.3 -0.2)
-			(stroke
-				(width 0.12)
-				(type solid)
-			)
-			(layer "F.Fab")
-		)
-		(fp_line
-			(start 1.3 0.2)
-			(end 1.3 -0.2)
-			(stroke
-				(width 0.12)
-				(type solid)
-			)
-			(layer "F.Fab")
-		)
-		(fp_text user "${REFERENCE}"
-			(at -0.07 -2.03 0)
-			(layer "F.Fab")
-			(effects
-				(font
-					(size 1 1)
-					(thickness 0.15)
-				)
-			)
-		)
-		(pad "1" thru_hole circle
-			(at 0 0)
-			(size 2 2)
-			(drill 1)
-			(layers "*.Cu" "*.Mask")
-			(remove_unused_layers no)
-			(net 3 "/Pi_Rx_MCU")
-			(pinfunction "1")
-			(pintype "passive")
-		)
-		(embedded_fonts no)
-		(model "${KICAD9_3DMODEL_DIR}/TestPoint.3dshapes/TestPoint_Loop_D2.50mm_Drill1.0mm.step"
-			(offset
-				(xyz 0 0 0)
-			)
-			(scale
-				(xyz 1 1 1)
-			)
-			(rotate
-				(xyz 0 0 0)
-			)
-		)
-	)
 	(footprint "MountingHole:MountingHole_3.2mm_M3"
 		(layer "F.Cu")
@@
 		)
 	)
+	(footprint "TestPoint:TestPoint_Loop_D2.50mm_Drill1.0mm"
+		(layer "F.Cu")
+		(at 60.2 52.38)
+		(descr "wire loop as test point, loop diameter 2.5mm, hole diameter 1.0mm")
+		(tags "test point wire loop bead")
+		(property "Reference" "TP6"
+			(at -0.04 -2.42 0)
+			(layer "F.SilkS")
+			(effects
+				(font
+					(size 1 1)
+					(thickness 0.15)
+				)
+			)
+		)
+		(property "Value" "TestPoint"
+			(at 0.6 -1.58 0)
+			(layer "F.Fab")
+			(effects
+				(font
+					(size 1 1)
+					(thickness 0.15)
+				)
+			)
+		)
+		(property "Datasheet" "~"
+			(at 0 0 0)
+			(unlocked yes)
+			(layer "F.Fab")
+			(hide yes)
+			(effects
+				(font
+					(size 1.27 1.27)
+					(thickness 0.15)
+				)
+			)
+		)
+		(property "Description" "test point"
+			(at 0 0 0)
+			(unlocked yes)
+			(layer "F.Fab")
+			(hide yes)
+			(effects
+				(font
+					(size 1.27 1.27)
+					(thickness 0.15)
+				)
+			)
+		)
+		(property ki_fp_filters "Pin* Test*")
+		(sheetname "/")
+		(sheetfile "ESP32S3_Snifar.kicad_sch")
+		(attr through_hole)
+		(fp_circle
+			(center 0 0)
+			(end 1.5 0)
+			(stroke
+				(width 0.12)
+				(type solid)
+			)
+			(fill no)
+			(layer "F.SilkS")
+		)
+		(fp_circle
+			(center 0 0)
+			(end 1.8 0)
+			(stroke
+				(width 0.05)
+				(type solid)
+			)
+			(fill no)
+			(layer "F.CrtYd")
+		)
+		(fp_line
+			(start -1.3 -0.2)
+			(end -1.3 0.2)
+			(stroke
+				(width 0.12)
+				(type solid)
+			)
+			(layer "F.Fab")
+		)
+		(fp_line
+			(start -1.3 0.2)
+			(end 1.3 0.2)
+			(stroke
+				(width 0.12)
+				(type solid)
+			)
+			(layer "F.Fab")
+		)
+		(fp_line
+			(start 1.3 -0.2)
+			(end -1.3 -0.2)
+			(stroke
+				(width 0.12)
+				(type solid)
+			)
+			(layer "F.Fab")
+		)
+		(fp_line
+			(start 1.3 0.2)
+			(end 1.3 -0.2)
+			(stroke
+				(width 0.12)
+				(type solid)
+			)
+			(layer "F.Fab")
+		)
+		(fp_text user "${REFERENCE}"
+			(at -0.02 1.88 0)
+			(layer "F.Fab")
+			(effects
+				(font
+					(size 1 1)
+					(thickness 0.15)
+				)
+			)
+		)
+		(pad "1" thru_hole circle
+			(at 0 0)
+			(size 2 2)
+			(drill 1)
+			(layers "*.Cu" "*.Mask")
+			(remove_unused_layers no)
+			(net 3 "/Pi_Rx_MCU")
+			(pinfunction "1")
+			(pintype "passive")
+		)
+		(embedded_fonts no)
+		(model "${KICAD9_3DMODEL_DIR}/TestPoint.3dshapes/TestPoint_Loop_D2.50mm_Drill1.0mm.step"
+			(offset
+				(xyz 0 0 0)
+			)
+			(scale
+				(xyz 1 1 1)
+			)
+			(rotate
+				(xyz 0 0 0)
+			)
+		)
+	)
 	(footprint "Connector_PinHeader_2.54mm:PinHeader_1x03_P2.54mm_Vertical"
 		(layer "F.Cu")
@@
 	)
 	(segment
-		(start 60.0392 52.1808)
-		(end 60.1784 52.0416)
-		(width 0.2)
-		(layer "F.Cu")
-		(net 3)
-	)
-	(segment
 		(start 62.39 52.32)
 		(end 62.36 52.35)
@@
 	)
 	(segment
-		(start 60.0392 52.1808)
-		(end 60.0808 52.1808)
-		(width 0.2)
-		(layer "F.Cu")
-		(net 3)
-	)
-	(segment
 		(start 70.0625 51.17)
 		(end 62.39 51.17)
@@
 	)
 	(segment
-		(start 60.0808 52.1808)
-		(end 60.25 52.35)
-		(width 0.2)
-		(layer "F.Cu")
-		(net 3)
-	)
-	(segment
 		(start 70.0625 53.6706)
 		(end 70.0625 51.17)
@@
 		(width 0.2)
 		(layer "F.Cu")
-		(net 3)
-	)
-	(segment
-		(start 59.9 52.32)
-		(end 60.0392 52.1808)
-		(width 0.2)
-		(layer "F.Cu")

Commit message: UPDATE
Parts:
- added C3: 101, Capacitor_THT:C_Disc_D5.0mm_W2.5mm_P5.00mm, F.Cu at (51.2, 42.0)
- moved R5 3.31 mm to (53.8, 37.2)
Routing:
- net /SIG_DIV: track 22.2 -> 29.6 mm
- net GND: track 237.6 -> 240.9 mm
Other:
- board text added: ">"
- board text added: "Do Not Populate"
Changed lines of the file:
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@@
 		)
 	)
+	(footprint "Capacitor_THT:C_Disc_D5.0mm_W2.5mm_P5.00mm"
+		(layer "F.Cu")
+		(at 51.17 42.02 180)
+		(descr "C, Disc series, Radial, pin pitch=5.00mm, diameter*width=5*2.5mm^2, Capacitor, http://cdn-reichelt.de/documents/datenblatt/B300/DS_KERKO_TC.pdf")
+		(tags "C Disc series Radial pin pitch 5.00mm diameter 5mm width 2.5mm Capacitor")
+		(property "Reference" "C3"
+			(at 2.66 2.35 0)
+			(layer "F.SilkS")
+			(effects
+				(font
+					(size 1 1)
+					(thickness 0.15)
+				)
+			)
+		)
+		(property "Value" "101"
+			(at 3.69 -2.38 0)
+			(layer "F.Fab")
+			(effects
+				(font
+					(size 1 1)
+					(thickness 0.15)
+				)
+			)
+		)
+		(property "Datasheet" "~"
+			(at 0 0 0)
+			(layer "F.Fab")
+			(hide yes)
+			(effects
+				(font
+					(size 1.27 1.27)
+					(thickness 0.15)
+				)
+			)
+		)
+		(property "Description" "Unpolarized capacitor"
+			(at 0 0 0)
+			(layer "F.Fab")
+			(hide yes)
+			(effects
+				(font
+					(size 1.27 1.27)
+					(thickness 0.15)
+				)
+			)
+		)
+		(property ki_fp_filters "C_*")
+		(sheetname "/")
+		(sheetfile "ESP32S3_Snifar.kicad_sch")
+		(attr through_hole)
+		(fp_line
+			(start 5.12 1.37)
+			(end -0.12 1.37)
+			(stroke
+				(width 0.12)
+				(type solid)
+			)
+			(layer "F.SilkS")
+		)
+		(fp_line
+			(start 5.12 1.033)
+			(end 5.12 1.37)
+			(stroke
+				(width 0.12)
+				(type solid)
+			)
+			(layer "F.SilkS")
+		)
+		(fp_line
+			(start 5.12 -1.37)
+			(end 5.12 -1.033)
+			(stroke
+				(width 0.12)
+				(type solid)
+			)
+			(layer "F.SilkS")
+		)
+		(fp_line
+			(start -0.12 1.37)
+			(end -0.12 1.033)
+			(stroke
+				(width 0.12)
+				(type solid)
+			)
+			(layer "F.SilkS")
+		)
+		(fp_line
+			(start -0.12 -1.033)
+			(end -0.12 -1.37)
+			(stroke
+				(width 0.12)
+				(type solid)
+			)
+			(layer "F.SilkS")
+		)
+		(fp_line
+			(start -0.12 -1.37)
+			(end 5.12 -1.37)
+			(stroke
+				(width 0.12)
+				(type solid)
+			)
+			(layer "F.SilkS")
+		)
+		(fp_rect
+			(start -1.05 -1.5)
+			(end 6.05 1.5)
+			(stroke
+				(width 0.05)
+				(type solid)
+			)
+			(fill no)
+			(layer "F.CrtYd")
+		)
+		(fp_rect
+			(start 0 -1.25)
+			(end 5 1.25)
+			(stroke
+				(width 0.1)
+				(type solid)
+			)
+			(fill no)
+			(layer "F.Fab")
+		)
+		(fp_text user "${REFERENCE}"
+			(at 2.5 0 0)
+			(layer "F.Fab")
+			(effects
+				(font
+					(size 1 1)
+					(thickness 0.15)
+				)
+			)
+		)
+		(pad "1" thru_hole circle
+			(at 0 0 180)
+			(size 1.6 1.6)
+			(drill 0.8)
+			(layers "*.Cu" "*.Mask")
+			(remove_unused_layers no)
+			(net 49 "/SIG_DIV")
+			(pintype "passive")
+		)
+		(pad "2" thru_hole circle
+			(at 5 0 180)
+			(size 1.6 1.6)
+			(drill 0.8)
+			(layers "*.Cu" "*.Mask")
+			(remove_unused_layers no)
+			(net 10 "GND")
+			(pintype "passive")
+		)
+		(embedded_fonts no)
+		(model "${KICAD9_3DMODEL_DIR}/Capacitor_THT.3dshapes/C_Disc_D5.0mm_W2.5mm_P5.00mm.step"
+			(offset
+				(xyz 0 0 0)
+			)
+			(scale
+				(xyz 1 1 1)
+			)
+			(rotate
+				(xyz 0 0 0)
+			)
+		)
+	)
 	(footprint "Diode_THT:D_DO-35_SOD27_P7.62mm_Horizontal"
 		(layer "F.Cu")
@@
 		(tags "Resistor Axial_DIN0207 series Axial Horizontal pin pitch 7.62mm 0.25W = 1/4W length 6.3mm diameter 2.5mm")
 		(property "Reference" "R2"
-			(at 3.81 -2.37 0)
+			(at 3.8 2.29 0)
 			(layer "F.SilkS")
 			(effects
@@
 		)
 		(property "Value" "100k"
-			(at 3.81 2.37 0)
+			(at 2.08 -2.33 0)
 			(layer "F.Fab")
 			(effects
@@
 	(footprint "Resistor_THT:R_Axial_DIN0207_L6.3mm_D2.5mm_P7.62mm_Horizontal"
 		(layer "F.Cu")
-		(at 53.75 40.51 180)
+		(at 53.76 37.2 180)
 		(descr "Resistor, Axial_DIN0207 series, Axial, Horizontal, pin pitch=7.62mm, 0.25W = 1/4W, length*diameter=6.3*2.5mm^2, http://cdn-reichelt.de/documents/datenblatt/B400/1_4W%23YAG.pdf")
 		(tags "Resistor Axial_DIN0207 series Axial Horizontal pin pitch 7.62mm 0.25W = 1/4W length 6.3mm diameter 2.5mm")
@@
 		)
 		(property "Value" "10k"
-			(at 3.59 -2.57 0)
+			(at 1.51 -2.42 0)
 			(layer "F.Fab")
 			(effects
@@
 		)
 	)
+	(gr_text ">"
+		(at 43.89 42.51 0)
+		(layer "F.SilkS")
+		(effects
+			(font
+				(size 1 1)
+				(thickness 0.1)
+			)
+			(justify left bottom)
+		)
+	)
+	(gr_text "Do Not Populate"
+		(at 43.84 46.65 90)
+		(layer "F.SilkS")
+		(effects
+			(font
+				(size 0.8 0.8)
+				(thickness 0.1)
+			)
+			(justify left bottom)
+		)
+	)
 	(gr_text "TC OC sniffer XIAO ESP32S3"
 		(at 184.76 175.83 0)
@@
 	)
 	(segment
-		(start 46.17 40.55)
-		(end 46.17 46.79)
-		(width 1)
-		(layer "B.Cu")
-		(net 10)
-	)
-	(segment
 		(start 53.96 68.8)
 		(end 52.28 68.8)
@@
 	)
 	(segment
-		(start 46.13 40.51)
-		(end 46.17 40.55)
-		(width 0.2)
-		(layer "B.Cu")
-		(net 10)
-	)
-	(segment
 		(start 67.06 77.43)
 		(end 67.06 78.63)
@@
 	)
 	(segment
+		(start 46.14 37.2)
+		(end 46.17 37.23)
+		(width 1)
+		(layer "B.Cu")
+		(net 10)
+	)
+	(segment
 		(start 37.96 53.05)
 		(end 37.96 61.725)
@@
 	)
 	(segment
+		(start 46.17 37.23)
+		(end 46.17 46.79)
+		(width 1)
+		(layer "B.Cu")
+		(net 10)
+	)
+	(segment
 		(start 42.52 66.65)
 		(end 42.52 59.16)
@@
 	)
 	(segment
+		(start 53.74 42.02)
+		(end 51.17 42.02)
+		(width 0.2)
+		(layer "F.Cu")
+		(net 49)
+	)
+	(segment
 		(start 67.01 46.7)
 		(end 67.02 46.71)
@@
 	)
 	(segment
+		(start 53.76 42)
+		(end 53.74 42.02)
+		(width 0.2)
+		(layer "F.Cu")
+		(net 49)
+	)
+	(segment
 		(start 60.2 40.49)
 		(end 53.77 40.49)
@@
 	)
 	(segment
-		(start 53.77 40.49)
-		(end 53.75 40.51)
+		(start 53.76 37.2)
+		(end 53.76 42)
 		(width 0.2)
 		(layer "F.Cu")

Commit message: UPDATE
Routing:
- added copper zone on B.Cu, net GND
Changed lines of the file:
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@@
 		(net 71)
+	)
+	(zone
+		(net 10)
+		(net_name "GND")
+		(layer "B.Cu")
+		(hatch edge 0.5)
+		(connect_pads
+			(clearance 0.5)
+		)
+		(min_thickness 0.25)
+		(filled_areas_thickness no)
+		(fill yes
+			(thermal_gap 0.5)
+			(thermal_bridge_width 0.5)
+		)
+		(polygon
+			(pts
+				(xy 32 31.68) (xy 32.11 98.43) (xy 124.11 98.1) (xy 124.33 31.68) (xy 31.89 31.57)
+			)
+		)
 	)
 	(embedded_fonts no)

Commit message: UPDATE
Connections:
- J1 pad 2: unconnected-(J1-Pin_2-Pad2) -> /TX
- J1 pad 3: Net-(J1-Pin_3) -> GND
- JP2 pad 1: Net-(J1-Pin_3) -> /TX
Routing:
- net /TX: track 0.00 -> 33.2 mm
- net Net-(J1-Pin_3): track 26.0 -> 0.00 mm
- net GND: track 240.9 -> 245.5 mm
- removed copper zone on B.Cu, net GND
