File: KiCad/TC_Interface_Board-Backup/TC_Interface_Board.kicad_pcb (KiCad board)
At the start: 2 copper layers, 68.9 x 121.6 mm, 30 parts, among them J10 Conn_01x05, J11 Conn_01x05, J1_24V_ROW1 Conn_01x04, J1_CN1_24V1 Conn_01x03, J2_CN2_9V_Main1 Conn_01x02, J3_CN3_9V_Main1 Conn_01x02, J4 Conn_01x05, J5 Conn_01x05, J6 Conn_01x05, J7 Conn_01x05, J8 Conn_01x05, J9 Conn_01x05, Q1 DTC143E, Q2 DTC143E, U1 MC34063AP

Commit message: UPDATE
Parts:
- D1: value 24V? -> 1N4148
- D2: value 630mV -> 1N4148
- D3: value 850mV -> 1N4148
- D4: value 630mV 1N5819 -> 1N5819
- D5: value 24V 1N4006 -> 1N4007
- R2: value 10K -> 10k
- R3: value 1.2K -> 1.2k
- R4: value 6.2K -> 6.2k
- R6: value 1K -> 1k
Connections:
- D1 pad 2: Net-(D1-A) -> GND
- J1_CN1_24V1 pad 3: Net-(D1-A) -> GND
- J2_CN2_9V_Main1 pad 1: Net-(D1-A) -> GND
- J3_CN3_9V_Main1 pad 1: Net-(D1-A) -> GND
- Q1 pad 1: Net-(D1-A) -> GND
- Q2 pad 1: Net-(D1-A) -> GND
- R1 pad 2: Net-(D1-A) -> GND
Routing:
- net GND: track 347.8 -> 509.0 mm
- net Net-(D1-A): track 119.9 -> 0.00 mm

Commit message: UPDATE
Parts:
- removed J1_CN1_24V1: Conn_01x03, Connector_JST:JST_VH_B3P-VH-B_1x03_P3.96mm_Vertical
- removed J2_CN2_9V_Main1, J3_CN3_9V_Main1: Conn_01x02, Connector_JST:JST_VH_B2P-VH-B_1x02_P3.96mm_Vertical
- added J1_CN1: JST_VH_01x03, Connector_JST:JST_VH_B3P-VH-B_1x03_P3.96mm_Vertical, F.Cu at (124.2, 141.1)
- added J2_CN2: JST_VH_01x02, Connector_JST:JST_VH_B2P-VH-B_1x02_P3.96mm_Vertical, F.Cu at (143.7, 140.9)
- added J3_CN3: JST_VH_01x02, Connector_JST:JST_VH_B2P-VH-B_1x02_P3.96mm_Vertical, F.Cu at (157.1, 141.0)
Connections:
- net Net-(D2-K) renamed /CMD_IN

Commit message: UPDATE
Other:
- board text added: "CMD_IN"
Changed lines of the file:
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@@
+		)
+	)
+	(gr_text "CMD_IN"
+		(at 164.28 137.06 270)
+		(layer "B.SilkS")
+		(effects
+			(font
+				(size 1 1)
+				(thickness 0.1)
+			)
+			(justify left bottom mirror)
 		)
 	)

Commit message: UPDATE
Parts:
- moved D2 0.35 mm to (166.3, 124.5)
- moved R2 0.27 mm to (169.8, 93.0)
- renumbered D2 to D1, D1 to D2
Connections:
- net -24V renamed +24V
- net Net-(D1-K) renamed /TC_CMD_BUS
Routing:
- net /TC_CMD_BUS: track 166.6 -> 167.8 mm
