File: KiCad/TC_Interface_Board-Backup/TC_Interface_Board.kicad_pcb (KiCad board)
At the start: 2 copper layers, 68.9 x 121.6 mm, 30 parts, among them J10 Conn_01x05, J11 Conn_01x05, J1_24V_ROW1 Conn_01x04, J1_CN1 JST_VH_01x03, J2_CN2 JST_VH_01x02, J3_CN3 JST_VH_01x02, J4 Conn_01x05, J5 Conn_01x05, J6 Conn_01x05, J7 Conn_01x05, J8 Conn_01x05, J9 Conn_01x05, Q1 DTC143E, Q2 DTC143E, U1 MC34063AP

Commit message: UPDATE
Connections:
- net Net-(J1_CN1-Pin_1) renamed /TC_TX_REP
Changed lines of the file:
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@@
 	(net 16 "unconnected-(J6-Pin_1-Pad1)")
 	(net 17 "unconnected-(J7-Pin_1-Pad1)")
-	(net 18 "Net-(J1_CN1-Pin_1)")
+	(net 18 "/TC_TX_REP")
 	(net 19 "/TC_CMD_BUS")
 	(net 20 "Net-(Q1-C)")
@@
 			(remove_unused_layers no)
 			(roundrect_rratio 0.092593)
-			(net 18 "Net-(J1_CN1-Pin_1)")
+			(net 18 "/TC_TX_REP")
 			(pinfunction "Pin_1")
 			(pintype "passive")
@@
 			(remove_unused_layers no)
 			(roundrect_rratio 0.092593)
-			(net 18 "Net-(J1_CN1-Pin_1)")
+			(net 18 "/TC_TX_REP")
 			(pinfunction "Pin_1")
 			(pintype "passive")

Commit message: UPDATE
Parts:
- D1: footprint Diode_THT:D_DO-41_SOD81_P7.62mm_Horizontal -> Diode_THT:D_DO-35_SOD27_P7.62mm_Horizontal
- D3: footprint Diode_THT:D_DO-41_SOD81_P10.16mm_Horizontal -> Diode_THT:D_DO-35_SOD27_P10.16mm_Horizontal
Changed lines of the file:
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@@
 		)
 	)
-	(footprint "Diode_THT:D_DO-41_SOD81_P7.62mm_Horizontal"
+	(footprint "Diode_THT:D_DO-35_SOD27_P7.62mm_Horizontal"
 		(layer "F.Cu")
 		(at 166.34 89.92 -90)
-		(descr "Diode, DO-41_SOD81 series, Axial, Horizontal, pin pitch=7.62mm, length*diameter=5.2*2.7mm^2, https://www.diodes.com/assets/Package-Files/DO-41-Plastic.pdf")
-		(tags "Diode DO-41_SOD81 series Axial Horizontal pin pitch 7.62mm  length 5.2mm diameter 2.7mm")
+		(descr "Diode, DO-35_SOD27 series, Axial, Horizontal, pin pitch=7.62mm, length*diameter=4*2mm^2, http://www.diodes.com/_files/packages/DO-35.pdf")
+		(tags "Diode DO-35_SOD27 series Axial Horizontal pin pitch 7.62mm  length 4mm diameter 2mm")
 		(property "Reference" "D1"
-			(at 6.37 3.71 90)
+			(at 3.81 -2.12 270)
 			(layer "F.SilkS")
 			(effects
@@
 		)
 		(property "Value" "1N4148"
-			(at 3.81 2.47 90)
+			(at 3.81 2.12 270)
 			(layer "F.Fab")
 			(effects
@@
 		)
 		(property "Datasheet" "~"
-			(at 0 0 90)
+			(at 0 0 270)
 			(layer "F.Fab")
 			(hide yes)
@@
 		)
 		(property "Description" "Diode"
-			(at 0 0 90)
+			(at 0 0 270)
 			(layer "F.Fab")
 			(hide yes)
@@
 		(attr through_hole)
 		(fp_line
-			(start 1.09 1.47)
-			(end 6.53 1.47)
-			(stroke
-				(width 0.12)
-				(type solid)
-			)
-			(layer "F.SilkS")
-		)
-		(fp_line
-			(start 6.53 1.47)
-			(end 6.53 1.34)
-			(stroke
-				(width 0.12)
-				(type solid)
-			)
-			(layer "F.SilkS")
-		)
-		(fp_line
-			(start 1.09 1.34)
-			(end 1.09 1.47)
-			(stroke
-				(width 0.12)
-				(type solid)
-			)
-			(layer "F.SilkS")
-		)
-		(fp_line
-			(start 1.09 -1.34)
-			(end 1.09 -1.47)
+			(start 1.04 0)
+			(end 1.69 0)
 			(stroke
 				(width 0.12)
@@
 		)
 		(fp_line
-			(start 1.09 -1.47)
-			(end 6.53 -1.47)
+			(start 6.58 0)
+			(end 5.93 0)
 			(stroke
 				(width 0.12)
@@
 		)
 		(fp_line
-			(start 1.87 -1.47)
-			(end 1.87 1.47)
+			(start 2.29 -1.12)
+			(end 2.29 1.12)
 			(stroke
 				(width 0.12)
@@
 		)
 		(fp_line
-			(start 1.99 -1.47)
-			(end 1.99 1.47)
+			(start 2.41 -1.12)
+			(end 2.41 1.12)
 			(stroke
 				(width 0.12)
@@
 		)
 		(fp_line
-			(start 2.11 -1.47)
-			(end 2.11 1.47)
+			(start 2.53 -1.12)
+			(end 2.53 1.12)
 			(stroke
 				(width 0.12)
@@
 			(layer "F.SilkS")
 		)
-		(fp_line
-			(start 6.53 -1.47)
-			(end 6.53 -1.34)
+		(fp_rect
+			(start 1.69 -1.12)
+			(end 5.93 1.12)
 			(stroke
 				(width 0.12)
 				(type solid)
 			)
+			(fill no)
 			(layer "F.SilkS")
 		)
 		(fp_rect
-			(start -1.35 -1.6)
-			(end 8.97 1.6)
+			(start -1.05 -1.25)
+			(end 8.67 1.25)
 			(stroke
 				(width 0.05)
@@
 		(fp_line
 			(start 0 0)
-			(end 1.21 0)
+			(end 1.81 0)
 			(stroke
 				(width 0.1)
@@
 		(fp_line
 			(start 7.62 0)
-			(end 6.41 0)
+			(end 5.81 0)
 			(stroke
 				(width 0.1)
@@
 		)
 		(fp_line
-			(start 1.89 -1.35)
-			(end 1.89 1.35)
+			(start 2.31 -1)
+			(end 2.31 1)
 			(stroke
 				(width 0.1)
@@
 		)
 		(fp_line
-			(start 1.99 -1.35)
-			(end 1.99 1.35)
+			(start 2.41 -1)
+			(end 2.41 1)
 			(stroke
 				(width 0.1)
@@
 		)
 		(fp_line
-			(start 2.09 -1.35)
-			(end 2.09 1.35)
+			(start 2.51 -1)
+			(end 2.51 1)
 			(stroke
 				(width 0.1)
@@
 		)
 		(fp_rect
-			(start 1.21 -1.35)
-			(end 6.41 1.35)
+			(start 1.81 -1)
+			(end 5.81 1)
 			(stroke
 				(width 0.1)
@@
 		)
 		(fp_text user "K"
-			(at 0.12 2.11 180)
+			(at 0 -1.8 270)
 			(layer "F.SilkS")
 			(effects
@@
 		)
 		(fp_text user "K"
-			(at 0 -2.1 90)
+			(at 0 -1.8 270)
 			(layer "F.Fab")
 			(effects
@@
 		)
 		(fp_text user "${REFERENCE}"
-			(at 4.2 0 90)
+			(at 4.11 0 270)
 			(layer "F.Fab")
 			(effects
 				(font
-					(size 1 1)
-					(thickness 0.15)
+					(size 0.8 0.8)
+					(thickness 0.12)
 				)
 			)
@@
 		(pad "1" thru_hole roundrect
 			(at 0 0 270)
-			(size 2.2 2.2)
-			(drill 1.1)
+			(size 1.6 1.6)
+			(drill 0.8)
 			(layers "*.Cu" "*.Mask")
 			(remove_unused_layers no)
-			(roundrect_rratio 0.113636)
+			(roundrect_rratio 0.15625)
 			(net 21 "/CMD_IN")
 			(pinfunction "K")
@@
 		(pad "2" thru_hole circle
 			(at 7.62 0 270)
-			(size 2.2 2.2)
-			(drill 1.1)
+			(size 1.6 1.6)
+			(drill 0.8)
 			(layers "*.Cu" "*.Mask")
 			(remove_unused_layers no)
@@
 		)
 		(embedded_fonts no)
-		(model "${KICAD9_3DMODEL_DIR}/Diode_THT.3dshapes/D_DO-41_SOD81_P7.62mm_Horizontal.step"
+		(model "${KICAD9_3DMODEL_DIR}/Diode_THT.3dshapes/D_DO-35_SOD27_P7.62mm_Horizontal.step"
 			(offset
 				(xyz 0 0 0)
@@
 		)
 	)
-	(footprint "Diode_THT:D_DO-41_SOD81_P10.16mm_Horizontal"
+	(footprint "Diode_THT:D_DO-35_SOD27_P10.16mm_Horizontal"
 		(layer "F.Cu")
 		(at 170.876428 80.29 90)
-		(descr "Diode, DO-41_SOD81 series, Axial, Horizontal, pin pitch=10.16mm, length*diameter=5.2*2.7mm^2, https://www.diodes.com/assets/Package-Files/DO-41-Plastic.pdf")
-		(tags "Diode DO-41_SOD81 series Axial Horizontal pin pitch 10.16mm  length 5.2mm diameter 2.7mm")
+		(descr "Diode, DO-35_SOD27 series, Axial, Horizontal, pin pitch=10.16mm, length*diameter=4*2mm^2, http://www.diodes.com/_files/packages/DO-35.pdf")
+		(tags "Diode DO-35_SOD27 series Axial Horizontal pin pitch 10.16mm  length 4mm diameter 2mm")
 		(property "Reference" "D3"
-			(at 5.17 4.07 90)
+			(at 5.08 -2.12 90)
 			(layer "F.SilkS")
 			(effects
@@
 		)
 		(property "Value" "1N4148"
-			(at 5.08 2.47 90)
+			(at 5.08 2.12 90)
 			(layer "F.Fab")
 			(effects
@@
 		(attr through_hole)
 		(fp_line
-			(start 3.38 -1.47)
-			(end 3.38 1.47)
+			(start 3.8 -1.12)
+			(end 3.8 1.12)
 			(stroke
 				(width 0.12)
@@
 		)
 		(fp_line
-			(start 3.26 -1.47)
-			(end 3.26 1.47)
+			(start 3.68 -1.12)
+			(end 3.68 1.12)
 			(stroke
 				(width 0.12)
@@
 		)
 		(fp_line
-			(start 3.14 -1.47)
-			(end 3.14 1.47)
+			(start 3.56 -1.12)
+			(end 3.56 1.12)
 			(stroke
 				(width 0.12)
@@
 		)
 		(fp_line
-			(start 8.82 0)
-			(end 7.8 0)
+			(start 9.12 0)
+			(end 7.2 0)
 			(stroke
 				(width 0.12)
@@
 		)
 		(fp_line
-			(start 1.34 0)
-			(end 2.36 0)
+			(start 1.04 0)
+			(end 2.96 0)
 			(stroke
 				(width 0.12)
@@
 		)
 		(fp_rect
-			(start 2.36 -1.47)
-			(end 7.8 1.47)
+			(start 2.96 -1.12)
+			(end 7.2 1.12)
 			(stroke
 				(width 0.12)
@@
 		)
 		(fp_rect
-			(start -1.35 -1.6)
-			(end 11.51 1.6)
+			(start -1.05 -1.25)
+			(end 11.21 1.25)
 			(stroke
 				(width 0.05)
@@
 		)
 		(fp_line
-			(start 3.36 -1.35)
-			(end 3.36 1.35)
+			(start 3.78 -1)
+			(end 3.78 1)
 			(stroke
 				(width 0.1)
@@
 		)
 		(fp_line
-			(start 3.26 -1.35)
-			(end 3.26 1.35)
+			(start 3.68 -1)
+			(end 3.68 1)
 			(stroke
 				(width 0.1)
@@
 		)
 		(fp_line
-			(start 3.16 -1.35)
-			(end 3.16 1.35)
+			(start 3.58 -1)
+			(end 3.58 1)
 			(stroke
 				(width 0.1)
@@
 		(fp_line
 			(start 10.16 0)
-			(end 7.68 0)
+			(end 7.08 0)
 			(stroke
 				(width 0.1)
@@
 		(fp_line
 			(start 0 0)
-			(end 2.48 0)
+			(end 3.08 0)
 			(stroke
 				(width 0.1)
@@
 		)
 		(fp_rect
-			(start 2.48 -1.35)
-			(end 7.68 1.35)
+			(start 3.08 -1)
+			(end 7.08 1)
 			(stroke
 				(width 0.1)
@@
 		)
 		(fp_text user "K"
-			(at -0.01 2.323572 90)
+			(at 0 -1.8 90)
 			(layer "F.SilkS")
 			(effects
@@
 		)
 		(fp_text user "${REFERENCE}"
-			(at 5.47 0 90)
+			(at 5.38 0 90)
 			(layer "F.Fab")
 			(effects
 				(font
-					(size 1 1)
-					(thickness 0.15)
+					(size 0.8 0.8)
+					(thickness 0.12)
 				)
 			)
 		)
 		(fp_text user "K"
-			(at 0 2.323572 90)
+			(at 0 -1.8 90)
 			(layer "F.Fab")
 			(effects
@@
 		(pad "1" thru_hole roundrect
 			(at 0 0 90)
-			(size 2.2 2.2)
-			(drill 1.1)
+			(size 1.6 1.6)
+			(drill 0.8)
 			(layers "*.Cu" "*.Mask")
 			(remove_unused_layers no)
-			(roundrect_rratio 0.113636)
+			(roundrect_rratio 0.15625)
 			(net 3 "Net-(D3-K)")
 			(pinfunction "K")
@@
 		(pad "2" thru_hole circle
 			(at 10.16 0 90)
-			(size 2.2 2.2)
-			(drill 1.1)
+			(size 1.6 1.6)
+			(drill 0.8)
 			(layers "*.Cu" "*.Mask")
 			(remove_unused_layers no)
@@
 		)
 		(embedded_fonts no)
-		(model "${KICAD9_3DMODEL_DIR}/Diode_THT.3dshapes/D_DO-41_SOD81_P10.16mm_Horizontal.step"
+		(model "${KICAD9_3DMODEL_DIR}/Diode_THT.3dshapes/D_DO-35_SOD27_P10.16mm_Horizontal.step"
 			(offset
 				(xyz 0 0 0)
