File: KiCad/TC_Interface_Board-Backup/TC_Interface_Board.kicad_sch (KiCad schematic)
At the start: 30 parts, among them J10 Conn_01x05, J11 Conn_01x05, J1_24V_ROW1 Conn_01x04, J1_CN1_24V1 Conn_01x03, J2_CN2_9V_Main1 Conn_01x02, J3_CN3_9V_Main1 Conn_01x02, J4 Conn_01x05, J5 Conn_01x05, J6 Conn_01x05, J7 Conn_01x05, J8 Conn_01x05, J9 Conn_01x05, Q1 DTC143E, Q2 DTC143E, U1 MC34063AP

Commit message: UPDATE
Connections:
- net GND: now also D1.2 (A), J1_CN1_24V1.3 (Pin_3), J2_CN2_9V_Main1.1 (Pin_1), J3_CN3_9V_Main1.1 (Pin_1), Q1.1 (B), Q2.1 (B), R1.2
Changed lines of the file:
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@@
-	)
-	(junction
-		(at 187.96 87.63)
-		(diameter 0)
-		(color 0 0 0 0)
 	)
 	(junction
@@
 	(junction
 		(at 138.43 109.22)
+		(diameter 0)
+		(color 0 0 0 0)
+	)
+	(junction
+		(at 144.78 31.75)
 		(diameter 0)
 		(color 0 0 0 0)
@@
 	(wire
 		(pts
-			(xy 170.18 96.52) (xy 187.96 96.52)
+			(xy 170.18 96.52) (xy 215.9 96.52)
 		)
 		(stroke
@@
 	(wire
 		(pts
-			(xy 187.96 87.63) (xy 187.96 96.52)
-		)
-		(stroke
-			(width 0)
-			(type default)
-		)
-	)
-	(wire
-		(pts
 			(xy 99.06 109.22) (xy 115.57 109.22)
 		)
@@
 	(wire
 		(pts
+			(xy 215.9 96.52) (xy 215.9 31.75)
+		)
+		(stroke
+			(width 0)
+			(type default)
+		)
+	)
+	(wire
+		(pts
 			(xy 66.04 124.46) (xy 69.85 124.46)
 		)
@@
 		(pts
 			(xy 69.85 124.46) (xy 69.85 133.35)
+		)
+		(stroke
+			(width 0)
+			(type default)
+		)
+	)
+	(wire
+		(pts
+			(xy 215.9 31.75) (xy 144.78 31.75)
 		)
 		(stroke
@@
 		)
 	)
+	(label "GND"
+		(at 63.5 26.67 0)
+		(effects
+			(font
+				(size 1.27 1.27)
+			)
+			(justify left bottom)
+		)
+	)

Commit message: UPDATE
Parts:
- J1_CN1: renamed from J1_CN1_24V1; value Conn_01x03 -> JST_VH_01x03
- J2_CN2: renamed from J2_CN2_9V_Main1; value Conn_01x02 -> JST_VH_01x02
- J3_CN3: renamed from J3_CN3_9V_Main1; value Conn_01x02 -> JST_VH_01x02
Connections:
- net CMD_IN: now reaches D2.1 (K), J2_CN2.2 (Pin_2), J3_CN3.2 (Pin_2), R3.1
- net at D2.2 (A), R1.1: now also Q2.2 (B); no longer Q2.3 (C)
- net TC_CMD_BUS: now reaches D1.1 (K), J10.2 (Pin_2), J11.2 (Pin_2), J4.2 (Pin_2), J5.2 (Pin_2), J6.2 (Pin_2), J7.2 (Pin_2), J8.2 (Pin_2), J9.2 (Pin_2)
- net TC_CMD_BUS: now also Q1.3 (C); no longer Q1.2 (E)
- new net: Q1.2 (B), Q2.3 (C), R2.1
Other:
- moved on the sheet: Q1, Q2

Commit message: UPDATE
Parts:
- renumbered D2 to D1, D1 to D2
Changed lines of the file:
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@@
 		(on_board yes)
 		(dnp no)
-		(property "Reference" "D1"
+		(property "Reference" "D2"
 			(at 76.454 37.338 0)
 			(effects
@@
 			(project ""
 				(path "/bd09a545-618a-47d2-a0b1-f0d03750b68a"
-					(reference "D1")
+					(reference "D2")
 					(unit 1)
 				)
@@
 		(on_board yes)
 		(dnp no)
-		(property "Reference" "D2"
+		(property "Reference" "D1"
 			(at 162.306 37.592 0)
 			(effects
@@
 			(project ""
 				(path "/bd09a545-618a-47d2-a0b1-f0d03750b68a"
-					(reference "D2")
-					(unit 1)
-				)
+					(reference "D1")
+					(unit 1)
+				)

Commit message: UPDATE
Connections:
- net -24V renamed +24V
Changed lines of the file:
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@@
 	(wire
 		(pts
-			(xy 45.72 45.72) (xy 44.45 45.72)
-		)
-		(stroke
-			(width 0)
-			(type default)
-		)
-	)
-	(wire
-		(pts
 			(xy 41.91 38.1) (xy 53.34 38.1)
 		)
@@
 	(wire
 		(pts
-			(xy 46.99 29.21) (xy 41.91 29.21)
+			(xy 44.45 29.21) (xy 41.91 29.21)
 		)
 		(stroke
@@
 	(wire
 		(pts
-			(xy 45.72 36.83) (xy 46.99 36.83)
-		)
-		(stroke
-			(width 0)
-			(type default)
-		)
-	)
-	(wire
-		(pts
 			(xy 153.67 111.76) (xy 153.67 137.16)
 		)
@@
 	(wire
 		(pts
-			(xy 44.45 45.72) (xy 44.45 93.98)
-		)
-		(stroke
-			(width 0)
-			(type default)
-		)
-	)
-	(wire
-		(pts
 			(xy 158.75 82.55) (xy 158.75 91.44)
 		)
@@
 	(wire
 		(pts
-			(xy 45.72 45.72) (xy 45.72 36.83)
+			(xy 44.45 29.21) (xy 44.45 93.98)
 		)
 		(stroke
@@
 	(wire
 		(pts
-			(xy 46.99 36.83) (xy 46.99 29.21)
-		)
-		(stroke
-			(width 0)
-			(type default)
-		)
-	)
-	(wire
-		(pts
 			(xy 147.32 59.69) (xy 118.11 59.69)
 		)
@@
 			)
 		)
-		(property "Value" "-24V"
+		(property "Value" "+24V"
 			(at 66.04 111.76 0)
 			(effects
@@
 			)
 		)
-		(property "Description" "Power symbol creates a global label with name \"-24V\""
+		(property "Description" "Power symbol creates a global label with name \"+24V\""
 			(at 66.04 116.84 0)
 			(effects

Commit message: UPDATE
Connections:
- net TC_CMD_BUS: now also Q1.2 (B); no longer Q1.3 (C)
- net at D1.2 (A), R1.1: now also Q2.3 (C); no longer Q2.2 (B)
- new net: Q1.3 (C), Q2.2 (B), R2.1
Other:
- moved on the sheet: Q1, Q2
Changed lines of the file:
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@@
 	)
 	(junction
-		(at 97.79 31.75)
-		(diameter 0)
-		(color 0 0 0 0)
-	)
-	(junction
 		(at 153.67 109.22)
 		(diameter 0)
@@
 	)
 	(junction
-		(at 115.57 116.84)
+		(at 130.81 31.75)
 		(diameter 0)
 		(color 0 0 0 0)
 	)
 	(junction
-		(at 125.73 31.75)
+		(at 115.57 116.84)
 		(diameter 0)
 		(color 0 0 0 0)
@@
 	)
 	(junction
+		(at 121.92 41.91)
+		(diameter 0)
+		(color 0 0 0 0)
+	)
+	(junction
 		(at 115.57 114.3)
 		(diameter 0)
@@
 	)
 	(junction
+		(at 82.55 36.83)
+		(diameter 0)
+		(color 0 0 0 0)
+	)
+	(junction
 		(at 133.35 109.22)
 		(diameter 0)
@@
 	)
 	(junction
+		(at 102.87 31.75)
+		(diameter 0)
+		(color 0 0 0 0)
+	)
+	(junction
 		(at 187.96 80.01)
 		(diameter 0)
@@
 	)
 	(junction
-		(at 125.73 41.91)
-		(diameter 0)
-		(color 0 0 0 0)
-	)
-	(junction
 		(at 83.82 139.7)
 		(diameter 0)
@@
 	)
 	(junction
-		(at 82.55 41.91)
-		(diameter 0)
-		(color 0 0 0 0)
-	)
-	(junction
 		(at 73.66 116.84)
 		(diameter 0)
@@
 	(wire
 		(pts
-			(xy 135.89 90.17) (xy 135.89 116.84)
-		)
-		(stroke
-			(width 0)
-			(type default)
-		)
-	)
-	(wire
-		(pts
-			(xy 134.62 36.83) (xy 138.43 36.83)
+			(xy 69.85 121.92) (xy 69.85 124.46)
 		)
 		(stroke
@@
 	(wire
 		(pts
-			(xy 69.85 121.92) (xy 69.85 124.46)
+			(xy 85.09 109.22) (xy 99.06 109.22)
 		)
 		(stroke
@@
 	(wire
 		(pts
-			(xy 85.09 109.22) (xy 99.06 109.22)
+			(xy 138.43 41.91) (xy 138.43 40.64)
 		)
 		(stroke
@@
 	(wire
 		(pts
-			(xy 67.31 31.75) (xy 97.79 31.75)
+			(xy 67.31 31.75) (xy 102.87 31.75)
 		)
 		(stroke
@@
 	(wire
 		(pts
-			(xy 147.32 59.69) (xy 147.32 69.85)
+			(xy 121.92 52.07) (xy 121.92 41.91)
 		)
 		(stroke
@@
 	(wire
 		(pts
-			(xy 41.91 48.26) (xy 53.34 48.26)
+			(xy 102.87 41.91) (xy 121.92 41.91)
 		)
 		(stroke
@@
 	(wire
 		(pts
-			(xy 187.96 87.63) (xy 147.32 87.63)
+			(xy 147.32 59.69) (xy 147.32 69.85)
 		)
 		(stroke
@@
 	(wire
 		(pts
-			(xy 80.01 34.29) (xy 82.55 34.29)
+			(xy 41.91 48.26) (xy 53.34 48.26)
 		)
 		(stroke
@@
 	(wire
 		(pts
-			(xy 147.32 69.85) (xy 147.32 72.39)
+			(xy 187.96 87.63) (xy 147.32 87.63)
 		)
 		(stroke
@@
 	(wire
 		(pts
-			(xy 125.73 31.75) (xy 144.78 31.75)
+			(xy 80.01 34.29) (xy 82.55 34.29)
 		)
 		(stroke
@@
 	(wire
 		(pts
-			(xy 115.57 137.16) (xy 133.35 137.16)
+			(xy 82.55 36.83) (xy 82.55 43.18)
 		)
 		(stroke
@@
 	(wire
 		(pts
-			(xy 85.09 111.76) (xy 99.06 111.76)
+			(xy 147.32 69.85) (xy 147.32 72.39)
 		)
 		(stroke
@@
 	(wire
 		(pts
-			(xy 53.34 45.72) (xy 168.91 45.72)
+			(xy 115.57 137.16) (xy 133.35 137.16)
 		)
 		(stroke
@@
 	(wire
 		(pts
-			(xy 140.97 52.07) (xy 125.73 52.07)
+			(xy 85.09 111.76) (xy 99.06 111.76)
 		)
 		(stroke
@@
 	(wire
 		(pts
-			(xy 57.15 116.84) (xy 57.15 57.15)
+			(xy 53.34 45.72) (xy 168.91 45.72)
 		)
 		(stroke
@@
 	(wire
 		(pts
-			(xy 52.07 80.01) (xy 52.07 133.35)
+			(xy 57.15 116.84) (xy 57.15 57.15)
 		)
 		(stroke
@@
 	(wire
 		(pts
-			(xy 82.55 41.91) (xy 97.79 41.91)
+			(xy 52.07 80.01) (xy 52.07 133.35)
 		)
 		(stroke
@@
 	(wire
 		(pts
-			(xy 82.55 41.91) (xy 82.55 43.18)
+			(xy 82.55 34.29) (xy 82.55 36.83)
 		)
 		(stroke
@@
 	(wire
 		(pts
-			(xy 115.57 41.91) (xy 125.73 41.91)
-		)
-		(stroke
-			(width 0)
-			(type default)
-		)
-	)
-	(wire
-		(pts
-			(xy 106.68 36.83) (xy 115.57 36.83)
+			(xy 102.87 31.75) (xy 130.81 31.75)
 		)
 		(stroke
@@
 	(wire
 		(pts
+			(xy 121.92 41.91) (xy 121.92 36.83)
+		)
+		(stroke
+			(width 0)
+			(type default)
+		)
+	)
+	(wire
+		(pts
 			(xy 153.67 111.76) (xy 153.67 137.16)
 		)
@@
 	(wire
 		(pts
+			(xy 140.97 52.07) (xy 121.92 52.07)
+		)
+		(stroke
+			(width 0)
+			(type default)
+		)
+	)
+	(wire
+		(pts
 			(xy 147.32 87.63) (xy 147.32 114.3)
 		)
@@
 	(wire
 		(pts
-			(xy 125.73 41.91) (xy 125.73 52.07)
+			(xy 130.81 31.75) (xy 144.78 31.75)
 		)
 		(stroke
@@
 	(wire
 		(pts
+			(xy 82.55 36.83) (xy 93.98 36.83)
+		)
+		(stroke
+			(width 0)
+			(type default)
+		)
+	)
+	(wire
+		(pts
 			(xy 208.28 40.64) (xy 208.28 110.49)
 		)
@@
 	(wire
 		(pts
-			(xy 158.75 72.39) (xy 158.75 80.01)
+			(xy 130.81 41.91) (xy 138.43 41.91)
 		)
 		(stroke
@@
 	(wire
 		(pts
-			(xy 73.66 119.38) (xy 73.66 116.84)
+			(xy 158.75 72.39) (xy 158.75 80.01)
 		)
 		(stroke
@@
 	(wire
 		(pts
-			(xy 44.45 93.98) (xy 138.43 93.98)
+			(xy 73.66 119.38) (xy 73.66 116.84)
 		)
 		(stroke
@@
 	(wire
 		(pts
-			(xy 83.82 142.24) (xy 99.06 142.24)
+			(xy 44.45 93.98) (xy 138.43 93.98)
 		)
 		(stroke
@@
 	(wire
 		(pts
-			(xy 46.99 52.07) (xy 58.42 52.07)
+			(xy 83.82 142.24) (xy 99.06 142.24)
 		)
 		(stroke
@@
 	(wire
 		(pts
-			(xy 115.57 36.83) (xy 115.57 41.91)
+			(xy 46.99 52.07) (xy 58.42 52.07)
 		)
 		(stroke
@@
 	(wire
 		(pts
-			(xy 138.43 36.83) (xy 138.43 40.64)
+			(xy 133.35 119.38) (xy 142.24 119.38)
 		)
 		(stroke
@@
 	(wire
 		(pts
-			(xy 133.35 119.38) (xy 142.24 119.38)
+			(xy 85.09 114.3) (xy 99.06 114.3)
 		)
 		(stroke
@@
 	(wire
 		(pts
-			(xy 85.09 114.3) (xy 99.06 114.3)
+			(xy 147.32 59.69) (xy 118.11 59.69)
 		)
 		(stroke
@@
 	(wire
 		(pts
-			(xy 147.32 59.69) (xy 118.11 59.69)
+			(xy 115.57 111.76) (xy 133.35 111.76)
 		)
 		(stroke
@@
 	(wire
 		(pts
-			(xy 115.57 111.76) (xy 133.35 111.76)
+			(xy 135.89 90.17) (xy 135.89 116.84)
 		)
 		(stroke
@@
 	(wire
 		(pts
-			(xy 97.79 31.75) (xy 125.73 31.75)
-		)
-		(stroke
-			(width 0)
-			(type default)
-		)
-	)
-	(wire
-		(pts
 			(xy 187.96 87.63) (xy 187.96 96.52)
 		)
@@
 	(wire
 		(pts
-			(xy 82.55 34.29) (xy 82.55 41.91)
-		)
-		(stroke
-			(width 0)
-			(type default)
-		)
-	)
-	(wire
-		(pts
 			(xy 187.96 74.93) (xy 187.96 80.01)
 		)
@@
 	(symbol
 		(lib_id "Transistor_BJT:DTC143E")
-		(at 128.27 36.83 180)
+		(at 128.27 36.83 0)
+		(mirror x)
 		(unit 1)
 		(exclude_from_sim no)
@@
 		(dnp no)
 		(property "Reference" "Q2"
-			(at 130.048 30.734 0)
+			(at 126.492 30.734 0)
 			(effects
 				(font
@@
 		)
 		(property "Value" "DTC143E"
-			(at 130.048 28.194 0)
+			(at 126.492 28.194 0)
 			(effects
 				(font
@@
 					(size 1.27 1.27)
 				)
+				(hide yes)
 			)
 		)
@@
 		(lib_name "DTC143E_1")
 		(lib_id "Transistor_BJT:DTC143E")
-		(at 100.33 36.83 180)
+		(at 100.33 36.83 0)
+		(mirror x)
 		(unit 1)
 		(exclude_from_sim no)
@@
 		(dnp no)
 		(property "Reference" "Q1"
-			(at 102.108 30.48 0)
+			(at 98.552 30.48 0)
 			(effects
 				(font
@@
 		)
 		(property "Value" "DTC143E"
-			(at 98.806 27.94 0)
+			(at 101.854 27.94 0)
 			(effects
 				(font
@@
 		)
 		(property "Footprint" "Package_TO_SOT_THT:TO-92_Inline"
-			(at 112.268 43.688 0)
+			(at 88.392 43.688 0)
 			(effects
 				(font
