File: KiCad/TC_Interface_Board-OLD/TC_Interface_Board.kicad_pcb (KiCad board)
At the start: 2 copper layers, 68.9 x 121.6 mm, 30 parts, among them J10 Conn_01x05, J11 Conn_01x05, J1_24V_ROW1 Conn_01x04, J1_CN1 JST_VH_01x03, J2_CN2 JST_VH_01x02, J3_CN3 JST_VH_01x02, J4 Conn_01x05, J5 Conn_01x05, J6 Conn_01x05, J7 Conn_01x05, J8 Conn_01x05, J9 Conn_01x05, Q1 DTC143E, Q2 DTC143E, U1 MC34063AP

Commit message: UPDATE
Parts:
- D2: renamed from D1; footprint Diode_THT:D_DO-35_SOD27_P7.62mm_Horizontal -> Diode_THT:D_DO-41_SOD81_P7.62mm_Horizontal
- D3: footprint Diode_THT:D_DO-35_SOD27_P10.16mm_Horizontal -> Diode_THT:D_DO-41_SOD81_P10.16mm_Horizontal
- J10, J11, J4, J5, J6, J7, J8, J9: value Conn_01x05 -> JST_VH_01x05
- J1_24V_ROW1: value Conn_01x04 -> JST_VH_01x04
- R1: value 220 -> 220R
- R2: value 10k -> 10kR
- R3: value 1.2k -> 1k2R
- R4: value 6.2k -> 6k2R
- R5: value 0.22 -> 0R22
- R6: value 1k -> 1kR
- moved J9 16.4 mm to (161.4, 108.5), turned to 180 degrees
- moved J10 16.2 mm to (161.6, 89.2), turned to 180 degrees
- moved J5 16.2 mm to (139.7, 108.3), turned to 180 degrees
- moved J11 16.0 mm to (161.1, 70.6), turned to 180 degrees
- moved J8 16.0 mm to (161.3, 127.8), turned to 180 degrees
- moved J7 15.9 mm to (139.8, 70.5), turned to 180 degrees
- moved J6 15.9 mm to (139.8, 89.2), turned to 180 degrees
- moved J4 15.7 mm to (139.4, 127.8), turned to 180 degrees
- moved Q1 2.73 mm to (168.3, 118.7), turned to 0 degrees
- moved Q2 2.40 mm to (166.1, 110.2), turned to 0 degrees
- moved J1_CN1 0.80 mm to (123.4, 141.2)
- moved J2_CN2 0.45 mm to (143.3, 140.8)
- moved D1 0.35 mm to (166.5, 124.8)
- moved J3_CN3 0.34 mm to (156.8, 140.8)
- moved R2 0.27 mm to (169.8, 93.3)
- renumbered D2 to D1
Connections:
- C3 pad 1: Net-(J10-Pin_4) -> /VCC_9V
- D1 pad 2: GND -> /CMD_IN
- D2 pad 1: /CMD_IN -> Net-(D2-K)
- D2 pad 2: Net-(D1-A) -> Net-(D2-A)
- D3 pad 2: +24V -> 24V
- D5 pad 2: +24V -> 24V
- J10 pad 1: unconnected-(J10-Pin_1-Pad1) -> 24V
- J10 pad 2: /TC_CMD_BUS -> /VCC_9V
- J10 pad 4: Net-(J10-Pin_4) -> /TC_CMD_BUS
- J10 pad 5: +24V -> unconnected-(J10-Pin_5-Pad5)
- J11 pad 1: unconnected-(J11-Pin_1-Pad1) -> 24V
- J11 pad 2: /TC_CMD_BUS -> /VCC_9V
- J11 pad 4: Net-(J10-Pin_4) -> /TC_CMD_BUS
- J11 pad 5: +24V -> unconnected-(J11-Pin_5-Pad5)
- J1_24V_ROW1 pad 3: +24V -> 24V
- J1_24V_ROW1 pad 4: +24V -> 24V
- J1_CN1 pad 1: /TC_TX_REP -> /TC_DATA_REP
- J1_CN1 pad 2: +24V -> 24V
- J1_CN1 pad 3: GND -> /CMD_IN
- J2_CN2 pad 1: GND -> /CMD_IN
- J2_CN2 pad 2: /CMD_IN -> Net-(D2-K)
- J3_CN3 pad 1: GND -> /CMD_IN
- J3_CN3 pad 2: /CMD_IN -> Net-(D2-K)
- J4 pad 1: /TC_TX_REP -> 24V
- J4 pad 2: /TC_CMD_BUS -> /VCC_9V
- J4 pad 4: Net-(J10-Pin_4) -> /TC_CMD_BUS
- J4 pad 5: +24V -> /TC_DATA_REP
- J5 pad 1: unconnected-(J5-Pin_1-Pad1) -> 24V
- J5 pad 2: /TC_CMD_BUS -> /VCC_9V
- J5 pad 4: Net-(J10-Pin_4) -> /TC_CMD_BUS
- J5 pad 5: +24V -> unconnected-(J5-Pin_5-Pad5)
- J6 pad 1: unconnected-(J6-Pin_1-Pad1) -> 24V
- J6 pad 2: /TC_CMD_BUS -> /VCC_9V
- J6 pad 4: Net-(J10-Pin_4) -> /TC_CMD_BUS
- J6 pad 5: +24V -> unconnected-(J6-Pin_5-Pad5)
- J7 pad 1: unconnected-(J7-Pin_1-Pad1) -> 24V
- J7 pad 2: /TC_CMD_BUS -> /VCC_9V
- J7 pad 4: Net-(J10-Pin_4) -> /TC_CMD_BUS
- J7 pad 5: +24V -> unconnected-(J7-Pin_5-Pad5)
- J8 pad 1: unconnected-(J8-Pin_1-Pad1) -> 24V
- J8 pad 2: /TC_CMD_BUS -> /VCC_9V
- J8 pad 4: Net-(J10-Pin_4) -> /TC_CMD_BUS
- J8 pad 5: +24V -> unconnected-(J8-Pin_5-Pad5)
- J9 pad 1: unconnected-(J9-Pin_1-Pad1) -> 24V
- J9 pad 2: /TC_CMD_BUS -> /VCC_9V
- J9 pad 4: Net-(J10-Pin_4) -> /TC_CMD_BUS
- J9 pad 5: +24V -> unconnected-(J9-Pin_5-Pad5)
- L1_Inductor1 pad 1: Net-(J10-Pin_4) -> /VCC_9V
- Q1 pad 3: Net-(Q1-C) -> /CMD_IN
- Q2 pad 2: Net-(Q1-C) -> /TC_CMD_BUS
- Q2 pad 3: Net-(D1-A) -> /CMD_IN
- R1 pad 1: Net-(D1-A) -> Net-(D2-A)
- R1 pad 2: GND -> /CMD_IN
- R2 pad 1: Net-(Q1-C) -> unconnected-(R2-Pad1)
- R2 pad 2: +24V -> 24V
- R3 pad 1: /CMD_IN -> Net-(D2-K)
- R4 pad 2: Net-(J10-Pin_4) -> /VCC_9V
- R6 pad 1: GND -> /CMD_IN
Routing:
- net 24V: track 0.00 -> 240.7 mm
- net +24V: track 240.7 -> 0.00 mm
- net Net-(J10-Pin_4): track 204.4 -> 0.00 mm, vias 2 -> 0
- net /VCC_9V: track 0.00 -> 204.4 mm, vias 0 -> 2
- net GND: track 509.0 -> 357.0 mm
- net /CMD_IN: track 71.2 -> 161.6 mm
- net Net-(D2-K): track 0.00 -> 71.2 mm
- net Net-(Q1-C): track 26.9 -> 0.00 mm
- net Net-(D1-A): track 13.3 -> 0.00 mm
- net /TC_TX_REP: track 13.2 -> 0.00 mm
- net /TC_DATA_REP: track 0.00 -> 13.2 mm
- net /TC_CMD_BUS: track 167.8 -> 175.8 mm
- net Net-(D2-A): track 0.00 -> 4.93 mm
Other:
- board text added: "GND"
- board text added: "SIG_BUS_RX"
- board text added: "TC_TX (ONLY CN4)"
- board text removed: "CMD_IN"
