File: KiCad/TC_Interface_Board-OLD/TC_Interface_Board.kicad_sch (KiCad schematic)
At the start: 30 parts, among them J10 Conn_01x05, J11 Conn_01x05, J1_24V_ROW1 Conn_01x04, J1_CN1 JST_VH_01x03, J2_CN2 JST_VH_01x02, J3_CN3 JST_VH_01x02, J4 Conn_01x05, J5 Conn_01x05, J6 Conn_01x05, J7 Conn_01x05, J8 Conn_01x05, J9 Conn_01x05, Q1 DTC143E, Q2 DTC143E, U1 MC34063AP

Commit message: UPDATE
Parts:
- D2: renamed from D1; footprint Diode_THT:D_DO-35_SOD27_P7.62mm_Horizontal -> Diode_THT:D_DO-41_SOD81_P7.62mm_Horizontal
- D3: footprint Diode_THT:D_DO-35_SOD27_P10.16mm_Horizontal -> Diode_THT:D_DO-41_SOD81_P10.16mm_Horizontal
- J10, J11, J4, J5, J6, J7, J8, J9: value Conn_01x05 -> JST_VH_01x05
- J1_24V_ROW1: value Conn_01x04 -> JST_VH_01x04
- R1: value 220 -> 220R
- R2: value 10k -> 10kR
- R3: value 1.2k -> 1k2R
- R4: value 6.2k -> 6k2R
- R5: value 0.22 -> 0R22
- R6: value 1k -> 1kR
- renumbered D2 to D1
Connections:
- net CMD_IN: now also D1.2 (A), J1_CN1.3 (Pin_3), J2_CN2.1 (Pin_1), J3_CN3.1 (Pin_1), Q1.3 (B), Q2.3 (B), R1.2, R6.1; no longer D2.1 (K), J2_CN2.2 (Pin_2), J3_CN3.2 (Pin_2), R3.1
- net GND: no longer D1.2 (A), J1_CN1.3 (Pin_3), J2_CN2.1 (Pin_1), J3_CN3.1 (Pin_1), R1.2, R6.1
- net TC_CMD_BUS: now also J10.4 (Pin_4), J11.4 (Pin_4), J4.4 (Pin_4), J5.4 (Pin_4), J6.4 (Pin_4), J7.4 (Pin_4), J8.4 (Pin_4), J9.4 (Pin_4), Q2.2 (C); no longer J10.2 (Pin_2), J11.2 (Pin_2), J4.2 (Pin_2), J5.2 (Pin_2), J6.2 (Pin_2), J7.2 (Pin_2), J8.2 (Pin_2), J9.2 (Pin_2)
- net at D2.2 (A), R1.1: no longer Q2.3 (C)
- net 24V: now reaches J9.1 (Pin_1)
- net 24V: now also D3.2 (A), D5.2 (A), J10.1 (Pin_1), J11.1 (Pin_1), J1_24V_ROW1.3 (Pin_3), J1_24V_ROW1.4 (Pin_4), J1_CN1.2 (Pin_2), J4.1 (Pin_1), J5.1 (Pin_1), J6.1 (Pin_1), J7.1 (Pin_1), J8.1 (Pin_1), R2.2
- removed net +24V: D3.2 (A), D5.2 (A), J10.5 (Pin_5), J11.5 (Pin_5), J1_24V_ROW1.3 (Pin_3), J1_24V_ROW1.4 (Pin_4), J1_CN1.2 (Pin_2), J4.5 (Pin_5), J5.5 (Pin_5), J6.5 (Pin_5), J7.5 (Pin_5), J8.5 (Pin_5), J9.5 (Pin_5), R2.2
- net TC_TX_REP renamed TC_DATA_REP
- net TC_DATA_REP: now also J4.5 (Pin_5); no longer J4.1 (Pin_1)
- new net: D2.1 (K), J2_CN2.2 (Pin_2), J3_CN3.2 (Pin_2), R3.1
- new net VCC_9V: C3.1, J10.2 (Pin_2), J11.2 (Pin_2), J4.2 (Pin_2), J5.2 (Pin_2), J6.2 (Pin_2), J7.2 (Pin_2), J8.2 (Pin_2), J9.2 (Pin_2), L1_Inductor1.1, R4.2
- now unconnected: R2.1
Other:
- moved on the sheet: J10, J11, J4, J5, J6, J7, J8, J9, Q1, Q2
