File: KiCad/TC_Interface_Board-Freerouting/TC_Interface_Board.kicad_sch (KiCad schematic)
At the start: 30 parts, among them J10 JST_VH_01x05, J11 JST_VH_01x05, J1_24V_ROW1 JST_VH_01x04, J1_CN1 JST_VH_01x03, J2_CN2 JST_VH_01x02, J3_CN3 JST_VH_01x02, J4 JST_VH_01x05, J5 JST_VH_01x05, J6 JST_VH_01x05, J7 JST_VH_01x05, J8 JST_VH_01x05, J9 JST_VH_01x05, Q1 DTC143E, Q2 DTC143E, U1 MC34063AP

Commit message: UPDATE
Parts:
- D2: footprint Diode_THT:D_DO-41_SOD81_P7.62mm_Horizontal -> Diode_THT:D_DO-35_SOD27_P7.62mm_Horizontal
- D5: renamed from D3; footprint Diode_THT:D_DO-41_SOD81_P10.16mm_Horizontal -> Diode_THT:D_DO-35_SOD27_P10.16mm_Horizontal
- L1_Inductor1: value L_Ferrite -> 330uH
- R1: renamed from R5; value 0R22 -> 220
- R2: renamed from R1; value 220R -> 10k
- R3: renamed from R2; value 10kR -> 1k2; footprint Resistor_THT:R_Axial_DIN0207_L6.3mm_D2.5mm_P7.62mm_Horizontal -> Resistor_THT:R_Axial_DIN0207_L6.3mm_D2.5mm_P10.16mm_Horizontal
- R4: value 6k2R -> 6k2
- R5: renamed from R6; value 1kR -> 0R22; footprint Resistor_THT:R_Axial_DIN0207_L6.3mm_D2.5mm_P7.62mm_Horizontal -> Resistor_THT:R_Axial_DIN0309_L9.0mm_D3.2mm_P12.70mm_Horizontal
- R6: renamed from R3; value 1k2R -> 1k; footprint Resistor_THT:R_Axial_DIN0207_L6.3mm_D2.5mm_P15.24mm_Horizontal -> Resistor_THT:R_Axial_DIN0204_L3.6mm_D1.6mm_P7.62mm_Horizontal
- renumbered C2 to C1, C1 to C2, D5 to D3, J5 to J1, J1_24V_ROW1 to J1_24V1, J8 to J2, J2_CN2 to J2_CN1, J7 to J3, J3_CN3 to J3_CN1, J6 to J5, J10 to J6, J9 to J7, J11 to J8, Q2 to Q1, Q1 to Q2
Connections:
- net CMD_IN: now also D1.1 (K), J2_CN1.2 (Pin_2), J3_CN1.2 (Pin_2), R3.1; no longer D1.2 (A), J1_CN1.3 (Pin_3), J2_CN1.1 (Pin_1), J3_CN1.1 (Pin_1), Q1.3 (B), Q2.3 (B), R2.2, R5.1
- net GND: now also D2.2 (A), J1_CN1.3 (Pin_3), J2_CN1.1 (Pin_1), J3_CN1.1 (Pin_1), R1.2, R6.2
- net TC_CMD_BUS: now also D2.1 (K); no longer D1.1 (K), Q2.2 (C)
- net +24V_FILT: now reaches D5.1 (K)
- net +24V_FILT: now also C2.1, R5.2, U1.6 (Vin); no longer R6.2
- net V_FB: now reaches R4.1, U1.5 (Vfb)
- net V_FB: now also R6.1; no longer R5.2
- net I_SENSE: now reaches U1.1 (SwC), U1.7 (Ipk), U1.8 (DC)
- net I_SENSE: now also R5.1; no longer R1.2
- net SW_OUT: now reaches D4.1 (K), L1_Inductor1.2, U1.2 (SwE)
- net MC34063_TC: now reaches U1.3 (TC)
- net MC34063_TC: now also C1.1; no longer C2.1
- net +24V: now reaches R2.1
- net +24V: now also D3.1 (K), D5.2 (A), J1.1 (Pin_1), J1_24V1.3 (Pin_3), J1_24V1.4 (Pin_4), J1_CN1.2 (Pin_2), J2.1 (Pin_1), J3.1 (Pin_1), J4.1 (Pin_1), J5.1 (Pin_1), J6.1 (Pin_1), J7.1 (Pin_1), J8.1 (Pin_1); no longer D2.2 (A)
- removed net 24V: D3.2 (A), D5.2 (A), J1.1 (Pin_1), J1_24V1.3 (Pin_3), J1_24V1.4 (Pin_4), J1_CN1.2 (Pin_2), J2.1 (Pin_1), J3.1 (Pin_1), J4.1 (Pin_1), J5.1 (Pin_1), J6.1 (Pin_1), J7.1 (Pin_1), J8.1 (Pin_1), R3.2
- net TC_DATA_REP renamed TC_TX_REP
- net VCC_9V renamed +5V_OUT
- new net CMD_IN_PROT: D3.2 (A), R3.2
- new net Q1_BASE: Q1.3 (B), Q2.2 (C), R2.2
- new net Q2_BASE: D1.2 (A), Q2.3 (B), R1.1
Other:
- note added: "2026.2.5"
- note added: "Pin 1 RX CN4のみ結線 Pin 2 TC_BUS Pin 3 GND Pin 4 +9V out Pin 5 +24V"
- note removed: "2026.2.1"
- note removed: "Pin 1 RX CN4のみ結線 Pin 2 不明(推定TX) Pin 3 GND Pin 4 +9V Pin 5 +24V D5通過後の24V太配線／外部供給実績あり"
- moved on the sheet: C1, C2, D1, D2, D3, D5, J1, J2, J3, J4, J5, J6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
