File: KiCad/ESP32S3_Snifar-Freerouting/ESP32S3_Snifar.kicad_pcb (KiCad board)
At the start: 2 copper layers, 95 x 70 mm, 22 parts, among them J1 Conn_01x04_Socket, Q1 2N7000, U1 MOUDLE-SEEEDUINO-XIAO-ESP32S3

Commit message: UPDATE
Parts:
- moved R5 27.7 mm to (72.5, 51.8), turned to 0 degrees
- moved R7 20.7 mm to (89.2, 63.8)
- moved R2 19.3 mm to (72.8, 43.5), turned to 0 degrees
- moved R8 16.6 mm to (83.8, 63.6)
- moved R4 15.4 mm to (57.0, 46.8)
- moved TP3 15.0 mm to (69.0, 61.2)
- moved TP2 14.7 mm to (68.8, 47.1)
- moved Q1 13.3 mm to (75.3, 64.8)
- moved R1 13.0 mm to (58.8, 38.6)
- moved R9 12.8 mm to (65.2, 50.0)
- moved D4 12.6 mm to (86.9, 57.0)
- moved R6 11.0 mm to (75.1, 47.1)
- moved D3 9.37 mm to (94.5, 50.8)
- moved TP1 9.37 mm to (69.6, 38.5)
- moved R3 7.39 mm to (75.3, 38.5)
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Routing:
- net Net-(D3-A): track 72.5 -> 34.7 mm
- net Net-(U1-PA6_A10_D10_MOSI): track 46.9 -> 17.5 mm
- net GND: track 199.5 -> 173.9 mm
- net Net-(D1-A): track 69.2 -> 44.0 mm
- net Net-(D1-K): track 60.2 -> 37.0 mm
- net Net-(R4-Pad2): track 34.4 -> 19.0 mm
- net Net-(R1-Pad2): track 25.2 -> 17.5 mm
- net Net-(J1-Pin_4): track 15.6 -> 22.7 mm
- net Net-(Q1-G): track 9.44 -> 14.1 mm
- net Net-(Q1-D): track 11.7 -> 14.9 mm
- net Net-(J1-Pin_3): track 16.6 -> 19.2 mm
- net Net-(J1-Pin_2): track 28.2 -> 27.7 mm, vias 1 -> 0

Commit message: UPDATE
Parts:
- moved R4 0.86 mm to (56.8, 46.0)
Routing:
- net GND: track 173.9 -> 160.7 mm
- net Net-(D1-K): track 37.0 -> 42.7 mm
- net Net-(D3-A): track 34.7 -> 38.2 mm
- net Net-(D1-A): track 44.0 -> 46.9 mm
- net Net-(R4-Pad2): track 19.0 -> 20.4 mm
- net Net-(R1-Pad2): track 17.5 -> 18.3 mm
