File: KiCad/ESP32S3_Snifar-backup/ESP32S3_Snifar.kicad_pcb (KiCad board)
At the start: 2 copper layers, 95 x 70 mm, 22 parts, among them J1 Conn_01x04_Socket, Q1 2N7000, U1 MOUDLE-SEEEDUINO-XIAO-ESP32S3

Commit message: Create
Parts:
- removed TP2: TestPoint, TestPoint:TestPoint_THTPad_D1.0mm_Drill0.5mm
- added JP1: Jumper_2_Open, Connector_Wire:SolderWire-0.25sqmm_1x02_P4.5mm_D0.65mm_OD2mm, F.Cu at (105.0, 41.8)
- added JP2: Jumper_2_Open, Connector_Wire:SolderWire-0.25sqmm_1x02_P4.5mm_D0.65mm_OD2mm, F.Cu at (105.1, 35.8)
- added JP3: Jumper_2_Open, Connector_Wire:SolderWire-0.25sqmm_1x02_P4.5mm_D0.65mm_OD2mm, F.Cu at (96.2, 72.1)
- added JP4: Jumper_2_Open, Connector_Wire:SolderWire-0.25sqmm_1x02_P4.5mm_D0.65mm_OD2mm, F.Cu at (94.3, 67.3)
- added JP5: Jumper_2_Open, Connector_Wire:SolderWire-0.25sqmm_1x02_P4.5mm_D0.65mm_OD2mm, F.Cu at (64.8, 60.8)
- added JP6: Jumper_2_Open, Connector_Wire:SolderWire-0.25sqmm_1x02_P4.5mm_D0.65mm_OD2mm, F.Cu at (71.5, 65.6)
- added M3: MountingHole_3.2mm_M3, MountingHole:MountingHole_3.2mm_M3, F.Cu at (121.0, 34.1)
- added M3: MountingHole_3.2mm_M3, MountingHole:MountingHole_3.2mm_M3, F.Cu at (121.1, 96.0)
- added M3: MountingHole_3.2mm_M3, MountingHole:MountingHole_3.2mm_M3, F.Cu at (34.1, 33.9)
- added M3: MountingHole_3.2mm_M3, MountingHole:MountingHole_3.2mm_M3, F.Cu at (34.1, 96.0)
- added Q2: 2N7000, Package_TO_SOT_THT:TO-92_Inline, F.Cu at (57.7, 68.0)
- added R10: 4k7, Resistor_THT:R_Axial_DIN0204_L3.6mm_D1.6mm_P5.08mm_Vertical, F.Cu at (63.3, 65.5)
- added R11: 100k, Resistor_THT:R_Axial_DIN0204_L3.6mm_D1.6mm_P5.08mm_Vertical, F.Cu at (62.0, 68.4)
- R5: value 3k3 -> 33k
- R6: value 2k2 -> 220R
- R9: value 100k -> 100R
- moved R5 34.0 mm to (76.1, 46.1)
- moved R4 29.8 mm to (71.0, 42.0)
- moved R6 20.4 mm to (51.0, 65.9), turned to 90 degrees
- moved R7 14.2 mm to (73.3, 54.1)
- moved R9 14.2 mm to (60.6, 45.6)
- moved TP3 14.2 mm to (60.8, 55.7)
- moved Q1 14.2 mm to (67.1, 55.4)
- moved R8 14.2 mm to (73.4, 57.3)
- moved D4 12.0 mm to (84.1, 57.2)
- moved D3 8.87 mm to (96.0, 51.5)
- moved A1 7.73 mm to (70.8, 93.7)
- moved D2 5.11 mm to (84.1, 43.7)
- moved TP5 4.97 mm to (81.3, 51.5)
- moved D1 2.09 mm to (94.3, 39.4)
- moved R2 1.50 mm to (53.5, 42.1)
Connections:
- net Net-(J1-Pin_2) renamed /SEND_BUS_OUT_FOR_CN2_2
- net Net-(J1-Pin_4) renamed /SIG_FOR_CN1_1
- net Net-(Q1-D) renamed /MOS_DRAIN
- net Net-(Q1-G) renamed /MOS_GATE
- net Net-(R1-Pad2) renamed /SIG_DIV
- net Net-(U1-PA6_A10_D10_MOSI) renamed /MCU_TX_TRIG
- A1 pad 13: unconnected-(A1-D10-Pad13) -> /SIG_FOR_Arduino_nano
- A1 pad 14: unconnected-(A1-MOSI-Pad14) -> /SEND_BUS_TO_Aruduino_nano
- D1 pad 2: Net-(D1-A) -> /MUC_RX
- D2 pad 1: Net-(D1-A) -> /MUC_RX
- D3 pad 1: Net-(D1-K) -> Net-(D3-K)
- J1 pad 3: Net-(J1-Pin_3) -> /SIG_FOR_Arduino_nano
- R3 pad 2: Net-(D1-A) -> /MUC_RX
- R4 pad 1: Net-(J1-Pin_3) -> /SIG_FOR_Arduino_nano
- R4 pad 2: Net-(R4-Pad2) -> Net-(D3-A)
- R5 pad 1: Net-(R4-Pad2) -> Net-(D3-A)
- R6 pad 1: Net-(R4-Pad2) -> Net-(Q2-G)
- R6 pad 2: Net-(D3-A) -> Net-(JP5-A)
- TP4 pad 1: Net-(D1-A) -> /MUC_RX
- U1 pad 12: Net-(D1-K) -> Net-(JP3-B)
- U1 pad 14: unconnected-(U1-5V-Pad14) -> Net-(JP6-B)
- U1 pad 4: Net-(D1-A) -> /MCU_RX
- U1 pad 6: Net-(D3-A) -> unconnected-(U1-PA9_A5_D5_SCL-Pad6)
Routing:
- net /SIG_FOR_Arduino_nano: track 0.00 -> 160.1 mm
- net /SEND_BUS_TO_Aruduino_nano: track 0.00 -> 74.7 mm
- net Net-(D1-A): track 69.2 -> 0.00 mm
- net Net-(JP6-B): track 0.00 -> 50.0 mm
- net /MUC_RX: track 0.00 -> 46.8 mm
- net Net-(R4-Pad2): track 34.4 -> 0.00 mm
- net Net-(D1-K): track 60.2 -> 27.8 mm
- net Net-(JP3-B): track 0.00 -> 32.1 mm
- net GND: track 199.5 -> 225.2 mm
- net Net-(D3-K): track 0.00 -> 20.6 mm
- net Net-(J1-Pin_3): track 16.6 -> 0.00 mm
- net Net-(JP5-A): track 0.00 -> 13.8 mm
- net Net-(Q2-G): track 0.00 -> 13.4 mm
- net /MCU_RX: track 0.00 -> 12.8 mm
- net Net-(D3-A): track 72.5 -> 61.0 mm
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