File: KiCad/TC106_Overall_circuit_diagram/TC_Interface_Board.kicad_sch (KiCad schematic)
At the start: 30 parts, among them J1 JST_VH_01x05, J1_24V1 JST_VH_01x04, J1_CN1 JST_VH_01x03, J2 JST_VH_01x05, J2_CN1 JST_VH_01x02, J3 JST_VH_01x05, J3_CN1 JST_VH_01x02, J4 JST_VH_01x05, J5 JST_VH_01x05, J6 JST_VH_01x05, J7 JST_VH_01x05, J8 JST_VH_01x05, Q1 DTC143E, Q2 DTC143E, U1 MC34063AP

Commit message: UPDATE
Parts:
- added C4, C5: 104, Capacitor_THT:C_Disc_D5.0mm_W2.5mm_P2.50mm, symbol Device:C
- added D6: HZ24, Diode_THT:D_DO-35_SOD27_P7.62mm_Horizontal, symbol Device:D_Zener
- added D7: D_TVS_Dual_AAC, symbol Device:D_TVS_Dual_AAC
- added J10: JST_VH_01x05, Connector_JST:JST_VH_B5P-VH-B_1x05_P3.96mm_Vertical, symbol Connector_Generic:Conn_01x05
- added J1_CN2: JST_VH_01x03, Connector_JST:JST_VH_B3P-VH-B_1x03_P3.96mm_Vertical, symbol Connector_Generic:Conn_01x03
- added J3_CN2: JST_VH_01x02, Connector_JST:JST_VH_B2P-VH-B_1x02_P3.96mm_Vertical, symbol Connector_Generic:Conn_01x02
- added J9: Conn_02x02_Odd_Even, symbol Connector_Generic:Conn_02x02_Odd_Even
- added JP1: Jumper_2_Open, symbol Jumper:Jumper_2_Open
- added Q3: 2SD1863, Package_TO_SOT_THT:TO-92_Inline, symbol Transistor_BJT:Q_NPN_ECB
- added Q4: Q_NPN_ECB, symbol Transistor_BJT:Q_NPN_ECB
- added R10, R13, R8, R9: 1k, Resistor_THT:R_Axial_DIN0204_L3.6mm_D1.6mm_P7.62mm_Horizontal, symbol Device:R
- added R11: 22k, Resistor_THT:R_Axial_DIN0204_L3.6mm_D1.6mm_P7.62mm_Horizontal, symbol Device:R
- added R12: 4k7, Resistor_THT:R_Axial_DIN0204_L3.6mm_D1.6mm_P7.62mm_Horizontal, symbol Device:R
- added R14: 10k, Resistor_THT:R_Axial_DIN0204_L3.6mm_D1.6mm_P7.62mm_Horizontal, symbol Device:R
- added R7: 330R, Resistor_THT:R_Axial_DIN0204_L3.6mm_D1.6mm_P7.62mm_Horizontal, symbol Device:R
- added U2: PIC16F73-ISP, symbol MCU_Microchip_PIC16:PIC16F73-ISP
Connections:
- net GND: now also C4.2, C5.2, D6.2 (A), D7.3 (common), J3_CN2.1 (Pin_1), J9.3 (Pin_3), JP1.2 (B), Q3.2 (C), Q4.1 (E), R14.2
- net CMD_IN renamed TC_RX
- net TC_TX_REP renamed TC_TX
- new net: C4.1, R8.2, R9.1
- new net: J1_CN2.3 (Pin_3), R10.1, R8.1
- new net: J9.2 (Pin_2), J9.4 (Pin_4), R10.2
- new net: J1_CN2.1 (Pin_1), JP1.1 (A)
- new net: R9.2, U2.18 (RC7/RX/DT)
- new net: R7.2, U2.11 (RC0/T10S0/T1CKI)
- new net +5V: R11.2, R12.2
- new net 5V: J9.1 (Pin_1)
- new net Pic33_RX: C5.1, R13.2, R14.1
- new net Pic33_TX: Q4.2 (C)
- new net TC_CMD_106: D7.1 (A1), J10.4 (Pin_4), R12.1, R13.1
- new net TC_RX_MAIN: D6.1 (K), J3_CN2.2 (Pin_2), Q3.1 (E), R7.1
- new net TC_TX_106: D7.2 (A2), J10.5 (Pin_5), Q4.3 (B), R11.1
Other:
- note added: "Main controller"
- note added: "TC106"
- note added: "To TC106"
- note removed: "Pin 1 RX CN4のみ結線 Pin 2 TC_BUS Pin 3 GND Pin 4 +9V out Pin 5 +24V"
