File: KiCad/TC106_Overall_circuit_diagram/TC106_Overall_circuit_diagram.kicad_sch (KiCad schematic)
At the start: 50 parts, among them J1 JST_VH_01x05, J10 JST_VH_01x05, J1_24V1 JST_VH_01x04, J1_CN1 JST_VH_01x03, J2 JST_VH_01x05, J2_CN1 JST_VH_01x02, J3 JST_VH_01x05, J3_CN1 JST_VH_01x02, J4 JST_VH_01x05, J4_CN2 JST_VH_01x02, J5 JST_VH_01x05, J5_CN2 JST_VH_01x03, J6 JST_VH_01x05, J7 JST_VH_01x05, J8 JST_VH_01x05, J9 Conn_02x02_Odd_Even, Q1 DTC143E, Q2 DTC143E, Q3 2SD1863, Q4 Q_NPN_ECB, U1 MC34063AP, U2 PIC16F73-ISP

Commit message: UPDATE
Parts:
- added U3: dsPIC33FJ16MC102, dsPIC33FJ16MC102:SOP65P780X200-28N, symbol MCU_Microchip_PIC16:PIC16F73-ISP
Connections:
- net Pic33_RX: no longer names the net of C5.1, R13.2, R14.1
- net Pic33_RX: now also U3.11 (RC0/T10S0/T1CKI)
- net Pic33_TX: no longer names the net of Q4.2 (C)
- net Pic33_TX: now also U3.12 (RC1/CCP2/T1OSI)
Changed lines of the file:
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@@
 	(wire
 		(pts
+			(xy 257.81 157.48) (xy 257.81 134.62)
+		)
+		(stroke
+			(width 0)
+			(type default)
+		)
+	)
+	(wire
+		(pts
 			(xy 55.88 119.38) (xy 66.04 119.38)
 		)
@@
 	(wire
 		(pts
+			(xy 260.35 132.08) (xy 243.84 132.08)
+		)
+		(stroke
+			(width 0)
+			(type default)
+		)
+	)
+	(wire
+		(pts
 			(xy 67.31 31.75) (xy 87.63 31.75)
 		)
@@
 	(wire
 		(pts
+			(xy 227.33 157.48) (xy 257.81 157.48)
+		)
+		(stroke
+			(width 0)
+			(type default)
+		)
+	)
+	(wire
+		(pts
 			(xy 74.93 186.69) (xy 80.01 186.69)
 		)
@@
 	(wire
 		(pts
-			(xy 199.39 154.94) (xy 204.47 154.94)
+			(xy 199.39 154.94) (xy 227.33 154.94)
 		)
 		(stroke
@@
 	(wire
 		(pts
-			(xy 243.84 138.43) (xy 243.84 143.51)
-		)
-		(stroke
-			(width 0)
-			(type default)
-		)
-	)
-	(wire
-		(pts
 			(xy 44.45 29.21) (xy 44.45 93.98)
 		)
@@
 	(wire
 		(pts
+			(xy 227.33 154.94) (xy 227.33 157.48)
+		)
+		(stroke
+			(width 0)
+			(type default)
+		)
+	)
+	(wire
+		(pts
 			(xy 204.47 31.75) (xy 158.75 31.75)
 		)
@@
 	(wire
 		(pts
+			(xy 257.81 134.62) (xy 260.35 134.62)
+		)
+		(stroke
+			(width 0)
+			(type default)
+		)
+	)
+	(wire
+		(pts
 			(xy 99.06 109.22) (xy 115.57 109.22)
 		)
@@
 	(wire
 		(pts
+			(xy 243.84 132.08) (xy 243.84 143.51)
+		)
+		(stroke
+			(width 0)
+			(type default)
+		)
+	)
+	(wire
+		(pts
 			(xy 151.13 142.24) (xy 151.13 116.84)
 		)
@@
 		)
 	)
-	(label "Pic33_RX"
-		(at 243.84 138.43 0)
-		(effects
-			(font
-				(size 1.27 1.27)
-			)
-			(justify left bottom)
-		)
-	)
 	(label "TC_RX"
 		(at 45.72 157.48 0)
@@
 		)
 	)
-	(label "Pic33_TX"
-		(at 204.47 154.94 0)
-		(effects
-			(font
-				(size 1.27 1.27)
-			)
-			(justify left bottom)
-		)
-	)
 	(label "TC_CMD_BUS"
 		(at 151.13 74.93 90)
@@
 					(unit 1)
 				)
+			)
+		)
+	)
+	(symbol
+		(lib_id "MCU_Microchip_PIC16:PIC16F73-ISP")
+		(at 280.67 132.08 0)
+		(unit 1)
+		(exclude_from_sim no)
+		(in_bom yes)
+		(on_board yes)
+		(dnp no)
+		(fields_autoplaced yes)
+		(property "Reference" "U3"
+			(at 282.8133 105.41 0)
+			(effects
+				(font
+					(size 1.27 1.27)
+				)
+				(justify left)
+			)
+		)
+		(property "Value" "dsPIC33FJ16MC102"
+			(at 282.8133 107.95 0)
+			(effects
+				(font
+					(size 1.27 1.27)
+				)
+				(justify left)
+			)
+		)
+		(property "Footprint" "dsPIC33FJ16MC102:SOP65P780X200-28N"
+			(at 280.67 132.08 0)
+			(effects
+				(font
+					(size 1.27 1.27)
+					(italic yes)
+				)
+				(hide yes)
+			)
+		)
+		(property "Datasheet" "http://ww1.microchip.com/downloads/en/DeviceDoc/30325b.pdf"
+			(at 280.67 132.08 0)
+			(effects
+				(font
+					(size 1.27 1.27)
+				)
+				(hide yes)
+			)
+		)
+		(property "Description" "PIC16F73, 4K Flash, 192B SRAM, ADC, PWM, SDIP28"
+			(at 280.67 132.08 0)
+			(effects
+				(font
+					(size 1.27 1.27)
+				)
+				(hide yes)
+			)
+		)
+		(pin "15"
+		)
+		(pin "7"
+		)
+		(pin "5"
+		)
+		(pin "1"
+		)
+		(pin "17"
+		)
+		(pin "20"
+		)
+		(pin "4"
+		)
+		(pin "8"
+		)
+		(pin "12"
+		)
+		(pin "18"
+		)
+		(pin "13"
+		)
+		(pin "9"
+		)
+		(pin "10"
+		)
+		(pin "14"
+		)
+		(pin "19"
+		)
+		(pin "2"
+		)
+		(pin "6"
+		)
+		(pin "16"
+		)
+		(pin "11"
+		)
+		(pin "3"
+		)
+		(pin "23"
+		)
+		(pin "25"
+		)
+		(pin "27"
+		)
+		(pin "22"
+		)
+		(pin "24"
+		)
+		(pin "26"
+		)
+		(pin "21"
+		)
+		(pin "28"
+		)
+		(instances
+			(project ""
+				(path "/bd09a545-618a-47d2-a0b1-f0d03750b68a"
+					(reference "U3")
+					(unit 1)
+				)

Commit message: UPDATE
Parts:
- removed U3: dsPIC33FJ16MC102, dsPIC33FJ16MC102:SOP65P780X200-28N, symbol MCU_Microchip_PIC16:PIC16F73-ISP
- added J11: Dummy dsPIC33FJ16MC102, dsPIC33FJ16MC102:SOP65P780X200-28N, symbol Connector:Conn_01x29_Pin
Connections:
- net at C5.1, R13.2, R14.1: now also J11.11 (Pin_11)
- net at Q4.2 (C): now also J11.12 (Pin_12)
Changed lines of the file:
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@@
 	(wire
 		(pts
-			(xy 257.81 157.48) (xy 257.81 134.62)
-		)
-		(stroke
-			(width 0)
-			(type default)
-		)
-	)
-	(wire
-		(pts
 			(xy 55.88 119.38) (xy 66.04 119.38)
 		)
@@
 	(wire
 		(pts
-			(xy 260.35 132.08) (xy 243.84 132.08)
-		)
-		(stroke
-			(width 0)
-			(type default)
-		)
-	)
-	(wire
-		(pts
 			(xy 67.31 31.75) (xy 87.63 31.75)
 		)
@@
 	(wire
 		(pts
+			(xy 236.22 123.19) (xy 236.22 132.08)
+		)
+		(stroke
+			(width 0)
+			(type default)
+		)
+	)
+	(wire
+		(pts
 			(xy 118.11 59.69) (xy 147.32 59.69)
 		)
@@
 	(wire
 		(pts
+			(xy 243.84 132.08) (xy 236.22 132.08)
+		)
+		(stroke
+			(width 0)
+			(type default)
+		)
+	)
+	(wire
+		(pts
 			(xy 99.06 116.84) (xy 115.57 116.84)
 		)
@@
 	(wire
 		(pts
+			(xy 257.81 130.81) (xy 257.81 157.48)
+		)
+		(stroke
+			(width 0)
+			(type default)
+		)
+	)
+	(wire
+		(pts
 			(xy 124.46 173.99) (xy 129.54 173.99)
 		)
@@
 	(wire
 		(pts
+			(xy 238.76 123.19) (xy 238.76 130.81)
+		)
+		(stroke
+			(width 0)
+			(type default)
+		)
+	)
+	(wire
+		(pts
 			(xy 72.39 34.29) (xy 72.39 44.45)
 		)
@@
 	(wire
 		(pts
-			(xy 257.81 134.62) (xy 260.35 134.62)
-		)
-		(stroke
-			(width 0)
-			(type default)
-		)
-	)
-	(wire
-		(pts
 			(xy 99.06 109.22) (xy 115.57 109.22)
 		)
@@
 		)
 	)
+	(wire
+		(pts
+			(xy 238.76 130.81) (xy 257.81 130.81)
+		)
+		(stroke
+			(width 0)
+			(type default)
+		)
+	)
 	(table
 		(column_count 3)
@@
 		(on_board yes)
 		(dnp no)
-		(fields_autoplaced yes)
 		(property "Reference" "R14"
-			(at 255.27 149.8599 0)
+			(at 253.746 144.272 0)
 			(effects
 				(font
@@
 		)
 		(property "Value" "10k"
-			(at 255.27 152.3999 0)
+			(at 253.746 146.812 0)
 			(effects
 				(font
@@
 	)
 	(symbol
+		(lib_id "Connector:Conn_01x29_Pin")
+		(at 246.38 128.27 90)
+		(unit 1)
+		(exclude_from_sim no)
+		(in_bom yes)
+		(on_board yes)
+		(dnp no)
+		(property "Reference" "J11"
+			(at 215.392 117.348 90)
+			(effects
+				(font
+					(size 1.27 1.27)
+				)
+			)
+		)
+		(property "Value" "Dummy dsPIC33FJ16MC102"
+			(at 216.154 120.142 90)
+			(effects
+				(font
+					(size 1.27 1.27)
+				)
+			)
+		)
+		(property "Footprint" "dsPIC33FJ16MC102:SOP65P780X200-28N"
+			(at 246.38 128.27 0)
+			(effects
+				(font
+					(size 1.27 1.27)
+				)
+				(hide yes)
+			)
+		)
+		(property "Datasheet" "~"
+			(at 246.38 128.27 0)
+			(effects
+				(font
+					(size 1.27 1.27)
+				)
+				(hide yes)
+			)
+		)
+		(property "Description" "Generic connector, single row, 01x29, script generated"
+			(at 246.38 128.27 0)
+			(effects
+				(font
+					(size 1.27 1.27)
+				)
+				(hide yes)
+			)
+		)
+		(pin "20"
+		)
+		(pin "2"
+		)
+		(pin "4"
+		)
+		(pin "5"
+		)
+		(pin "7"
+		)
+		(pin "6"
+		)
+		(pin "9"
+		)
+		(pin "10"
+		)
+		(pin "11"
+		)
+		(pin "12"
+		)
+		(pin "13"
+		)
+		(pin "8"
+		)
+		(pin "14"
+		)
+		(pin "15"
+		)
+		(pin "16"
+		)
+		(pin "17"
+		)
+		(pin "18"
+		)
+		(pin "3"
+		)
+		(pin "19"
+		)
+		(pin "1"
+		)
+		(pin "28"
+		)
+		(pin "23"
+		)
+		(pin "25"
+		)
+		(pin "26"
+		)
+		(pin "21"
+		)
+		(pin "24"
+		)
+		(pin "27"
+		)
+		(pin "22"
+		)
+		(pin "29"
+		)
+		(instances
+			(project ""
+				(path "/bd09a545-618a-47d2-a0b1-f0d03750b68a"
+					(reference "J11")
+					(unit 1)
+				)
+			)
+		)
+	)
+	(symbol
 		(lib_id "Device:R")
 		(at 227.33 139.7 180)
@@
 		(on_board yes)
 		(dnp no)
-		(fields_autoplaced yes)
 		(property "Reference" "C5"
-			(at 247.65 149.8599 0)
+			(at 237.744 149.606 0)
 			(effects
 				(font
@@
 		)
 		(property "Value" "104"
-			(at 247.65 152.3999 0)
+			(at 237.744 152.146 0)
 			(effects
 				(font
@@
 					(unit 1)
 				)
-			)
-		)
-	)
-	(symbol
-		(lib_id "MCU_Microchip_PIC16:PIC16F73-ISP")
-		(at 280.67 132.08 0)
-		(unit 1)
-		(exclude_from_sim no)
-		(in_bom yes)
-		(on_board yes)
-		(dnp no)
-		(fields_autoplaced yes)
-		(property "Reference" "U3"
-			(at 282.8133 105.41 0)
-			(effects
-				(font
-					(size 1.27 1.27)
-				)
-				(justify left)
-			)
-		)
-		(property "Value" "dsPIC33FJ16MC102"
-			(at 282.8133 107.95 0)
-			(effects
-				(font
-					(size 1.27 1.27)
-				)
-				(justify left)
-			)
-		)
-		(property "Footprint" "dsPIC33FJ16MC102:SOP65P780X200-28N"
-			(at 280.67 132.08 0)
-			(effects
-				(font
-					(size 1.27 1.27)
-					(italic yes)
-				)
-				(hide yes)
-			)
-		)
-		(property "Datasheet" "http://ww1.microchip.com/downloads/en/DeviceDoc/30325b.pdf"
-			(at 280.67 132.08 0)
-			(effects
-				(font
-					(size 1.27 1.27)
-				)
-				(hide yes)
-			)
-		)
-		(property "Description" "PIC16F73, 4K Flash, 192B SRAM, ADC, PWM, SDIP28"
-			(at 280.67 132.08 0)
-			(effects
-				(font
-					(size 1.27 1.27)
-				)
-				(hide yes)
-			)
-		)
-		(pin "15"
-		)
-		(pin "7"
-		)
-		(pin "5"
-		)
-		(pin "1"
-		)
-		(pin "17"
-		)
-		(pin "20"
-		)
-		(pin "4"
-		)
-		(pin "8"
-		)
-		(pin "12"
-		)
-		(pin "18"
-		)
-		(pin "13"
-		)
-		(pin "9"
-		)
-		(pin "10"
-		)
-		(pin "14"
-		)
-		(pin "19"
-		)
-		(pin "2"
-		)
-		(pin "6"
-		)
-		(pin "16"
-		)
-		(pin "11"
-		)
-		(pin "3"
-		)
-		(pin "23"
-		)
-		(pin "25"
-		)
-		(pin "27"
-		)
-		(pin "22"
-		)
-		(pin "24"
-		)
-		(pin "26"
-		)
-		(pin "21"
-		)
-		(pin "28"
-		)
-		(instances
-			(project ""
-				(path "/bd09a545-618a-47d2-a0b1-f0d03750b68a"
-					(reference "U3")
-					(unit 1)
-				)

Commit message: UPDATE
Parts:
- removed Q4: Q_NPN_ECB, Package_TO_SOT_THT:TO-92_Inline, symbol Transistor_BJT:Q_NPN_ECB
- added Q5: DTC143E, Package_TO_SOT_SMD:SOT-23, symbol Transistor_BJT:DTC143E
Connections:
- net GND: now also Q5.1 (B)
- net TC_TX: now also Q5.3 (C)
- net at J11.12 (Pin_12): now also Q5.2 (E)
Changed lines of the file:
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@@
 	)
 	(junction
-		(at 66.04 116.84)
+		(at 194.31 147.32)
 		(diameter 0)
 		(color 0 0 0 0)
 	)
 	(junction
-		(at 99.06 142.24)
+		(at 66.04 116.84)
 		(diameter 0)
 		(color 0 0 0 0)
 	)
 	(junction
-		(at 194.31 147.32)
+		(at 99.06 142.24)
 		(diameter 0)
 		(color 0 0 0 0)
@@
 	(wire
 		(pts
+			(xy 262.89 162.56) (xy 262.89 130.81)
+		)
+		(stroke
+			(width 0)
+			(type default)
+		)
+	)
+	(wire
+		(pts
 			(xy 57.15 57.15) (xy 64.77 57.15)
 		)
@@
 	(wire
 		(pts
-			(xy 184.15 154.94) (xy 184.15 160.02)
+			(xy 180.34 152.4) (xy 180.34 157.48)
 		)
 		(stroke
@@
 	(wire
 		(pts
-			(xy 189.23 154.94) (xy 184.15 154.94)
-		)
-		(stroke
-			(width 0)
-			(type default)
-		)
-	)
-	(wire
-		(pts
 			(xy 80.01 34.29) (xy 80.01 43.18)
 		)
@@
 	(wire
 		(pts
-			(xy 227.33 157.48) (xy 257.81 157.48)
-		)
-		(stroke
-			(width 0)
-			(type default)
-		)
-	)
-	(wire
-		(pts
 			(xy 74.93 186.69) (xy 80.01 186.69)
 		)
@@
 	(wire
 		(pts
+			(xy 238.76 130.81) (xy 238.76 123.19)
+		)
+		(stroke
+			(width 0)
+			(type default)
+		)
+	)
+	(wire
+		(pts
 			(xy 147.32 59.69) (xy 147.32 69.85)
 		)
@@
 	(wire
 		(pts
+			(xy 194.31 157.48) (xy 194.31 162.56)
+		)
+		(stroke
+			(width 0)
+			(type default)
+		)
+	)
+	(wire
+		(pts
 			(xy 130.81 41.91) (xy 151.13 41.91)
 		)
@@
 	(wire
 		(pts
-			(xy 138.43 93.98) (xy 138.43 109.22)
+			(xy 180.34 152.4) (xy 185.42 152.4)
 		)
 		(stroke
@@
 	(wire
 		(pts
-			(xy 44.45 29.21) (xy 41.91 29.21)
+			(xy 138.43 93.98) (xy 138.43 109.22)
 		)
 		(stroke
@@
 	(wire
 		(pts
-			(xy 194.31 143.51) (xy 194.31 147.32)
+			(xy 44.45 29.21) (xy 41.91 29.21)
 		)
 		(stroke
@@
 	(wire
 		(pts
-			(xy 115.57 139.7) (xy 129.54 139.7)
+			(xy 194.31 143.51) (xy 194.31 147.32)
 		)
 		(stroke
@@
 	(wire
 		(pts
-			(xy 63.5 34.29) (xy 67.31 34.29)
+			(xy 194.31 162.56) (xy 262.89 162.56)
 		)
 		(stroke
@@
 	(wire
 		(pts
-			(xy 73.66 109.22) (xy 85.09 109.22)
+			(xy 115.57 139.7) (xy 129.54 139.7)
 		)
 		(stroke
@@
 	(wire
 		(pts
-			(xy 147.32 72.39) (xy 147.32 74.93)
+			(xy 63.5 34.29) (xy 67.31 34.29)
 		)
 		(stroke
@@
 	(wire
 		(pts
-			(xy 168.91 91.44) (xy 182.88 91.44)
+			(xy 73.66 109.22) (xy 85.09 109.22)
 		)
 		(stroke
@@
 	(wire
 		(pts
-			(xy 257.81 130.81) (xy 257.81 157.48)
+			(xy 147.32 72.39) (xy 147.32 74.93)
 		)
 		(stroke
@@
 	(wire
 		(pts
-			(xy 124.46 173.99) (xy 129.54 173.99)
+			(xy 168.91 91.44) (xy 182.88 91.44)
 		)
 		(stroke
@@
 	(wire
 		(pts
-			(xy 168.91 123.19) (xy 185.42 123.19)
+			(xy 124.46 173.99) (xy 129.54 173.99)
 		)
 		(stroke
@@
 	(wire
 		(pts
-			(xy 238.76 123.19) (xy 238.76 130.81)
+			(xy 168.91 123.19) (xy 185.42 123.19)
 		)
 		(stroke
@@
 	(wire
 		(pts
-			(xy 199.39 154.94) (xy 227.33 154.94)
-		)
-		(stroke
-			(width 0)
-			(type default)
-		)
-	)
-	(wire
-		(pts
 			(xy 147.32 87.63) (xy 147.32 114.3)
 		)
@@
 	(wire
 		(pts
-			(xy 227.33 154.94) (xy 227.33 157.48)
+			(xy 204.47 31.75) (xy 158.75 31.75)
 		)
 		(stroke
@@
 	(wire
 		(pts
-			(xy 204.47 31.75) (xy 158.75 31.75)
+			(xy 64.77 73.66) (xy 64.77 93.98)
 		)
 		(stroke
@@
 	(wire
 		(pts
-			(xy 64.77 73.66) (xy 64.77 93.98)
+			(xy 153.67 110.49) (xy 153.67 109.22)
 		)
 		(stroke
@@
 	(wire
 		(pts
-			(xy 153.67 110.49) (xy 153.67 109.22)
+			(xy 33.02 191.77) (xy 48.26 191.77)
 		)
 		(stroke
@@
 	(wire
 		(pts
-			(xy 33.02 191.77) (xy 48.26 191.77)
+			(xy 85.09 116.84) (xy 99.06 116.84)
 		)
 		(stroke
@@
 	(wire
 		(pts
-			(xy 85.09 116.84) (xy 99.06 116.84)
+			(xy 99.06 109.22) (xy 115.57 109.22)
 		)
 		(stroke
@@
 	(wire
 		(pts
-			(xy 99.06 109.22) (xy 115.57 109.22)
+			(xy 262.89 130.81) (xy 238.76 130.81)
 		)
 		(stroke
@@
 		)
 	)
-	(wire
-		(pts
-			(xy 238.76 130.81) (xy 257.81 130.81)
-		)
-		(stroke
-			(width 0)
-			(type default)
-		)
-	)
 	(table
 		(column_count 3)
@@
 	(symbol
 		(lib_id "power:GND")
-		(at 184.15 160.02 0)
+		(at 180.34 157.48 0)
 		(unit 1)
 		(exclude_from_sim no)
@@
 		(dnp no)
 		(property "Reference" "#PWR0102"
-			(at 184.15 166.37 0)
+			(at 180.34 163.83 0)
 			(effects
 				(font
@@
 		)
 		(property "Value" "GND"
-			(at 181.864 163.83 0)
+			(at 178.054 161.29 0)
 			(effects
 				(font
@@
 		)
 		(property "Footprint" ""
-			(at 184.15 160.02 0)
+			(at 180.34 157.48 0)
 			(effects
 				(font
@@
 		)
 		(property "Datasheet" ""
-			(at 184.15 160.02 0)
+			(at 180.34 157.48 0)
 			(effects
 				(font
@@
 		)
 		(property "Description" "Power symbol creates a global label with name \"GND\" , ground"
-			(at 184.15 160.02 0)
+			(at 180.34 157.48 0)
 			(effects
 				(font
@@
 	)
 	(symbol
+		(lib_name "DTC143E_2")
+		(lib_id "Transistor_BJT:DTC143E")
+		(at 191.77 152.4 0)
+		(unit 1)
+		(exclude_from_sim no)
+		(in_bom yes)
+		(on_board yes)
+		(dnp no)
+		(fields_autoplaced yes)
+		(property "Reference" "Q5"
+			(at 196.85 151.1299 0)
+			(effects
+				(font
+					(size 1.27 1.27)
+				)
+				(justify left)
+			)
+		)
+		(property "Value" "DTC143E"
+			(at 196.85 153.6699 0)
+			(effects
+				(font
+					(size 1.27 1.27)
+				)
+				(justify left)
+			)
+		)
+		(property "Footprint" "Package_TO_SOT_SMD:SOT-23"
+			(at 191.77 152.4 0)
+			(effects
+				(font
+					(size 1.27 1.27)
+				)
+				(justify left)
+				(hide yes)
+			)
+		)
+		(property "Datasheet" ""
+			(at 191.77 152.4 0)
+			(effects
+				(font
+					(size 1.27 1.27)
+				)
+				(justify left)
+				(hide yes)
+			)
+		)
+		(property "Description" "Digital NPN Transistor, 4k7/4k7, SOT-23"
+			(at 191.77 152.4 0)
+			(effects
+				(font
+					(size 1.27 1.27)
+				)
+				(hide yes)
+			)
+		)
+		(pin "3"
+		)
+		(pin "1"
+		)
+		(pin "2"
+		)
+		(instances
+			(project ""
+				(path "/bd09a545-618a-47d2-a0b1-f0d03750b68a"
+					(reference "Q5")
+					(unit 1)
+				)
+			)
+		)
+	)
+	(symbol
 		(lib_id "Device:D")
 		(at 76.2 34.29 0)
@@
 					(unit 1)
 				)
-			)
-		)
-	)
-	(symbol
-		(lib_id "Transistor_BJT:Q_NPN_ECB")
-		(at 194.31 152.4 270)
-		(unit 1)
-		(exclude_from_sim no)
-		(in_bom yes)
-		(on_board yes)
-		(dnp no)
-		(fields_autoplaced yes)
-		(property "Reference" "Q4"
-			(at 194.31 158.75 90)
-			(effects
-				(font
-					(size 1.27 1.27)
-				)
-			)
-		)
-		(property "Value" "Q_NPN_ECB"
-			(at 194.31 161.29 90)
-			(effects
-				(font
-					(size 1.27 1.27)
-				)
-			)
-		)
-		(property "Footprint" "Package_TO_SOT_THT:TO-92_Inline"
-			(at 196.85 157.48 0)
-			(effects
-				(font
-					(size 1.27 1.27)
-				)
-				(hide yes)
-			)
-		)
-		(property "Datasheet" "~"
-			(at 194.31 152.4 0)
-			(effects
-				(font
-					(size 1.27 1.27)
-				)
-				(hide yes)
-			)
-		)
-		(property "Description" "NPN transistor, emitter/collector/base"
-			(at 194.31 152.4 0)
-			(effects
-				(font
-					(size 1.27 1.27)
-				)
-				(hide yes)
-			)
-		)
-		(property "Sim.Device" "NPN"
-			(at 194.31 152.4 0)
-			(effects
-				(font
-					(size 1.27 1.27)
-				)
-				(hide yes)
-			)
-		)
-		(property "Sim.Pins" "1=E 2=C 3=B"
-			(at 194.31 152.4 0)
-			(effects
-				(font
-					(size 1.27 1.27)
-				)
-				(hide yes)
-			)
-		)
-		(pin "3"
-		)
-		(pin "1"
-		)
-		(pin "2"
-		)
-		(instances
-			(project ""
-				(path "/bd09a545-618a-47d2-a0b1-f0d03750b68a"
-					(reference "Q4")
-					(unit 1)
-				)
