File: KiCad/TC106_Overall_circuit_diagram/TC106_Overall_circuit_diagram.kicad_sch (KiCad schematic)
At the start: 51 parts, among them J1 JST_VH_01x05, J10 JST_VH_01x05, J11 Dummy dsPIC33FJ16MC102, J1_24V1 JST_VH_01x04, J1_CN1 JST_VH_01x03, J2 JST_VH_01x05, J2_CN1 JST_VH_01x02, J3 JST_VH_01x05, J3_CN1 JST_VH_01x02, J4 JST_VH_01x05, J4_CN2 JST_VH_01x02, J5 JST_VH_01x05, J5_CN2 JST_VH_01x03, J6 JST_VH_01x05, J7 JST_VH_01x05, J8 JST_VH_01x05, J9 Conn_02x02_Odd_Even, Q1 DTC143E, Q2 DTC143E, Q3 2SD1863, Q5 DTC143E, U1 MC34063AP, U2 PIC16F73-ISP

Commit message: UPDATE
Parts:
- removed J11: Dummy dsPIC33FJ16MC102, dsPIC33FJ16MC102:SOP65P780X200-28N, symbol Connector:Conn_01x29_Pin
- added U3: Dummy dsPic33FJ16MC102, dsPIC33FJ16MC102:SOP65P780X200-28N, symbol Connector:Conn_01x28_Pin
Connections:
- net at C5.1, R13.2, R14.1: now also U3.12 (Pin_12)
- net at Q5.2 (E): now also U3.11 (Pin_11)
Changed lines of the file:
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@@
 	(wire
 		(pts
+			(xy 254 132.08) (xy 254 128.27)
+		)
+		(stroke
+			(width 0)
+			(type default)
+		)
+	)
+	(wire
+		(pts
 			(xy 41.91 40.64) (xy 67.31 40.64)
 		)
@@
 	(wire
 		(pts
-			(xy 74.93 186.69) (xy 80.01 186.69)
+			(xy 243.84 132.08) (xy 254 132.08)
 		)
 		(stroke
@@
 	(wire
 		(pts
-			(xy 64.77 93.98) (xy 138.43 93.98)
+			(xy 74.93 186.69) (xy 80.01 186.69)
 		)
 		(stroke
@@
 	(wire
 		(pts
-			(xy 102.87 46.99) (xy 74.93 46.99)
+			(xy 64.77 93.98) (xy 138.43 93.98)
 		)
 		(stroke
@@
 	(wire
 		(pts
-			(xy 58.42 191.77) (xy 62.23 191.77)
+			(xy 102.87 46.99) (xy 74.93 46.99)
 		)
 		(stroke
@@
 	(wire
 		(pts
-			(xy 236.22 123.19) (xy 236.22 132.08)
+			(xy 58.42 191.77) (xy 62.23 191.77)
 		)
 		(stroke
@@
 	(wire
 		(pts
-			(xy 238.76 130.81) (xy 238.76 123.19)
-		)
-		(stroke
-			(width 0)
-			(type default)
-		)
-	)
-	(wire
-		(pts
 			(xy 147.32 59.69) (xy 147.32 69.85)
 		)
@@
 	(wire
 		(pts
-			(xy 243.84 132.08) (xy 236.22 132.08)
-		)
-		(stroke
-			(width 0)
-			(type default)
-		)
-	)
-	(wire
-		(pts
 			(xy 99.06 116.84) (xy 115.57 116.84)
 		)
@@
 	(wire
 		(pts
+			(xy 262.89 130.81) (xy 256.54 130.81)
+		)
+		(stroke
+			(width 0)
+			(type default)
+		)
+	)
+	(wire
+		(pts
 			(xy 194.31 162.56) (xy 262.89 162.56)
 		)
@@
 	(wire
 		(pts
+			(xy 256.54 130.81) (xy 256.54 128.27)
+		)
+		(stroke
+			(width 0)
+			(type default)
+		)
+	)
+	(wire
+		(pts
 			(xy 44.45 29.21) (xy 44.45 93.98)
 		)
@@
 	(wire
 		(pts
+			(xy 243.84 132.08) (xy 243.84 143.51)
+		)
+		(stroke
+			(width 0)
+			(type default)
+		)
+	)
+	(wire
+		(pts
 			(xy 153.67 114.3) (xy 153.67 137.16)
 		)
@@
 	(wire
 		(pts
-			(xy 262.89 130.81) (xy 238.76 130.81)
-		)
-		(stroke
-			(width 0)
-			(type default)
-		)
-	)
-	(wire
-		(pts
 			(xy 41.91 31.75) (xy 58.42 31.75)
 		)
@@
 	(wire
 		(pts
-			(xy 243.84 132.08) (xy 243.84 143.51)
-		)
-		(stroke
-			(width 0)
-			(type default)
-		)
-	)
-	(wire
-		(pts
 			(xy 151.13 142.24) (xy 151.13 116.84)
 		)
@@
 	)
 	(symbol
-		(lib_id "Device:D_Zener")
-		(at 58.42 161.29 270)
+		(lib_id "Connector:Conn_01x28_Pin")
+		(at 248.92 123.19 270)
 		(unit 1)
 		(exclude_from_sim no)
@@
 		(on_board yes)
 		(dnp no)
-		(fields_autoplaced yes)
-		(property "Reference" "D6"
-			(at 60.96 160.0199 90)
+		(property "Reference" "U3"
+			(at 214.884 118.364 90)
 			(effects
 				(font
 					(size 1.27 1.27)
 				)
-				(justify left)
 			)
 		)
-		(property "Value" "HZ24"
-			(at 60.96 162.5599 90)
+		(property "Value" "Dummy dsPic33FJ16MC102"
+			(at 214.884 120.904 90)
 			(effects
 				(font
 					(size 1.27 1.27)
 				)
-				(justify left)
 			)
 		)
-		(property "Footprint" "Diode_THT:D_DO-35_SOD27_P7.62mm_Horizontal"
-			(at 58.42 161.29 0)
+		(property "Footprint" "dsPIC33FJ16MC102:SOP65P780X200-28N"
+			(at 248.92 123.19 0)
 			(effects
 				(font
@@
 		)
 		(property "Datasheet" "~"
-			(at 58.42 161.29 0)
+			(at 248.92 123.19 0)
 			(effects
 				(font
@@
 			)
 		)
-		(property "Description" "Zener diode"
-			(at 58.42 161.29 0)
+		(property "Description" "Generic connector, single row, 01x28, script generated"
+			(at 248.92 123.19 0)
 			(effects
 				(font
@@
 			)
 		)
-		(pin "2"
+		(pin "28"
+		)
+		(pin "9"
+		)
+		(pin "7"
 		)
 		(pin "1"
 		)
+		(pin "6"
+		)
+		(pin "5"
+		)
+		(pin "8"
+		)
+		(pin "2"
+		)
+		(pin "3"
+		)
+		(pin "4"
+		)
+		(pin "11"
+		)
+		(pin "10"
+		)
+		(pin "24"
+		)
+		(pin "25"
+		)
+		(pin "26"
+		)
+		(pin "27"
+		)
+		(pin "18"
+		)
+		(pin "16"
+		)
+		(pin "21"
+		)
+		(pin "20"
+		)
+		(pin "19"
+		)
+		(pin "15"
+		)
+		(pin "14"
+		)
+		(pin "12"
+		)
+		(pin "13"
+		)
+		(pin "17"
+		)
+		(pin "22"
+		)
+		(pin "23"
+		)
 		(instances
 			(project ""
 				(path "/bd09a545-618a-47d2-a0b1-f0d03750b68a"
-					(reference "D6")
+					(reference "U3")
 					(unit 1)
 				)
@@
 	)
 	(symbol
-		(lib_id "Connector:Conn_01x29_Pin")
-		(at 246.38 128.27 90)
+		(lib_id "Device:D_Zener")
+		(at 58.42 161.29 270)
 		(unit 1)
 		(exclude_from_sim no)
@@
 		(on_board yes)
 		(dnp no)
-		(property "Reference" "J11"
-			(at 215.392 117.348 90)
+		(fields_autoplaced yes)
+		(property "Reference" "D6"
+			(at 60.96 160.0199 90)
 			(effects
 				(font
 					(size 1.27 1.27)
 				)
+				(justify left)
 			)
 		)
-		(property "Value" "Dummy dsPIC33FJ16MC102"
-			(at 216.154 120.142 90)
+		(property "Value" "HZ24"
+			(at 60.96 162.5599 90)
 			(effects
 				(font
 					(size 1.27 1.27)
 				)
+				(justify left)
 			)
 		)
-		(property "Footprint" "dsPIC33FJ16MC102:SOP65P780X200-28N"
-			(at 246.38 128.27 0)
+		(property "Footprint" "Diode_THT:D_DO-35_SOD27_P7.62mm_Horizontal"
+			(at 58.42 161.29 0)
 			(effects
 				(font
@@
 		)
 		(property "Datasheet" "~"
-			(at 246.38 128.27 0)
+			(at 58.42 161.29 0)
 			(effects
 				(font
@@
 			)
 		)
-		(property "Description" "Generic connector, single row, 01x29, script generated"
-			(at 246.38 128.27 0)
+		(property "Description" "Zener diode"
+			(at 58.42 161.29 0)
 			(effects
 				(font
@@
 			)
 		)
-		(pin "20"
-		)
 		(pin "2"
 		)
-		(pin "4"
-		)
-		(pin "5"
-		)
-		(pin "7"
-		)
-		(pin "6"
-		)
-		(pin "9"
-		)
-		(pin "10"
-		)
-		(pin "11"
-		)
-		(pin "12"
-		)
-		(pin "13"
-		)
-		(pin "8"
-		)
-		(pin "14"
-		)
-		(pin "15"
-		)
-		(pin "16"
-		)
-		(pin "17"
-		)
-		(pin "18"
-		)
-		(pin "3"
-		)
-		(pin "19"
-		)
 		(pin "1"
 		)
-		(pin "28"
-		)
-		(pin "23"
-		)
-		(pin "25"
-		)
-		(pin "26"
-		)
-		(pin "21"
-		)
-		(pin "24"
-		)
-		(pin "27"
-		)
-		(pin "22"
-		)
-		(pin "29"
-		)
 		(instances
 			(project ""
 				(path "/bd09a545-618a-47d2-a0b1-f0d03750b68a"
-					(reference "J11")
+					(reference "D6")
 					(unit 1)
 				)
@@
 		(on_board yes)
 		(dnp no)
-		(fields_autoplaced yes)
 		(property "Reference" "JP1"
-			(at 53.34 185.42 0)
+			(at 53.34 192.532 0)
 			(effects
 				(font
@@
 		)
 		(property "Value" "Jumper_2_Open"
-			(at 53.34 187.96 0)
+			(at 53.34 195.072 0)
 			(effects
 				(font

Commit message: UPDATE
Connections:
- net TC_RX: no longer R7.1
- net at Q3.3 (B): now also R7.1
Changed lines of the file:
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@@
-	)
-	(junction
-		(at 85.09 157.48)
-		(diameter 0)
-		(color 0 0 0 0)
 	)
 	(junction
@@
 	(wire
 		(pts
+			(xy 92.71 162.56) (xy 110.49 162.56)
+		)
+		(stroke
+			(width 0)
+			(type default)
+		)
+	)
+	(wire
+		(pts
 			(xy 73.66 116.84) (xy 73.66 109.22)
 		)
@@
 	(wire
 		(pts
-			(xy 110.49 157.48) (xy 110.49 162.56)
-		)
-		(stroke
-			(width 0)
-			(type default)
-		)
-	)
-	(wire
-		(pts
 			(xy 252.73 143.51) (xy 252.73 147.32)
 		)
@@
 		)
 		(stroke
-			(width 0)
-			(type default)
-		)
-	)
-	(wire
-		(pts
-			(xy 85.09 157.48) (xy 110.49 157.48)
-		)
-		(stroke
