File: KiCad/TC106_Overall_circuit_diagram/TC106_Overall_circuit_diagram.kicad_sch (KiCad schematic)
At the start: 51 parts, among them J1 JST_VH_01x05, J10 JST_VH_01x05, J1_24V1 JST_VH_01x04, J1_CN1 JST_VH_01x03, J2 JST_VH_01x05, J2_CN1 JST_VH_01x02, J3 JST_VH_01x05, J3_CN1 JST_VH_01x02, J4 JST_VH_01x05, J4_CN2 JST_VH_01x02, J5 JST_VH_01x05, J5_CN2 JST_VH_01x03, J6 JST_VH_01x05, J7 JST_VH_01x05, J8 JST_VH_01x05, J9 Conn_02x02_Odd_Even, Q1 DTC143E, Q2 DTC143E, Q3 2SD1863, Q5 DTC143E, U1 MC34063AP, U2 PIC16F73-ISP, U3 Dummy dsPic33FJ16MC102

Commit message: UPDATE
Connections:
- removed net +5V: J9.1 (Pin_1), R11.2, R12.2

Commit message: UPDATE
Parts:
- added U5: DC-DC_Converter, symbol Connector:Conn_01x01_Pin
- J9: footprint Connector_PinHeader_1.00mm:PinHeader_2x02_P1.00mm_Vertical -> (none)
Connections:
- net +24V: now also U5.1 (Pin_1)
- no-connect marks 9 -> 61

Commit message: UPDATE
Parts:
- U3: footprint dsPIC33FJ16MC102:SOP65P780X200-28N -> dsPic33FJ16MC102:SOP65P780X200-28N
Changed lines of the file:
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@@
 	(wire
 		(pts
+			(xy 194.31 134.62) (xy 194.31 135.89)
+		)
+		(stroke
+			(width 0)
+			(type default)
+		)
+	)
+	(wire
+		(pts
 			(xy 129.54 142.24) (xy 151.13 142.24)
 		)
@@
 	(wire
 		(pts
+			(xy 227.33 133.35) (xy 227.33 135.89)
+		)
+		(stroke
+			(width 0)
+			(type default)
+		)
+	)
+	(wire
+		(pts
 			(xy 142.24 91.44) (xy 46.99 91.44)
 		)
@@
 	(symbol
 		(lib_id "power:PWR_FLAG")
-		(at 227.33 135.89 0)
+		(at 227.33 133.35 0)
 		(unit 1)
 		(exclude_from_sim no)
@@
 		(dnp no)
 		(property "Reference" "#U11_POWER_5V01"
-			(at 227.33 133.985 0)
+			(at 227.33 131.445 0)
 			(effects
 				(font
@@
 		)
 		(property "Value" "+5V"
-			(at 233.426 133.858 0)
+			(at 233.426 131.318 0)
 			(effects
 				(font
@@
 		)
 		(property "Footprint" ""
-			(at 227.33 135.89 0)
+			(at 227.33 133.35 0)
 			(effects
 				(font
@@
 		)
 		(property "Datasheet" "~"
-			(at 227.33 135.89 0)
+			(at 227.33 133.35 0)
 			(effects
 				(font
@@
 		)
 		(property "Description" "Special symbol for telling ERC where power comes from"
-			(at 227.33 135.89 0)
+			(at 227.33 133.35 0)
 			(effects
 				(font
@@
 			)
 		)
-		(property "Footprint" "dsPIC33FJ16MC102:SOP65P780X200-28N"
+		(property "Footprint" "dsPic33FJ16MC102:SOP65P780X200-28N"
 			(at 248.92 123.19 0)
 			(effects
@@
 	(symbol
 		(lib_id "power:PWR_FLAG")
-		(at 194.31 135.89 0)
+		(at 194.31 134.62 0)
 		(unit 1)
 		(exclude_from_sim no)
@@
 		(dnp no)
 		(property "Reference" "#U11_POWER_5V0101"
-			(at 194.31 133.985 0)
+			(at 194.31 132.715 0)
 			(effects
 				(font
@@
 		)
 		(property "Value" "+5V"
-			(at 200.406 133.858 0)
+			(at 200.406 132.588 0)
 			(effects
 				(font
@@
 		)
 		(property "Footprint" ""
-			(at 194.31 135.89 0)
+			(at 194.31 134.62 0)
 			(effects
 				(font
@@
 		)
 		(property "Datasheet" "~"
-			(at 194.31 135.89 0)
+			(at 194.31 134.62 0)
 			(effects
 				(font
@@
 		)
 		(property "Description" "Special symbol for telling ERC where power comes from"
-			(at 194.31 135.89 0)
+			(at 194.31 134.62 0)
 			(effects
 				(font

Commit message: UPDATE
Connections:
- net GND: now also Q5.2 (E); no longer Q5.1 (B)
- net TC_TX_U3: now also Q5.1 (B); no longer Q5.2 (E)
Other:
- moved on the sheet: Q5
Changed lines of the file:
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@@
 	)
 	(junction
+		(at 189.23 147.32)
+		(diameter 0)
+		(color 0 0 0 0)
+	)
+	(junction
 		(at 147.32 114.3)
 		(diameter 0)
@@
 	)
 	(junction
-		(at 194.31 147.32)
-		(diameter 0)
-		(color 0 0 0 0)
-	)
-	(junction
 		(at 66.04 116.84)
 		(diameter 0)
@@
 	(wire
 		(pts
-			(xy 180.34 152.4) (xy 180.34 157.48)
-		)
-		(stroke
-			(width 0)
-			(type default)
-		)
-	)
-	(wire
-		(pts
 			(xy 190.5 123.19) (xy 190.5 120.65)
 		)
@@
 	(wire
 		(pts
+			(xy 203.2 152.4) (xy 198.12 152.4)
+		)
+		(stroke
+			(width 0)
+			(type default)
+		)
+	)
+	(wire
+		(pts
 			(xy 58.42 191.77) (xy 62.23 191.77)
 		)
@@
 	(wire
 		(pts
-			(xy 184.15 147.32) (xy 194.31 147.32)
+			(xy 184.15 147.32) (xy 189.23 147.32)
 		)
 		(stroke
@@
 	(wire
 		(pts
-			(xy 194.31 157.48) (xy 194.31 162.56)
+			(xy 130.81 41.91) (xy 151.13 41.91)
 		)
 		(stroke
@@
 	(wire
 		(pts
-			(xy 130.81 41.91) (xy 151.13 41.91)
+			(xy 62.23 184.15) (xy 62.23 191.77)
 		)
 		(stroke
@@
 	(wire
 		(pts
-			(xy 62.23 184.15) (xy 62.23 191.77)
+			(xy 83.82 66.04) (xy 81.28 66.04)
 		)
 		(stroke
@@
 	(wire
 		(pts
-			(xy 83.82 66.04) (xy 81.28 66.04)
+			(xy 63.5 34.29) (xy 63.5 26.67)
 		)
 		(stroke
@@
 	(wire
 		(pts
-			(xy 63.5 34.29) (xy 63.5 26.67)
+			(xy 58.42 31.75) (xy 58.42 52.07)
 		)
 		(stroke
@@
 	(wire
 		(pts
-			(xy 58.42 31.75) (xy 58.42 52.07)
+			(xy 189.23 147.32) (xy 194.31 147.32)
 		)
 		(stroke
@@
 	(wire
 		(pts
-			(xy 102.87 31.75) (xy 130.81 31.75)
+			(xy 262.89 162.56) (xy 203.2 162.56)
 		)
 		(stroke
@@
 	(wire
 		(pts
-			(xy 100.33 54.61) (xy 100.33 62.23)
+			(xy 102.87 31.75) (xy 130.81 31.75)
 		)
 		(stroke
@@
 	(wire
 		(pts
-			(xy 58.42 157.48) (xy 85.09 157.48)
+			(xy 100.33 54.61) (xy 100.33 62.23)
 		)
 		(stroke
@@
 	(wire
 		(pts
-			(xy 252.73 143.51) (xy 252.73 147.32)
+			(xy 58.42 157.48) (xy 85.09 157.48)
 		)
 		(stroke
@@
 	(wire
 		(pts
-			(xy 106.68 80.01) (xy 106.68 66.04)
+			(xy 252.73 143.51) (xy 252.73 147.32)
 		)
 		(stroke
@@
 	(wire
 		(pts
-			(xy 180.34 152.4) (xy 185.42 152.4)
+			(xy 106.68 80.01) (xy 106.68 66.04)
 		)
 		(stroke
@@
 	(wire
 		(pts
-			(xy 194.31 162.56) (xy 262.89 162.56)
-		)
-		(stroke
-			(width 0)
-			(type default)
-		)
-	)
-	(wire
-		(pts
 			(xy 115.57 139.7) (xy 129.54 139.7)
 		)
@@
 	(wire
 		(pts
+			(xy 189.23 157.48) (xy 189.23 161.29)
+		)
+		(stroke
+			(width 0)
+			(type default)
+		)
+	)
+	(wire
+		(pts
+			(xy 203.2 162.56) (xy 203.2 152.4)
+		)
+		(stroke
+			(width 0)
+			(type default)
+		)
+	)
+	(wire
+		(pts
 			(xy 147.32 87.63) (xy 147.32 114.3)
 		)
@@
 	(symbol
 		(lib_id "power:GND")
-		(at 180.34 157.48 0)
+		(at 189.23 161.29 0)
 		(unit 1)
 		(exclude_from_sim no)
@@
 		(dnp no)
 		(property "Reference" "#PWR0102"
-			(at 180.34 163.83 0)
+			(at 189.23 167.64 0)
 			(effects
 				(font
@@
 		)
 		(property "Value" "GND"
-			(at 178.054 161.29 0)
+			(at 185.674 161.798 0)
 			(effects
 				(font
@@
 		)
 		(property "Footprint" ""
-			(at 180.34 157.48 0)
+			(at 189.23 161.29 0)
 			(effects
 				(font
@@
 		)
 		(property "Datasheet" ""
-			(at 180.34 157.48 0)
+			(at 189.23 161.29 0)
 			(effects
 				(font
@@
 		)
 		(property "Description" "Power symbol creates a global label with name \"GND\" , ground"
-			(at 180.34 157.48 0)
+			(at 189.23 161.29 0)
 			(effects
 				(font
@@
 		(lib_id "Transistor_BJT:DTC143E")
 		(at 191.77 152.4 0)
+		(mirror y)
 		(unit 1)
 		(exclude_from_sim no)
@@
 		(on_board yes)
 		(dnp no)
-		(fields_autoplaced yes)
 		(property "Reference" "Q5"
-			(at 196.85 151.1299 0)
+			(at 186.69 151.1299 0)
 			(effects
 				(font
@@
 		)
 		(property "Value" "DTC143E"
-			(at 196.85 153.6699 0)
+			(at 186.69 153.6699 0)
 			(effects
 				(font

Commit message: UPDATE
Connections:
- net Q1_BASE is gone; now on net TC_RX: Q1.3 (B), Q2.2 (C), R2.2
- net Q2_BASE is gone; now on net TC_RX: D1.2 (A), Q2.3 (B), R1.1
- net TC_CMD_BUS: no longer D2.1 (K), J1.4 (Pin_4), J2.4 (Pin_4), J3.4 (Pin_4), J4.4 (Pin_4), J5.4 (Pin_4), J6.4 (Pin_4), J7.4 (Pin_4), J8.4 (Pin_4), Q1.2 (C)
- net TC_RX: now also D2.1 (K), J1.4 (Pin_4), J2.4 (Pin_4), J3.4 (Pin_4), J4.4 (Pin_4), J5.4 (Pin_4), J6.4 (Pin_4), J7.4 (Pin_4), J8.4 (Pin_4), Q1.2 (C)
Changed lines of the file:
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@@
 		)
 	)
-	(label "TC_CMD_BUS"
+	(label "TC_RX"
 		(at 139.7 41.91 0)
+		(effects
+			(font
+				(size 1.27 1.27)
+			)
+			(justify left bottom)
+		)
+	)
+	(label "TC_RX"
+		(at 106.68 41.91 0)
 		(effects
 			(font
@@
 		)
 	)
-	(label "Q1_BASE"
+	(label "TC_RX"
 		(at 93.98 46.99 0)
 		(effects
@@
 		)
 	)
-	(label "TC_CMD_BUS"
+	(label "TC_RX"
 		(at 106.68 142.24 0)
 		(effects
@@
 		)
 	)
-	(label "Q2_BASE"
+	(label "TC_RX"
 		(at 88.9 36.83 0)
 		(effects
@@
 		)
 	)
-	(label "TC_CMD_BUS"
+	(label "TC_RX"
 		(at 151.13 74.93 90)
 		(effects
@@
 		)
 	)
-	(label "TC_CMD_BUS"
+	(label "TC_RX"
 		(at 106.68 116.84 0)
 		(effects

Commit message: UPDATE
Connections:
- net TC_CMD_BUS is gone; now on net TC_RX: D7.1 (A1), J10.4 (Pin_4), R12.1, R13.1
- net TC_CMD_U3 renamed TC_RX_U3
Changed lines of the file:
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@@
 		)
 	)
-	(label "TC_CMD_U3"
+	(label "TC_RX_U3"
 		(at 243.84 134.62 0)
 		(effects
@@
 		)
 	)
-	(label "TC_CMD_BUS"
+	(label "TC_RX"
 		(at 195.58 130.81 0)
 		(effects

Commit message: UPDATE
Connections:
- net TC_RX renamed TC_RX_BUS
- net TC_RX_BUS: no longer D1.1 (K), D1.2 (A), D6.1 (K), J2_CN1.2 (Pin_2), J3_CN1.2 (Pin_2), J4_CN2.2 (Pin_2), Q1.3 (B), Q2.2 (C), Q2.3 (B), Q3.1 (E), R1.1, R2.2, R3.1
- new net INT_TC_S2: D1.1 (K), D6.1 (K), J2_CN1.2 (Pin_2), J3_CN1.2 (Pin_2), J4_CN2.2 (Pin_2), Q1.3 (B), Q2.2 (C), Q3.1 (E), R2.2, R3.1
- new net TC_RX_IN: D1.2 (A), Q2.3 (B), R1.1
Changed lines of the file:
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@@
 		)
 	)
-	(label "TC_RX"
+	(label "TC_RX_BUS"
 		(at 139.7 41.91 0)
 		(effects
@@
 		)
 	)
-	(label "TC_RX"
+	(label "INT_TC_S2"
 		(at 106.68 41.91 0)
 		(effects
@@
 		)
 	)
-	(label "TC_RX"
+	(label "TC_RX_BUS"
 		(at 106.68 142.24 0)
 		(effects
@@
 		)
 	)
-	(label "TC_RX"
+	(label "TC_RX_BUS"
 		(at 195.58 130.81 0)
 		(effects
@@
 		)
 	)
-	(label "TC_RX"
+	(label "TC_RX_IN"
 		(at 88.9 36.83 0)
 		(effects
@@
 		)
 	)
-	(label "TC_RX"
+	(label "TC_RX_BUS"
 		(at 151.13 74.93 90)
 		(effects
@@
 		)
 	)
-	(label "TC_RX"
+	(label "TC_RX_BUS"
 		(at 106.68 116.84 0)
 		(effects

Commit message: UPDATE
Connections:
- net IN_Q_MAIN: now reaches Q3.3 (B), R7.1
- net TC_MAIN_U: now reaches R7.2, U2.11 (RC0/T10S0/T1CKI)
- net INT_TC_S2 renamed TC_RX
- net TC_RX: no longer Q1.3 (B), Q2.2 (C), R2.2
- new net TC_RX_24V: Q1.3 (B), Q2.2 (C), R2.2
Changed lines of the file:
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@@
 	(wire
 		(pts
-			(xy 114.3 36.83) (xy 121.92 36.83)
+			(xy 119.38 36.83) (xy 121.92 36.83)
 		)
 		(stroke
@@
 	(wire
 		(pts
-			(xy 102.87 41.91) (xy 114.3 41.91)
+			(xy 102.87 41.91) (xy 119.38 41.91)
 		)
 		(stroke
@@
 	(wire
 		(pts
-			(xy 114.3 41.91) (xy 114.3 36.83)
+			(xy 119.38 41.91) (xy 119.38 36.83)
 		)
 		(stroke
@@
 		)
 	)
+	(label "TC_MAIN_U"
+		(at 124.46 172.72 90)
+		(effects
+			(font
+				(size 1.27 1.27)
+			)
+			(justify left bottom)
+		)
+	)
 	(label "MC34063_TC"
 		(at 107.95 80.01 0)
@@
 		)
 	)
-	(label "INT_TC_S2"
-		(at 106.68 41.91 0)
+	(label "TC_RX_CLAMP"
+		(at 105.41 41.91 0)
 		(effects
 			(font
@@
 		)
 	)
-	(label "TC_RX"
+	(label "TC_RX_24V"
 		(at 93.98 46.99 0)
 		(effects
@@
 			)
 			(justify left bottom)
+		)
+	)
+	(label "IN_Q_MAIN"
+		(at 96.52 162.56 0)
+		(effects
+			(font
+				(size 1.27 1.27)
+			)
+			(justify left bottom)
