File: KiCad/TC106_Overall_circuit_diagram/TC106_Overall_circuit_diagram.kicad_sch (KiCad schematic)
At the start: 52 parts, among them J1 JST_VH_01x05, J10 JST_VH_01x05, J1_24V1 JST_VH_01x04, J1_CN1 JST_VH_01x03, J2 JST_VH_01x05, J2_CN1 JST_VH_01x02, J3 JST_VH_01x05, J3_CN1 JST_VH_01x02, J4 JST_VH_01x05, J4_CN2 JST_VH_01x02, J5 JST_VH_01x05, J5_CN2 JST_VH_01x03, J6 JST_VH_01x05, J7 JST_VH_01x05, J8 JST_VH_01x05, J9 Conn_02x02_Odd_Even, Q1 DTC143E, Q2 DTC143E, Q3 2SD1863, Q5 DTC143E, U1 MC34063AP, U2 PIC16F73-ISP, U3 Dummy dsPic33FJ16MC102, U5 DC-DC_Inverter

Commit message: UPDATE
Changed lines of the file:
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@@
-	)
-	(symbol
-		(lib_id "power:PWR_FLAG")
-		(at 190.5 134.62 0)
-		(unit 1)
-		(exclude_from_sim no)
-		(in_bom yes)
-		(on_board yes)
-		(dnp no)
-		(property "Reference" "#FLG04"
-			(at 190.5 132.715 0)
-			(effects
-				(font
-					(size 1.27 1.27)
-				)
-				(hide yes)
-			)
-		)
-		(property "Value" "PWR_5V_INT"
-			(at 189.738 136.398 0)
-			(effects
-				(font
-					(size 1 1)
-				)
-			)
-		)
-		(property "Footprint" ""
-			(at 190.5 134.62 0)
-			(effects
-				(font
-					(size 1.27 1.27)
-				)
-				(hide yes)
-			)
-		)
-		(property "Datasheet" "~"
-			(at 190.5 134.62 0)
-			(effects
-				(font
-					(size 1.27 1.27)
-				)
-				(hide yes)
-			)
-		)
-		(property "Description" "Special symbol for telling ERC where power comes from"
-			(at 190.5 134.62 0)
-			(effects
-				(font
-					(size 1.27 1.27)
-				)
-				(hide yes)
-			)
-		)
-		(pin "1"
-		)
-		(instances
-			(project ""
-				(path "/bd09a545-618a-47d2-a0b1-f0d03750b68a"
-					(reference "#FLG04")
-					(unit 1)
-				)
-			)
-		)
 	)
 	(symbol
@@
 					(unit 1)
 				)
+			)
+		)
+	)
+	(symbol
+		(lib_id "power:PWR_FLAG")
+		(at 190.5 134.62 0)
+		(unit 1)
+		(exclude_from_sim no)
+		(in_bom yes)
+		(on_board yes)
+		(dnp no)
+		(property "Reference" "#FLG04"
+			(at 190.5 132.715 0)
+			(effects
+				(font
+					(size 1.27 1.27)
+				)
+				(hide yes)
+			)
+		)
+		(property "Value" "PWR_FLAG"
+			(at 189.484 135.89 0)
+			(effects
+				(font
+					(size 1.27 1.27)
+				)
+			)
+		)
+		(property "Footprint" ""
+			(at 190.5 134.62 0)
+			(effects
+				(font
+					(size 1.27 1.27)
+				)
+				(hide yes)
+			)
+		)
+		(property "Datasheet" "~"
+			(at 190.5 134.62 0)
+			(effects
+				(font
+					(size 1.27 1.27)
+				)
+				(hide yes)
+			)
+		)
+		(property "Description" "Special symbol for telling ERC where power comes from"
+			(at 190.5 134.62 0)
+			(effects
+				(font
+					(size 1.27 1.27)
+				)
+				(hide yes)
+			)
+		)
+		(pin "1"
+		)
+		(instances
+			(project ""
+				(path "/bd09a545-618a-47d2-a0b1-f0d03750b68a"
+					(reference "#FLG04")
+					(unit 1)
+				)

Commit message: UPDATE
Parts:
- added J11, J12: Conn_01x01_Socket, symbol Connector:Conn_01x01_Socket
Connections:
- net +5V_INT: now also J11.1 (Pin_1)
- net at J9.1 (Pin_1): now also J12.1 (Pin_1)
Changed lines of the file:
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@@
 	)
 	(junction
+		(at 190.5 134.62)
+		(diameter 0)
+		(color 0 0 0 0)
+	)
+	(junction
 		(at 115.57 137.16)
 		(diameter 0)
@@
 	)
 	(junction
+		(at 40.64 175.26)
+		(diameter 0)
+		(color 0 0 0 0)
+	)
+	(junction
 		(at 129.54 139.7)
 		(diameter 0)
@@
 	(wire
 		(pts
+			(xy 189.23 134.62) (xy 190.5 134.62)
+		)
+		(stroke
+			(width 0)
+			(type default)
+		)
+	)
+	(wire
+		(pts
 			(xy 99.06 134.62) (xy 115.57 134.62)
 		)
@@
 	(wire
 		(pts
+			(xy 36.83 175.26) (xy 40.64 175.26)
+		)
+		(stroke
+			(width 0)
+			(type default)
+		)
+	)
+	(wire
+		(pts
 			(xy 130.81 41.91) (xy 151.13 41.91)
 		)
@@
 	)
 	(symbol
+		(lib_id "Connector:Conn_01x01_Socket")
+		(at 36.83 170.18 90)
+		(unit 1)
+		(exclude_from_sim no)
+		(in_bom yes)
+		(on_board yes)
+		(dnp no)
+		(fields_autoplaced yes)
+		(property "Reference" "J12"
+			(at 38.1 169.5449 90)
+			(effects
+				(font
+					(size 1.27 1.27)
+				)
+				(justify right)
+			)
+		)
+		(property "Value" "Conn_01x01_Socket"
+			(at 38.1 172.0849 90)
+			(effects
+				(font
+					(size 1.27 1.27)
+				)
+				(justify right)
+				(hide yes)
+			)
+		)
+		(property "Footprint" ""
+			(at 36.83 170.18 0)
+			(effects
+				(font
+					(size 1.27 1.27)
+				)
+				(hide yes)
+			)
+		)
+		(property "Datasheet" "~"
+			(at 36.83 170.18 0)
+			(effects
+				(font
+					(size 1.27 1.27)
+				)
+				(hide yes)
+			)
+		)
+		(property "Description" "Generic connector, single row, 01x01, script generated"
+			(at 36.83 170.18 0)
+			(effects
+				(font
+					(size 1.27 1.27)
+				)
+				(hide yes)
+			)
+		)
+		(pin "1"
+		)
+		(instances
+			(project "TC106_Overall_circuit_diagram"
+				(path "/bd09a545-618a-47d2-a0b1-f0d03750b68a"
+					(reference "J12")
+					(unit 1)
+				)
+			)
+		)
+	)
+	(symbol
 		(lib_id "Device:R")
 		(at 227.33 139.7 180)
@@
 					(unit 1)
 				)
+			)
+		)
+	)
+	(symbol
+		(lib_id "Connector:Conn_01x01_Socket")
+		(at 189.23 129.54 90)
+		(unit 1)
+		(exclude_from_sim no)
+		(in_bom yes)
+		(on_board yes)
+		(dnp no)
+		(fields_autoplaced yes)
+		(property "Reference" "J11"
+			(at 190.5 128.9049 90)
+			(effects
+				(font
+					(size 1.27 1.27)
+				)
+				(justify right)
+			)
+		)
+		(property "Value" "Conn_01x01_Socket"
+			(at 190.5 131.4449 90)
+			(effects
+				(font
+					(size 1.27 1.27)
+				)
+				(justify right)
+				(hide yes)
+			)
+		)
+		(property "Footprint" ""
+			(at 189.23 129.54 0)
+			(effects
+				(font
+					(size 1.27 1.27)
+				)
+				(hide yes)
+			)
+		)
+		(property "Datasheet" "~"
+			(at 189.23 129.54 0)
+			(effects
+				(font
+					(size 1.27 1.27)
+				)
+				(hide yes)
+			)
+		)
+		(property "Description" "Generic connector, single row, 01x01, script generated"
+			(at 189.23 129.54 0)
+			(effects
+				(font
+					(size 1.27 1.27)
+				)
+				(hide yes)
+			)
+		)
+		(pin "1"
+		)
+		(instances
+			(project ""
+				(path "/bd09a545-618a-47d2-a0b1-f0d03750b68a"
+					(reference "J11")
+					(unit 1)
+				)

Commit message: UPDATE
Parts:
- J11, J12: footprint (none) -> TestPoint:TestPoint_Keystone_5000-5004_Miniature
Changed lines of the file:
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@@
 			)
 		)
-		(property "Footprint" ""
+		(property "Footprint" "TestPoint:TestPoint_Keystone_5000-5004_Miniature"
 			(at 36.83 170.18 0)
 			(effects
@@
 			)
 		)
-		(property "Footprint" ""
+		(property "Footprint" "TestPoint:TestPoint_Keystone_5000-5004_Miniature"
 			(at 189.23 129.54 0)
 			(effects

Commit message: UPDATE
Parts:
- renumbered C4 to C2, C2 to C3, C3 to C4, D6 to D1, D3 to D2, D1 to D3, D5 to D4, D2 to D5, D4 to D6, J12 to J1, J8 to J10, J10 to J11, J11 to J12, J9 to J2, J5 to J3, J1 to J4, J4_CN2 to J4_CN1, J2 to J5, J5_CN2 to J5_CN1, J7 to J6, J3 to J7, J6 to J8, J4 to J9, Q3 to Q1, Q1 to Q3, Q5 to Q4, R2 to R1, R6 to R10, R10 to R2, R1 to R4, R8 to R5, R9 to R6, R5 to R7, R7 to R8, R4 to R9, U5 to U3, U3 to U4

Commit message: UPDATE
Parts:
- renumbered D5 to D1, D3 to D2, D2 to D3, D1 to D5
Changed lines of the file:
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@@
 		(on_board yes)
 		(dnp no)
-		(property "Reference" "D2"
+		(property "Reference" "D3"
 			(at 68.326 54.61 0)
 			(effects
@@
 			(project ""
 				(path "/bd09a545-618a-47d2-a0b1-f0d03750b68a"
-					(reference "D2")
+					(reference "D3")
 					(unit 1)
 				)
@@
 		(on_board yes)
 		(dnp no)
-		(property "Reference" "D3"
+		(property "Reference" "D2"
 			(at 76.2 27.432 0)
 			(effects
@@
 			(project ""
 				(path "/bd09a545-618a-47d2-a0b1-f0d03750b68a"
-					(reference "D3")
+					(reference "D2")
 					(unit 1)
 				)
@@
 		(on_board yes)
 		(dnp no)
-		(property "Reference" "D5"
+		(property "Reference" "D1"
 			(at 161.798 36.576 0)
 			(effects
@@
 			(project ""
 				(path "/bd09a545-618a-47d2-a0b1-f0d03750b68a"
-					(reference "D5")
+					(reference "D1")
 					(unit 1)
 				)
@@
 		(dnp no)
 		(fields_autoplaced yes)
-		(property "Reference" "D1"
+		(property "Reference" "D5"
 			(at 60.96 160.0199 90)
 			(effects
@@
 			(project ""
 				(path "/bd09a545-618a-47d2-a0b1-f0d03750b68a"
-					(reference "D1")
-					(unit 1)
-				)
+					(reference "D5")
+					(unit 1)
+				)

Commit message: UPDATE
Parts:
- removed C2, C5: 104, Capacitor_THT:C_Disc_D5.0mm_W2.5mm_P2.50mm, symbol Device:C
- removed D5: HZ24, Diode_THT:D_DO-35_SOD27_P7.62mm_Horizontal, symbol Device:D_Zener
- removed D7: D_TVS_Dual_AAC, Package_TO_SOT_SMD:SOT-23, symbol Device:D_TVS_Dual_AAC
- removed J1, J12: Conn_01x01_Socket, TestPoint:TestPoint_Keystone_5000-5004_Miniature, symbol Connector:Conn_01x01_Socket
- removed J11: JST_VH_01x05, Connector_JST:JST_VH_B5P-VH-B_1x05_P3.96mm_Vertical, symbol Connector_Generic:Conn_01x05
- removed J2: Conn_02x02_Odd_Even, symbol Connector_Generic:Conn_02x02_Odd_Even
- removed J4_CN1: JST_VH_01x02, Connector_JST:JST_VH_B2P-VH-B_1x02_P3.96mm_Vertical, symbol Connector_Generic:Conn_01x02
- removed J5_CN1: JST_VH_01x03, Connector_JST:JST_VH_B3P-VH-B_1x03_P3.96mm_Vertical, symbol Connector_Generic:Conn_01x03
- removed JP1: Jumper_2_Open, Connector_PinHeader_1.00mm:PinHeader_1x02_P1.00mm_Vertical, symbol Jumper:Jumper_2_Open
- removed Q1: 2SD1863, Package_TO_SOT_THT:TO-92_Inline, symbol Transistor_BJT:Q_NPN_ECB
- removed Q4: DTC143E, Package_TO_SOT_SMD:SOT-23, symbol Transistor_BJT:DTC143E
- removed R11: 22k, Resistor_THT:R_Axial_DIN0204_L3.6mm_D1.6mm_P7.62mm_Horizontal, symbol Device:R
- removed R12: 4k7, Resistor_THT:R_Axial_DIN0204_L3.6mm_D1.6mm_P7.62mm_Horizontal, symbol Device:R
- removed R13, R2, R5, R6: 1k, Resistor_THT:R_Axial_DIN0204_L3.6mm_D1.6mm_P7.62mm_Horizontal, symbol Device:R
- removed R14: 10k, Resistor_THT:R_Axial_DIN0204_L3.6mm_D1.6mm_P7.62mm_Horizontal, symbol Device:R
- removed R8: 330R, Resistor_THT:R_Axial_DIN0204_L3.6mm_D1.6mm_P7.62mm_Horizontal, symbol Device:R
- removed U2: PIC16F73-ISP, Package_DIP:DIP-28_W15.24mm, symbol MCU_Microchip_PIC16:PIC16F73-ISP
- removed U3: DC-DC_Inverter, symbol Connector:Conn_01x01_Pin
- removed U4: Dummy dsPic33FJ16MC102, dsPic33FJ16MC102:SOP65P780X200-28N, symbol Connector:Conn_01x28_Pin
- renumbered J4 to J1, J5 to J2, J7 to J3, J9 to J4, J10 to J5, J8 to J6, J6 to J7, J3 to J8, Q3 to Q1
Connections:
- no-connect marks 60 -> 7
Other:
- note removed: "Main controller"
- note removed: "TC106"

Commit message: UPDATE
Parts:
- C3: footprint Capacitor_THT:CP_Radial_D12.5mm_P5.00mm -> Capacitor_THT:CP_Radial_D10.0mm_P7.50mm
- C4: footprint Capacitor_THT:CP_Radial_D8.0mm_P3.50mm -> Capacitor_THT:CP_Radial_D8.0mm_P5.00mm
- renumbered D6 to D4, D4 to D5, R4 to R1, R1 to R2, R9 to R4, R7 to R5, R10 to R6
Connections:
- net TC_RX_24V renamed TC_RX_CLAMP
Changed lines of the file:
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@@
 		)
 	)
-	(label "+24V"
-		(at 116.84 93.98 0)
-		(effects
-			(font
-				(size 1.27 1.27)
-			)
-			(justify left bottom)
-		)
-	)
-	(label "TC_RX_24V"
+	(label "TC_RX_CLAMP"
 		(at 93.98 46.99 0)
 		(effects
@@
 		)
 	)
-	(label "+24V"
-		(at 67.31 116.84 0)
-		(effects
-			(font
-				(size 1.27 1.27)
-			)
-			(justify left bottom)
-		)
-	)
 	(symbol
 		(lib_id "Device:R")
@@
 		(on_board yes)
 		(dnp no)
-		(property "Reference" "R10"
+		(property "Reference" "R6"
 			(at 167.386 99.06 90)
 			(effects
@@
 			(project ""
 				(path "/bd09a545-618a-47d2-a0b1-f0d03750b68a"
-					(reference "R10")
+					(reference "R6")
 					(unit 1)
 				)
@@
 		(on_board yes)
 		(dnp no)
-		(property "Reference" "R9"
+		(property "Reference" "R4"
 			(at 168.91 92.456 90)
 			(effects
@@
 			(project ""
 				(path "/bd09a545-618a-47d2-a0b1-f0d03750b68a"
-					(reference "R9")
+					(reference "R4")
 					(unit 1)
 				)
@@
 			)
 		)
-		(property "Footprint" "Capacitor_THT:CP_Radial_D12.5mm_P5.00mm"
+		(property "Footprint" "Capacitor_THT:CP_Radial_D10.0mm_P7.50mm"
 			(at 104.394 79.248 0)
 			(effects
@@
 		(dnp no)
 		(fields_autoplaced yes)
-		(property "Reference" "R1"
+		(property "Reference" "R2"
 			(at 67.31 68.5799 0)
 			(effects
@@
 			(project ""
 				(path "/bd09a545-618a-47d2-a0b1-f0d03750b68a"
-					(reference "R1")
+					(reference "R2")
 					(unit 1)
 				)
@@
 		(on_board yes)
 		(dnp no)
-		(property "Reference" "R7"
+		(property "Reference" "R5"
 			(at 113.284 62.484 90)
 			(effects
@@
 			(project ""
 				(path "/bd09a545-618a-47d2-a0b1-f0d03750b68a"
-					(reference "R7")
+					(reference "R5")
 					(unit 1)
 				)
@@
 			)
 		)
-		(property "Footprint" "Capacitor_THT:CP_Radial_D8.0mm_P3.50mm"
+		(property "Footprint" "Capacitor_THT:CP_Radial_D8.0mm_P5.00mm"
 			(at 178.562 77.724 0)
 			(effects
@@
 		(on_board yes)
 		(dnp no)
-		(property "Reference" "R4"
+		(property "Reference" "R1"
 			(at 83.058 40.894 90)
 			(effects
@@
 			(project ""
 				(path "/bd09a545-618a-47d2-a0b1-f0d03750b68a"
-					(reference "R4")
+					(reference "R1")
 					(unit 1)
 				)
@@
 		(dnp no)
 		(fields_autoplaced yes)
-		(property "Reference" "D6"
+		(property "Reference" "D4"
 			(at 162.56 73.66 0)
 			(effects
@@
 			(project ""
 				(path "/bd09a545-618a-47d2-a0b1-f0d03750b68a"
-					(reference "D6")
+					(reference "D4")
 					(unit 1)
 				)
@@
 		(dnp no)
 		(fields_autoplaced yes)
-		(property "Reference" "D4"
+		(property "Reference" "D5"
 			(at 114.3 48.26 0)
 			(effects
@@
 			(project ""
 				(path "/bd09a545-618a-47d2-a0b1-f0d03750b68a"
-					(reference "D4")
-					(unit 1)
-				)
+					(reference "D5")
+					(unit 1)
+				)
