File: KiCad/TC106_Overall_circuit_diagram/TC106_Overall_circuit_diagram.kicad_pcb (KiCad board)
At the start: 2 copper layers, 68.9 x 121.6 mm, 30 parts, among them J1 JST_VH_01x05, J1_24V1 JST_VH_01x04, J1_CN1 JST_VH_01x03, J2 JST_VH_01x05, J2_CN1 JST_VH_01x02, J3 JST_VH_01x05, J3_CN1 JST_VH_01x02, J4 JST_VH_01x05, J5 JST_VH_01x05, J6 JST_VH_01x05, J7 JST_VH_01x05, J8 JST_VH_01x05, Q1 DTC143E, Q2 DTC143E, U1 MC34063AP

Commit message: UPDATE
Parts:
- added C4: 104, Capacitor_THT:C_Disc_D5.0mm_W2.5mm_P2.50mm, F.Cu at (74.3, 104.1)
- added C5: 104, Capacitor_THT:C_Disc_D5.0mm_W2.5mm_P2.50mm, F.Cu at (74.3, 108.1)
- added D6: HZ24, Diode_THT:D_DO-35_SOD27_P7.62mm_Horizontal, F.Cu at (72.2, 120.4)
- added D7: D_TVS_Dual_AAC, Package_TO_SOT_SMD:SOT-23, F.Cu at (64.2, 140.9)
- added J10: JST_VH_01x05, Connector_JST:JST_VH_B5P-VH-B_1x05_P3.96mm_Vertical, F.Cu at (94.6, 135.1)
- added J4_CN2: JST_VH_01x02, Connector_JST:JST_VH_B2P-VH-B_1x02_P3.96mm_Vertical, F.Cu at (143.8, 162.8)
- added J5_CN2: JST_VH_01x03, Connector_JST:JST_VH_B3P-VH-B_1x03_P3.96mm_Vertical, F.Cu at (123.7, 162.6)
- added J9: Conn_02x02_Odd_Even, Connector_PinHeader_1.00mm:PinHeader_2x02_P1.00mm_Vertical, F.Cu at (47.6, 138.4)
- added JP1: Jumper_2_Open, Connector_PinHeader_1.00mm:PinHeader_1x02_P1.00mm_Vertical, F.Cu at (77.7, 154.2)
- added Q3: 2SD1863, Package_TO_SOT_THT:TO-92_Inline, F.Cu at (76.8, 134.6)
- added Q4: Q_NPN_ECB, Package_TO_SOT_THT:TO-92_Inline, F.Cu at (67.0, 131.8)
- added R10: 1k, Resistor_THT:R_Axial_DIN0204_L3.6mm_D1.6mm_P7.62mm_Horizontal, F.Cu at (38.7, 105.7)
- added R11: 22k, Resistor_THT:R_Axial_DIN0204_L3.6mm_D1.6mm_P7.62mm_Horizontal, F.Cu at (38.0, 110.3)
- added R12: 4k7, Resistor_THT:R_Axial_DIN0204_L3.6mm_D1.6mm_P7.62mm_Horizontal, F.Cu at (38.0, 115.3)
- added R13: 1k, Resistor_THT:R_Axial_DIN0204_L3.6mm_D1.6mm_P7.62mm_Horizontal, F.Cu at (45.5, 122.2)
- added R14: 10k, Resistor_THT:R_Axial_DIN0204_L3.6mm_D1.6mm_P7.62mm_Horizontal, F.Cu at (52.2, 128.8)
- added R7: 330R, Resistor_THT:R_Axial_DIN0204_L3.6mm_D1.6mm_P7.62mm_Horizontal, F.Cu at (56.1, 91.3)
- added R8: 1k, Resistor_THT:R_Axial_DIN0204_L3.6mm_D1.6mm_P7.62mm_Horizontal, F.Cu at (39.3, 97.6)
- added R9: 1k, Resistor_THT:R_Axial_DIN0204_L3.6mm_D1.6mm_P7.62mm_Horizontal, F.Cu at (50.5, 110.6)
- added U2: PIC16F73-ISP, Package_DIP:DIP-28_W15.24mm, F.Cu at (71.1, 51.1)
- moved J1_CN1 0.81 mm to (123.7, 141.8)
- moved J2_CN1 0.32 mm to (143.5, 140.8)
Connections:
- net /CMD_IN renamed /TC_RX
- net /TC_TX_REP renamed /TC_TX

Commit message: UPDATE
Parts:
- added U3: dsPIC33FJ16MC102, dsPIC33FJ16MC102:SOP65P780X200-28N, F.Cu at (75.3, 178.4)
Connections:
- net /Pic33_RX renamed Net-(U3-RC0/T10S0/T1CKI)
- Q4 pad 2: /Pic33_TX -> Net-(Q4-C)

Commit message: UPDATE
Parts:
- removed U3: dsPIC33FJ16MC102, dsPIC33FJ16MC102:SOP65P780X200-28N
- added J11: Dummy dsPIC33FJ16MC102, dsPIC33FJ16MC102:SOP65P780X200-28N, F.Cu at (60.7, 164.3)

Commit message: UPDATE
Parts:
- removed Q4: Q_NPN_ECB, Package_TO_SOT_THT:TO-92_Inline
- added Q5: DTC143E, Package_TO_SOT_SMD:SOT-23, F.Cu at (47.5, 154.2)

Commit message: UPDATE
Parts:
- removed J11: Dummy dsPIC33FJ16MC102, dsPIC33FJ16MC102:SOP65P780X200-28N
- added U3: Dummy dsPic33FJ16MC102, dsPIC33FJ16MC102:SOP65P780X200-28N, F.Cu at (93.5, 164.3)

Commit message: UPDATE
Connections:
- net Net-(Q5-E) renamed /TC_TX_U3
- net Net-(U3-Pin_12) renamed /TC_CMD_U3
- J9 pad 1: +5V -> Net-(J9-Pin_1)
- Q3 pad 3: unconnected-(Q3-B-Pad3) -> Net-(Q3-B)
- R11 pad 2: +5V -> Net-(R11-Pad2)
- R12 pad 2: +5V -> Net-(R12-Pad2)
- R7 pad 1: /TC_RX -> Net-(Q3-B)
Changed lines of the file:
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@@
 	(net 23 "unconnected-(J5_CN2-Pin_2-Pad2)")
 	(net 24 "unconnected-(J10-Pin_2-Pad2)")
-	(net 25 "unconnected-(Q3-B-Pad3)")
+	(net 25 "/TC_CMD_U3")
 	(net 26 "Net-(U2-RC0{slash}T10S0{slash}T1CKI)")
 	(net 27 "Net-(U2-RC7{slash}RX{slash}DT)")
 	(net 28 "Net-(J9-Pin_2)")
-	(net 29 "+5V")
+	(net 29 "Net-(J9-Pin_1)")
 	(net 30 "unconnected-(U2-RB4-Pad25)")
 	(net 31 "unconnected-(U2-VSS-Pad19)")
@@
 	(net 55 "unconnected-(U2-VSS-Pad8)")
 	(net 56 "Net-(J5_CN2-Pin_3)")
-	(net 57 "Net-(U3-Pin_12)")
-	(net 58 "Net-(Q5-E)")
+	(net 57 "Net-(Q3-B)")
+	(net 58 "/TC_TX_U3")
 	(net 59 "unconnected-(U3-Pin_4-Pad4)")
 	(net 60 "unconnected-(U3-Pin_13-Pad13)")
@@
 	(net 83 "unconnected-(U3-Pin_16-Pad16)")
 	(net 84 "unconnected-(U3-Pin_27-Pad27)")
+	(net 85 "Net-(R11-Pad2)")
+	(net 86 "Net-(R12-Pad2)")
 	(footprint "Resistor_THT:R_Axial_DIN0204_L3.6mm_D1.6mm_P7.62mm_Horizontal"
 		(layer "F.Cu")
@@
 			(layers "*.Cu" "*.Mask")
 			(remove_unused_layers no)
-			(net 29 "+5V")
+			(net 86 "Net-(R12-Pad2)")
 			(pintype "passive")
 		)
@@
 			(layers "*.Cu" "*.Mask")
 			(remove_unused_layers no)
-			(net 25 "unconnected-(Q3-B-Pad3)")
+			(net 57 "Net-(Q3-B)")
 			(pinfunction "B")
 			(pintype "input")
@@
 			(layers "F.Cu" "F.Mask" "F.Paste")
 			(roundrect_rratio 0.25)
-			(net 58 "Net-(Q5-E)")
+			(net 58 "/TC_TX_U3")
 			(pinfunction "E")
 			(pintype "passive")
@@
 			(layers "*.Cu" "*.Mask")
 			(remove_unused_layers no)
-			(net 29 "+5V")
+			(net 29 "Net-(J9-Pin_1)")
 			(pinfunction "Pin_1")
 			(pintype "passive")
@@
 			(layers "*.Cu" "*.Mask")
 			(remove_unused_layers no)
-			(net 21 "/TC_RX")
+			(net 57 "Net-(Q3-B)")
 			(pintype "passive")
 		)
@@
 			(layers "*.Cu" "*.Mask")
 			(remove_unused_layers no)
-			(net 57 "Net-(U3-Pin_12)")
+			(net 25 "/TC_CMD_U3")
 			(pintype "passive")
 		)
@@
 			(size 1.9 0.48)
 			(layers "F.Cu" "F.Paste")
-			(net 58 "Net-(Q5-E)")
+			(net 58 "/TC_TX_U3")
 			(pinfunction "Pin_11")
 			(pintype "passive")
@@
 			(size 1.9 0.48)
 			(layers "F.Cu" "F.Paste")
-			(net 57 "Net-(U3-Pin_12)")
+			(net 25 "/TC_CMD_U3")
 			(pinfunction "Pin_12")
 			(pintype "passive")
@@
 			(layers "*.Cu" "*.Mask")
 			(remove_unused_layers no)
-			(net 57 "Net-(U3-Pin_12)")
+			(net 25 "/TC_CMD_U3")
 			(pintype "passive")
 		)
@@
 			(layers "*.Cu" "*.Mask")
 			(remove_unused_layers no)
-			(net 57 "Net-(U3-Pin_12)")
+			(net 25 "/TC_CMD_U3")
 			(pintype "passive")
 		)
@@
 			(layers "*.Cu" "*.Mask")
 			(remove_unused_layers no)
-			(net 29 "+5V")
+			(net 85 "Net-(R11-Pad2)")
 			(pintype "passive")
 		)

Commit message: UPDATE
Parts:
- U3: footprint dsPIC33FJ16MC102:SOP65P780X200-28N -> dsPic33FJ16MC102:SOP65P780X200-28N
Connections:
- Q5 pad 1: GND -> /TC_TX_U3
- Q5 pad 2: /TC_TX_U3 -> GND
Changed lines of the file:
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@@
 			(layers "F.Cu" "F.Mask" "F.Paste")
 			(roundrect_rratio 0.25)
-			(net 4 "GND")
+			(net 58 "/TC_TX_U3")
 			(pinfunction "B")
 			(pintype "input")
@@
 			(layers "F.Cu" "F.Mask" "F.Paste")
 			(roundrect_rratio 0.25)
-			(net 58 "/TC_TX_U3")
+			(net 4 "GND")
 			(pinfunction "E")
 			(pintype "passive")
@@
 		)
 	)
-	(footprint "dsPIC33FJ16MC102:SOP65P780X200-28N"
+	(footprint "dsPic33FJ16MC102:SOP65P780X200-28N"
 		(layer "F.Cu")
 		(at 93.495 164.275)
@@
 			(net 66 "unconnected-(U3-Pin_1-Pad1)")
 			(pinfunction "Pin_1")
-			(pintype "passive")
+			(pintype "passive+no_connect")
 		)
 		(pad "2" smd rect
@@
 			(net 73 "unconnected-(U3-Pin_2-Pad2)")
 			(pinfunction "Pin_2")
-			(pintype "passive")
+			(pintype "passive+no_connect")
 		)
 		(pad "3" smd rect
@@
 			(net 61 "unconnected-(U3-Pin_3-Pad3)")
 			(pinfunction "Pin_3")
-			(pintype "passive")
+			(pintype "passive+no_connect")
 		)
 		(pad "4" smd rect
@@
 			(net 59 "unconnected-(U3-Pin_4-Pad4)")
 			(pinfunction "Pin_4")
-			(pintype "passive")
+			(pintype "passive+no_connect")
 		)
 		(pad "5" smd rect
@@
 			(net 62 "unconnected-(U3-Pin_5-Pad5)")
 			(pinfunction "Pin_5")
-			(pintype "passive")
+			(pintype "passive+no_connect")
 		)
 		(pad "6" smd rect
@@
 			(net 80 "unconnected-(U3-Pin_6-Pad6)")
 			(pinfunction "Pin_6")
-			(pintype "passive")
+			(pintype "passive+no_connect")
 		)
 		(pad "7" smd rect
@@
 			(net 63 "unconnected-(U3-Pin_7-Pad7)")
 			(pinfunction "Pin_7")
-			(pintype "passive")
+			(pintype "passive+no_connect")
 		)
 		(pad "8" smd rect
@@
 			(net 64 "unconnected-(U3-Pin_8-Pad8)")
 			(pinfunction "Pin_8")
-			(pintype "passive")
+			(pintype "passive+no_connect")
 		)
 		(pad "9" smd rect
@@
 			(net 77 "unconnected-(U3-Pin_9-Pad9)")
 			(pinfunction "Pin_9")
-			(pintype "passive")
+			(pintype "passive+no_connect")
 		)
 		(pad "10" smd rect
@@
 			(net 65 "unconnected-(U3-Pin_10-Pad10)")
 			(pinfunction "Pin_10")
-			(pintype "passive")
+			(pintype "passive+no_connect")
 		)
 		(pad "11" smd rect
@@
 			(net 60 "unconnected-(U3-Pin_13-Pad13)")
 			(pinfunction "Pin_13")
-			(pintype "passive")
+			(pintype "passive+no_connect")
 		)
 		(pad "14" smd rect
@@
 			(net 67 "unconnected-(U3-Pin_14-Pad14)")
 			(pinfunction "Pin_14")
-			(pintype "passive")
+			(pintype "passive+no_connect")
 		)
 		(pad "15" smd rect
@@
 			(net 79 "unconnected-(U3-Pin_15-Pad15)")
 			(pinfunction "Pin_15")
-			(pintype "passive")
+			(pintype "passive+no_connect")
 		)
 		(pad "16" smd rect
@@
 			(net 83 "unconnected-(U3-Pin_16-Pad16)")
 			(pinfunction "Pin_16")
-			(pintype "passive")
+			(pintype "passive+no_connect")
 		)
 		(pad "17" smd rect
@@
 			(net 82 "unconnected-(U3-Pin_17-Pad17)")
 			(pinfunction "Pin_17")
-			(pintype "passive")
+			(pintype "passive+no_connect")
 		)
 		(pad "18" smd rect
@@
 			(net 76 "unconnected-(U3-Pin_18-Pad18)")
 			(pinfunction "Pin_18")
-			(pintype "passive")
+			(pintype "passive+no_connect")
 		)
 		(pad "19" smd rect
@@
 			(net 70 "unconnected-(U3-Pin_19-Pad19)")
 			(pinfunction "Pin_19")
-			(pintype "passive")
+			(pintype "passive+no_connect")
 		)
 		(pad "20" smd rect
@@
 			(net 69 "unconnected-(U3-Pin_20-Pad20)")
 			(pinfunction "Pin_20")
-			(pintype "passive")
+			(pintype "passive+no_connect")
 		)
 		(pad "21" smd rect
@@
 			(net 75 "unconnected-(U3-Pin_21-Pad21)")
 			(pinfunction "Pin_21")
-			(pintype "passive")
+			(pintype "passive+no_connect")
 		)
 		(pad "22" smd rect
@@
 			(net 72 "unconnected-(U3-Pin_22-Pad22)")
 			(pinfunction "Pin_22")
-			(pintype "passive")
+			(pintype "passive+no_connect")
 		)
 		(pad "23" smd rect
@@
 			(net 81 "unconnected-(U3-Pin_23-Pad23)")
 			(pinfunction "Pin_23")
-			(pintype "passive")
+			(pintype "passive+no_connect")
 		)
 		(pad "24" smd rect
@@
 			(net 74 "unconnected-(U3-Pin_24-Pad24)")
 			(pinfunction "Pin_24")
-			(pintype "passive")
+			(pintype "passive+no_connect")
 		)
 		(pad "25" smd rect
@@
 			(net 78 "unconnected-(U3-Pin_25-Pad25)")
 			(pinfunction "Pin_25")
-			(pintype "passive")
+			(pintype "passive+no_connect")
 		)
 		(pad "26" smd rect
@@
 			(net 68 "unconnected-(U3-Pin_26-Pad26)")
 			(pinfunction "Pin_26")
-			(pintype "passive")
+			(pintype "passive+no_connect")
 		)
 		(pad "27" smd rect
@@
 			(net 84 "unconnected-(U3-Pin_27-Pad27)")
 			(pinfunction "Pin_27")
-			(pintype "passive")
+			(pintype "passive+no_connect")
 		)
 		(pad "28" smd rect
@@
 			(net 71 "unconnected-(U3-Pin_28-Pad28)")
 			(pinfunction "Pin_28")
-			(pintype "passive")
+			(pintype "passive+no_connect")
 		)
 		(embedded_fonts no)
@@
 			(net 48 "unconnected-(U2-~{MCLR}{slash}Vpp-Pad1)")
 			(pinfunction "~{MCLR}/Vpp")
-			(pintype "input")
+			(pintype "input+no_connect")
 		)
 		(pad "2" thru_hole circle
@@
 			(net 45 "unconnected-(U2-AN0{slash}RA0-Pad2)")
 			(pinfunction "AN0/RA0")
-			(pintype "bidirectional")
+			(pintype "bidirectional+no_connect")
 		)
 		(pad "3" thru_hole circle
@@
 			(net 50 "unconnected-(U2-AN1{slash}RA1-Pad3)")
 			(pinfunction "AN1/RA1")
-			(pintype "bidirectional")
+			(pintype "bidirectional+no_connect")
 		)
 		(pad "4" thru_hole circle
@@
 			(net 33 "unconnected-(U2-AN2{slash}RA2-Pad4)")
 			(pinfunction "AN2/RA2")
-			(pintype "bidirectional")
+			(pintype "bidirectional+no_connect")
 		)
 		(pad "5" thru_hole circle
@@
 			(net 35 "unconnected-(U2-Vref{slash}AN3{slash}RA3-Pad5)")
 			(pinfunction "Vref/AN3/RA3")
-			(pintype "bidirectional")
+			(pintype "bidirectional+no_connect")
 		)
 		(pad "6" thru_hole circle
@@
 			(net 34 "unconnected-(U2-T0CKI{slash}RA4-Pad6)")
 			(pinfunction "T0CKI/RA4")
-			(pintype "bidirectional")
+			(pintype "bidirectional+no_connect")
 		)
 		(pad "7" thru_hole circle
@@
 			(net 36 "unconnected-(U2-~{SS}{slash}AN4{slash}RA5-Pad7)")
 			(pinfunction "~{SS}/AN4/RA5")
-			(pintype "bidirectional")
+			(pintype "bidirectional+no_connect")
 		)
 		(pad "8" thru_hole circle
@@
 			(net 55 "unconnected-(U2-VSS-Pad8)")
 			(pinfunction "VSS")
-			(pintype "power_in")
+			(pintype "power_in+no_connect")
 		)
 		(pad "9" thru_hole circle
@@
 			(net 46 "unconnected-(U2-OSC1{slash}CLKIN-Pad9)")
 			(pinfunction "OSC1/CLKIN")
-			(pintype "input")
+			(pintype "input+no_connect")
 		)
 		(pad "10" thru_hole circle
@@
 			(net 43 "unconnected-(U2-OSC2{slash}CLKOUT-Pad10)")
 			(pinfunction "OSC2/CLKOUT")
-			(pintype "output")
+			(pintype "output+no_connect")
 		)
 		(pad "11" thru_hole circle
@@
 			(net 42 "unconnected-(U2-RC1{slash}CCP2{slash}T1OSI-Pad12)")
 			(pinfunction "RC1/CCP2/T1OSI")
-			(pintype "bidirectional")
+			(pintype "bidirectional+no_connect")
 		)
 		(pad "13" thru_hole circle
@@
 			(net 37 "unconnected-(U2-RC2{slash}CCP1-Pad13)")
 			(pinfunction "RC2/CCP1")
-			(pintype "bidirectional")
+			(pintype "bidirectional+no_connect")
 		)
 		(pad "14" thru_hole circle
@@
 			(net 47 "unconnected-(U2-RC3{slash}SCK{slash}SCL-Pad14)")
 			(pinfunction "RC3/SCK/SCL")
-			(pintype "bidirectional")
+			(pintype "bidirectional+no_connect")
 		)
 		(pad "15" thru_hole circle
@@
 			(net 52 "unconnected-(U2-RC4{slash}SDI{slash}SDA-Pad15)")
 			(pinfunction "RC4/SDI/SDA")
-			(pintype "bidirectional")
+			(pintype "bidirectional+no_connect")
 		)
 		(pad "16" thru_hole circle
@@
 			(net 54 "unconnected-(U2-RC5{slash}SDO-Pad16)")
 			(pinfunction "RC5/SDO")
-			(pintype "bidirectional")
+			(pintype "bidirectional+no_connect")
 		)
 		(pad "17" thru_hole circle
@@
 			(net 41 "unconnected-(U2-RC6{slash}TX{slash}CK-Pad17)")
 			(pinfunction "RC6/TX/CK")
-			(pintype "bidirectional")
+			(pintype "bidirectional+no_connect")
 		)
 		(pad "18" thru_hole circle
@@
 			(net 31 "unconnected-(U2-VSS-Pad19)")
 			(pinfunction "VSS")
-			(pintype "power_in")
+			(pintype "power_in+no_connect")
 		)
 		(pad "20" thru_hole circle
@@
 			(net 38 "unconnected-(U2-VDD-Pad20)")
 			(pinfunction "VDD")
-			(pintype "power_in")
+			(pintype "power_in+no_connect")
 		)
 		(pad "21" thru_hole circle
@@
 			(net 39 "unconnected-(U2-INT{slash}RB0-Pad21)")
 			(pinfunction "INT/RB0")
-			(pintype "bidirectional")
+			(pintype "bidirectional+no_connect")
 		)
 		(pad "22" thru_hole circle
@@
 			(net 44 "unconnected-(U2-RB1-Pad22)")
 			(pinfunction "RB1")
-			(pintype "bidirectional")
+			(pintype "bidirectional+no_connect")
 		)
 		(pad "23" thru_hole circle
@@
 			(net 49 "unconnected-(U2-RB2-Pad23)")
 			(pinfunction "RB2")
-			(pintype "bidirectional")
+			(pintype "bidirectional+no_connect")
 		)
 		(pad "24" thru_hole circle
@@
 			(net 40 "unconnected-(U2-PGM{slash}RB3-Pad24)")
 			(pinfunction "PGM/RB3")
-			(pintype "bidirectional")
+			(pintype "bidirectional+no_connect")
 		)
 		(pad "25" thru_hole circle
@@
 			(net 30 "unconnected-(U2-RB4-Pad25)")
 			(pinfunction "RB4")
-			(pintype "bidirectional")
+			(pintype "bidirectional+no_connect")
 		)
 		(pad "26" thru_hole circle
@@
 			(net 51 "unconnected-(U2-RB5-Pad26)")
 			(pinfunction "RB5")
-			(pintype "bidirectional")
+			(pintype "bidirectional+no_connect")
 		)
 		(pad "27" thru_hole circle
@@
 			(net 53 "unconnected-(U2-PGC{slash}RB6-Pad27)")
 			(pinfunction "PGC/RB6")
-			(pintype "bidirectional")
+			(pintype "bidirectional+no_connect")
 		)
 		(pad "28" thru_hole circle
@@
 			(net 32 "unconnected-(U2-PGD{slash}RB7-Pad28)")
 			(pinfunction "PGD/RB7")
-			(pintype "bidirectional")
+			(pintype "bidirectional+no_connect")
 		)
 		(embedded_fonts no)

Commit message: UPDATE
Connections:
- net /Q1_BASE renamed /TC_RX_24V
- net /Q2_BASE renamed /TC_RX_IN
- net /TC_CMD_BUS renamed /TC_RX_BUS
- net /TC_CMD_U3 renamed /TC_RX_U3
- net Net-(Q3-B) renamed /IN_Q_MAIN
- net Net-(U2-RC0/T10S0/T1CKI) renamed /TC_MAIN_U
