File: KiCad/TC106_Overall_circuit_diagram/TC106_Overall_circuit_diagram.kicad_pcb (KiCad board)
At the start: 2 copper layers, 68.9 x 121.6 mm, 51 parts, among them J1 JST_VH_01x05, J10 JST_VH_01x05, J1_24V1 JST_VH_01x04, J1_CN1 JST_VH_01x03, J2 JST_VH_01x05, J2_CN1 JST_VH_01x02, J3 JST_VH_01x05, J3_CN1 JST_VH_01x02, J4 JST_VH_01x05, J4_CN2 JST_VH_01x02, J5 JST_VH_01x05, J5_CN2 JST_VH_01x03, J6 JST_VH_01x05, J7 JST_VH_01x05, J8 JST_VH_01x05, J9 Conn_02x02_Odd_Even, Q1 DTC143E, Q2 DTC143E, Q3 2SD1863, Q5 DTC143E, U1 MC34063AP, U2 PIC16F73-ISP, U3 Dummy dsPic33FJ16MC102

Commit message: UPDATE
Connections:
- D1 pad 1: /TC_RX -> /TC_RX_IN
- D1 pad 2: /TC_RX_IN -> /TC_RX
Changed lines of the file:
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@@
 			(remove_unused_layers no)
 			(roundrect_rratio 0.113636)
-			(net 21 "/TC_RX")
+			(net 17 "/TC_RX_IN")
 			(pinfunction "K")
 			(pintype "passive")
@@
 			(layers "*.Cu" "*.Mask")
 			(remove_unused_layers no)
-			(net 17 "/TC_RX_IN")
+			(net 21 "/TC_RX")
 			(pinfunction "A")
 			(pintype "passive")

Commit message: UPDATE
Parts:
- added J11: Conn_01x01_Socket, TestPoint:TestPoint_Keystone_5000-5004_Miniature, F.Cu at (48.9, 72.2)
- added J12: Conn_01x01_Socket, TestPoint:TestPoint_Keystone_5000-5004_Miniature, F.Cu at (48.9, 76.5)
Connections:
- net +24V renamed +24V_EXT
- Q3 pad 1: /TC_RX -> GND
- Q3 pad 2: GND -> /TC_RX
- R11 pad 2: Net-(R11-Pad2) -> +5V_INT
- R12 pad 2: Net-(R12-Pad2) -> +5V_INT
- U3 pad 1: unconnected-(U3-Pin_1-Pad1) -> +3.3V
Other:
- board text added: "2026.2.19"
- board text removed: "2026.2.11"

Commit message: UPDATE
Parts:
- removed J4_CN2: JST_VH_01x02, Connector_JST:JST_VH_B2P-VH-B_1x02_P3.96mm_Vertical
- removed J5_CN2: JST_VH_01x03, Connector_JST:JST_VH_B3P-VH-B_1x03_P3.96mm_Vertical
- removed Q5: DTC143E, Package_TO_SOT_SMD:SOT-23
- added J4_CN1: JST_VH_01x02, Connector_JST:JST_VH_B2P-VH-B_1x02_P3.96mm_Vertical, F.Cu at (187.0, 141.7)
- added J5_CN1: JST_VH_01x03, Connector_JST:JST_VH_B3P-VH-B_1x03_P3.96mm_Vertical, F.Cu at (191.7, 122.6)
- added Q4: DTC143E, Package_TO_SOT_SMD:SOT-23, F.Cu at (208.2, 134.2)
- C2: value 1000uF 35V -> 104; footprint Capacitor_THT:CP_Radial_D12.5mm_P5.00mm -> Capacitor_THT:C_Disc_D5.0mm_W2.5mm_P2.50mm
- C3: value 470uF 16V -> 1000uF 35V; footprint Capacitor_THT:CP_Radial_D8.0mm_P3.50mm -> Capacitor_THT:CP_Radial_D12.5mm_P5.00mm
- C4: value 104 -> 470uF 16V; footprint Capacitor_THT:C_Disc_D5.0mm_W2.5mm_P2.50mm -> Capacitor_THT:CP_Radial_D8.0mm_P3.50mm
- D1: value 1N4148 -> HZ24; footprint Diode_THT:D_DO-41_SOD81_P7.62mm_Horizontal -> Diode_THT:D_DO-35_SOD27_P7.62mm_Horizontal
- D2: value 1N4148 -> 1N4007; footprint Diode_THT:D_DO-35_SOD27_P7.62mm_Horizontal -> Diode_THT:D_DO-41_SOD81_P7.62mm_Horizontal
- D3: value 1N4007 -> 1N4148
- D4: value 1N5819 -> 1N4148; footprint Diode_THT:D_DO-41_SOD81_P7.62mm_Horizontal -> Diode_THT:D_DO-35_SOD27_P10.16mm_Horizontal
- D5: footprint Diode_THT:D_DO-35_SOD27_P10.16mm_Horizontal -> Diode_THT:D_DO-35_SOD27_P7.62mm_Horizontal
- D6: value HZ24 -> 1N5819; footprint Diode_THT:D_DO-35_SOD27_P7.62mm_Horizontal -> Diode_THT:D_DO-41_SOD81_P7.62mm_Horizontal
- J1: value JST_VH_01x05 -> Conn_01x01_Socket; footprint Connector_JST:JST_VH_B5P-VH-B_1x05_P3.96mm_Vertical -> TestPoint:TestPoint_Keystone_5000-5004_Miniature
- J11: value Conn_01x01_Socket -> JST_VH_01x05; footprint TestPoint:TestPoint_Keystone_5000-5004_Miniature -> Connector_JST:JST_VH_B5P-VH-B_1x05_P3.96mm_Vertical
- J2: value JST_VH_01x05 -> Conn_02x02_Odd_Even
- J9: value Conn_02x02_Odd_Even -> JST_VH_01x05; footprint Connector_PinHeader_1.00mm:PinHeader_2x02_P1.00mm_Vertical -> Connector_JST:JST_VH_B5P-VH-B_1x05_P3.96mm_Vertical
- Q1: value DTC143E -> 2SD1863
- Q3: value 2SD1863 -> DTC143E
- R1: value 220 -> 10k; footprint Resistor_THT:R_Axial_DIN0207_L6.3mm_D2.5mm_P10.16mm_Horizontal -> Resistor_THT:R_Axial_DIN0207_L6.3mm_D2.5mm_P7.62mm_Horizontal
- R2: value 10k -> 1k; footprint Resistor_THT:R_Axial_DIN0207_L6.3mm_D2.5mm_P7.62mm_Horizontal -> Resistor_THT:R_Axial_DIN0204_L3.6mm_D1.6mm_P7.62mm_Horizontal
- R4: value 6k2 -> 220; footprint Resistor_THT:R_Axial_DIN0207_L6.3mm_D2.5mm_P7.62mm_Horizontal -> Resistor_THT:R_Axial_DIN0207_L6.3mm_D2.5mm_P10.16mm_Horizontal
- R5: value 0R22 -> 1k; footprint Resistor_THT:R_Axial_DIN0309_L9.0mm_D3.2mm_P12.70mm_Horizontal -> Resistor_THT:R_Axial_DIN0204_L3.6mm_D1.6mm_P7.62mm_Horizontal
- R7: value 330R -> 0R22; footprint Resistor_THT:R_Axial_DIN0204_L3.6mm_D1.6mm_P7.62mm_Horizontal -> Resistor_THT:R_Axial_DIN0309_L9.0mm_D3.2mm_P12.70mm_Horizontal
- R8: value 1k -> 330R
- R9: value 1k -> 6k2; footprint Resistor_THT:R_Axial_DIN0204_L3.6mm_D1.6mm_P7.62mm_Horizontal -> Resistor_THT:R_Axial_DIN0207_L6.3mm_D2.5mm_P7.62mm_Horizontal
- U3: value Dummy dsPic33FJ16MC102 -> DC-DC_Inverter
Connections:
- C2 pad 1: /+24V_FILT -> Net-(C2-Pad1)
- C3 pad 1: /+9V -> /+24V_FILT
- C4 pad 1: Net-(C4-Pad1) -> /+9V
- D1 pad 1: /TC_RX_IN -> /TC_RX
- D1 pad 2: /TC_RX -> GND
- D2 pad 1: /TC_RX_BUS -> +24V_EXT
- D2 pad 2: GND -> /CMD_IN_PROT
- D3 pad 1: +24V_EXT -> /TC_RX_IN
- D3 pad 2: /CMD_IN_PROT -> /TC_RX
- D4 pad 1: /SW_OUT -> /+24V_FILT
- D4 pad 2: GND -> +24V_EXT
- D5 pad 1: /+24V_FILT -> /TC_RX_BUS
- D5 pad 2: +24V_EXT -> GND
- D6 pad 1: /TC_RX -> /SW_OUT
- J1 pad 1: +24V_EXT -> Net-(J1-Pin_1)
- J10 pad 2: unconnected-(J10-Pin_2-Pad2) -> /+9V
- J10 pad 5: /TC_TX -> unconnected-(J10-Pin_5-Pad5)
- J11 pad 1: +5V_INT -> +24V_EXT
- J12 pad 1: Net-(J12-Pin_1) -> +5V_INT
- J2 pad 1: +24V_EXT -> Net-(J1-Pin_1)
- J2 pad 2: /+9V -> Net-(J2-Pin_2)
- J2 pad 4: /TC_RX_BUS -> Net-(J2-Pin_2)
- J2 pad 5: unconnected-(J2-Pin_5-Pad5) -> (no net)
- J4 pad 5: /TC_TX -> unconnected-(J4-Pin_5-Pad5)
- J9 pad 1: Net-(J12-Pin_1) -> +24V_EXT
- J9 pad 2: Net-(J9-Pin_2) -> /+9V
- J9 pad 4: Net-(J9-Pin_2) -> /TC_RX_BUS
- Q1 pad 2: /TC_RX_BUS -> /TC_RX
- Q1 pad 3: /TC_RX_24V -> /IN_Q_MAIN
- Q3 pad 2: /TC_RX -> /TC_RX_BUS
- Q3 pad 3: /IN_Q_MAIN -> /TC_RX_24V
- R1 pad 1: /TC_RX_IN -> +24V_EXT
- R1 pad 2: GND -> /TC_RX_24V
- R10 pad 1: /TC_TX -> /V_FB
- R10 pad 2: Net-(J9-Pin_2) -> GND
- R2 pad 1: +24V_EXT -> /TC_TX
- R2 pad 2: /TC_RX_24V -> Net-(J2-Pin_2)
- R4 pad 1: /V_FB -> /TC_RX_IN
- R4 pad 2: /+9V -> GND
- R5 pad 1: /I_SENSE -> /TC_TX
- R5 pad 2: /+24V_FILT -> Net-(C2-Pad1)
- R6 pad 1: /V_FB -> Net-(C2-Pad1)
- R6 pad 2: GND -> Net-(U2-RC7/RX/DT)
- R7 pad 1: /IN_Q_MAIN -> /I_SENSE
- R7 pad 2: /TC_MAIN_U -> /+24V_FILT
- R8 pad 1: /TC_TX -> /IN_Q_MAIN
- R8 pad 2: Net-(C4-Pad1) -> /TC_MAIN_U
- R9 pad 1: Net-(C4-Pad1) -> /V_FB
- R9 pad 2: Net-(U2-RC7/RX/DT) -> /+9V
- U3 pad 1: +3.3V -> +24V_EXT
- U3 pad 10: unconnected-(U3-Pin_10-Pad10) -> (no net)
- U3 pad 11: /TC_TX_U3 -> (no net)
- U3 pad 12: /TC_RX_U3 -> (no net)
- U3 pad 13: unconnected-(U3-Pin_13-Pad13) -> (no net)
- U3 pad 14: unconnected-(U3-Pin_14-Pad14) -> (no net)
- U3 pad 15: unconnected-(U3-Pin_15-Pad15) -> (no net)
- U3 pad 16: unconnected-(U3-Pin_16-Pad16) -> (no net)
- U3 pad 17: unconnected-(U3-Pin_17-Pad17) -> (no net)
- U3 pad 18: unconnected-(U3-Pin_18-Pad18) -> (no net)
- U3 pad 19: unconnected-(U3-Pin_19-Pad19) -> (no net)
- U3 pad 2: unconnected-(U3-Pin_2-Pad2) -> (no net)
- U3 pad 20: unconnected-(U3-Pin_20-Pad20) -> (no net)
- U3 pad 21: unconnected-(U3-Pin_21-Pad21) -> (no net)
- U3 pad 22: unconnected-(U3-Pin_22-Pad22) -> (no net)
- U3 pad 23: unconnected-(U3-Pin_23-Pad23) -> (no net)
- U3 pad 24: unconnected-(U3-Pin_24-Pad24) -> (no net)
- U3 pad 25: unconnected-(U3-Pin_25-Pad25) -> (no net)
- U3 pad 26: unconnected-(U3-Pin_26-Pad26) -> (no net)
- U3 pad 27: unconnected-(U3-Pin_27-Pad27) -> (no net)
- U3 pad 28: unconnected-(U3-Pin_28-Pad28) -> (no net)
- U3 pad 3: unconnected-(U3-Pin_3-Pad3) -> (no net)
- U3 pad 4: unconnected-(U3-Pin_4-Pad4) -> (no net)
- U3 pad 5: unconnected-(U3-Pin_5-Pad5) -> (no net)
- U3 pad 6: unconnected-(U3-Pin_6-Pad6) -> (no net)
- U3 pad 7: unconnected-(U3-Pin_7-Pad7) -> (no net)
- U3 pad 8: unconnected-(U3-Pin_8-Pad8) -> (no net)
- U3 pad 9: unconnected-(U3-Pin_9-Pad9) -> (no net)

Commit message: UPDATE
Parts:
- D1: value HZ24 -> 1N4148
- D2: value 1N4007 -> 1N4148
- D3: value 1N4148 -> 1N4007
- D5: value 1N4148 -> HZ24
- moved D1 34.5 mm to (166.5, 124.4)
- moved D2 26.2 mm to (166.3, 98.3), turned to 90 degrees
Connections:
- D1 pad 1: /TC_RX -> /TC_RX_BUS
- D2 pad 1: +24V_EXT -> /TC_RX_IN
- D2 pad 2: /CMD_IN_PROT -> /TC_RX
- D3 pad 1: /TC_RX_IN -> +24V_EXT
- D3 pad 2: /TC_RX -> /CMD_IN_PROT
- D5 pad 1: /TC_RX_BUS -> /TC_RX
Changed lines of the file:
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@@
 	(footprint "Diode_THT:D_DO-41_SOD81_P7.62mm_Horizontal"
 		(layer "F.Cu")
-		(at 166.3446 124.5108 -90)
+		(at 166.32 98.32 90)
 		(descr "Diode, DO-41_SOD81 series, Axial, Horizontal, pin pitch=7.62mm, length*diameter=5.2*2.7mm^2, https://www.diodes.com/assets/Package-Files/DO-41-Plastic.pdf")
 		(tags "Diode DO-41_SOD81 series Axial Horizontal pin pitch 7.62mm  length 5.2mm diameter 2.7mm")
 		(property "Reference" "D2"
-			(at 3.81 -2.47 270)
+			(at 3.81 -2.47 90)
 			(layer "F.SilkS")
 			(effects
@@
 			)
 		)
-		(property "Value" "1N4007"
-			(at 3.81 2.47 270)
+		(property "Value" "1N4148"
+			(at 3.81 2.47 90)
 			(layer "F.Fab")
 			(effects
@@
 		)
 		(property "Datasheet" "~"
-			(at 0 0 270)
+			(at 0 0 90)
 			(layer "F.Fab")
 			(hide yes)
@@
 		)
 		(property "Description" "Diode"
-			(at 0 0 270)
+			(at 0 0 90)
 			(layer "F.Fab")
 			(hide yes)
@@
 		)
 		(property "Sim.Device" "D"
-			(at 0 0 270)
+			(at 0 0 90)
 			(unlocked yes)
 			(layer "F.Fab")
@@
 		)
 		(property "Sim.Pins" "1=K 2=A"
-			(at 0 0 270)
+			(at 0 0 90)
 			(unlocked yes)
 			(layer "F.Fab")
@@
 		(attr through_hole)
 		(fp_line
-			(start 1.09 1.47)
-			(end 6.53 1.47)
+			(start 6.53 -1.47)
+			(end 6.53 -1.34)
 			(stroke
 				(width 0.12)
@@
 		)
 		(fp_line
-			(start 6.53 1.47)
-			(end 6.53 1.34)
+			(start 2.11 -1.47)
+			(end 2.11 1.47)
 			(stroke
 				(width 0.12)
@@
 		)
 		(fp_line
-			(start 1.09 1.34)
-			(end 1.09 1.47)
+			(start 1.99 -1.47)
+			(end 1.99 1.47)
 			(stroke
 				(width 0.12)
@@
 		)
 		(fp_line
-			(start 1.09 -1.34)
-			(end 1.09 -1.47)
+			(start 1.87 -1.47)
+			(end 1.87 1.47)
 			(stroke
 				(width 0.12)
@@
 		)
 		(fp_line
-			(start 1.87 -1.47)
-			(end 1.87 1.47)
+			(start 1.09 -1.34)
+			(end 1.09 -1.47)
 			(stroke
 				(width 0.12)
@@
 		)
 		(fp_line
-			(start 1.99 -1.47)
-			(end 1.99 1.47)
+			(start 1.09 1.34)
+			(end 1.09 1.47)
 			(stroke
 				(width 0.12)
@@
 		)
 		(fp_line
-			(start 2.11 -1.47)
-			(end 2.11 1.47)
+			(start 6.53 1.47)
+			(end 6.53 1.34)
 			(stroke
 				(width 0.12)
@@
 		)
 		(fp_line
-			(start 6.53 -1.47)
-			(end 6.53 -1.34)
+			(start 1.09 1.47)
+			(end 6.53 1.47)
 			(stroke
 				(width 0.12)
@@
 		)
 		(fp_line
-			(start 0 0)
-			(end 1.21 0)
+			(start 2.09 -1.35)
+			(end 2.09 1.35)
 			(stroke
 				(width 0.1)
@@
 		)
 		(fp_line
-			(start 7.62 0)
-			(end 6.41 0)
+			(start 1.99 -1.35)
+			(end 1.99 1.35)
 			(stroke
 				(width 0.1)
@@
 		)
 		(fp_line
-			(start 1.99 -1.35)
-			(end 1.99 1.35)
+			(start 7.62 0)
+			(end 6.41 0)
 			(stroke
 				(width 0.1)
@@
 		)
 		(fp_line
-			(start 2.09 -1.35)
-			(end 2.09 1.35)
+			(start 0 0)
+			(end 1.21 0)
 			(stroke
 				(width 0.1)
@@
 		)
 		(fp_text user "K"
-			(at 0 -2.1 270)
+			(at 0 -2.1 90)
 			(layer "F.SilkS")
 			(effects
@@
 		)
 		(fp_text user "K"
-			(at 0 -2.1 270)
+			(at 0 -2.1 90)
 			(layer "F.Fab")
 			(effects
@@
 		)
 		(fp_text user "${REFERENCE}"
-			(at 4.2 0 270)
+			(at 4.2 0 90)
 			(layer "F.Fab")
 			(effects
@@
 		)
 		(pad "1" thru_hole roundrect
-			(at 0 0 270)
+			(at 0 0 90)
 			(size 2.2 2.2)
 			(drill 1.1)
@@
 			(remove_unused_layers no)
 			(roundrect_rratio 0.113636)
-			(net 1 "+24V_EXT")
+			(net 15 "/TC_RX_IN")
 			(pinfunction "K")
 			(pintype "passive")
 		)
 		(pad "2" thru_hole circle
-			(at 7.62 0 270)
+			(at 7.62 0 90)
 			(size 2.2 2.2)
 			(drill 1.1)
 			(layers "*.Cu" "*.Mask")
 			(remove_unused_layers no)
-			(net 3 "/CMD_IN_PROT")
+			(net 19 "/TC_RX")
 			(pinfunction "A")
 			(pintype "passive")
@@
 	(footprint "Diode_THT:D_DO-35_SOD27_P7.62mm_Horizontal"
 		(layer "F.Cu")
-		(at 166.34 89.92 -90)
+		(at 166.51 124.4 -90)
 		(descr "Diode, DO-35_SOD27 series, Axial, Horizontal, pin pitch=7.62mm, length*diameter=4*2mm^2, http://www.diodes.com/_files/packages/DO-35.pdf")
 		(tags "Diode DO-35_SOD27 series Axial Horizontal pin pitch 7.62mm  length 4mm diameter 2mm")
@@
 			)
 		)
-		(property "Value" "HZ24"
+		(property "Value" "1N4148"
 			(at 3.81 2.12 270)
 			(layer "F.Fab")
@@
 			)
 		)
-		(property "Description" "Zener diode"
+		(property "Description" "Diode"
 			(at 0 0 270)
 			(layer "F.Fab")
@@
 			)
 		)
+		(property "Sim.Device" "D"
+			(at 0 0 270)
+			(unlocked yes)
+			(layer "F.Fab")
+			(hide yes)
+			(effects
+				(font
+					(size 1 1)
+					(thickness 0.15)
+				)
+			)
+		)
+		(property "Sim.Pins" "1=K 2=A"
+			(at 0 0 270)
+			(unlocked yes)
+			(layer "F.Fab")
+			(hide yes)
+			(effects
+				(font
+					(size 1 1)
+					(thickness 0.15)
+				)
+			)
+		)
 		(property ki_fp_filters "TO-???* *_Diode_* *SingleDiode* D_*")
 		(sheetname "/")
@@
 			(remove_unused_layers no)
 			(roundrect_rratio 0.15625)
-			(net 19 "/TC_RX")
+			(net 16 "/TC_RX_BUS")
 			(pinfunction "K")
 			(pintype "passive")
@@
 			)
 		)
-		(property "Value" "1N4148"
+		(property "Value" "1N4007"
 			(at 3.81 2.47 90)
 			(layer "F.Fab")
@@
 			(remove_unused_layers no)
 			(roundrect_rratio 0.113636)
-			(net 15 "/TC_RX_IN")
+			(net 1 "+24V_EXT")
 			(pinfunction "K")
 			(pintype "passive")
@@
 			(layers "*.Cu" "*.Mask")
 			(remove_unused_layers no)
-			(net 19 "/TC_RX")
+			(net 3 "/CMD_IN_PROT")
 			(pinfunction "A")
 			(pintype "passive")
@@
 			)
 		)
-		(property "Value" "1N4148"
+		(property "Value" "HZ24"
 			(at 3.81 2.12 180)
 			(layer "F.Fab")
@@
 			)
 		)
-		(property "Description" "Diode"
+		(property "Description" "Zener diode"
 			(at 0 0 180)
 			(layer "F.Fab")
@@
 			(remove_unused_layers no)
 			(roundrect_rratio 0.15625)
-			(net 16 "/TC_RX_BUS")
+			(net 19 "/TC_RX")
 			(pinfunction "K")
 			(pintype "passive")

Commit message: UPDATE
Parts:
- removed C2, C5: 104, Capacitor_THT:C_Disc_D5.0mm_W2.5mm_P2.50mm
- removed D5: HZ24, Diode_THT:D_DO-35_SOD27_P7.62mm_Horizontal
- removed D7: D_TVS_Dual_AAC, Package_TO_SOT_SMD:SOT-23
- removed J10, J11, J9: JST_VH_01x05, Connector_JST:JST_VH_B5P-VH-B_1x05_P3.96mm_Vertical
- removed J12: Conn_01x01_Socket, TestPoint:TestPoint_Keystone_5000-5004_Miniature
- removed J4_CN1: JST_VH_01x02, Connector_JST:JST_VH_B2P-VH-B_1x02_P3.96mm_Vertical
- removed J5_CN1: JST_VH_01x03, Connector_JST:JST_VH_B3P-VH-B_1x03_P3.96mm_Vertical
- removed JP1: Jumper_2_Open, Connector_PinHeader_1.00mm:PinHeader_1x02_P1.00mm_Vertical
- removed Q3: DTC143E, Package_TO_SOT_THT:TO-92_Inline
- removed Q4: DTC143E, Package_TO_SOT_SMD:SOT-23
- removed R11: 22k, Resistor_THT:R_Axial_DIN0204_L3.6mm_D1.6mm_P7.62mm_Horizontal
- removed R12: 4k7, Resistor_THT:R_Axial_DIN0204_L3.6mm_D1.6mm_P7.62mm_Horizontal
- removed R13, R2, R5, R6: 1k, Resistor_THT:R_Axial_DIN0204_L3.6mm_D1.6mm_P7.62mm_Horizontal
- removed R14: 10k, Resistor_THT:R_Axial_DIN0204_L3.6mm_D1.6mm_P7.62mm_Horizontal
- removed R8: 330R, Resistor_THT:R_Axial_DIN0204_L3.6mm_D1.6mm_P7.62mm_Horizontal
- removed U2: PIC16F73-ISP, Package_DIP:DIP-28_W15.24mm
- removed U3: DC-DC_Inverter, dsPic33FJ16MC102:SOP65P780X200-28N
- J1: value Conn_01x01_Socket -> JST_VH_01x05; footprint TestPoint:TestPoint_Keystone_5000-5004_Miniature -> Connector_JST:JST_VH_B5P-VH-B_1x05_P3.96mm_Vertical
- J2: value Conn_02x02_Odd_Even -> JST_VH_01x05
- Q1: value 2SD1863 -> DTC143E
- moved R7 131.9 mm to (184.8, 62.4), turned to 90 degrees
- moved C4 114.6 mm to (167.1, 36.8), turned to 90 degrees
- moved D6 26.2 mm to (92.2, 103.3)
- moved R10 26.2 mm to (58.6, 88.6)
- moved R9 26.2 mm to (70.5, 93.6)
- moved J2 0.20 mm to (139.6, 88.7)
Connections:
- J1 pad 1: Net-(J1-Pin_1) -> +24V_EXT
- J2 pad 1: Net-(J1-Pin_1) -> +24V_EXT
- J2 pad 2: Net-(J2-Pin_2) -> /+9V
- J2 pad 4: Net-(J2-Pin_2) -> /TC_RX_BUS
- J2 pad 5: (no net) -> unconnected-(J2-Pin_5-Pad5)
- J4 pad 5: unconnected-(J4-Pin_5-Pad5) -> /TC_TX
- Q1 pad 2: /TC_RX -> /TC_RX_BUS
- Q1 pad 3: /IN_Q_MAIN -> /TC_RX_24V

Commit message: UPDATE
Parts:
- removed D6: 1N5819, Diode_THT:D_DO-41_SOD81_P7.62mm_Horizontal
- removed R10: 1k, Resistor_THT:R_Axial_DIN0204_L3.6mm_D1.6mm_P7.62mm_Horizontal
- removed R7: 0R22, Resistor_THT:R_Axial_DIN0309_L9.0mm_D3.2mm_P12.70mm_Horizontal
- removed R9: 6k2, Resistor_THT:R_Axial_DIN0207_L6.3mm_D2.5mm_P7.62mm_Horizontal
- added D5: 1N4148, Diode_THT:D_DO-35_SOD27_P10.16mm_Horizontal, F.Cu at (144.2, 37.1)
- added R2: 10k, Resistor_THT:R_Axial_DIN0207_L6.3mm_D2.5mm_P7.62mm_Horizontal, F.Cu at (169.9, 85.5)
- added R5: 0R22, Resistor_THT:R_Axial_DIN0309_L9.0mm_D3.2mm_P12.70mm_Horizontal, F.Cu at (162.4, 59.8)
- added R6: 1k, Resistor_THT:R_Axial_DIN0204_L3.6mm_D1.6mm_P7.62mm_Horizontal, F.Cu at (166.6, 60.1)
- C3: footprint Capacitor_THT:CP_Radial_D12.5mm_P5.00mm -> Capacitor_THT:CP_Radial_D10.0mm_P7.50mm
- C4: footprint Capacitor_THT:CP_Radial_D8.0mm_P3.50mm -> Capacitor_THT:CP_Radial_D8.0mm_P5.00mm
- D4: value 1N4148 -> 1N5819; footprint Diode_THT:D_DO-35_SOD27_P10.16mm_Horizontal -> Diode_THT:D_DO-41_SOD81_P7.62mm_Horizontal
- R1: value 10k -> 220; footprint Resistor_THT:R_Axial_DIN0207_L6.3mm_D2.5mm_P7.62mm_Horizontal -> Resistor_THT:R_Axial_DIN0207_L6.3mm_D2.5mm_P10.16mm_Horizontal
- R4: value 220 -> 6k2; footprint Resistor_THT:R_Axial_DIN0207_L6.3mm_D2.5mm_P10.16mm_Horizontal -> Resistor_THT:R_Axial_DIN0207_L6.3mm_D2.5mm_P7.62mm_Horizontal
- moved C3 8.90 mm to (166.2, 45.4), turned to 0 degrees
- moved C4 3.47 mm to (164.3, 38.9)
- moved D4 0.35 mm to (151.0, 50.6)
Connections:
- D4 pad 1: /+24V_FILT -> /SW_OUT
- D4 pad 2: +24V_EXT -> GND
- Q1 pad 3: /TC_RX_24V -> /TC_RX_CLAMP
- Q2 pad 2: /TC_RX_24V -> /TC_RX_CLAMP
- R1 pad 1: +24V_EXT -> /TC_RX_IN
- R1 pad 2: /TC_RX_24V -> GND
- R4 pad 1: /TC_RX_IN -> /V_FB
- R4 pad 2: GND -> /+9V
Routing:
- net /TC_RX_CLAMP: track 0.00 -> 26.9 mm
- net /TC_RX_24V: track 26.9 -> 0.00 mm
- net /+24V_FILT: track 65.0 -> 62.0 mm
- net GND: track 509.6 -> 506.6 mm
