File: KiCad/TC106_Pi_READY_RESET_Breadboard_v0.3_20260902/TC106_Pi_READY_RESET_Breadboard.kicad_pcb (KiCad board)
At the start: 2 copper layers, 7 parts, among them J1 Pi_GPIO, J2 XIAO_ESP32S3, Q1 2N7000, Q2 2N7000

Commit message: UPDATE
Other:
- board outline added: 90 x 70 mm
Changed lines of the file:
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@@
 		)
+	)
+	(gr_rect
+		(start 80 60)
+		(end 170 130)
+		(stroke
+			(width 0.05)
+			(type solid)
+		)
+		(fill no)
+		(layer "Edge.Cuts")
 	)
 	(embedded_fonts no)

Commit message: Summary
Parts:
- moved R2 13.1 mm to (124.2, 98.5), turned to -90 degrees
- moved Q1 2.72 mm to (147.0, 90.2)
- moved J1 0.36 mm to (94.6, 92.5)
- moved R3 0.11 mm to (111.0, 92.5)
Routing:
- net /GND: track 0.00 -> 100.6 mm
- net /Q2_GATE: track 0.00 -> 37.4 mm
- net /HOLD: track 0.00 -> 28.5 mm
- net /XIAO_3V3: track 0.00 -> 20.1 mm
- net /CHIP_PU_RESET: track 0.00 -> 18.5 mm
- net /ESP_RUN_BCM17: track 0.00 -> 16.4 mm

Commit message: Summary
Parts:
- moved Q1 0.88 mm to (147.9, 90.0)
Routing:
- net /HOLD: track 28.5 -> 33.2 mm
- net /GND: track 100.6 -> 104.1 mm
- net /XIAO_3V3: track 20.1 -> 23.0 mm
Changed lines of the file:
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@@
 	(footprint "Package_TO_SOT_THT:TO-92_Inline"
 		(layer "F.Cu")
-		(at 147 90.15 180)
+		(at 147.86 89.96 180)
 		(descr "TO-92 leads in-line, narrow, oval pads, drill 0.75mm (see NXP sot054_po.pdf)")
 		(tags "to-92 sc-43 sc-43a sot54 PA33 transistor")
@@
 	(segment
 		(start 124.24 106.14)
-		(end 144.5317 106.14)
+		(end 132.2 114.1)
 		(width 0.2)
 		(layer "F.Cu")
@@
 	)
 	(segment
-		(start 144.5317 106.14)
-		(end 148 109.6083)
+		(start 132.2 114.1)
+		(end 148 114.1)
 		(width 0.2)
 		(layer "F.Cu")
@@
 	)
 	(segment
-		(start 148 110.66)
-		(end 148 109.6083)
+		(start 147.8267 72.3167)
+		(end 147.23 71.72)
 		(width 0.2)
 		(layer "F.Cu")
@@
 	)
 	(segment
+		(start 148 110.538274)
+		(end 148 110.66)
+		(width 0.2)
+		(layer "F.Cu")
+		(net "/GND")
+	)
+	(segment
+		(start 147.8267 90.15)
+		(end 147.8267 72.3167)
+		(width 0.2)
+		(layer "F.Cu")
+		(net "/GND")
+	)
+	(segment
+		(start 148 110.66)
+		(end 148 90.3233)
+		(width 0.2)
+		(layer "F.Cu")
+		(net "/GND")
+	)
+	(segment
+		(start 148 114.1)
+		(end 148 110.66)
+		(width 0.2)
+		(layer "F.Cu")
+		(net "/GND")
+	)
+	(segment
 		(start 148 90.3233)
 		(end 147.8267 90.15)
@@
 	)
 	(segment
-		(start 147.8267 72.4233)
-		(end 147.88 72.37)
-		(width 0.2)
-		(layer "B.Cu")
-		(net "/GND")
-	)
-	(segment
-		(start 147.8267 90.15)
-		(end 147.8267 72.4233)
-		(width 0.2)
-		(layer "B.Cu")
-		(net "/GND")
-	)
-	(segment
-		(start 147 90.15)
-		(end 147.8267 90.15)
-		(width 0.2)
-		(layer "B.Cu")
-		(net "/GND")
-	)
-	(segment
-		(start 148 110.66)
-		(end 148 90.3233)
-		(width 0.2)
-		(layer "B.Cu")
-		(net "/GND")
-	)
-	(segment
-		(start 147.23 71.72)
-		(end 147.88 72.37)
-		(width 0.2)
-		(layer "B.Cu")
-		(net "/GND")
-	)
-	(segment
 		(start 137.4317 111.7117)
 		(end 124.24 98.52)
 		(width 0.2)
+		(layer "F.Cu")
+		(net "/Q2_GATE")
+	)
+	(segment
+		(start 124.24 98.52)
+		(end 118.6 92.88)
+		(width 0.2)
+		(layer "F.Cu")
+		(net "/Q2_GATE")
+	)
+	(segment
+		(start 146.73 111.7117)
+		(end 137.4317 111.7117)
+		(width 0.2)
+		(layer "F.Cu")
+		(net "/Q2_GATE")
+	)
+	(segment
+		(start 146.73 110.66)
+		(end 146.73 111.7117)
+		(width 0.2)
+		(layer "F.Cu")
+		(net "/Q2_GATE")
+	)
+	(segment
+		(start 118.6 92.88)
+		(end 118.6 92.46)
+		(width 0.2)
 		(layer "B.Cu")
 		(net "/Q2_GATE")
 	)
 	(segment
-		(start 124.24 98.52)
-		(end 118.6 92.88)
-		(width 0.2)
-		(layer "B.Cu")
-		(net "/Q2_GATE")
-	)
-	(segment
-		(start 118.6 92.88)
-		(end 118.6 92.46)
-		(width 0.2)
-		(layer "B.Cu")
-		(net "/Q2_GATE")
-	)
-	(segment
-		(start 146.73 111.7117)
-		(end 137.4317 111.7117)
-		(width 0.2)
-		(layer "B.Cu")
-		(net "/Q2_GATE")
-	)
-	(segment
-		(start 146.73 110.66)
-		(end 146.73 111.7117)
-		(width 0.2)
-		(layer "B.Cu")
-		(net "/Q2_GATE")
-	)
-	(segment
 		(start 139.5817 97.35)
 		(end 139.5817 105.6084)
 		(width 0.2)
-		(layer "B.Cu")
-		(net "/HOLD")
-	)
-	(segment
-		(start 139.5817 97.35)
-		(end 145.73 91.2017)
-		(width 0.2)
-		(layer "B.Cu")
+		(layer "F.Cu")
 		(net "/HOLD")
 	)
@@
 		(end 144.6333 110.66)
 		(width 0.2)
-		(layer "B.Cu")
-		(net "/HOLD")
-	)
-	(segment
-		(start 145.73 90.15)
-		(end 145.73 91.2017)
-		(width 0.2)
-		(layer "B.Cu")
+		(layer "F.Cu")
 		(net "/HOLD")
 	)
@@
 		(end 144.6333 110.66)
 		(width 0.2)
-		(layer "B.Cu")
+		(layer "F.Cu")
+		(net "/HOLD")
+	)
+	(segment
+		(start 146.59 97.35)
+		(end 146.59 89.96)
+		(width 0.2)
+		(layer "F.Cu")
+		(net "/HOLD")
+	)
+	(segment
+		(start 139.5817 97.35)
+		(end 146.59 97.35)
+		(width 0.2)
+		(layer "F.Cu")
 		(net "/HOLD")
 	)
@@
 		(end 139.5817 97.35)
 		(width 0.2)
-		(layer "B.Cu")
+		(layer "F.Cu")
 		(net "/HOLD")
 	)
 	(segment
-		(start 142.15 71.72)
-		(end 142.15 72.8717)
-		(width 0.2)
-		(layer "B.Cu")
-		(net "/XIAO_3V3")
-	)
-	(segment
-		(start 142.15 72.8717)
-		(end 137.03 77.9917)
-		(width 0.2)
-		(layer "B.Cu")
+		(start 142.15 77.74)
+		(end 142.01 77.88)
+		(width 0.2)
+		(layer "F.Cu")
 		(net "/XIAO_3V3")
 	)
@@
 		(end 137.03 89.73)
 		(width 0.2)
-		(layer "B.Cu")
+		(layer "F.Cu")
+		(net "/XIAO_3V3")
+	)
+	(segment
+		(start 142.01 77.88)
+		(end 137.1417 77.88)
+		(width 0.2)
+		(layer "F.Cu")
+		(net "/XIAO_3V3")
+	)
+	(segment
+		(start 142.15 71.72)
+		(end 142.15 77.74)
+		(width 0.2)
+		(layer "F.Cu")
+		(net "/XIAO_3V3")
+	)
+	(segment
+		(start 137.1417 77.88)
+		(end 137.03 77.9917)
+		(width 0.2)
+		(layer "F.Cu")
 		(net "/XIAO_3V3")
 	)
@@
 	)
 	(segment
-		(start 144.69 88.8683)
-		(end 144.46 89.0983)
-		(width 0.2)
-		(layer "B.Cu")
+		(start 144.69 71.72)
+		(end 145.32 72.35)
+		(width 0.2)
+		(layer "F.Cu")
 		(net "/CHIP_PU_RESET")
 	)
 	(segment
-		(start 144.69 71.72)
-		(end 144.69 88.8683)
-		(width 0.2)
-		(layer "B.Cu")
+		(start 145.32 72.35)
+		(end 145.32 89.96)
+		(width 0.2)
+		(layer "F.Cu")
 		(net "/CHIP_PU_RESET")
 	)
-	(segment
-		(start 144.46 90.15)
-		(end 144.46 89.0983)
-		(width 0.2)
-		(layer "B.Cu")
-		(net "/CHIP_PU_RESET")
-	)
