File: KiCad/106_circuit/TC106-MainController/TC106_Main_Comm_Reconstruction.kicad_sch (KiCad schematic)
At the start: 22 parts, among them CN1 ch1-TX(53259-0210), CN2 ch2-TX(53259-0210), CN4 ch1-LENGTH(53259-0310), CN6 ch2-LENGTH(53259-0310), Q1 D1863, Q2 D1863, U1 X24C00, U2 PIC16C62A (Main Controller MC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, Y1 10MHz

Commit message: UpDATE
Connections:
- net GND: no longer C1.2, C2.2, CN2.1, CN6.3 (LENGTH), U1.VCC_pin (VCC)
- net NET_CH1_FILT: no longer C1.1
- net NET_CH2_FILT: no longer C2.1, R6.1, R8.2
- net NET_CH2_LEN_J: no longer JP2.2, R8.1
- net NET_CH2_LEN_RAW: no longer CN6.1 (GND), JP2.1
- net NET_OSC1: no longer Y1.1
- net NET_OSC2: no longer Y1.2
- net NET_PIC_RC3_pin14_SCL_DERIVED: no longer U1.5 (DA(SDA))
- net NET_PIC_RC4_pin15_SDA_DERIVED: no longer R11.2, U1.6 (CL(SCL))
- net NET_PIC_RC6_pin17_rxch2_DERIVED: no longer R6.2
- net VCC: no longer R11.1, U1.GND_pin (GND)
Other:
- moved on the sheet: R11
Changed lines of the file:
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@@
 	(text "DERIVED -> pin15(RC4/SDA)"
 		(exclude_from_sim no)
-		(at 280.42 295.97 0)
+		(at 294.64 294.894 0)
 		(effects
 			(font
@@
 	(text "UNRESOLVED: wired, source unknown"
 		(exclude_from_sim no)
-		(at 414.04 198.43 0)
+		(at 434.086 198.628 0)
 		(effects
 			(font
@@
 	(text "DERIVED -> pin14(RC3/SCL)"
 		(exclude_from_sim no)
-		(at 280.42 298.51 0)
+		(at 294.894 297.942 0)
 		(effects
 			(font
@@
 	(text "pin2 = NC (3-pin original)"
 		(exclude_from_sim no)
-		(at 203.72 244.78 0)
+		(at 208.788 248.92 0)
 		(effects
 			(font
@@
 	(text "SOFTENED: no source found on this sheet"
 		(exclude_from_sim no)
-		(at 414.04 206.05 0)
+		(at 436.626 205.994 0)
 		(effects
 			(font
@@
 	(wire
 		(pts
-			(xy 309.88 294.64) (xy 307.34 294.64)
+			(xy 320.04 294.64) (xy 317.5 294.64)
 		)
 		(stroke
@@
 	(wire
 		(pts
-			(xy 299.72 294.64) (xy 302.26 294.64)
+			(xy 309.88 294.64) (xy 312.42 294.64)
 		)
 		(stroke
@@
 	(global_label "NET_CH2_LEN_J"
 		(shape passive)
-		(at 270.26 239.64 0)
+		(at 264.16 247.65 0)
 		(effects
 			(font
@@
 		)
 		(property "Intersheetrefs" "${INTERSHEET_REFS}"
-			(at 270.26 239.64 0)
+			(at 264.16 247.65 0)
 			(hide yes)
 			(show_name no)
@@
 	(global_label "NET_CH2_LEN_RAW"
 		(shape passive)
-		(at 203.72 242.18 0)
+		(at 172.72 242.57 0)
 		(effects
 			(font
@@
 		)
 		(property "Intersheetrefs" "${INTERSHEET_REFS}"
-			(at 203.72 242.18 0)
+			(at 172.72 242.57 0)
 			(hide yes)
 			(show_name no)
@@
 	(global_label "NET_CH2_FILT"
 		(shape passive)
-		(at 302.26 239.64 0)
+		(at 292.1 247.65 0)
 		(effects
 			(font
@@
 		)
 		(property "Intersheetrefs" "${INTERSHEET_REFS}"
-			(at 302.26 239.64 0)
+			(at 292.1 247.65 0)
 			(hide yes)
 			(show_name no)
@@
 	(global_label "NET_CH1_FILT"
 		(shape passive)
-		(at 270.26 206.64 0)
+		(at 256.54 201.93 0)
 		(effects
 			(font
@@
 		)
 		(property "Intersheetrefs" "${INTERSHEET_REFS}"
-			(at 270.26 206.64 0)
+			(at 256.54 201.93 0)
 			(hide yes)
 			(show_name no)
@@
 	(global_label "VCC"
 		(shape passive)
-		(at 265.18 295.91 0)
+		(at 252.73 295.91 0)
 		(effects
 			(font
@@
 		)
 		(property "Intersheetrefs" "${INTERSHEET_REFS}"
-			(at 265.18 295.91 0)
+			(at 252.73 295.91 0)
 			(hide yes)
 			(show_name no)
@@
 	(global_label "NET_OSC1"
 		(shape passive)
-		(at 238.26 339.64 0)
+		(at 219.71 340.36 0)
 		(effects
 			(font
@@
 		)
 		(property "Intersheetrefs" "${INTERSHEET_REFS}"
-			(at 238.26 339.64 0)
+			(at 219.71 340.36 0)
 			(hide yes)
 			(show_name no)
@@
 	(global_label "NET_OSC2"
 		(shape passive)
-		(at 243.34 339.64 0)
+		(at 254 340.36 0)
 		(effects
 			(font
@@
 		)
 		(property "Intersheetrefs" "${INTERSHEET_REFS}"
-			(at 243.34 339.64 0)
+			(at 254 340.36 0)
 			(hide yes)
 			(show_name no)
@@
 	(global_label "GND"
 		(shape passive)
-		(at 206.26 134.64 0)
+		(at 196.85 133.35 0)
 		(effects
 			(font
@@
 		)
 		(property "Intersheetrefs" "${INTERSHEET_REFS}"
-			(at 206.26 134.64 0)
+			(at 196.85 133.35 0)
 			(hide yes)
 			(show_name no)
@@
 	(global_label "NET_CH2_FILT"
 		(shape passive)
-		(at 275.34 239.64 0)
+		(at 280.67 233.68 0)
 		(effects
 			(font
@@
 		)
 		(property "Intersheetrefs" "${INTERSHEET_REFS}"
-			(at 275.34 239.64 0)
+			(at 280.67 233.68 0)
 			(hide yes)
 			(show_name no)
@@
 	(global_label "NET_PIC_RC3_pin14_SCL_DERIVED"
 		(shape passive)
-		(at 280.42 295.91 0)
+		(at 298.45 302.26 0)
 		(effects
 			(font
@@
 		)
 		(property "Intersheetrefs" "${INTERSHEET_REFS}"
-			(at 280.42 295.91 0)
+			(at 298.45 302.26 0)
 			(hide yes)
 			(show_name no)
@@
 	(global_label "NET_PIC_RC4_pin15_SDA_DERIVED"
 		(shape passive)
-		(at 307.34 294.64 0)
+		(at 339.09 294.64 0)
 		(effects
 			(font
@@
 		)
 		(property "Intersheetrefs" "${INTERSHEET_REFS}"
-			(at 307.34 294.64 0)
+			(at 339.09 294.64 0)
 			(hide yes)
 			(show_name no)
@@
 	(global_label "GND"
 		(shape passive)
-		(at 203.72 237.1 0)
+		(at 186.69 236.22 0)
 		(effects
 			(font
@@
 		)
 		(property "Intersheetrefs" "${INTERSHEET_REFS}"
-			(at 203.72 237.1 0)
+			(at 186.69 236.22 0)
 			(hide yes)
 			(show_name no)
@@
 	(global_label "GND"
 		(shape passive)
-		(at 265.18 293.37 0)
+		(at 252.73 290.83 0)
 		(effects
 			(font
@@
 		)
 		(property "Intersheetrefs" "${INTERSHEET_REFS}"
-			(at 265.18 293.37 0)
+			(at 252.73 290.83 0)
 			(hide yes)
 			(show_name no)
@@
 	(global_label "NET_CH2_FILT"
 		(shape passive)
-		(at 270.26 261.64 0)
+		(at 256.54 255.27 0)
 		(effects
 			(font
@@
 		)
 		(property "Intersheetrefs" "${INTERSHEET_REFS}"
-			(at 270.26 261.64 0)
+			(at 256.54 255.27 0)
 			(hide yes)
 			(show_name no)
@@
 	(global_label "NET_CH2_LEN_J"
 		(shape passive)
-		(at 243.34 239.64 0)
+		(at 247.65 233.68 0)
 		(effects
 			(font
@@
 		)
 		(property "Intersheetrefs" "${INTERSHEET_REFS}"
-			(at 243.34 239.64 0)
+			(at 247.65 233.68 0)
 			(hide yes)
 			(show_name no)
@@
 	(global_label "VCC"
 		(shape passive)
-		(at 302.26 294.64 0)
+		(at 312.42 294.64 0)
 		(effects
 			(font
@@
 		)
 		(property "Intersheetrefs" "${INTERSHEET_REFS}"
-			(at 302.26 294.64 0)
+			(at 312.42 294.64 0)
 			(hide yes)
 			(show_name no)
@@
 	(global_label "GND"
 		(shape passive)
-		(at 275.34 206.64 0)
+		(at 281.94 210.82 0)
 		(effects
 			(font
@@
 		)
 		(property "Intersheetrefs" "${INTERSHEET_REFS}"
-			(at 275.34 206.64 0)
+			(at 281.94 210.82 0)
 			(hide yes)
 			(show_name no)
@@
 	(global_label "NET_PIC_RC4_pin15_SDA_DERIVED"
 		(shape passive)
-		(at 280.42 293.37 0)
+		(at 298.45 289.56 0)
 		(effects
 			(font
@@
 		)
 		(property "Intersheetrefs" "${INTERSHEET_REFS}"
-			(at 280.42 293.37 0)
+			(at 298.45 289.56 0)
 			(hide yes)
 			(show_name no)
@@
 	(global_label "NET_CH2_LEN_RAW"
 		(shape passive)
-		(at 238.26 239.64 0)
+		(at 232.41 247.65 0)
 		(effects
 			(font
@@
 		)
 		(property "Intersheetrefs" "${INTERSHEET_REFS}"
-			(at 238.26 239.64 0)
+			(at 232.41 247.65 0)
 			(hide yes)
 			(show_name no)
@@
 	(global_label "GND"
 		(shape passive)
-		(at 275.34 261.64 0)
+		(at 284.48 265.43 0)
 		(effects
 			(font
@@
 		)
 		(property "Intersheetrefs" "${INTERSHEET_REFS}"
-			(at 275.34 261.64 0)
+			(at 284.48 265.43 0)
 			(hide yes)
 			(show_name no)
@@
 	(global_label "NET_PIC_RC6_pin17_rxch2_DERIVED"
 		(shape passive)
-		(at 307.34 239.64 0)
+		(at 325.12 234.95 0)
 		(effects
 			(font
@@
 		)
 		(property "Intersheetrefs" "${INTERSHEET_REFS}"
-			(at 307.34 239.64 0)
+			(at 325.12 234.95 0)
 			(hide yes)
 			(show_name no)
@@
 		)
 		(property "Value" "ch2-LENGTH(53259-0310)"
-			(at 208.8 242.84 0)
+			(at 208.788 246.126 0)
 			(show_name no)
 			(do_not_autoplace no)
@@
 	(symbol
 		(lib_id "GEN_R")
-		(at 304.8 294.64 0)
+		(at 306.07 283.21 0)
 		(unit 1)
 		(body_style 1)
@@
 		(dnp no)
 		(property "Reference" "R11"
-			(at 304.8 291.44 0)
+			(at 306.07 280.01 0)
 			(show_name no)
 			(do_not_autoplace no)
@@
 		)
 		(property "Value" "1k (pullup)"
-			(at 304.8 297.84 0)
+			(at 306.07 286.41 0)
 			(show_name no)
 			(do_not_autoplace no)
@@
 		)
 		(property "Footprint" ""
-			(at 304.8 294.64 0)
+			(at 306.07 283.21 0)
 			(hide yes)
 			(show_name no)
@@
 		)
 		(property "Datasheet" ""
-			(at 304.8 294.64 0)
+			(at 306.07 283.21 0)
 			(show_name no)
 			(do_not_autoplace no)
@@
 		)
 		(property "Description" ""
-			(at 304.8 294.64 0)
+			(at 306.07 283.21 0)
 			(show_name no)
 			(do_not_autoplace no)
@@
 		(dnp no)
 		(property "Reference" "U1"
-			(at 272.8 291.44 0)
+			(at 271.78 294.64 0)
 			(show_name no)
 			(do_not_autoplace no)
@@
 		)
 		(property "Value" "X24C00"
-			(at 272.8 297.84 0)
+			(at 273.05 299.974 0)
 			(show_name no)
 			(do_not_autoplace no)
@@
 		)
 		(property "Value" "PIC16C62A (Main Controller MCU)"
-			(at 398.8 202.84 0)
+			(at 398.526 214.376 0)
 			(show_name no)
 			(do_not_autoplace no)
