File: KiCad/ESP32S3_Snifar_#2/ESP32S3_Snifar.kicad_pcb (KiCad board)
At the start: 2 copper layers, 95 x 70 mm, 46 parts, among them J1 Conn_01x04_Socket, J2 J2_Pi_01x06_Socket, Q2 2N7000, U1 XIAO-ESP32S3

Commit message: Summary
Other:
- board text added: "FOR Pi UART"
- board text added: "GND RX TX"
- board text added: "TC106 Snidar ESP32S3 Ver 2.1 2026.10.26"
- board text removed: "FOR RaspberyPi UART PORT"
- board text removed: "TC106 Snidar ESP32S3 Ver 2.0 2026.10.26"
Changed lines of the file:
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@@
 		(tags "Through hole socket strip THT 1x06 2.54mm single row")
 		(property "Reference" "J2"
-			(at 0 -2.77 180)
+			(at -0.025 15.23 180)
 			(layer "F.SilkS")
 			(effects
@@
 		)
 	)
-	(gr_text "FOR RaspberyPi UART PORT"
-		(at 35.45 55.09 90)
+	(gr_text "FOR Pi UART"
+		(at 34.65 56.06 0)
+		(layer "F.SilkS")
+		(effects
+			(font
+				(size 0.8 0.8)
+				(thickness 0.1)
+			)
+			(justify left bottom)
+		)
+	)
+	(gr_text "GND         RX  TX"
+		(at 35.84 54.14 90)
 		(layer "F.SilkS")
 		(effects
@@
 		)
 	)
-	(gr_text "TC106 Snidar ESP32S3\nVer 2.0 2026.10.26"
+	(gr_text "TC106 Snidar ESP32S3\nVer 2.1 2026.10.26"
 		(at 39.5 91.68 90)
 		(layer "F.SilkS")

Commit message: Update
Other:
- board text removed: ">"
- board text removed: "Do Not Populate"
Changed lines of the file:
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@@
-		)
-	)
-	(gr_text "Do Not Populate"
-		(at 43.84 46.65 90)
-		(layer "F.SilkS")
-		(effects
-			(font
-				(size 0.8 0.8)
-				(thickness 0.1)
-			)
-			(justify left bottom)
-		)
-	)
-	(gr_text ">"
-		(at 43.89 42.51 0)
-		(layer "F.SilkS")
-		(effects
-			(font
-				(size 1 1)
-				(thickness 0.1)
-			)
-			(justify left bottom)
 		)
 	)

Commit message: Update PCB
Parts:
- moved TP1 0.44 mm to (65.9, 71.3)
Routing:
- net /SIG_5V_LOW_FOR_TC106: track 78.5 -> 77.1 mm
Other:
- board text added: "2026.10.26"
- board text added: "Ver2.1"
- board text removed: "2026.08.18"
- board text removed: "Ver2.0"
Changed lines of the file:
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@@
 	(footprint "TestPoint:TestPoint_Loop_D2.50mm_Drill1.0mm"
 		(layer "F.Cu")
-		(at 65.97 70.85)
+		(at 65.94 71.29)
 		(descr "wire loop as test point, loop diameter 2.5mm, hole diameter 1.0mm")
 		(tags "test point wire loop bead")
@@
 		)
 	)
-	(gr_text "2026.08.18"
+	(gr_text "2026.10.26"
 		(at 207 193.81 0)
 		(layer "Cmts.User")
@@
 		)
 	)
-	(gr_text "Ver2.0"
+	(gr_text "Ver2.1"
 		(at 269.09 193.72 0)
 		(layer "Cmts.User")
@@
 	)
 	(segment
-		(start 65.97 72.21)
-		(end 65.97 70.85)
+		(start 37.98 69.365)
+		(end 37.975 69.36)
 		(width 0.2)
 		(layer "F.Cu")
@@
 	)
 	(segment
-		(start 85.74 72.21)
-		(end 65.97 72.21)
+		(start 37.98 71.31)
+		(end 37.98 69.365)
+		(width 0.2)
+		(layer "F.Cu")
+		(net "/SIG_5V_LOW_FOR_TC106")
+	)
+	(segment
+		(start 67.33 72.21)
+		(end 66.41 71.29)
 		(width 0.2)
 		(layer "F.Cu")
@@
 	)
 	(segment
-		(start 65.97 72.21)
-		(end 37.98 72.21)
+		(start 85.74 72.21)
+		(end 67.33 72.21)
 		(width 0.2)
 		(layer "F.Cu")
@@
 	)
 	(segment
-		(start 37.98 69.365)
-		(end 37.975 69.36)
+		(start 65.97 71.31)
+		(end 37.98 71.31)
 		(width 0.2)
 		(layer "F.Cu")
@@
 	)
 	(segment
-		(start 37.98 72.21)
-		(end 37.98 69.365)
+		(start 66.41 71.29)
+		(end 65.94 71.29)
+		(width 0.2)
+		(layer "F.Cu")
+		(net "/SIG_5V_LOW_FOR_TC106")
+	)
+	(segment
+		(start 65.97 70.85)
+		(end 65.97 71.31)
 		(width 0.2)
 		(layer "F.Cu")
