File: KiCad/ESP32S3_Snifar_#2/ESP32S3_Snifar.kicad_pcb (KiCad board)
At the start: 2 copper layers, 95 x 70 mm, 46 parts, among them J1 Conn_01x04_Socket, J2 J2_Pi_01x06_Socket, Q2 2N7000, U1 XIAO-ESP32S3

Commit message: Summary
Other:
- board text added: "From TC Interface Board or Arduino nano every ESP32S3 relay circuit"
- board text removed: "ESP32S3 TC106 Snifar"
Changed lines of the file:
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@@
 		)
 	)
-	(gr_text "ESP32S3 TC106 Snifar"
+	(gr_text "From TC Interface Board or Arduino nano every ESP32S3 relay circuit"
 		(at 188.59 190.5 0)
 		(layer "Cmts.User")
