File: KiCad/ESP32S3_Snifar_#2/ESP32S3_Snifar.kicad_sch (KiCad schematic)
At the start: 46 parts, among them J1 Conn_01x04_Socket, J2 J2_Pi_01x06_Socket, Q2 2N7000, U1 XIAO-ESP32S3

Commit message: Summry
Connections:
- net GND: no longer TP1.1
- net SIG_5V_LOW_FOR_TC106: now also TP1.1
Other:
- moved on the sheet: TP1
Changed lines of the file:
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@@
 	)
 	(junction
-		(at 104.14 55.88)
-		(diameter 0)
-		(color 0 0 0 0)
-	)
-	(junction
 		(at 139.7 96.52)
 		(diameter 0)
@@
 	)
 	(junction
+		(at 78.74 34.29)
+		(diameter 0)
+		(color 0 0 0 0)
+	)
+	(junction
 		(at 104.14 34.29)
 		(diameter 0)
@@
 	(wire
 		(pts
-			(xy 64.77 34.29) (xy 82.55 34.29)
+			(xy 64.77 34.29) (xy 78.74 34.29)
 		)
 		(stroke
@@
 	(wire
 		(pts
-			(xy 104.14 45.72) (xy 104.14 55.88)
-		)
-		(stroke
-			(width 0)
-			(type default)
-		)
-	)
-	(wire
-		(pts
 			(xy 167.64 139.7) (xy 212.09 139.7)
 		)
@@
 	(wire
 		(pts
+			(xy 78.74 34.29) (xy 82.55 34.29)
+		)
+		(stroke
+			(width 0)
+			(type default)
+		)
+	)
+	(wire
+		(pts
 			(xy 238.76 30.48) (xy 238.76 40.64)
 		)
@@
 	(wire
 		(pts
-			(xy 104.14 55.88) (xy 104.14 69.85)
+			(xy 104.14 45.72) (xy 104.14 69.85)
 		)
 		(stroke
@@
 	(symbol
 		(lib_id "Connector:TestPoint")
-		(at 104.14 55.88 90)
+		(at 78.74 34.29 180)
 		(unit 1)
 		(body_style 1)
@@
 		(dnp no)
 		(property "Reference" "TP1"
-			(at 96.52 64.516 0)
+			(at 81.026 39.878 0)
 			(show_name no)
 			(do_not_autoplace no)
@@
 		)
 		(property "Value" "TestPoint"
-			(at 99.06 64.516 0)
+			(at 86.36 41.91 0)
 			(show_name no)
 			(do_not_autoplace no)
@@
 		)
 		(property "Footprint" "TestPoint:TestPoint_Loop_D2.50mm_Drill1.0mm"
-			(at 104.14 50.8 0)
+			(at 73.66 34.29 0)
 			(hide yes)
 			(show_name no)
@@
 		)
 		(property "Datasheet" ""
-			(at 104.14 50.8 0)
+			(at 73.66 34.29 0)
 			(hide yes)
 			(show_name no)
@@
 		)
 		(property "Description" "test point"
-			(at 104.14 55.88 0)
+			(at 78.74 34.29 0)
 			(hide yes)
 			(show_name no)

Commit message: Summary
Other:
- note added: "Ver 2.1"
- note removed: "Ver 2.0"
Changed lines of the file:
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@@
 		)
 	)
-	(text "Ver 2.0"
+	(text "Ver 2.1"
 		(exclude_from_sim no)
 		(at 274.828 193.294 0)

Commit message: Summary
Other:
- note added: "From TC Interface Board or Arduino nano every ESP32S3 relay circuit"
- note removed: "From TC Intterface Borad or Arduino nano every ESP32S3 relay circuit"
Changed lines of the file:
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@@
 	(generator_version "10.0")
 	(paper "A4")
-	(text "From TC Intterface Borad or Arduino nano every ESP32S3 relay circuit"
+	(text "From TC Interface Board or Arduino nano every ESP32S3 relay circuit"
 		(exclude_from_sim no)
 		(at 223.774 189.738 0)
